File: components_predev/output_driver/hardware/output_driver.sch (KiCad schematic (older format))
At the start: 20 parts

Commit message: Output Driver Schematic
Parts:
- added C? (x6): CP1, symbol CP1
- added D? (x2): D, symbol D
- added P?: CONN_01X04, symbol CONN_01X04
- added Q? (x2): Q_PNP_BCE, symbol Q_PNP_BCE
- added Q? (x2): Q_NPN_BCE, symbol Q_NPN_BCE
- added Q?: Q_PMOS_DGS, symbol Q_PMOS_DGS
- added R? (x8): R, symbol R
Connections:
- net VDD: now also Q?.1 (D), R?.1, R?.1
- net VSS: now also R?.2, R?.2
- net at R?.2: now also Q?.2 (C), Q?.2 (C)
- new net: Q?.1 (B), Q?.2 (C), R?.2
- new net: Q?.3 (E), R?.2 (x2)
- new net: Q?.1 (B), Q?.2 (C), R?.1
- new net: Q?.3 (E), R?.1 (x2)
- new net: R?.1, R?.2
- new net: D?.2 (A), Q?.1 (B), R?.2
- new net: D?.1 (K), Q?.1 (B), R?.1
- new net: C?.1, C?.1, C?.1, Q?.3 (S)
- new net +5V: R?.1
- new net offset_adj: D?.1 (K), D?.2 (A)
Other:
- moved on the sheet: R?

Commit message: Inrush Current Limit
Parts:
- added D? (x2): D_Zener, symbol D_Zener
- added Q? (x3): Q_NMOS_DGS, symbol Q_NMOS_DGS
- added R? (x6): R, symbol R
Connections:
- net GNDPWR: now also C?.2, C?.2, C?.2, C?.2, C?.2, C?.2, P?.3 (P3), P?.4 (P4), Q?.3 (S), Q?.3 (S)
- net VDD: now also C?.1, C?.1, C?.1, R?.1
- net VSS: now also C?.1, C?.1, C?.1, Q?.1 (D), R?.1
- net v_sense_ext+: now reaches P?.1 (P1)
- net v_sense+: now reaches P?.2 (P2), Q?.3 (E), Q?.3 (E), R?.1, R?.2
- net i_sense+: now reaches P?.3 (P3), R?.1
- net v_sense_ext-: now reaches P?.4 (P4)
- net drv_input: now reaches R?.1, R?.2
- net at P?.1 (P1): now also Q?.3 (S), D?.1 (K), R?.2, R?.2
- net at P?.2 (P2): now also D?.2 (A), Q?.3 (S), R?.2, R?.2
- net at Q?.2 (G): now also D?.2 (A), R?.1, R?.2
- new net: Q?.1 (D), R?.1 (x2)
- new net: D?.1 (K), Q?.2 (G), R?.1, R?.2
- new net pwr_enable: Q?.2 (G), Q?.2 (G)
Other:
- moved on the sheet: C?, D?, P?, Q?, R?, RV?

Commit message: .gitignore, Component Selection for Inrush Current Limiter
Parts:
- removed Q? (x2): Q_NMOS_DGS, symbol Q_NMOS_DGS
- added Q? (x2): MMBT5550L, symbol Q_NPN_BCE
- added R? (x2): 68k, symbol R
- added R? (x2): R, symbol R
- C? (x6): value CP1 -> 100u; Digikey (none) -> 493-1165-ND; Manufacturer (none) -> Nichicon; Part Number (none) -> UVR2C101MHD
- D? (x2): value D_Zener -> 10V
- Q?: value Q_PMOS_DGS -> FDMS86263P; Digikey (none) -> FDMS86263PCT-ND; Manufacturer (none) -> Fairchild; Mouser (none) -> 512-FDMS86263P
- Q?: value Q_NMOS_DGS -> FDMS86252; Digikey (none) -> FDMS86252CT-ND; Manufacturer (none) -> Fairchild; Part Number (none) -> FDMS86252
- R? (x2): value R -> 18k
- R? (x2): value R -> 68k
- R? (x2): value R -> 220
Connections:
- net GNDPWR: now also C?.1, C?.1, C?.1, Q?.3 (E), Q?.3 (E); no longer C?.2, C?.2, C?.2
- net VDD: now also R?.1; no longer C?.1, C?.1, C?.1, Q?.1 (D), R?.1
- net VSS: now also R?.1; no longer C?.1, C?.1, C?.1, Q?.1 (D), R?.1
- net pwr_enable: now also R?.2, R?.2
- net at R?.1: now also Q?.2 (C) (x2)
- new net: Q?.1 (B), R?.1 (x2)
- new net in-: C?.2, C?.2, C?.2, Q?.1 (D), R?.1, R?.2
- new net ip+: C?.1, C?.1, C?.1, Q?.1 (D), R?.1, R?.2
Other:
- note added: "-25V - -100V"
- note added: "25V - 100V"
- note added: "To Do:\n-----------------------------------------------------------\nOutput Current/Voltage Measurement\nSupply Current/Voltage Measurement\nAnalog Supply\nDigital Supply\n"
- moved on the sheet: C?

Commit message: Checked Transistor Power Dissipation
Parts:
- Q?: value Q_PNP_BCE -> 2SA1962OTU; Digikey (none) -> 2SA1962OTU-ND; Manufacturer (none) -> Fairchild; Part Number (none) -> 2SA1962OTU
- Q? (x3): value Q_NPN_BCE -> MMBT5550L; Digikey (none) -> MMBT5550LT1GOSCT-ND; Manufacturer (none) -> OnSemi; Part Number (none) -> MMBT5550L
- Q?: value Q_NPN_BCE -> MMBT5550L; Part Number (none) -> MMBT5550L
- Q? (x3): value Q_PNP_BCE -> MMBT5401-7-F; Manufacturer (none) -> Diodes; Part Number (none) -> MMBT5401-7-F
- Q?: value Q_NPN_BCE -> 2SC5242OTU; Digikey (none) -> 2SC5242OTU-ND; Manufacturer (none) -> Fairchild; Part Number (none) -> 2SC5242OTU
- Q?: value Q_PNP_BCE -> MJD350T4G; Digikey (none) -> MJD350T4GOSCT-ND; Manufacturer (none) -> OnSemi; Part Number (none) -> MJD350T4G
- Q?: value Q_NPN_BCE -> MJD340T4G; Digikey (none) -> MJD340T4GOSCT-ND; Manufacturer (none) -> OnSemi; Part Number (none) -> MJD340T4G
- R? (x4): value R -> 1k
- R? (x2): value R -> 200m
- R? (x2): value R -> 3k3
- R? (x2): value R -> 520
- R?: value R -> 68k
- R?: value R -> 33
- R? (x2): value R -> 100
- R? (x2): value R -> 10
- R? (x2): value R -> 680
- R? (x2): value R -> 10m
- RV?: value POT_TRIM -> 500
Changed lines of the file:
@@
 P 12950 2100
 F 0 "Q?" H 13150 2150 50  0000 L CNN
-F 1 "Q_PNP_BCE" H 13150 2050 50  0000 L CNN
+F 1 "2SA1962OTU" H 13150 2050 50  0000 L CNN
 F 2 "" H 13150 2200 50  0000 C CNN
 F 3 "" H 12950 2100 50  0000 C CNN
+F 4 "Fairchild" H 12950 2100 60  0001 C CNN "Manufacturer"
+F 5 "2SA1962OTU-ND" H 12950 2100 60  0001 C CNN "Digikey"
+F 6 "2SA1962OTU" H 12950 2100 60  0001 C CNN "Part Number"
 	1    12950 2100
 	1    0    0    1
@@
 P 12350 2500
 F 0 "Q?" H 12550 2550 50  0000 L CNN
-F 1 "Q_NPN_BCE" H 12550 2450 50  0000 L CNN
+F 1 "MMBT5550L" H 12550 2450 50  0000 L CNN
 F 2 "" H 12550 2600 50  0000 C CNN
 F 3 "" H 12350 2500 50  0000 C CNN
+F 4 "OnSemi" H 12350 2500 60  0001 C CNN "Manufacturer"
+F 5 "MMBT5550LT1GOSCT-ND" H 12350 2500 60  0001 C CNN "Digikey"
+F 6 "MMBT5550L" H 12350 2500 60  0001 C CNN "Part Number"
 	1    12350 2500
 	1    0    0    -1
@@
 P 12450 1750
 F 0 "R?" V 12530 1750 50  0000 C CNN
-F 1 "R" V 12450 1750 50  0000 C CNN
+F 1 "1k" V 12450 1750 50  0000 C CNN
 F 2 "" V 12380 1750 50  0000 C CNN
 F 3 "" H 12450 1750 50  0000 C CNN
@@
 P 13050 3750
 F 0 "R?" V 13130 3750 50  0000 C CNN
-F 1 "R" V 13050 3750 50  0000 C CNN
+F 1 "200m" V 13050 3750 50  0000 C CNN
 F 2 "" V 12980 3750 50  0000 C CNN
 F 3 "" H 13050 3750 50  0000 C CNN
@@
 P 12750 3500
 F 0 "Q?" H 12950 3550 50  0000 L CNN
-F 1 "Q_NPN_BCE" H 12950 3450 50  0000 L CNN
+F 1 "MMBT5550L" H 12950 3450 50  0000 L CNN
 F 2 "" H 12950 3600 50  0000 C CNN
 F 3 "" H 12750 3500 50  0000 C CNN
+F 4 "MMBT5550L" H 12750 3500 60  0001 C CNN "Part Number"
 	1    12750 3500
 	-1   0    0    -1
@@
 P 13050 4350
 F 0 "R?" V 13130 4350 50  0000 C CNN
-F 1 "R" V 13050 4350 50  0000 C CNN
+F 1 "200m" V 13050 4350 50  0000 C CNN
 F 2 "" V 12980 4350 50  0000 C CNN
 F 3 "" H 13050 4350 50  0000 C CNN
@@
 P 12750 4650
 F 0 "Q?" H 12950 4700 50  0000 L CNN
-F 1 "Q_PNP_BCE" H 12950 4600 50  0000 L CNN
+F 1 "MMBT5401-7-F" H 12950 4600 50  0000 L CNN
 F 2 "" H 12950 4750 50  0000 C CNN
 F 3 "" H 12750 4650 50  0000 C CNN
+F 4 "Diodes" H 12750 4650 60  0001 C CNN "Manufacturer"
+F 5 "MMBT5401-7-F" H 12750 4650 60  0001 C CNN "Part Number"
 	1    12750 4650
 	-1   0    0    1
@@
 P 12400 5600
 F 0 "Q?" H 12600 5650 50  0000 L CNN
-F 1 "Q_PNP_BCE" H 12600 5550 50  0000 L CNN
+F 1 "MMBT5401-7-F" H 12600 5550 50  0000 L CNN
 F 2 "" H 12600 5700 50  0000 C CNN
 F 3 "" H 12400 5600 50  0000 C CNN
+F 4 "Diodes" H 12400 5600 60  0001 C CNN "Manufacturer"
+F 5 "MMBT5401-7-F" H 12400 5600 60  0001 C CNN "Part Number"
 	1    12400 5600
 	1    0    0    1
@@
 P 12950 6000
 F 0 "Q?" H 13150 6050 50  0000 L CNN
-F 1 "Q_NPN_BCE" H 13150 5950 50  0000 L CNN
+F 1 "2SC5242OTU" H 13150 5950 50  0000 L CNN
 F 2 "" H 13150 6100 50  0000 C CNN
 F 3 "" H 12950 6000 50  0000 C CNN
+F 4 "Fairchild" H 12950 6000 60  0001 C CNN "Manufacturer"
+F 5 "2SC5242OTU-ND" H 12950 6000 60  0001 C CNN "Digikey"
+F 6 "2SC5242OTU" H 12950 6000 60  0001 C CNN "Part Number"
 	1    12950 6000
 	1    0    0    -1
@@
 P 12500 6350
 F 0 "R?" V 12580 6350 50  0000 C CNN
-F 1 "R" V 12500 6350 50  0000 C CNN
+F 1 "1k" V 12500 6350 50  0000 C CNN
 F 2 "" V 12430 6350 50  0000 C CNN
 F 3 "" H 12500 6350 50  0000 C CNN
@@
 P 11800 2500
 F 0 "R?" V 11880 2500 50  0000 C CNN
-F 1 "R" V 11800 2500 50  0000 C CNN
+F 1 "3k3" V 11800 2500 50  0000 C CNN
 F 2 "" V 11730 2500 50  0000 C CNN
 F 3 "" H 11800 2500 50  0000 C CNN
@@
 P 11900 5600
 F 0 "R?" V 11980 5600 50  0000 C CNN
-F 1 "R" V 11900 5600 50  0000 C CNN
+F 1 "3k3" V 11900 5600 50  0000 C CNN
 F 2 "" V 11830 5600 50  0000 C CNN
 F 3 "" H 11900 5600 50  0000 C CNN
@@
 P 11300 4050
 F 0 "Q?" H 11500 4100 50  0000 L CNN
-F 1 "Q_NPN_BCE" H 11500 4000 50  0000 L CNN
+F 1 "MMBT5550L" H 11500 4000 50  0000 L CNN
 F 2 "" H 11500 4150 50  0000 C CNN
 F 3 "" H 11300 4050 50  0000 C CNN
+F 4 "OnSemi" H 11300 4050 60  0001 C CNN "Manufacturer"
+F 5 "MMBT5550LT1GOSCT-ND" H 11300 4050 60  0001 C CNN "Digikey"
+F 6 "MMBT5550L" H 11300 4050 60  0001 C CNN "Part Number"
 	1    11300 4050
 	1    0    0    -1
@@
 P 10750 4050
 F 0 "RV?" V 10575 4050 50  0000 C CNN
-F 1 "POT_TRIM" V 10650 4050 50  0000 C CNN
+F 1 "500" V 10650 4050 50  0000 C CNN
 F 2 "" H 10750 4050 50  0000 C CNN
 F 3 "" H 10750 4050 50  0000 C CNN
@@
 P 10750 3600
 F 0 "R?" V 10830 3600 50  0000 C CNN
-F 1 "R" V 10750 3600 50  0000 C CNN
+F 1 "520" V 10750 3600 50  0000 C CNN
 F 2 "" V 10680 3600 50  0000 C CNN
 F 3 "" H 10750 3600 50  0000 C CNN
@@
 P 10750 4500
 F 0 "R?" V 10830 4500 50  0000 C CNN
-F 1 "R" V 10750 4500 50  0000 C CNN
+F 1 "520" V 10750 4500 50  0000 C CNN
 F 2 "" V 10680 4500 50  0000 C CNN
 F 3 "" H 10750 4500 50  0000 C CNN
@@
 P 11400 6350
 F 0 "R?" V 11480 6350 50  0000 C CNN
-F 1 "R" V 11400 6350 50  0000 C CNN
+F 1 "68k" V 11400 6350 50  0000 C CNN
 F 2 "" V 11330 6350 50  0000 C CNN
 F 3 "" H 11400 6350 50  0000 C CNN
@@
 P 10200 2800
 F 0 "R?" V 10280 2800 50  0000 C CNN
-F 1 "R" V 10200 2800 50  0000 C CNN
+F 1 "33" V 10200 2800 50  0000 C CNN
 F 2 "" V 10130 2800 50  0000 C CNN
 F 3 "" H 10200 2800 50  0000 C CNN
@@
 P 9250 2500
 F 0 "Q?" H 9450 2550 50  0000 L CNN
-F 1 "Q_PNP_BCE" H 9450 2450 50  0000 L CNN
+F 1 "MJD350T4G" H 9450 2450 50  0000 L CNN
 F 2 "" H 9450 2600 50  0000 C CNN
 F 3 "" H 9250 2500 50  0000 C CNN
+F 4 "OnSemi" H 9250 2500 60  0001 C CNN "Manufacturer"
+F 5 "MJD350T4GOSCT-ND" H 9250 2500 60  0001 C CNN "Digikey"
+F 6 "MJD350T4G" H 9250 2500 60  0001 C CNN "Part Number"
 	1    9250 2500
 	1    0    0    1
@@
 P 9250 3100
 F 0 "Q?" H 9450 3150 50  0000 L CNN
-F 1 "Q_NPN_BCE" H 9450 3050 50  0000 L CNN
+F 1 "MJD340T4G" H 9450 3050 50  0000 L CNN
 F 2 "" H 9450 3200 50  0000 C CNN
 F 3 "" H 9250 3100 50  0000 C CNN
+F 4 "OnSemi" H 9250 3100 60  0001 C CNN "Manufacturer"
+F 5 "MJD340T4GOSCT-ND" H 9250 3100 60  0001 C CNN "Digikey"
+F 6 "MJD340T4G" H 9250 3100 60  0001 C CNN "Part Number"
 	1    9250 3100
 	1    0    0    -1
@@
 P 9350 2050
 F 0 "R?" V 9430 2050 50  0000 C CNN
-F 1 "R" V 9350 2050 50  0000 C CNN
+F 1 "100" V 9350 2050 50  0000 C CNN
 F 2 "" V 9280 2050 50  0000 C CNN
 F 3 "" H 9350 2050 50  0000 C CNN
@@
 P 9350 3550
 F 0 "R?" V 9430 3550 50  0000 C CNN
-F 1 "R" V 9350 3550 50  0000 C CNN
+F 1 "100" V 9350 3550 50  0000 C CNN
 F 2 "" V 9280 3550 50  0000 C CNN
 F 3 "" H 9350 3550 50  0000 C CNN
@@
 P 7600 2550
 F 0 "R?" V 7680 2550 50  0000 C CNN
-F 1 "R" V 7600 2550 50  0000 C CNN
+F 1 "10" V 7600 2550 50  0000 C CNN
 F 2 "" V 7530 2550 50  0000 C CNN
 F 3 "" H 7600 2550 50  0000 C CNN
@@
 P 7600 3050
 F 0 "R?" V 7680 3050 50  0000 C CNN
-F 1 "R" V 7600 3050 50  0000 C CNN
+F 1 "10" V 7600 3050 50  0000 C CNN
 F 2 "" V 7530 3050 50  0000 C CNN
 F 3 "" H 7600 3050 50  0000 C CNN
@@
 P 7700 2050
 F 0 "Q?" H 7900 2100 50  0000 L CNN
-F 1 "Q_NPN_BCE" H 7900 2000 50  0000 L CNN
+F 1 "MMBT5550L" H 7900 2000 50  0000 L CNN
 F 2 "" H 7900 2150 50  0000 C CNN
 F 3 "" H 7700 2050 50  0000 C CNN
+F 4 "OnSemi" H 7700 2050 60  0001 C CNN "Manufacturer"
+F 5 "MMBT5550LT1GOSCT-ND" H 7700 2050 60  0001 C CNN "Digikey"
+F 6 "MMBT5550L" H 7700 2050 60  0001 C CNN "Part Number"
 	1    7700 2050
 	-1   0    0    -1
@@
 P 7700 3550
 F 0 "Q?" H 7900 3600 50  0000 L CNN
-F 1 "Q_PNP_BCE" H 7900 3500 50  0000 L CNN
+F 1 "MMBT5401-7-F" H 7900 3500 50  0000 L CNN
 F 2 "" H 7900 3650 50  0000 C CNN
 F 3 "" H 7700 3550 50  0000 C CNN
+F 4 "Diodes" H 7700 3550 60  0001 C CNN "Manufacturer"
+F 5 "MMBT5401-7-F" H 7700 3550 60  0001 C CNN "Part Number"
 	1    7700 3550
 	-1   0    0    1
@@
 P 7600 1550
 F 0 "R?" V 7680 1550 50  0000 C CNN
-F 1 "R" V 7600 1550 50  0000 C CNN
+F 1 "1k" V 7600 1550 50  0000 C CNN
 F 2 "" V 7530 1550 50  0000 C CNN
 F 3 "" H 7600 1550 50  0000 C CNN
@@
 P 7600 4050
 F 0 "R?" V 7680 4050 50  0000 C CNN
-F 1 "R" V 7600 4050 50  0000 C CNN
+F 1 "1k" V 7600 4050 50  0000 C CNN
 F 2 "" V 7530 4050 50  0000 C CNN
 F 3 "" H 7600 4050 50  0000 C CNN
@@
 P 8350 2050
 F 0 "R?" V 8430 2050 50  0000 C CNN
-F 1 "R" V 8350 2050 50  0000 C CNN
+F 1 "680" V 8350 2050 50  0000 C CNN
 F 2 "" V 8280 2050 50  0000 C CNN
 F 3 "" H 8350 2050 50  0000 C CNN
@@
 P 8350 3550
 F 0 "R?" V 8430 3550 50  0000 C CNN
-F 1 "R" V 8350 3550 50  0000 C CNN
+F 1 "680" V 8350 3550 50  0000 C CNN
 F 2 "" V 8280 3550 50  0000 C CNN
 F 3 "" H 8350 3550 50  0000 C CNN
@@
 P 5300 1200
 F 0 "R?" V 5380 1200 50  0000 C CNN
-F 1 "R" V 5300 1200 50  0000 C CNN
+F 1 "10m" V 5300 1200 50  0000 C CNN
 F 2 "" V 5230 1200 50  0000 C CNN
 F 3 "" H 5300 1200 50  0000 C CNN
@@
 P 5300 3250
 F 0 "R?" V 5380 3250 50  0000 C CNN
-F 1 "R" V 5300 3250 50  0000 C CNN
+F 1 "10m" V 5300 3250 50  0000 C CNN
 F 2 "" V 5230 3250 50  0000 C CNN
 F 3 "" H 5300 3250 50  0000 C CNN

Commit message: Moved ICL to now Sheet
Parts:
- removed C? (x6): 100u, symbol CP1
- removed D? (x2): 10V, symbol D_Zener
- removed Q?: FDMS86263P, symbol Q_PMOS_DGS
- removed Q?: FDMS86252, symbol Q_NMOS_DGS
- removed Q? (x2): MMBT5550L, symbol Q_NPN_BCE
- removed R? (x2): 18k, symbol R
- removed R? (x4): 68k, symbol R
- removed R? (x2): 220, symbol R
- removed R? (x2): 10m, symbol R
- added K?: PE014005, symbol PE014005
- added R?: R, symbol R
Connections:
- net GNDPWR: now also R?.2
- net Inrush Current Limiter/VIn+: now reaches P?.1 (P1)
- net Inrush Current Limiter/VIn-: now reaches P?.2 (P2)
- net i_sense+ renamed il_sense+
- net il_sense+: now also K?.12; no longer P?.3 (P3)
- new net GND: K?.2
- new net i_range_rel: K?.1
- new net ih_sense+: K?.14, R?.1
- new net v_sense-: K?.11, P?.3 (P3)
Other:
- note removed: "-25V - -100V"
- note removed: "25V - 100V"
- moved on the sheet: R?

Commit message: Moved output stage to new schematic sheet
Parts:
- removed D? (x2): D, symbol D
- removed Q?: 2SA1962OTU, symbol Q_PNP_BCE
- removed Q? (x4): MMBT5550L, symbol Q_NPN_BCE
- removed Q? (x3): MMBT5401-7-F, symbol Q_PNP_BCE
- removed Q?: 2SC5242OTU, symbol Q_NPN_BCE
- removed Q?: MJD350T4G, symbol Q_PNP_BCE
- removed Q?: MJD340T4G, symbol Q_NPN_BCE
- removed R? (x4): 1k, symbol R
- removed R? (x2): 200m, symbol R
- removed R? (x2): 3k3, symbol R
- removed R? (x2): 520, symbol R
- removed R?: 68k, symbol R
- removed R?: 33, symbol R
- removed R? (x2): 100, symbol R
- removed R? (x2): 10, symbol R
- removed R? (x2): 680, symbol R
- removed RV?: 500, symbol POT_TRIM
Other:
- moved on the sheet: K?, P?, R?

Commit message: Added Subsheets to structure Circuit
Parts:
- added P?: CONN_01X02, symbol CONN_01X02
- added P?: CONN_01X24, symbol CONN_01X24
Connections:
- net GND: now also P?.2 (P2)
- new net supplies/v_supply: P?.1 (P1)
Other:
- moved on the sheet: P?
Changed lines of the file:
@@
 $Descr A4 11693 8268
 encoding utf-8
-Sheet 1 3
+Sheet 1 6
 Title "openSMU - Output Driver PreDev v1"
 Date "2018-05-24"
@@
 L CONN_01X04 P?
 U 1 1 5B06FF0C
-P 1300 1350
-F 0 "P?" H 1300 1600 50  0000 C CNN
-F 1 "CONN_01X04" V 1400 1350 50  0000 C CNN
-F 2 "" H 1300 1350 50  0000 C CNN
-F 3 "" H 1300 1350 50  0000 C CNN
-	1    1300 1350
+P 900 6250
+F 0 "P?" H 900 6500 50  0000 C CNN
+F 1 "CONN_01X04" V 1000 6250 50  0000 C CNN
+F 2 "" H 900 6250 50  0000 C CNN
+F 3 "" H 900 6250 50  0000 C CNN
+	1    900  6250
 	-1   0    0    -1
 $EndComp
@@
 L VDD #PWR?
 U 1 1 5B07094E
-P 3500 1200
-F 0 "#PWR?" H 3500 1050 50  0001 C CNN
-F 1 "VDD" H 3500 1350 50  0000 C CNN
-F 2 "" H 3500 1200 50  0000 C CNN
-F 3 "" H 3500 1200 50  0000 C CNN
-	1    3500 1200
+P 4800 6100
+F 0 "#PWR?" H 4800 5950 50  0001 C CNN
+F 1 "VDD" H 4800 6250 50  0000 C CNN
+F 2 "" H 4800 6100 50  0000 C CNN
+F 3 "" H 4800 6100 50  0000 C CNN
+	1    4800 6100
 	0    1    1    0
 $EndComp
@@
 L VSS #PWR?
 U 1 1 5B084BEC
-P 3500 1550
-F 0 "#PWR?" H 3500 1400 50  0001 C CNN
-F 1 "VSS" H 3500 1700 50  0000 C CNN
-F 2 "" H 3500 1550 50  0000 C CNN
-F 3 "" H 3500 1550 50  0000 C CNN
-	1    3500 1550
+P 4800 6450
+F 0 "#PWR?" H 4800 6300 50  0001 C CNN
+F 1 "VSS" H 4800 6600 50  0000 C CNN
+F 2 "" H 4800 6450 50  0000 C CNN
+F 3 "" H 4800 6450 50  0000 C CNN
+	1    4800 6450
 	0    1    1    0
 $EndComp
@@
 L GNDPWR #PWR?
 U 1 1 5B08A530
-P 1650 1700
-F 0 "#PWR?" H 1650 1500 50  0001 C CNN
-F 1 "GNDPWR" H 1650 1570 50  0000 C CNN
-F 2 "" H 1650 1650 50  0000 C CNN
-F 3 "" H 1650 1650 50  0000 C CNN
-	1    1650 1700
+P 1250 6600
+F 0 "#PWR?" H 1250 6400 50  0001 C CNN
+F 1 "GNDPWR" H 1250 6470 50  0000 C CNN
+F 2 "" H 1250 6550 50  0000 C CNN
+F 3 "" H 1250 6550 50  0000 C CNN
+	1    1250 6600
 	1    0    0    -1
 $EndComp
 Wire Wire Line
-	1650 1400 1650 1700
-Wire Wire Line
-	1650 1500 1500 1500
-Wire Wire Line
-	1500 1400 1650 1400
-Connection ~ 1650 1500
+	1250 6300 1250 6600
+Wire Wire Line
+	1250 6400 1100 6400
+Wire Wire Line
+	1100 6300 1250 6300
+Connection ~ 1250 6400
 Text GLabel 9950 1550 1    60   Output ~ 0
 v_sense_ext+
@@
 	10200 3050 10200 3450
 $Sheet
-S 2250 1000 1100 1600
+S 3550 5900 1100 1600
 U 5B0C28A9
 F0 "Inrush Current Limiter" 60
 F1 "inrush_limiter.sch" 60
-F2 "VIn+" I L 2250 1200 60
-F3 "VIn-" I L 2250 1300 60
-F4 "VDD" O R 3350 1200 60
-F5 "VSS" O R 3350 1550 60
-F6 "pwr_enable" I L 2250 2350 60
-F7 "ip+" O R 3350 1950 60
-F8 "ip-" O R 3350 2050 60
-F9 "in+" O R 3350 2250 60
-F10 "in-" O R 3350 2350 60
-$EndSheet
-Wire Wire Line
-	3350 1550 3500 1550
-Wire Wire Line
-	3350 1200 3500 1200
-Wire Wire Line
-	2250 1200 1500 1200
-Wire Wire Line
-	2250 1300 1500 1300
-$Sheet
-S 5950 1000 2150 1550
+F2 "VIn+" I L 3550 6100 60
+F3 "VIn-" I L 3550 6200 60
+F4 "VDD" O R 4650 6100 60
+F5 "VSS" O R 4650 6450 60
+F6 "pwr_enable" I L 3550 7250 60
+F7 "ip+" O R 4650 6850 60
+F8 "ip-" O R 4650 6950 60
+F9 "in+" O R 4650 7150 60
+F10 "in-" O R 4650 7250 60
+$EndSheet
+Wire Wire Line
+	4650 6450 4800 6450
+Wire Wire Line
+	4650 6100 4800 6100
+Wire Wire Line
+	1100 6100 3550 6100
+Wire Wire Line
+	1100 6200 3550 6200
+$Sheet
+S 7000 1000 1100 1650
 U 5B0E9220
 F0 "output_stage" 60
 F1 "output_stage.sch" 60
-F2 "VDD" I L 5950 1150 60
-F3 "VSS" I L 5950 1300 60
+F2 "VDD" I L 7000 1150 60
+F3 "VSS" I L 7000 1300 60
 F4 "output" O R 8100 1800 60
 $EndSheet
@@
 L VDD #PWR?
 U 1 1 5B0EC83F
-P 5600 1150
-F 0 "#PWR?" H 5600 1000 50  0001 C CNN
-F 1 "VDD" H 5600 1300 50  0000 C CNN
-F 2 "" H 5600 1150 50  0000 C CNN
-F 3 "" H 5600 1150 50  0000 C CNN
-	1    5600 1150
+P 6650 1150
+F 0 "#PWR?" H 6650 1000 50  0001 C CNN
+F 1 "VDD" H 6650 1300 50  0000 C CNN
+F 2 "" H 6650 1150 50  0000 C CNN
+F 3 "" H 6650 1150 50  0000 C CNN
+	1    6650 1150
 	0    -1   -1   0
 $EndComp
@@
 L VSS #PWR?
 U 1 1 5B0EC997
-P 5600 1300
-F 0 "#PWR?" H 5600 1150 50  0001 C CNN
-F 1 "VSS" H 5600 1450 50  0000 C CNN
-F 2 "" H 5600 1300 50  0000 C CNN
-F 3 "" H 5600 1300 50  0000 C CNN
-	1    5600 1300
+P 6650 1300
+F 0 "#PWR?" H 6650 1150 50  0001 C CNN
+F 1 "VSS" H 6650 1450 50  0000 C CNN
+F 2 "" H 6650 1300 50  0000 C CNN
+F 3 "" H 6650 1300 50  0000 C CNN
+	1    6650 1300
 	0    -1   -1   0
 $EndComp
 Wire Wire Line
-	5600 1300 5950 1300
-Wire Wire Line
-	5950 1150 5600 1150
+	6650 1300 7000 1300
+Wire Wire Line
+	7000 1150 6650 1150
 Wire Wire Line
 	10500 5000 10350 5000
@@
 Wire Wire Line
 	10350 3050 10200 3050
+$Sheet
+S 1800 6600 1100 900
+U 5B1543EF
+F0 "supplies" 60
+F1 "supplies.sch" 60
+F2 "v_supply" I L 1800 6800 60
+$EndSheet
+$Comp
+L CONN_01X02 P?
+U 1 1 5B1544A1
+P 900 6850
+F 0 "P?" H 900 7000 50  0000 C CNN
+F 1 "CONN_01X02" V 1000 6850 50  0000 C CNN
+F 2 "" H 900 6850 50  0000 C CNN
+F 3 "" H 900 6850 50  0000 C CNN
+	1    900  6850
+	-1   0    0    -1
+$EndComp
+Wire Wire Line
+	1100 6900 1250 6900
+$Comp
+L GND #PWR?
+U 1 1 5B15483E
+P 1250 7200
+F 0 "#PWR?" H 1250 6950 50  0001 C CNN
+F 1 "GND" H 1250 7050 50  0000 C CNN
+F 2 "" H 1250 7200 50  0000 C CNN
+F 3 "" H 1250 7200 50  0000 C CNN
+	1    1250 7200
+	1    0    0    -1
+$EndComp
+Wire Wire Line
+	1800 6800 1100 6800
+$Sheet
+S 7000 3400 1100 2400
+U 5B156993
+F0 "vi_filter" 60
+F1 "vi_filter.sch" 60
+$EndSheet
+Wire Wire Line
+	1250 6900 1250 7200
+$Sheet
+S 3550 1000 1100 1650
+U 5B158093
+F0 "DAC" 60
+F1 "DAC.sch" 60
+$EndSheet
+$Sheet
+S 3550 3400 1100 1650
+U 5B1582A3
+F0 "ADC" 60
+F1 "ADC.sch" 60
+$EndSheet
+$Comp
+L CONN_01X24 P?
+U 1 1 5B15842C
+P 900 2500
+F 0 "P?" H 900 3750 50  0000 C CNN
+F 1 "CONN_01X24" V 1000 2500 50  0000 C CNN
+F 2 "" H 900 2500 50  0000 C CNN
+F 3 "" H 900 2500 50  0000 C CNN
+	1    900  2500
+	-1   0    0    -1
+$EndComp
 $EndSCHEMATC

Commit message: Interface Wiring
Parts:
- added D?: D, symbol D
- added Q?: Q_NMOS_DGS, symbol Q_NMOS_DGS
- added R?: R, symbol R
Connections:
- net Inrush Current Limiter/VIn- is gone; now on net Inrush Current Limiter/VIn+: P?.2 (P2)
- net GND: now also P?.24 (P24), Q?.3 (S), R?.2; no longer K?.2
- net v_range: now reaches P?.20 (P20)
- net i_range: now reaches P?.21 (P21)
- net i_range: now also Q?.2 (G), R?.1
- net v_extern: now reaches P?.22 (P22)
- net i_range_rel renamed +12V
- net +12V: now also D?.1 (K)
- net il_sense+ renamed vi_filter/il_sense+
- new net: D?.2 (A), K?.2, Q?.1 (D)
Other:
- note removed: "To Do:\n-----------------------------------------------------------\nOutput Current/Voltage Measurement\nSupply Current/Voltage Measurement\nAnalog Supply\nDigital Supply\n"
- moved on the sheet: K?
