File: components_predev/output_driver/hardware/output_driver.sch (KiCad schematic (older format))
At the start: 10 parts

Commit message: Added ADC Symbol, Started Wiring
Connections:
- net ADC/DINA: now reaches P?.11 (P11)
- net ADC/DINB: now reaches P?.12 (P12)
- net ADC/DOUTA: now reaches P?.13 (P13)
- net ADC/DOUTB: now reaches P?.14 (P14)
- net ADC/SCLK: now reaches P?.15 (P15)
- net ADC/CNVSTA: now reaches P?.17 (P17)
- net ADC/CNVSTB: now reaches P?.18 (P18)
Changed lines of the file:
@@
 F8 "ip" I R 4650 4450 60
 F9 "in" I R 4650 4550 60
+F10 "DINA" I L 3550 3600 60
+F11 "DINB" I L 3550 3700 60
+F12 "DOUTA" O L 3550 3800 60
+F13 "DOUTB" O L 3550 3900 60
+F14 "SCLK" I L 3550 4000 60
+F15 "CNVSTA" I L 3550 4200 60
+F16 "CNVSTB" I L 3550 4300 60
 $EndSheet
 $Comp
@@
 Wire Wire Line
 	7000 5300 6600 5300
+Wire Wire Line
+	3550 4300 2100 4300
+Wire Wire Line
+	2100 4300 2100 3050
+Wire Wire Line
+	2100 3050 1100 3050
+Wire Wire Line
+	3550 4200 2200 4200
+Wire Wire Line
+	2200 4200 2200 2950
+Wire Wire Line
+	2200 2950 1100 2950
+Wire Wire Line
+	3550 4000 2400 4000
+Wire Wire Line
+	2400 4000 2400 2750
+Wire Wire Line
+	2400 2750 1100 2750
+Wire Wire Line
+	3550 3900 2500 3900
+Wire Wire Line
+	2500 3900 2500 2650
+Wire Wire Line
+	2500 2650 1100 2650
+Wire Wire Line
+	3550 3800 2600 3800
+Wire Wire Line
+	2600 3800 2600 2550
+Wire Wire Line
+	2600 2550 1100 2550
+Wire Wire Line
+	3550 3700 2700 3700
+Wire Wire Line
+	2700 3700 2700 2450
+Wire Wire Line
+	2700 2450 1100 2450
+Wire Wire Line
+	3550 3600 2800 3600
+Wire Wire Line
+	2800 3600 2800 2350
+Wire Wire Line
+	2800 2350 1100 2350
 $EndSCHEMATC

Commit message: Added DAC, added disengage relay
Parts:
- removed P?: CONN_01X24, symbol CONN_01X24
- added P?: CONN_01X32, symbol CONN_01X32
Connections:
- net ADC/CNVSTA: now also P?.19 (P19)
- net ADC/CNVSTB: now also P?.20 (P20)
- net ADC/DINA: now also P?.13 (P13)
- net ADC/DINB: now also P?.14 (P14)
- net ADC/DOUTA: now also P?.15 (P15)
- net ADC/DOUTB: now also P?.16 (P16)
- net ADC/SCLK: now also P?.17 (P17)
- net GND: now also P?.18 (P18), P?.26 (P26)
- net i_range: now also P?.23 (P23)
- net v_extern: now also P?.24 (P24)
- net v_range: now also P?.22 (P22)
- new net DAC/DIN: P?.8 (P8)
- new net DAC/DOUT: P?.9 (P9)
- new net DAC/PD: P?.2 (P2)
- new net DAC/SCLK: P?.7 (P7)
- new net DAC/~BUSY: P?.1 (P1)
- new net DAC/~CS: P?.6 (P6)
- new net DAC/~LDAC: P?.4 (P4)
- new net DAC/~READY: P?.5 (P5)
- new net DAC/~RST: P?.3 (P3)
- new net output_stage/disengage: P?.25 (P25)
- new net pwr_enable: P?.27 (P27)

Commit message: Put opamp gain stage into schematic
Connections:
- net output_stage/temp: now reaches P?.11 (P11)
Changed lines of the file:
@@
 F5 "drv_input" I L 7000 1800 60
 F6 "disengage" I L 7000 2400 60
+F7 "v_ref_2" I L 7000 1950 60
+F8 "temp" O L 7000 2250 60
 $EndSheet
 $Comp
@@
 Wire Wire Line
 	1500 3750 1100 3750
+Wire Wire Line
+	4650 4850 5200 4850
+Wire Wire Line
+	5200 4850 5200 1950
+Wire Wire Line
+	5200 1950 7000 1950
+Wire Wire Line
+	7000 2250 5300 2250
+Wire Wire Line
+	5300 2250 5300 2950
+Wire Wire Line
+	5300 2950 2900 2950
+Wire Wire Line
+	2900 2950 2900 2150
+Wire Wire Line
+	2900 2150 1100 2150
 $EndSCHEMATC

Commit message: Removed Supply Sensing from vi_filter.sch
Parts:
- gave numbers to parts that had none: 10
Connections:
- net GND: now also P101.30 (P30)
- net ip: now reaches P101.28 (P28)
- net in: now reaches P101.29 (P29)
- net vp: now reaches P101.31 (P31)
- net vn: now reaches P101.32 (P32)
