File: components_predev/output_driver/hardware/DAC.sch (KiCad schematic (older format))
At the start: 0 parts

Commit message: Added DAC, added disengage relay
Parts:
- added JP? (x2): Jumper_NC_Dual, symbol Jumper_NC_Dual
- added R?: 2k, symbol R_Small
- added R?: R_Small, symbol R_Small
- added RN? (x2): R_Pack06, symbol R_Pack06
- added U?: MAX5318, symbol MAX5318
Connections:
- new net: RN?.8 (R5.2), U?.1 (~RST)
- new net: RN?.10 (R3.2), U?.10 (TS/~SB)
- new net: RN?.9 (R4.2), U?.11 (PD)
- new net: RN?.12 (R1.2), U?.2 (~READY)
- new net: JP?.3, JP?.3, R?.1, U?.24 (VDDIO)
- new net: RN?.11 (R2.2), U?.3 (M/~Z)
- new net: R?.2, RN?.12 (R1.2), U?.4 (~BUSY)
- new net: RN?.7 (R6.2), U?.5 (~LDAC)
- new net: RN?.8 (R5.2), U?.6 (DOUT)
- new net: RN?.9 (R4.2), U?.7 (DIN)
- new net: RN?.10 (R3.2), U?.8 (SCLK)
- new net: RN?.11 (R2.2), U?.9 (~CS)
- new net: JP?.2, RN?.2 (R2.1)
- new net: JP?.2, RN?.3 (R3.1)
- new net DIN: RN?.4 (R4.1)
- new net DOUT: RN?.5 (R5.1)
- new net GND: JP?.1, JP?.1, U?.23 (DGND)
- new net PD: RN?.4 (R4.1)
- new net SCLK: RN?.3 (R3.1)
- new net v_ref: U?.18 (REF)
- new net ~BUSY: RN?.1 (R1.1)
- new net ~CS: R?.2, RN?.2 (R2.1)
- new net ~LDAC: RN?.6 (R6.1)
- new net ~READY: RN?.1 (R1.1)
- new net ~RST: RN?.5 (R5.1)
- no-connect marks 0 -> 2
Changed lines of the file:
@@
 $Descr A4 11693 8268
 encoding utf-8
-Sheet 1 7
+Sheet 6 7
 Title ""
 Date ""
@@
 Comment4 ""
 $EndDescr
+$Comp
+L MAX5318 U?
+U 1 1 5B296E71
+P 5150 3800
+F 0 "U?" H 5950 4550 60  0000 C CNN
+F 1 "MAX5318" H 5300 3800 60  0000 C CNN
+F 2 "" H 5150 3800 60  0001 C CNN
+F 3 "" H 5150 3800 60  0001 C CNN
+	1    5150 3800
+	1    0    0    -1
+$EndComp
+Text HLabel 7300 3400 2    60   Input ~ 0
+v_ref
+Wire Wire Line
+	6350 3400 7300 3400
+$Comp
+L GND #PWR?
+U 1 1 5B299996
+P 4900 4950
+F 0 "#PWR?" H 4900 4700 50  0001 C CNN
+F 1 "GND" H 4900 4800 50  0000 C CNN
+F 2 "" H 4900 4950 50  0000 C CNN
+F 3 "" H 4900 4950 50  0000 C CNN
+	1    4900 4950
+	1    0    0    -1
+$EndComp
+Wire Wire Line
+	4900 4950 4900 4750
+$Comp
+L R_Pack06 RN?
+U 1 1 5B2999B0
+P 3350 3400
+F 0 "RN?" V 2950 3400 50  0000 C CNN
+F 1 "R_Pack06" V 3650 3400 50  0000 C CNN
+F 2 "" V 3725 3400 50  0001 C CNN
+F 3 "" H 3350 3400 50  0000 C CNN
+	1    3350 3400
+	0    1    1    0
+$EndComp
+$Comp
+L R_Pack06 RN?
+U 1 1 5B299A19
+P 3350 4300
+F 0 "RN?" V 2950 4300 50  0000 C CNN
+F 1 "R_Pack06" V 3650 4300 50  0000 C CNN
+F 2 "" V 3725 4300 50  0001 C CNN
+F 3 "" H 3350 4300 50  0000 C CNN
+	1    3350 4300
+	0    1    1    0
+$EndComp
+Wire Wire Line
+	3950 2950 3950 3300
+Wire Wire Line
+	3950 3300 4250 3300
+Wire Wire Line
+	3900 3200 3900 3400
+Wire Wire Line
+	3900 3400 4250 3400
+Wire Wire Line
+	3850 3300 3850 3500
+Wire Wire Line
+	3850 3500 4250 3500
+Wire Wire Line
+	3800 3400 3800 3600
+Wire Wire Line
+	3800 3600 4250 3600
+Wire Wire Line
+	3750 3500 3750 3700
+Wire Wire Line
+	3750 3700 4250 3700
+Wire Wire Line
+	3700 3600 3700 3800
+Wire Wire Line
+	3700 3800 4250 3800
+Wire Wire Line
+	3700 3900 4250 3900
+Wire Wire Line
+	3550 4100 4250 4100
+Wire Wire Line
+	3550 4200 4250 4200
+Wire Wire Line
+	3550 4300 4250 4300
+Wire Wire Line
+	3550 4400 4250 4400
+Wire Wire Line
+	3700 3600 3550 3600
+Wire Wire Line
+	3550 3500 3750 3500
+Wire Wire Line
+	3550 3400 3800 3400
+Wire Wire Line
+	3550 3300 3850 3300
+Wire Wire Line
+	3550 3200 3900 3200
+Wire Wire Line
+	3550 3100 3950 3100
+Wire Wire Line
+	3550 4000 3700 4000
+Wire Wire Line
+	3700 4000 3700 3900
+NoConn ~ 3550 4500
+NoConn ~ 3150 4500
+Text HLabel 2000 3100 0    60   BiDi ~ 0
+~BUSY
+Wire Wire Line
+	2000 3100 3150 3100
+$Comp
+L R_Small R?
+U 1 1 5B29C829
+P 3950 2850
+F 0 "R?" H 3980 2870 50  0000 L CNN
+F 1 "2k" H 3980 2810 50  0000 L CNN
+F 2 "" H 3950 2850 50  0000 C CNN
+F 3 "" H 3950 2850 50  0000 C CNN
+	1    3950 2850
+	1    0    0    -1
+$EndComp
+Wire Wire Line
+	4900 2600 4900 2950
+Wire Wire Line
+	3100 2600 4900 2600
+Wire Wire Line
+	3950 2600 3950 2750
+Connection ~ 3950 3100
+$Comp
+L Jumper_NC_Dual JP?
+U 1 1 5B29C8D3
+P 2850 2600
+F 0 "JP?" H 2900 2500 50  0000 L CNN
+F 1 "Jumper_NC_Dual" H 2850 2700 50  0000 C BNN
+F 2 "" H 2850 2600 50  0000 C CNN
+F 3 "" H 2850 2600 50  0000 C CNN
+	1    2850 2600
+	1    0    0    -1
+$EndComp
+Connection ~ 3950 2600
+Wire Wire Line
+	3150 3200 2850 3200
+Wire Wire Line
+	2850 3200 2850 2700
+$Comp
+L GND #PWR?
+U 1 1 5B29C959
+P 2500 2800
+F 0 "#PWR?" H 2500 2550 50  0001 C CNN
+F 1 "GND" H 2500 2650 50  0000 C CNN
+F 2 "" H 2500 2800 50  0000 C CNN
+F 3 "" H 2500 2800 50  0000 C CNN
+	1    2500 2800
+	1    0    0    -1
+$EndComp
+$Comp
+L Jumper_NC_Dual JP?
+U 1 1 5B29C9AC
+P 2850 2150
+F 0 "JP?" H 2900 2050 50  0000 L CNN
+F 1 "Jumper_NC_Dual" H 2850 2250 50  0000 C BNN
+F 2 "" H 2850 2150 50  0000 C CNN
+F 3 "" H 2850 2150 50  0000 C CNN
+	1    2850 2150
+	1    0    0    -1
+$EndComp
+Wire Wire Line
+	3150 3300 2300 3300
+Wire Wire Line
+	2300 3300 2300 2350
+Wire Wire Line
+	2300 2350 2850 2350
+Wire Wire Line
+	2850 2350 2850 2250
+Wire Wire Line
+	3100 2150 3350 2150
+Wire Wire Line
+	3350 2150 3350 2600
+Connection ~ 3350 2600
+Wire Wire Line
+	2500 2150 2500 2800
+Wire Wire Line
+	2500 2600 2600 2600
+Wire Wire Line
+	2500 2150 2600 2150
+Connection ~ 2500 2600
+Text HLabel 2000 3400 0    60   Input ~ 0
+PD
+Wire Wire Line
+	2000 3400 3150 3400
+Text HLabel 2000 3500 0    60   Input ~ 0
+~RST
+Wire Wire Line
+	2000 3500 3150 3500
+Text HLabel 2000 3600 0    60   Input ~ 0
+~LDAC
+Wire Wire Line
+	2000 3600 3150 3600
+Text HLabel 2000 4000 0    60   Output ~ 0
+~READY
+Wire Wire Line
+	2000 4000 3150 4000
+Text HLabel 2000 4100 0    60   Input ~ 0
+~CS
+Wire Wire Line
+	2000 4100 3150 4100
+Text HLabel 2000 4200 0    60   Input ~ 0
+SCLK
+Wire Wire Line
+	2000 4200 3150 4200
+Text HLabel 2000 4300 0    60   Input ~ 0
+DIN
+Wire Wire Line
+	2000 4300 3150 4300
+Text HLabel 2000 4400 0    60   Output ~ 0
+DOUT
+Wire Wire Line
+	2000 4400 3150 4400
+$Comp
+L R_Small R?
+U 1 1 5B29D046
+P 2600 3800
+F 0 "R?" H 2630 3820 50  0000 L CNN
+F 1 "R_Small" H 2630 3760 50  0000 L CNN
+F 2 "" H 2600 3800 50  0000 C CNN
+F 3 "" H 2600 3800 50  0000 C CNN
+	1    2600 3800
+	0    1    1    0
+$EndComp
+Wire Wire Line
+	2500 3800 2300 3800
+Wire Wire Line
+	2300 3800 2300 4100
+Connection ~ 2300 4100
+Text HLabel 10500 3800 2    60   Output ~ 0
+output
 $EndSCHEMATC

Commit message: Put opamp gain stage into schematic
Parts:
- removed RN? (x2): R_Pack06, symbol R_Pack06
- added RN? (x3): R_Pack04, symbol R_Pack04
Connections:
- net DIN: now also RN?.3 (R3.1)
- net DOUT: now also RN?.4 (R4.1)
- net PD: now also RN?.4 (R4.1)
- net SCLK: now also RN?.2 (R2.1)
- net ~BUSY: now also RN?.1 (R1.1)
- net ~CS: now also RN?.1 (R1.1); no longer R?.2
- net ~LDAC: now also RN?.3 (R3.1)
- net ~READY: now also RN?.4 (R4.1)
- net ~RST: now also R?.1, RN?.2 (R2.1)
- net at U?.1 (~RST): now also RN?.7 (R2.2)
- net at U?.10 (TS/~SB): now also RN?.6 (R3.2)
- net at U?.11 (PD): now also RN?.5 (R4.2)
- net at U?.2 (~READY): now also RN?.5 (R4.2)
- net at U?.3 (M/~Z): now also RN?.7 (R2.2)
- net at R?.2, U?.4 (~BUSY): now also RN?.8 (R1.2)
- net at U?.5 (~LDAC): now also RN?.6 (R3.2)
- net at U?.6 (DOUT): now also RN?.5 (R4.2)
- net at U?.7 (DIN): now also RN?.6 (R3.2)
- net at U?.8 (SCLK): now also RN?.7 (R2.2)
- net at U?.9 (~CS): now also RN?.8 (R1.2)
- net at JP?.2: now also RN?.2 (R2.1)
- net at JP?.2: now also RN?.3 (R3.1)
Other:
- moved on the sheet: R?
Changed lines of the file:
@@
 Wire Wire Line
 	4900 4950 4900 4750
-$Comp
-L R_Pack06 RN?
-U 1 1 5B2999B0
-P 3350 3400
-F 0 "RN?" V 2950 3400 50  0000 C CNN
-F 1 "R_Pack06" V 3650 3400 50  0000 C CNN
-F 2 "" V 3725 3400 50  0001 C CNN
-F 3 "" H 3350 3400 50  0000 C CNN
-	1    3350 3400
-	0    1    1    0
-$EndComp
-$Comp
-L R_Pack06 RN?
-U 1 1 5B299A19
-P 3350 4300
-F 0 "RN?" V 2950 4300 50  0000 C CNN
-F 1 "R_Pack06" V 3650 4300 50  0000 C CNN
-F 2 "" V 3725 4300 50  0001 C CNN
-F 3 "" H 3350 4300 50  0000 C CNN
-	1    3350 4300
-	0    1    1    0
-$EndComp
 Wire Wire Line
 	3950 2950 3950 3300
@@
 	3800 3600 4250 3600
 Wire Wire Line
-	3750 3500 3750 3700
-Wire Wire Line
-	3750 3700 4250 3700
-Wire Wire Line
-	3700 3600 3700 3800
-Wire Wire Line
-	3700 3800 4250 3800
-Wire Wire Line
-	3700 3900 4250 3900
+	3100 3700 4250 3700
+Wire Wire Line
+	3100 3800 4250 3800
+Wire Wire Line
+	3100 3900 4250 3900
 Wire Wire Line
 	3550 4100 4250 4100
@@
 	3550 4400 4250 4400
 Wire Wire Line
-	3700 3600 3550 3600
-Wire Wire Line
-	3550 3500 3750 3500
-Wire Wire Line
 	3550 3400 3800 3400
 Wire Wire Line
@@
 Wire Wire Line
 	3550 3100 3950 3100
-Wire Wire Line
-	3550 4000 3700 4000
-Wire Wire Line
-	3700 4000 3700 3900
-NoConn ~ 3550 4500
-NoConn ~ 3150 4500
+NoConn ~ 3100 3600
+NoConn ~ 2700 3600
 Text HLabel 2000 3100 0    60   BiDi ~ 0
 ~BUSY
-Wire Wire Line
-	2000 3100 3150 3100
 $Comp
 L R_Small R?
@@
 Connection ~ 3950 2600
 Wire Wire Line
-	3150 3200 2850 3200
-Wire Wire Line
 	2850 3200 2850 2700
 $Comp
@@
 $EndComp
 Wire Wire Line
-	3150 3300 2300 3300
-Wire Wire Line
 	2300 3300 2300 2350
 Wire Wire Line
@@
 Text HLabel 2000 3400 0    60   Input ~ 0
 PD
-Wire Wire Line
-	2000 3400 3150 3400
-Text HLabel 2000 3500 0    60   Input ~ 0
+Text HLabel 2000 3700 0    60   Input ~ 0
 ~RST
-Wire Wire Line
-	2000 3500 3150 3500
-Text HLabel 2000 3600 0    60   Input ~ 0
+Text HLabel 2000 3800 0    60   Input ~ 0
 ~LDAC
-Wire Wire Line
-	2000 3600 3150 3600
-Text HLabel 2000 4000 0    60   Output ~ 0
+Text HLabel 2000 3900 0    60   Output ~ 0
 ~READY
-Wire Wire Line
-	2000 4000 3150 4000
 Text HLabel 2000 4100 0    60   Input ~ 0
 ~CS
-Wire Wire Line
-	2000 4100 3150 4100
 Text HLabel 2000 4200 0    60   Input ~ 0
 SCLK
-Wire Wire Line
-	2000 4200 3150 4200
 Text HLabel 2000 4300 0    60   Input ~ 0
 DIN
-Wire Wire Line
-	2000 4300 3150 4300
 Text HLabel 2000 4400 0    60   Output ~ 0
 DOUT
-Wire Wire Line
-	2000 4400 3150 4400
 $Comp
 L R_Small R?
 U 1 1 5B29D046
-P 2600 3800
-F 0 "R?" H 2630 3820 50  0000 L CNN
-F 1 "R_Small" H 2630 3760 50  0000 L CNN
-F 2 "" H 2600 3800 50  0000 C CNN
-F 3 "" H 2600 3800 50  0000 C CNN
-	1    2600 3800
-	0    1    1    0
-$EndComp
-Wire Wire Line
-	2500 3800 2300 3800
-Wire Wire Line
-	2300 3800 2300 4100
-Connection ~ 2300 4100
+P 2100 2700
+F 0 "R?" H 2130 2720 50  0000 L CNN
+F 1 "R_Small" H 2130 2660 50  0000 L CNN
+F 2 "" H 2100 2700 50  0000 C CNN
+F 3 "" H 2100 2700 50  0000 C CNN
+	1    2100 2700
+	-1   0    0    1
+$EndComp
 Text HLabel 10500 3800 2    60   Output ~ 0
 output
+$Comp
+L R_Pack04 RN?
+U 1 1 5B2A27DD
+P 3350 3300
+F 0 "RN?" V 3050 3300 50  0000 C CNN
+F 1 "R_Pack04" V 3550 3300 50  0000 C CNN
+F 2 "" V 3625 3300 50  0001 C CNN
+F 3 "" H 3350 3300 50  0000 C CNN
+	1    3350 3300
+	0    1    1    0
+$EndComp
+$Comp
+L R_Pack04 RN?
+U 1 1 5B2A2862
+P 3350 4300
+F 0 "RN?" V 3050 4300 50  0000 C CNN
+F 1 "R_Pack04" V 3550 4300 50  0000 C CNN
+F 2 "" V 3625 4300 50  0001 C CNN
+F 3 "" H 3350 4300 50  0000 C CNN
+	1    3350 4300
+	0    1    1    0
+$EndComp
+$Comp
+L R_Pack04 RN?
+U 1 1 5B2A28B9
+P 2900 3800
+F 0 "RN?" V 2600 3800 50  0000 C CNN
+F 1 "R_Pack04" V 3100 3800 50  0000 C CNN
+F 2 "" V 3175 3800 50  0001 C CNN
+F 3 "" H 2900 3800 50  0000 C CNN
+	1    2900 3800
+	0    1    1    0
+$EndComp
+Wire Wire Line
+	2000 3700 2700 3700
+Wire Wire Line
+	2700 3800 2000 3800
+Wire Wire Line
+	2000 3900 2700 3900
+Wire Wire Line
+	2000 3100 3150 3100
+Wire Wire Line
+	3150 3200 2850 3200
+Wire Wire Line
+	3150 3300 2300 3300
+Wire Wire Line
+	3150 3400 2000 3400
+Wire Wire Line
+	3150 4400 2000 4400
+Wire Wire Line
+	2000 4300 3150 4300
+Wire Wire Line
+	3150 4200 2000 4200
+Wire Wire Line
+	2000 4100 3150 4100
+Wire Wire Line
+	2100 2800 2100 3700
+Connection ~ 2100 3700
 $EndSCHEMATC

Commit message: Removed Supply Sensing from vi_filter.sch
Parts:
- gave numbers to parts that had none: 8
Changed lines of the file:
@@
 $EndDescr
 $Comp
-L MAX5318 U?
+L MAX5318 U601
 U 1 1 5B296E71
 P 5150 3800
-F 0 "U?" H 5950 4550 60  0000 C CNN
+F 0 "U601" H 5950 4550 60  0000 C CNN
 F 1 "MAX5318" H 5300 3800 60  0000 C CNN
 F 2 "" H 5150 3800 60  0001 C CNN
@@
 	6350 3400 7300 3400
 $Comp
-L GND #PWR?
+L GND #PWR047
 U 1 1 5B299996
 P 4900 4950
-F 0 "#PWR?" H 4900 4700 50  0001 C CNN
+F 0 "#PWR047" H 4900 4700 50  0001 C CNN
 F 1 "GND" H 4900 4800 50  0000 C CNN
 F 2 "" H 4900 4950 50  0000 C CNN
@@
 ~BUSY
 $Comp
-L R_Small R?
+L R_Small R602
 U 1 1 5B29C829
 P 3950 2850
-F 0 "R?" H 3980 2870 50  0000 L CNN
+F 0 "R602" H 3980 2870 50  0000 L CNN
 F 1 "2k" H 3980 2810 50  0000 L CNN
 F 2 "" H 3950 2850 50  0000 C CNN
@@
 Connection ~ 3950 3100
 $Comp
-L Jumper_NC_Dual JP?
+L Jumper_NC_Dual JP602
 U 1 1 5B29C8D3
 P 2850 2600
-F 0 "JP?" H 2900 2500 50  0000 L CNN
+F 0 "JP602" H 2900 2500 50  0000 L CNN
 F 1 "Jumper_NC_Dual" H 2850 2700 50  0000 C BNN
 F 2 "" H 2850 2600 50  0000 C CNN
@@
 	2850 3200 2850 2700
 $Comp
-L GND #PWR?
+L GND #PWR048
 U 1 1 5B29C959
 P 2500 2800
-F 0 "#PWR?" H 2500 2550 50  0001 C CNN
+F 0 "#PWR048" H 2500 2550 50  0001 C CNN
 F 1 "GND" H 2500 2650 50  0000 C CNN
 F 2 "" H 2500 2800 50  0000 C CNN
@@
 $EndComp
 $Comp
-L Jumper_NC_Dual JP?
+L Jumper_NC_Dual JP601
 U 1 1 5B29C9AC
 P 2850 2150
-F 0 "JP?" H 2900 2050 50  0000 L CNN
+F 0 "JP601" H 2900 2050 50  0000 L CNN
 F 1 "Jumper_NC_Dual" H 2850 2250 50  0000 C BNN
 F 2 "" H 2850 2150 50  0000 C CNN
@@
 DOUT
 $Comp
-L R_Small R?
+L R_Small R601
 U 1 1 5B29D046
 P 2100 2700
-F 0 "R?" H 2130 2720 50  0000 L CNN
+F 0 "R601" H 2130 2720 50  0000 L CNN
 F 1 "R_Small" H 2130 2660 50  0000 L CNN
 F 2 "" H 2100 2700 50  0000 C CNN
@@
 output
 $Comp
-L R_Pack04 RN?
+L R_Pack04 RN602
 U 1 1 5B2A27DD
 P 3350 3300
-F 0 "RN?" V 3050 3300 50  0000 C CNN
+F 0 "RN602" V 3050 3300 50  0000 C CNN
 F 1 "R_Pack04" V 3550 3300 50  0000 C CNN
 F 2 "" V 3625 3300 50  0001 C CNN
@@
 $EndComp
 $Comp
-L R_Pack04 RN?
+L R_Pack04 RN603
 U 1 1 5B2A2862
 P 3350 4300
-F 0 "RN?" V 3050 4300 50  0000 C CNN
+F 0 "RN603" V 3050 4300 50  0000 C CNN
 F 1 "R_Pack04" V 3550 4300 50  0000 C CNN
 F 2 "" V 3625 4300 50  0001 C CNN
@@
 $EndComp
 $Comp
-L R_Pack04 RN?
+L R_Pack04 RN601
 U 1 1 5B2A28B9
 P 2900 3800
-F 0 "RN?" V 2600 3800 50  0000 C CNN
+F 0 "RN601" V 2600 3800 50  0000 C CNN
 F 1 "R_Pack04" V 3100 3800 50  0000 C CNN
 F 2 "" V 3175 3800 50  0001 C CNN
