File: components_predev/output_driver/hardware/ADC.sch (KiCad schematic (older format))
At the start: 0 parts

Commit message: Added ADC Symbol, Started Wiring
Parts:
- added C? (x4): 10u, symbol C_Small
- added RN?: 33, symbol R_Pack08
- added U?: MAX11960, symbol MAX11960
Connections:
- new net: RN?.13 (R4.2), U?.11 (SCLK)
- new net: RN?.10 (R7.2), U?.12 (CNVSTB)
- new net: RN?.14 (R3.2), U?.13 (CNVSTA)
- new net: RN?.11 (R6.2), U?.14 (DINB)
- new net: RN?.15 (R2.2), U?.15 (DINA)
- new net: C?.2, U?.24 (REF1A)
- new net: C?.2, U?.25 (REF1B)
- new net: C?.2, U?.26 (REF2A)
- new net: C?.2, U?.27 (REF2B)
- new net: RN?.12 (R5.2), U?.6 (DOUTB)
- new net: RN?.16 (R1.2), U?.7 (DOUTA)
- new net CNVSTA: RN?.3 (R3.1)
- new net CNVSTB: RN?.7 (R7.1)
- new net DINA: RN?.2 (R2.1)
- new net DINB: RN?.6 (R6.1)
- new net DOUTA: RN?.1 (R1.1)
- new net DOUTB: RN?.5 (R5.1)
- new net GND: C?.1, C?.1, C?.1, C?.1, U?.28 (REFGND), U?.29 (REFGND), U?.3 (DGND), U?.30 (REFGND), U?.8 (DGND)
- new net GNDPWR: U?.16 (AGND), U?.19 (AGND), U?.20 (AGND), U?.33 (AGND)
- new net SCLK: RN?.4 (R4.1)
Changed lines of the file:
@@
 Comment4 ""
 $EndDescr
+$Comp
+L MAX11960 U?
+U 1 1 5B1A4BE8
+P 5550 3900
+F 0 "U?" H 6050 5000 60  0000 C CNN
+F 1 "MAX11960" H 5500 3900 60  0000 C CNN
+F 2 "" H 7875 5325 60  0001 C CNN
+F 3 "" H 7875 5325 60  0001 C CNN
+	1    5550 3900
+	1    0    0    -1
+$EndComp
+$Comp
+L GNDPWR #PWR?
+U 1 1 5B1A5AC8
+P 4850 5250
+F 0 "#PWR?" H 4850 5050 50  0001 C CNN
+F 1 "GNDPWR" H 4850 5120 50  0000 C CNN
+F 2 "" H 4850 5200 50  0000 C CNN
+F 3 "" H 4850 5200 50  0000 C CNN
+	1    4850 5250
+	1    0    0    -1
+$EndComp
+$Comp
+L GND #PWR?
+U 1 1 5B1A5ADE
+P 5400 5250
+F 0 "#PWR?" H 5400 5000 50  0001 C CNN
+F 1 "GND" H 5400 5100 50  0000 C CNN
+F 2 "" H 5400 5250 50  0000 C CNN
+F 3 "" H 5400 5250 50  0000 C CNN
+	1    5400 5250
+	1    0    0    -1
+$EndComp
+$Comp
+L GND #PWR?
+U 1 1 5B1A5AF4
+P 5650 5250
+F 0 "#PWR?" H 5650 5000 50  0001 C CNN
+F 1 "GND" H 5650 5100 50  0000 C CNN
+F 2 "" H 5650 5250 50  0000 C CNN
+F 3 "" H 5650 5250 50  0000 C CNN
+	1    5650 5250
+	1    0    0    -1
+$EndComp
+Wire Wire Line
+	5650 5250 5650 5100
+Wire Wire Line
+	5400 5250 5400 5100
+Wire Wire Line
+	4850 5250 4850 5100
+Wire Wire Line
+	4850 5200 5150 5200
+Wire Wire Line
+	5150 5200 5150 5100
+Connection ~ 4850 5200
+Wire Wire Line
+	5050 5100 5050 5200
+Connection ~ 5050 5200
+Wire Wire Line
+	4950 5100 4950 5200
+Connection ~ 4950 5200
+Wire Wire Line
+	5400 5200 5500 5200
+Wire Wire Line
+	5500 5200 5500 5100
+Connection ~ 5400 5200
+Wire Wire Line
+	5650 5200 5850 5200
+Wire Wire Line
+	5850 5200 5850 5100
+Connection ~ 5650 5200
+Wire Wire Line
+	5750 5100 5750 5200
+Connection ~ 5750 5200
+$Comp
+L C_Small C?
+U 1 1 5B1A5BE6
+P 6800 4500
+F 0 "C?" H 6810 4570 50  0000 L CNN
+F 1 "10u" H 6810 4420 50  0000 L CNN
+F 2 "" H 6800 4500 50  0000 C CNN
+F 3 "" H 6800 4500 50  0000 C CNN
+	1    6800 4500
+	0    1    1    0
+$EndComp
+$Comp
+L C_Small C?
+U 1 1 5B1A5C2F
+P 7100 4600
+F 0 "C?" H 7110 4670 50  0000 L CNN
+F 1 "10u" H 7110 4520 50  0000 L CNN
+F 2 "" H 7100 4600 50  0000 C CNN
+F 3 "" H 7100 4600 50  0000 C CNN
+	1    7100 4600
+	0    1    1    0
+$EndComp
+Wire Wire Line
+	6700 4500 6500 4500
+Wire Wire Line
+	7000 4600 6500 4600
+$Comp
+L GND #PWR?
+U 1 1 5B1A5C9E
+P 7450 4550
+F 0 "#PWR?" H 7450 4300 50  0001 C CNN
+F 1 "GND" H 7450 4400 50  0000 C CNN
+F 2 "" H 7450 4550 50  0000 C CNN
+F 3 "" H 7450 4550 50  0000 C CNN
+	1    7450 4550
+	0    -1   -1   0
+$EndComp
+Wire Wire Line
+	7450 4550 7350 4550
+Wire Wire Line
+	7350 4500 7350 4600
+Wire Wire Line
+	7350 4500 6900 4500
+Wire Wire Line
+	7350 4600 7200 4600
+Connection ~ 7350 4550
+$Comp
+L C_Small C?
+U 1 1 5B1A5D50
+P 6800 3250
+F 0 "C?" H 6810 3320 50  0000 L CNN
+F 1 "10u" H 6810 3170 50  0000 L CNN
+F 2 "" H 6800 3250 50  0000 C CNN
+F 3 "" H 6800 3250 50  0000 C CNN
+	1    6800 3250
+	0    1    1    0
+$EndComp
+$Comp
+L C_Small C?
+U 1 1 5B1A5D56
+P 7100 3350
+F 0 "C?" H 7110 3420 50  0000 L CNN
+F 1 "10u" H 7110 3270 50  0000 L CNN
+F 2 "" H 7100 3350 50  0000 C CNN
+F 3 "" H 7100 3350 50  0000 C CNN
+	1    7100 3350
+	0    1    1    0
+$EndComp
+Wire Wire Line
+	6700 3250 6500 3250
+Wire Wire Line
+	7000 3350 6500 3350
+$Comp
+L GND #PWR?
+U 1 1 5B1A5D5E
+P 7450 3300
+F 0 "#PWR?" H 7450 3050 50  0001 C CNN
+F 1 "GND" H 7450 3150 50  0000 C CNN
+F 2 "" H 7450 3300 50  0000 C CNN
+F 3 "" H 7450 3300 50  0000 C CNN
+	1    7450 3300
+	0    -1   -1   0
+$EndComp
+Wire Wire Line
+	7450 3300 7350 3300
+Wire Wire Line
+	7350 3250 7350 3350
+Wire Wire Line
+	7350 3250 6900 3250
+Wire Wire Line
+	7350 3350 7200 3350
+Connection ~ 7350 3300
+$Comp
+L R_Pack08 RN?
+U 1 1 5B1A6087
+P 3750 4000
+F 0 "RN?" V 3250 4000 50  0000 C CNN
+F 1 "33" V 4150 4000 50  0000 C CNN
+F 2 "" V 4225 4000 50  0001 C CNN
+F 3 "" H 3750 4000 50  0000 C CNN
+	1    3750 4000
+	0    1    1    0
+$EndComp
+Wire Wire Line
+	3950 3600 4450 3600
+Wire Wire Line
+	4450 3700 3950 3700
+Wire Wire Line
+	3950 3800 4450 3800
+Wire Wire Line
+	4450 3900 3950 3900
+Wire Wire Line
+	3950 4000 4450 4000
+Wire Wire Line
+	3950 4100 4450 4100
+Wire Wire Line
+	3950 4200 4450 4200
+Text HLabel 2550 3700 0    60   Input ~ 0
+DINA
+Text HLabel 2550 4100 0    60   Input ~ 0
+DINB
+Text HLabel 2550 3600 0    60   Output ~ 0
+DOUTA
+Text HLabel 2550 4000 0    60   Output ~ 0
+DOUTB
+Text HLabel 2550 4200 0    60   Input ~ 0
+CNVSTB
+Text HLabel 2550 3800 0    60   Input ~ 0
+CNVSTA
+Text HLabel 2550 3900 0    60   Input ~ 0
+SCLK
+Wire Wire Line
+	2550 3600 3550 3600
+Wire Wire Line
+	3550 3700 2550 3700
+Wire Wire Line
+	2550 3800 3550 3800
+Wire Wire Line
+	3550 3900 2550 3900
+Wire Wire Line
+	2550 4000 3550 4000
+Wire Wire Line
+	3550 4100 2550 4100
+Wire Wire Line
+	2550 4200 3550 4200
 $EndSCHEMATC

Commit message: Added reference voltage circuit
Parts:
- added C? (x5): C_Small, symbol C_Small
- added C? (x2): CP1_Small, symbol CP1_Small
- added L? (x2): L_Small, symbol L_Small
- added R? (x2): R_Small, symbol R_Small
- added RN?: Voltage_Divider, symbol Voltage_Divider
- added U?: AD54xx, symbol AD54xx
- added U? (x2): LTC2055, symbol LTC2055
Connections:
- net GND: now also C?.1, C?.1, C?.1, C?.1, C?.2, C?.2, RN?.3, U?.4 (GND), U?.4 (V-)
- net v_meas-: now reaches U?.1 (AINA-)
- net v_meas+: now reaches U?.2 (AINA+)
- net V_ref: now reaches U?.23 (REFIN)
- net V_ref: now also RN?.1, U?.1, U?.2 (-)
- net i_meas-: now reaches U?.31 (AINB-)
- net i_meas+: now reaches U?.32 (AINB+)
- net at U?.4 (OVDD): now also U?.5 (OVDD), C?.2, C?.2, C?.2, L?.2
- new net: C?.2, L?.2, U?.2 (VIn)
- new net: R?.1, R?.1, U?.6 (VOut)
- new net: C?.1, R?.2, U?.3 (+)
- new net: C?.1, C?.2, R?.2
- new net: RN?.2, U?.6 (+)
- new net +3V3: L?.1
- new net +5V: C?.1, L?.1, U?.8 (V+)
- new net v_ref_2: U?.5 (-), U?.7
- no-connect marks 0 -> 2
Other:
- moved on the sheet: C?, RN?, U?

Commit message: Added ADC Voltage Regulation and Reference Heater
Parts:
- added C? (x10): C_Small, symbol C_Small
- added C? (x2): CP1_Small, symbol CP1_Small
- added Q?: Q_NMOS_DGS, symbol Q_NMOS_DGS
- added R?: R, symbol R
- added R? (x2): R_Small, symbol R_Small
- added RV?: POT_TRIM, symbol POT_TRIM
- added U? (x3): NCP508, symbol NCP508
- added U?: LMT88, symbol LMT88
- added U?: MIC7211, symbol MIC7211
- U?: value AD54xx -> ADR5433
Connections:
- net +3V3: now also C?.1, C?.1, U?.1 (In), U?.1 (In), U?.3 (En), U?.3 (En)
- net +5V: now also C?.1, C?.1, C?.1, C?.2, R?.1, U?.1 (In), U?.2 (V+), U?.3 (En), U?.4 (V+)
- net GND: now also C?.1, C?.2, C?.2, C?.2, C?.2, C?.2, C?.2, C?.2, C?.2, C?.2, C?.2, C?.2, Q?.3 (S), R?.2, RV?.3, U?.2 (GND), U?.2 (GND), U?.2 (GND), U?.2 (GND), U?.5 (GND), U?.5 (V-)
- net at U?.10 (DVDD): now also U?.9 (DVDD), C?.1, C?.1, U?.5 (Out)
- net at U?.17 (REFVDD): now also U?.18 (REFVDD), C?.1, C?.1, U?.5 (Out)
- net at U?.21 (AVDD): now also U?.22 (AVDD), C?.1, C?.1, U?.5 (Out)
- new net: Q?.1 (D), R?.2
- new net: Q?.2 (G), R?.1, U?.1
- new net: U?.3 (V_out), U?.4 (_)
- new net: RV?.2, U?.3 (+)
- new net: R?.2, RV?.1
- new net +12V: R?.1
Other:
- moved on the sheet: C?, L?, R?, RN?, U?, U?A, U?B

Commit message: Added DAC, added disengage relay
Parts:
- U?: value ADR5433 -> ADR4533
Connections:
- no-connect marks 2 -> 4
Changed lines of the file:
@@
 P 2500 8650
 F 0 "U?" H 2600 8800 60  0000 C CNN
-F 1 "ADR5433" H 2700 8250 60  0000 C CNN
+F 1 "ADR4533" H 2700 8250 60  0000 C CNN
 F 2 "" H 2500 8650 60  0001 C CNN
 F 3 "" H 2500 8650 60  0001 C CNN
@@
 $EndComp
 $Comp
-L GND #PWR?
-U 1 1 5B227F91
-P 0 5050
-F 0 "#PWR?" H 0   4800 50  0001 C CNN
-F 1 "GND" H 0   4900 50  0000 C CNN
-F 2 "" H 0   5050 50  0000 C CNN
-F 3 "" H 0   5050 50  0000 C CNN
-	1    0    5050
-	0    1    1    0
-$EndComp
-$Comp
 L +5V #PWR?
 U 1 1 5B22994C
@@
 	6550 9150 6700 9150
 Wire Wire Line
-	6600 9150 6600 8700
+	6600 8700 6600 9550
 Wire Wire Line
 	6600 8700 5750 8700
@@
 Wire Wire Line
 	2450 6500 3350 6500
+NoConn ~ 3050 5650
+NoConn ~ 2650 5650
+Text HLabel 6700 8300 2    60   Output ~ 0
+v_ref
+Wire Wire Line
+	6700 8300 6300 8300
+Wire Wire Line
+	6300 8300 6300 8550
+Connection ~ 6300 8550
+Text HLabel 6700 9550 2    60   Output ~ 0
+v_ref_2
+Wire Wire Line
+	6600 9550 6700 9550
 $EndSCHEMATC

Commit message: Removed Supply Sensing from vi_filter.sch
Parts:
- gave numbers to parts that had none: 42

Commit message: Added Supply Schematic
Changed lines of the file:
@@
 $EndComp
 Wire Wire Line
-	4750 6450 4750 6550
-Wire Wire Line
-	4750 6550 4750 6600
-Wire Wire Line
-	4500 6450 4500 6550
-Wire Wire Line
-	4500 6550 4500 6600
-Wire Wire Line
-	3950 6450 3950 6550
-Wire Wire Line
-	3950 6550 3950 6600
-Wire Wire Line
-	3950 6550 4050 6550
-Wire Wire Line
-	4050 6550 4150 6550
-Wire Wire Line
-	4150 6550 4250 6550
+	4750 6450 4750 6600
+Wire Wire Line
+	4500 6450 4500 6600
+Wire Wire Line
+	3950 6450 3950 6600
+Wire Wire Line
+	3950 6550 4250 6550
 Wire Wire Line
 	4250 6550 4250 6450
@@
 Connection ~ 4500 6550
 Wire Wire Line
-	4750 6550 4850 6550
-Wire Wire Line
-	4850 6550 4950 6550
+	4750 6550 4950 6550
 Wire Wire Line
 	4950 6550 4950 6450
@@
 	6550 5900 6450 5900
 Wire Wire Line
-	6450 5850 6450 5900
-Wire Wire Line
-	6450 5900 6450 5950
+	6450 5850 6450 5950
 Wire Wire Line
 	6450 5850 6000 5850
@@
 	6550 4650 6450 4650
 Wire Wire Line
-	6450 4600 6450 4650
-Wire Wire Line
-	6450 4650 6450 4700
+	6450 4600 6450 4700
 Wire Wire Line
 	6450 4600 6000 4600
@@
 	3750 9550 3750 9350
 Wire Wire Line
-	3750 8950 3750 9050
-Wire Wire Line
-	3750 9050 3750 9150
+	3750 8950 3750 9150
 Wire Wire Line
 	3550 9050 3750 9050
@@
 	3750 8750 3750 8650
 Wire Wire Line
-	3550 8650 3750 8650
-Wire Wire Line
-	3750 8650 4600 8650
-Wire Wire Line
-	3000 8650 3200 8650
-Wire Wire Line
-	3200 8650 3350 8650
+	3550 8650 4600 8650
+Wire Wire Line
+	3000 8650 3350 8650
 Wire Wire Line
 	3350 9050 3200 9050
@@
 	1850 9000 1850 8650
 Wire Wire Line
-	1750 8650 1850 8650
-Wire Wire Line
-	1850 8650 2000 8650
+	1750 8650 2000 8650
 Connection ~ 1850 8650
 Wire Wire Line
@@
 Connection ~ 3750 8650
 Wire Wire Line
-	5200 8550 5500 8550
-Wire Wire Line
-	5500 8550 6300 8550
-Wire Wire Line
-	6300 8550 6800 8550
-Wire Wire Line
-	5500 7800 5500 8550
-Wire Wire Line
-	5500 8550 5500 9000
+	5200 8550 6800 8550
+Wire Wire Line
+	5500 7800 5500 9000
 Wire Wire Line
 	5500 7800 4250 7800
@@
 Connection ~ 5500 8550
 Wire Wire Line
-	6550 9150 6600 9150
-Wire Wire Line
-	6600 9150 6700 9150
-Wire Wire Line
-	6600 8700 6600 9150
-Wire Wire Line
-	6600 9150 6600 9550
+	6550 9150 6700 9150
+Wire Wire Line
+	6600 8700 6600 9550
 Wire Wire Line
 	6600 8700 5750 8700
@@
 	5950 9250 5650 9250
 Wire Wire Line
-	4850 8050 4850 8150
-Wire Wire Line
-	4850 8150 4850 8250
+	4850 8050 4850 8250
 Wire Wire Line
 	4950 8150 4850 8150
@@
 	6400 5250 5600 5250
 Wire Wire Line
-	3250 3550 3350 3550
-Wire Wire Line
-	3350 3550 3550 3550
-Wire Wire Line
-	3550 3550 3750 3550
-Wire Wire Line
-	3750 3550 3950 3550
-Wire Wire Line
-	3950 3550 4050 3550
+	3250 3550 4050 3550
 Wire Wire Line
 	3350 3700 3350 3550
@@
 	3450 4050 3450 4000
 Wire Wire Line
-	3350 4000 3450 4000
-Wire Wire Line
-	3450 4000 3550 4000
-Wire Wire Line
-	3550 4000 3750 4000
+	3350 4000 3750 4000
 Wire Wire Line
 	3550 4000 3550 3900
@@
 	2850 2950 2850 2850
 Wire Wire Line
-	4350 2350 4350 3550
-Wire Wire Line
-	4350 3550 4350 4050
-Wire Wire Line
-	3300 2350 3550 2350
-Wire Wire Line
-	3550 2350 3750 2350
-Wire Wire Line
-	3750 2350 4350 2350
+	4350 2350 4350 4050
+Wire Wire Line
+	3300 2350 4350 2350
 Wire Wire Line
 	3750 2500 3750 2350
@@
 	3650 2950 3650 2900
 Wire Wire Line
-	3550 2900 3650 2900
-Wire Wire Line
-	3650 2900 3750 2900
+	3550 2900 3750 2900
 Wire Wire Line
 	3550 2900 3550 2700
@@
 	2850 1900 2850 1800
 Wire Wire Line
-	3300 1300 3550 1300
-Wire Wire Line
-	3550 1300 3750 1300
-Wire Wire Line
-	3750 1300 4650 1300
+	3300 1300 4650 1300
 Wire Wire Line
 	3750 1450 3750 1300
@@
 	3650 1900 3650 1850
 Wire Wire Line
-	3550 1850 3650 1850
-Wire Wire Line
-	3650 1850 3750 1850
+	3550 1850 3750 1850
 Wire Wire Line
 	3550 1850 3550 1650
@@
 Connection ~ 3650 1850
 Wire Wire Line
-	4650 1300 4650 3550
-Wire Wire Line
-	4650 3550 4650 4050
+	4650 1300 4650 4050
 Wire Wire Line
 	4550 3550 4550 4050
@@
 Connection ~ 4650 3550
 Wire Wire Line
-	1250 1300 1500 1300
-Wire Wire Line
-	1500 1300 2050 1300
-Wire Wire Line
-	2050 1300 2300 1300
-Wire Wire Line
-	2300 1300 2400 1300
+	1250 1300 2400 1300
 Wire Wire Line
 	2050 1300 2050 2350
 Wire Wire Line
-	2050 2350 2300 2350
-Wire Wire Line
-	2300 2350 2400 2350
+	2050 2350 2400 2350
 Wire Wire Line
 	1500 1300 1500 1450
 Connection ~ 2050 1300
 Wire Wire Line
-	1250 1200 1250 1300
-Wire Wire Line
-	1250 1300 1250 1450
+	1250 1200 1250 1450
 Connection ~ 1500 1300
 Connection ~ 1250 1300
@@
 Connection ~ 2300 2350
 Wire Wire Line
-	1250 1650 1250 1750
-Wire Wire Line
-	1250 1750 1250 1850
+	1250 1650 1250 1850
 Wire Wire Line
 	1250 1750 1500 1750
@@
 	5400 1900 5400 1850
 Wire Wire Line
-	5300 1850 5400 1850
-Wire Wire Line
-	5400 1850 5500 1850
+	5300 1850 5500 1850
 Wire Wire Line
 	5500 1850 5500 1650
@@
 Connection ~ 5400 1850
 Wire Wire Line
-	6650 1300 6750 1300
-Wire Wire Line
-	6750 1300 7000 1300
-Wire Wire Line
-	7000 1300 7250 1300
+	6650 1300 7250 1300
 Wire Wire Line
 	6650 1450 6750 1450
@@
 Connection ~ 6750 1300
 Wire Wire Line
-	4950 1300 4950 3550
-Wire Wire Line
-	4950 3550 4950 4050
-Wire Wire Line
-	4950 1300 5300 1300
-Wire Wire Line
-	5300 1300 5500 1300
-Wire Wire Line
-	5500 1300 5750 1300
+	4950 1300 4950 4050
+Wire Wire Line
+	4950 1300 5750 1300
 Wire Wire Line
 	4850 4050 4850 3550
@@
 	7000 1300 7000 1450
 Wire Wire Line
-	7250 1200 7250 1300
-Wire Wire Line
-	7250 1300 7250 1450
+	7250 1200 7250 1450
 Connection ~ 7000 1300
 Connection ~ 7250 1300
 Wire Wire Line
-	7250 1650 7250 1750
-Wire Wire Line
-	7250 1750 7250 1850
+	7250 1650 7250 1850
 Wire Wire Line
 	7250 1750 7000 1750
@@
 Connection ~ 7250 1750
 Wire Wire Line
-	1300 7800 1300 7900
-Wire Wire Line
-	1300 7900 1300 8050
+	1300 7800 1300 8050
 Wire Wire Line
 	1850 7900 2500 7900
@@
 	3350 6850 3250 6850
 Wire Wire Line
-	3350 6350 3350 6500
-Wire Wire Line
-	3350 6500 3350 6850
+	3350 6350 3350 6850
 Wire Wire Line
 	1300 7900 1450 7900
@@
 	1300 7550 1650 7550
 Wire Wire Line
-	1650 7450 1650 7550
-Wire Wire Line
-	1650 7550 1650 7600
+	1650 7450 1650 7600
 Connection ~ 1650 7550
 Wire Wire Line
@@
 	2300 7200 2300 7050
 Wire Wire Line
-	2250 7050 2300 7050
-Wire Wire Line
-	2300 7050 2350 7050
+	2250 7050 2350 7050
 Connection ~ 2300 7050
 Wire Wire Line
-	1950 7050 2000 7050
-Wire Wire Line
-	2000 7050 2050 7050
+	1950 7050 2050 7050
 Wire Wire Line
 	2000 7000 2000 7050
@@
 $EndComp
 Wire Wire Line
-	1050 7150 1050 7050
-Wire Wire Line
-	1050 7050 1050 6500
+	1050 6500 1050 7150
 Wire Wire Line
 	1050 6500 1400 6500

Commit message: Added test points
Parts:
- added W? (x7): TEST_1P, symbol TEST_1P
Connections:
- net V_ref: now also W?.1
- net at C708.1, C711.1, U705.5 (Out)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: now also W?.1
- net at C716.1, C717.1, U706.17 (REFVDD)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: now also W?.1
- net at C707.1, C710.1, U704.5 (Out)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: now also W?.1
- net at C705.2, C709.2, C712.2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: now also W?.1
- net at R704.1, R705.1, U702.6 (VOut): now also W?.1
- net at C713.1, R704.2, U707.3 (+): now also W?.1
Changed lines of the file:
@@
 Connection ~ 3750 9050
 Wire Wire Line
-	3750 8750 3750 8650
+	3750 8400 3750 8750
 Wire Wire Line
 	3550 8650 4600 8650
@@
 	3000 8650 3350 8650
 Wire Wire Line
-	3350 9050 3200 9050
-Wire Wire Line
-	3200 9050 3200 8650
+	3200 9050 3350 9050
+Wire Wire Line
+	3200 8400 3200 9050
 Connection ~ 3200 8650
 Wire Wire Line
@@
 	2850 3550 2850 3400
 Wire Wire Line
-	4050 3550 4050 4050
+	4050 3400 4050 4050
 Connection ~ 3950 3550
 Wire Wire Line
@@
 	2850 2950 2850 2850
 Wire Wire Line
-	4350 2350 4350 4050
+	4350 2200 4350 4050
 Wire Wire Line
 	3300 2350 4350 2350
@@
 Connection ~ 3650 1850
 Wire Wire Line
-	4650 1300 4650 4050
+	4650 1150 4650 4050
 Wire Wire Line
 	4550 3550 4550 4050
@@
 Connection ~ 6750 1300
 Wire Wire Line
-	4950 1300 4950 4050
+	4950 1150 4950 4050
 Wire Wire Line
 	4950 1300 5750 1300
@@
 	6800 8300 6300 8300
 Wire Wire Line
-	6300 8300 6300 8550
+	6300 8150 6300 8550
 Connection ~ 6300 8550
 Text HLabel 6700 9550 2    60   Output ~ 0
@@
 Wire Wire Line
 	6600 9550 6700 9550
+$Comp
+L TEST_1P W?
+U 1 1 5B3ACD8A
+P 4050 3400
+F 0 "W?" H 4050 3670 50  0000 C CNN
+F 1 "TEST_1P" H 4050 3600 50  0000 C CNN
+F 2 "" H 4250 3400 50  0000 C CNN
+F 3 "" H 4250 3400 50  0000 C CNN
+	1    4050 3400
+	1    0    0    -1
+$EndComp
+$Comp
+L TEST_1P W?
+U 1 1 5B3ACE6F
+P 4350 2200
+F 0 "W?" H 4350 2470 50  0000 C CNN
+F 1 "TEST_1P" H 4350 2400 50  0000 C CNN
+F 2 "" H 4550 2200 50  0000 C CNN
+F 3 "" H 4550 2200 50  0000 C CNN
+	1    4350 2200
+	1    0    0    -1
+$EndComp
+$Comp
+L TEST_1P W?
+U 1 1 5B3ACF61
+P 4650 1150
+F 0 "W?" H 4650 1420 50  0000 C CNN
+F 1 "TEST_1P" H 4650 1350 50  0000 C CNN
+F 2 "" H 4850 1150 50  0000 C CNN
+F 3 "" H 4850 1150 50  0000 C CNN
+	1    4650 1150
+	1    0    0    -1
+$EndComp
+$Comp
+L TEST_1P W?
+U 1 1 5B3AD029
+P 4950 1150
+F 0 "W?" H 4950 1420 50  0000 C CNN
+F 1 "TEST_1P" H 4950 1350 50  0000 C CNN
+F 2 "" H 5150 1150 50  0000 C CNN
+F 3 "" H 5150 1150 50  0000 C CNN
+	1    4950 1150
+	1    0    0    -1
+$EndComp
+Connection ~ 4950 1300
+Connection ~ 4650 1300
+Connection ~ 4350 2350
+Connection ~ 4050 3550
+$Comp
+L TEST_1P W?
+U 1 1 5B3AD5C7
+P 6300 8150
+F 0 "W?" H 6300 8420 50  0000 C CNN
+F 1 "TEST_1P" H 6300 8350 50  0000 C CNN
+F 2 "" H 6500 8150 50  0000 C CNN
+F 3 "" H 6500 8150 50  0000 C CNN
+	1    6300 8150
+	1    0    0    -1
+$EndComp
+Connection ~ 6300 8300
+$Comp
+L TEST_1P W?
+U 1 1 5B3AD82A
+P 3750 8400
+F 0 "W?" H 3750 8670 50  0000 C CNN
+F 1 "TEST_1P" H 3750 8600 50  0000 C CNN
+F 2 "" H 3950 8400 50  0000 C CNN
+F 3 "" H 3950 8400 50  0000 C CNN
+	1    3750 8400
+	1    0    0    -1
+$EndComp
+$Comp
+L TEST_1P W?
+U 1 1 5B3ADA32
+P 3200 8400
+F 0 "W?" H 3200 8670 50  0000 C CNN
+F 1 "TEST_1P" H 3200 8600 50  0000 C CNN
+F 2 "" H 3400 8400 50  0000 C CNN
+F 3 "" H 3400 8400 50  0000 C CNN
+	1    3200 8400
+	1    0    0    -1
+$EndComp
 $EndSCHEMATC
