File: components_predev/output_driver/hardware/inrush_limiter.sch (KiCad schematic (older format))
At the start: 22 parts

Commit message: Moved output stage to new schematic sheet
Changed lines of the file:
@@
 $Descr A4 11693 8268
 encoding utf-8
-Sheet 2 2
+Sheet 2 3
 Title ""
 Date ""
@@
 	3650 2500 3500 2500
 Wire Wire Line
-	3500 2100 3500 2500
-Wire Wire Line
-	3500 2500 3500 2750
+	3500 2100 3500 2750
 Connection ~ 3500 2100
 Wire Wire Line
 	3950 2500 4100 2500
 Wire Wire Line
-	4100 2400 4100 2500
-Wire Wire Line
-	4100 2500 4100 2750
+	4100 2400 4100 2750
 Wire Wire Line
 	3500 2750 3650 2750
@@
 $EndComp
 Wire Wire Line
-	5450 2850 5450 2750
-Wire Wire Line
-	5450 2750 5450 2500
-Wire Wire Line
-	5450 2750 5750 2750
-Wire Wire Line
-	5750 2750 6050 2750
+	5450 2500 5450 2850
+Wire Wire Line
+	5450 2750 6050 2750
 Wire Wire Line
 	6050 2750 6050 2500
@@
 	6050 4150 6050 4250
 Wire Wire Line
-	5750 4250 5750 4150
+	5750 4150 5750 4250
 Connection ~ 6050 4150
 Connection ~ 5750 4150
@@
 	3950 4600 4100 4600
 Wire Wire Line
-	4100 4450 4100 4600
-Wire Wire Line
-	4100 4600 4100 4850
+	4100 4450 4100 4850
 Wire Wire Line
 	3350 4600 3650 4600
 Wire Wire Line
-	4250 2750 4100 2750
-Wire Wire Line
-	4100 2750 3950 2750
+	3950 2750 4250 2750
 $Comp
 L R R?
@@
 $EndComp
 Wire Wire Line
-	3950 4850 4100 4850
-Wire Wire Line
-	4100 4850 4250 4850
+	3950 4850 4250 4850
 Connection ~ 4100 4600
 Connection ~ 4100 4850
@@
 	4850 5550 4850 5450
 Wire Wire Line
-	4300 4150 4350 4150
-Wire Wire Line
-	4350 4150 5450 4150
-Wire Wire Line
-	5450 4150 5750 4150
-Wire Wire Line
-	5750 4150 6050 4150
-Wire Wire Line
-	6050 4150 6550 4150
-Wire Wire Line
-	6550 4150 6650 4150
-Wire Wire Line
-	3900 2100 3850 2100
-Wire Wire Line
-	3850 2100 3500 2100
-Wire Wire Line
-	3500 2100 3000 2100
+	4300 4150 6650 4150
+Wire Wire Line
+	3000 2100 3900 2100
 Wire Wire Line
 	3000 2200 3350 2200
 Wire Wire Line
-	6650 2100 6550 2100
-Wire Wire Line
-	6550 2100 6050 2100
-Wire Wire Line
-	6050 2100 5750 2100
-Wire Wire Line
-	5750 2100 5450 2100
-Wire Wire Line
-	5450 2100 4350 2100
-Wire Wire Line
-	4350 2100 4300 2100
-Wire Wire Line
-	5450 4550 5450 4800
-Wire Wire Line
-	5450 4800 5450 4900
-Wire Wire Line
-	5450 4800 5750 4800
-Wire Wire Line
-	5750 4800 6050 4800
+	4300 2100 6650 2100
+Wire Wire Line
+	5450 4550 5450 4900
+Wire Wire Line
+	5450 4800 6050 4800
 Wire Wire Line
 	6050 4800 6050 4550
@@
 Connection ~ 5450 4800
 Wire Wire Line
-	3350 4150 3850 4150
-Wire Wire Line
-	3850 4150 3900 4150
+	3350 4150 3900 4150
 $Comp
 L R R?
@@
 Connection ~ 4350 4150
 Wire Wire Line
-	3350 2200 3350 4150
-Wire Wire Line
-	3350 4150 3350 4600
-Wire Wire Line
-	3350 4600 3350 4850
+	3350 2200 3350 4850
 Connection ~ 3350 4600
 Connection ~ 3350 4150
@@
 $EndComp
 Wire Wire Line
-	6950 4150 7050 4150
-Wire Wire Line
-	7050 4150 7700 4150
-Wire Wire Line
-	6950 2100 7050 2100
-Wire Wire Line
-	7050 2100 7700 2100
+	6950 4150 7700 4150
+Wire Wire Line
+	6950 2100 7700 2100
 Wire Wire Line
 	6550 2300 6550 2100

Commit message: Removed Supply Sensing from vi_filter.sch
Parts:
- Q201: renamed from Q?; Part Number (none) -> FDMS86263P
- gave numbers to parts that had none: 21
Connections:
- net labels removed: in+, in-, ip+, ip-
Changed lines of the file:
@@
 $EndDescr
 $Comp
-L CP1 C?
+L CP1 C201
 U 1 1 5B0C3B3C
 P 5450 2350
-F 0 "C?" H 5475 2450 50  0000 L CNN
+F 0 "C201" H 5475 2450 50  0000 L CNN
 F 1 "100u" H 5475 2250 50  0000 L CNN
 F 2 "" H 5450 2350 50  0000 C CNN
@@
 $EndComp
 $Comp
-L CP1 C?
+L CP1 C203
 U 1 1 5B0C3B46
 P 5750 2350
-F 0 "C?" H 5775 2450 50  0000 L CNN
+F 0 "C203" H 5775 2450 50  0000 L CNN
 F 1 "100u" H 5775 2250 50  0000 L CNN
 F 2 "" H 5750 2350 50  0000 C CNN
@@
 $EndComp
 $Comp
-L CP1 C?
+L CP1 C205
 U 1 1 5B0C3B50
 P 6050 2350
-F 0 "C?" H 6075 2450 50  0000 L CNN
+F 0 "C205" H 6075 2450 50  0000 L CNN
 F 1 "100u" H 6075 2250 50  0000 L CNN
 F 2 "" H 6050 2350 50  0000 C CNN
@@
 $EndComp
 $Comp
-L CP1 C?
+L CP1 C202
 U 1 1 5B0C3B5A
 P 5450 4400
-F 0 "C?" H 5475 4500 50  0000 L CNN
+F 0 "C202" H 5475 4500 50  0000 L CNN
 F 1 "100u" H 5475 4300 50  0000 L CNN
 F 2 "" H 5450 4400 50  0000 C CNN
@@
 $EndComp
 $Comp
-L CP1 C?
+L CP1 C204
 U 1 1 5B0C3B64
 P 5750 4400
-F 0 "C?" H 5775 4500 50  0000 L CNN
+F 0 "C204" H 5775 4500 50  0000 L CNN
 F 1 "100u" H 5775 4300 50  0000 L CNN
 F 2 "" H 5750 4400 50  0000 C CNN
@@
 $EndComp
 $Comp
-L CP1 C?
+L CP1 C206
 U 1 1 5B0C3B6E
 P 6050 4400
-F 0 "C?" H 6075 4500 50  0000 L CNN
+F 0 "C206" H 6075 4500 50  0000 L CNN
 F 1 "100u" H 6075 4300 50  0000 L CNN
 F 2 "" H 6050 4400 50  0000 C CNN
@@
 $EndComp
 $Comp
-L Q_PMOS_DGS Q?
+L Q_PMOS_DGS Q201
 U 1 1 5B0C3B78
 P 4100 2200
-F 0 "Q?" V 4100 2400 50  0000 L CNN
+F 0 "Q201" V 4100 2400 50  0000 L CNN
 F 1 "FDMS86263P" V 4000 2400 50  0000 L CNN
 F 2 "" H 4300 2300 50  0000 C CNN
@@
 F 4 "Fairchild" H 4100 2200 60  0001 C CNN "Manufacturer"
 F 5 "FDMS86263PCT-ND" H 4100 2200 60  0001 C CNN "Digikey"
-F 6 "512-FDMS86263P" H 4100 2200 60  0001 C CNN "Mouser"
+F 6 "FDMS86263P" H 4100 2200 60  0001 C CNN "Part Number"
+F 7 "512-FDMS86263P" H 4100 2200 60  0001 C CNN "Mouser"
 	1    4100 2200
 	0    1    -1   0
@@
 	6050 2200 6050 2100
 $Comp
-L D_Zener D?
+L D_Zener D201
 U 1 1 5B0C3B82
 P 3800 2500
-F 0 "D?" H 3800 2600 50  0000 C CNN
+F 0 "D201" H 3800 2600 50  0000 C CNN
 F 1 "10V" H 3800 2400 50  0000 C CNN
 F 2 "" H 3800 2500 50  0000 C CNN
@@
 $EndComp
 $Comp
-L R R?
+L R R201
 U 1 1 5B0C3B89
 P 3800 2750
-F 0 "R?" V 3880 2750 50  0000 C CNN
+F 0 "R201" V 3880 2750 50  0000 C CNN
 F 1 "18k" V 3800 2750 50  0000 C CNN
 F 2 "" V 3730 2750 50  0000 C CNN
@@
 Connection ~ 4100 2500
 $Comp
-L R R?
+L R R207
 U 1 1 5B0C3B9A
 P 4400 2750
-F 0 "R?" V 4480 2750 50  0000 C CNN
+F 0 "R207" V 4480 2750 50  0000 C CNN
 F 1 "68k" V 4400 2750 50  0000 C CNN
 F 2 "" V 4330 2750 50  0000 C CNN
@@
 	4850 3450 4850 3350
 $Comp
-L GNDPWR #PWR?
+L GNDPWR #PWR022
 U 1 1 5B0C3BA5
 P 4850 3450
-F 0 "#PWR?" H 4850 3250 50  0001 C CNN
+F 0 "#PWR022" H 4850 3250 50  0001 C CNN
 F 1 "GNDPWR" H 4850 3320 50  0000 C CNN
 F 2 "" H 4850 3400 50  0000 C CNN
@@
 Connection ~ 5750 2100
 $Comp
-L GNDPWR #PWR?
+L GNDPWR #PWR023
 U 1 1 5B0C3BAD
 P 5450 2850
-F 0 "#PWR?" H 5450 2650 50  0001 C CNN
+F 0 "#PWR023" H 5450 2650 50  0001 C CNN
 F 1 "GNDPWR" H 5450 2720 50  0000 C CNN
 F 2 "" H 5450 2800 50  0000 C CNN
@@
 Connection ~ 5750 4150
 $Comp
-L Q_NMOS_DGS Q?
+L Q_NMOS_DGS Q202
 U 1 1 5B0C3BC2
 P 4100 4250
-F 0 "Q?" H 4300 4300 50  0000 L CNN
+F 0 "Q202" H 4300 4300 50  0000 L CNN
 F 1 "FDMS86252" V 4050 4400 50  0000 L CNN
 F 2 "" H 4300 4350 50  0000 C CNN
@@
 $EndComp
 $Comp
-L D_Zener D?
+L D_Zener D202
 U 1 1 5B0C3BC9
 P 3800 4600
-F 0 "D?" H 3800 4700 50  0000 C CNN
+F 0 "D202" H 3800 4700 50  0000 C CNN
 F 1 "10V" H 3800 4500 50  0000 C CNN
 F 2 "" H 3800 4600 50  0000 C CNN
@@
 	3950 2750 4250 2750
 $Comp
-L R R?
+L R R202
 U 1 1 5B0C3BD6
 P 3800 4850
-F 0 "R?" V 3880 4850 50  0000 C CNN
+F 0 "R202" V 3880 4850 50  0000 C CNN
 F 1 "18k" V 3800 4850 50  0000 C CNN
 F 2 "" V 3730 4850 50  0000 C CNN
@@
 $EndComp
 $Comp
-L R R?
+L R R208
 U 1 1 5B0C3BDD
 P 4400 4850
-F 0 "R?" V 4480 4850 50  0000 C CNN
+F 0 "R208" V 4480 4850 50  0000 C CNN
 F 1 "68k" V 4400 4850 50  0000 C CNN
 F 2 "" V 4330 4850 50  0000 C CNN
@@
 	4850 5050 4850 4850
 $Comp
-L GNDPWR #PWR?
+L GNDPWR #PWR024
 U 1 1 5B0C3BEC
 P 4850 5550
-F 0 "#PWR?" H 4850 5350 50  0001 C CNN
+F 0 "#PWR024" H 4850 5350 50  0001 C CNN
 F 1 "GNDPWR" H 4850 5420 50  0000 C CNN
 F 2 "" H 4850 5500 50  0000 C CNN
@@
 Connection ~ 5750 4800
 $Comp
-L GNDPWR #PWR?
+L GNDPWR #PWR025
 U 1 1 5B0C3C0A
 P 5450 4900
-F 0 "#PWR?" H 5450 4700 50  0001 C CNN
+F 0 "#PWR025" H 5450 4700 50  0001 C CNN
 F 1 "GNDPWR" H 5450 4770 50  0000 C CNN
 F 2 "" H 5450 4850 50  0000 C CNN
@@
 	3350 4150 3900 4150
 $Comp
-L R R?
+L R R203
 U 1 1 5B0C3C13
 P 4100 1750
-F 0 "R?" V 4180 1750 50  0000 C CNN
+F 0 "R203" V 4180 1750 50  0000 C CNN
 F 1 "220" V 4100 1750 50  0000 C CNN
 F 2 "" V 4030 1750 50  0000 C CNN
@@
 Connection ~ 4350 2100
 $Comp
-L R R?
+L R R204
 U 1 1 5B0C3C20
 P 4100 3800
-F 0 "R?" V 4180 3800 50  0000 C CNN
+F 0 "R204" V 4180 3800 50  0000 C CNN
 F 1 "220" V 4100 3800 50  0000 C CNN
 F 2 "" V 4030 3800 50  0000 C CNN
@@
 -25V - -100V
 $Comp
-L Q_NPN_BCE Q?
+L Q_NPN_BCE Q203
 U 1 1 5B0C3C37
 P 4750 3150
-F 0 "Q?" H 4950 3200 50  0000 L CNN
+F 0 "Q203" H 4950 3200 50  0000 L CNN
 F 1 "MMBT5550L" H 4950 3100 50  0000 L CNN
 F 2 "" H 4950 3250 50  0000 C CNN
@@
 $EndComp
 $Comp
-L Q_NPN_BCE Q?
+L Q_NPN_BCE Q204
 U 1 1 5B0C3C41
 P 4750 5250
-F 0 "Q?" H 4950 5300 50  0000 L CNN
+F 0 "Q204" H 4950 5300 50  0000 L CNN
 F 1 "MMBT5550L" H 4950 5200 50  0000 L CNN
 F 2 "" H 4950 5350 50  0000 C CNN
@@
 $EndComp
 $Comp
-L R R?
+L R R205
 U 1 1 5B0C3C48
 P 4300 3150
-F 0 "R?" V 4380 3150 50  0000 C CNN
+F 0 "R205" V 4380 3150 50  0000 C CNN
 F 1 "68k" V 4300 3150 50  0000 C CNN
 F 2 "" V 4230 3150 50  0000 C CNN
@@
 $EndComp
 $Comp
-L R R?
+L R R206
 U 1 1 5B0C3C4F
 P 4300 5250
-F 0 "R?" V 4380 5250 50  0000 C CNN
+F 0 "R206" V 4380 5250 50  0000 C CNN
 F 1 "68k" V 4300 5250 50  0000 C CNN
 F 2 "" V 4230 5250 50  0000 C CNN
@@
 Connection ~ 5450 4150
 $Comp
-L R R?
+L R R209
 U 1 1 5B0C3C5E
 P 6800 2100
-F 0 "R?" V 6880 2100 50  0000 C CNN
+F 0 "R209" V 6880 2100 50  0000 C CNN
 F 1 "10m" V 6800 2100 50  0000 C CNN
 F 2 "" V 6730 2100 50  0000 C CNN
@@
 $EndComp
 $Comp
-L R R?
+L R R210
 U 1 1 5B0C3C65
 P 6800 4150
-F 0 "R?" V 6880 4150 50  0000 C CNN
+F 0 "R210" V 6880 4150 50  0000 C CNN
 F 1 "10m" V 6800 4150 50  0000 C CNN
 F 2 "" V 6730 4150 50  0000 C CNN
@@
 Text HLabel 4050 5250 0    60   Input ~ 0
 pwr_enable
-Text HLabel 6550 2300 3    60   Output ~ 0
-ip+
-Text HLabel 7050 2300 3    60   Output ~ 0
-ip-
-Text HLabel 6550 4350 3    60   Output ~ 0
-in+
-Text HLabel 7050 4350 3    60   Output ~ 0
-in-
 $EndSCHEMATC

Commit message: Added test points
Parts:
- added W? (x2): TEST_1P, symbol TEST_1P
Connections:
- wire segments 55 -> 57
Changed lines of the file:
@@
 Text HLabel 4050 5250 0    60   Input ~ 0
 pwr_enable
+$Comp
+L TEST_1P W?
+U 1 1 5B3AB7FE
+P 7500 2000
+F 0 "W?" H 7500 2270 50  0000 C CNN
+F 1 "TEST_1P" H 7500 2200 50  0000 C CNN
+F 2 "" H 7700 2000 50  0000 C CNN
+F 3 "" H 7700 2000 50  0000 C CNN
+	1    7500 2000
+	1    0    0    -1
+$EndComp
+$Comp
+L TEST_1P W?
+U 1 1 5B3AB87D
+P 7500 4050
+F 0 "W?" H 7500 4320 50  0000 C CNN
+F 1 "TEST_1P" H 7500 4250 50  0000 C CNN
+F 2 "" H 7700 4050 50  0000 C CNN
+F 3 "" H 7700 4050 50  0000 C CNN
+	1    7500 4050
+	1    0    0    -1
+$EndComp
+Wire Wire Line
+	7500 4050 7500 4150
+Connection ~ 7500 4150
+Wire Wire Line
+	7500 2000 7500 2100
+Connection ~ 7500 2100
 $EndSCHEMATC
