File: components_predev/output_driver/hardware/output_stage.sch (KiCad schematic (older format))
At the start: 36 parts

Commit message: Interface Wiring
Changed lines of the file:
@@
 $Descr A4 11693 8268
 encoding utf-8
-Sheet 3 6
+Sheet 3 7
 Title ""
 Date ""
@@
 Text GLabel 5000 2400 2    60   Input ~ 0
 offset_adj
-Text GLabel 3950 2400 0    60   Input ~ 0
-drv_input
 Wire Wire Line
 	9150 1700 9450 1700
@@
 	5300 3150 5200 3150
 Wire Wire Line
-	3950 2400 4300 2400
+	1250 2400 4300 2400
 Connection ~ 4300 2400
 Wire Wire Line
@@
 Wire Wire Line
 	10350 3650 10600 3650
+Text HLabel 1250 2400 0    60   Input ~ 0
+drv_input
 $EndSCHEMATC

Commit message: Added DAC, added disengage relay
Parts:
- added D?: D, symbol D
- added K?: PE014005, symbol PE014005
- added Q?: Q_NMOS_DGS, symbol Q_NMOS_DGS
- added R?: R_Small, symbol R_Small
Connections:
- net at Q?.3 (E), Q?.3 (E), R?.1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: now also K?.11; no longer L?.2
- new net: K?.14, L?.2
- new net: D?.2 (A), K?.2, Q?.1 (D)
- new net +12V: D?.1 (K), K?.1
- new net GND: Q?.3 (S), R?.2
- new net disengage: Q?.2 (G), R?.1
- no-connect marks 0 -> 1
Other:
- moved on the sheet: C?, D?, L?, Q?, R?, RV?

Commit message: Put opamp gain stage into schematic
Parts:
- removed D? (x2): D, symbol D
- removed Q?: MJD350T4G, symbol Q_PNP_BCE
- removed Q?: MJD340T4G, symbol Q_NPN_BCE
- removed Q?: MMBT5550L, symbol Q_NPN_BCE
- removed Q?: MMBT5401-7-F, symbol Q_PNP_BCE
- removed R? (x2): 100, symbol R
- removed R? (x2): 10, symbol R
- removed R? (x2): 1k, symbol R
- removed R? (x2): 680, symbol R
- added C? (x2): 100n, symbol C_Small
- added D?: LED, symbol LED
- added R? (x2): 120k, symbol R
- added R? (x2): 100k, symbol R
- added R?: 2k, symbol R
- added R?: 132k, symbol R
- added R?: R, symbol R
- added U?: LTC6090-5, symbol LTC6090
- added U? (x2): LTC6091, symbol LTC6091
- R?: value 33 -> 68
Connections:
- net +5V: now also D?.2 (A)
- net GND: now also C?.1, C?.1, U?.1 (COM), U?.14 (V+B), U?.16 (COMB), U?.4 (COMB), U?.7 (V-)
- net VDD: now also C?.2, R?.2, U?.10 (V+B)
- net VSS: now also C?.2, R?.1, U?.3 (V-)
- net drv_input: now also R?.2
- net output: now also R?.1
- net at R?.2: now also R?.1, R?.2, U?.6 (Out)
- net at L?.2: now also K?.12; no longer K?.14
- new net: R?.1, R?.2, U?.2 (-IN)
- new net: U?.1 (-IN), U?.13 (OutB), U?.4 (V-)
- new net: U?.5 (-IN), U?.7 (V+), U?.9 (OutB)
- new net: R?.1, R?.2, U?.2 (+IN)
- new net: R?.1, R?.2, U?.6 (+IN)
- new net: D?.1 (K), R?.2
- new net V-: U?.9 (V-)
- new net temp: R?.1, U?.11 (~ODB), U?.12 (~TFLAGB), U?.15 (~ODB), U?.5 (~TFLAG), U?.8 (~OD), U?.8 (~TFLAGB)
- new net v_ref_2: U?.3 (+IN)
Other:
- moved on the sheet: C?, D?, K?, L?, Q?, R?, RV?

Commit message: Removed Supply Sensing from vi_filter.sch
Parts:
- gave numbers to parts that had none: 38

Commit message: Added test points
Parts:
- added W? (x5): TEST_1P, symbol TEST_1P
Connections:
- net at K301.11, Q304.3 (E), Q305.3 (E)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: now also W?.1
- net at C303.1, Q301.2 (C), R308.1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: now also W?.1
- net at R304.2, R305.1, R308.2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: now also W?.1
- net at U301.4 (V-), U302.1 (-IN), U302.13 (OutB): now also W?.1
- net at U301.7 (V+), U302.5 (-IN), U302.9 (OutB): now also W?.1
Changed lines of the file:
@@
 Connection ~ 6650 5150
 Wire Wire Line
-	6650 2050 6650 3400
+	6650 1950 6650 3400
 Connection ~ 6000 2850
 Wire Wire Line
@@
 	4100 3000 2800 3000
 Wire Wire Line
-	2800 3000 2800 3350
+	2800 2900 2800 3350
 Connection ~ 4100 4750
 $Comp
@@
 Wire Wire Line
 	1350 4600 1750 4600
+$Comp
+L TEST_1P W?
+U 1 1 5B3ABE63
+P 4800 3650
+F 0 "W?" H 4800 3920 50  0000 C CNN
+F 1 "TEST_1P" H 4800 3850 50  0000 C CNN
+F 2 "" H 5000 3650 50  0000 C CNN
+F 3 "" H 5000 3650 50  0000 C CNN
+	1    4800 3650
+	1    0    0    -1
+$EndComp
+Wire Wire Line
+	4800 3650 4800 3800
+Connection ~ 4800 3800
+$Comp
+L TEST_1P W?
+U 1 1 5B3ABFD1
+P 2800 2900
+F 0 "W?" H 2800 3170 50  0000 C CNN
+F 1 "TEST_1P" H 2800 3100 50  0000 C CNN
+F 2 "" H 3000 2900 50  0000 C CNN
+F 3 "" H 3000 2900 50  0000 C CNN
+	1    2800 2900
+	1    0    0    -1
+$EndComp
+$Comp
+L TEST_1P W?
+U 1 1 5B3AC0BA
+P 1700 2900
+F 0 "W?" H 1700 3170 50  0000 C CNN
+F 1 "TEST_1P" H 1700 3100 50  0000 C CNN
+F 2 "" H 1900 2900 50  0000 C CNN
+F 3 "" H 1900 2900 50  0000 C CNN
+	1    1700 2900
+	1    0    0    -1
+$EndComp
+Wire Wire Line
+	1700 2900 1700 3000
+Wire Wire Line
+	1700 3000 2050 3000
+Connection ~ 2050 3000
+Connection ~ 2800 3000
+$Comp
+L TEST_1P W?
+U 1 1 5B3AC35A
+P 8850 3500
+F 0 "W?" H 8850 3770 50  0000 C CNN
+F 1 "TEST_1P" H 8850 3700 50  0000 C CNN
+F 2 "" H 9050 3500 50  0000 C CNN
+F 3 "" H 9050 3500 50  0000 C CNN
+	1    8850 3500
+	1    0    0    -1
+$EndComp
+Wire Wire Line
+	8850 3500 8850 3600
+Connection ~ 8850 3600
+$Comp
+L TEST_1P W?
+U 1 1 5B3AC54F
+P 6650 1950
+F 0 "W?" H 6650 2220 50  0000 C CNN
+F 1 "TEST_1P" H 6650 2150 50  0000 C CNN
+F 2 "" H 6850 1950 50  0000 C CNN
+F 3 "" H 6850 1950 50  0000 C CNN
+	1    6650 1950
+	1    0    0    -1
+$EndComp
+Connection ~ 6650 2050
 $EndSCHEMATC
