File: components_predev/output_driver/hardware/supplies.sch (KiCad schematic (older format))
At the start: 0 parts

Commit message: Added ADC Symbol, Started Wiring
Parts:
- added C?: CP1, symbol CP1
- added C?: C, symbol C
- added L?: Ferrite_Bead, symbol Ferrite_Bead
Connections:
- new net +12V: C?.1, C?.1, L?.1
- new net GND: C?.2, C?.2
- new net v_supply: L?.2
Changed lines of the file:
@@
 Comment4 ""
 $EndDescr
+Text HLabel 1650 1400 0    60   Input ~ 0
+v_supply
+$Comp
+L Ferrite_Bead L?
+U 1 1 5B19AAF9
+P 2100 1400
+F 0 "L?" V 1950 1425 50  0000 C CNN
+F 1 "Ferrite_Bead" V 2250 1400 50  0000 C CNN
+F 2 "" V 2030 1400 50  0000 C CNN
+F 3 "" H 2100 1400 50  0000 C CNN
+	1    2100 1400
+	0    1    1    0
+$EndComp
+Wire Wire Line
+	1950 1400 1650 1400
+$Comp
+L +12V #PWR?
+U 1 1 5B19AB24
+P 3700 1300
+F 0 "#PWR?" H 3700 1150 50  0001 C CNN
+F 1 "+12V" H 3700 1440 50  0000 C CNN
+F 2 "" H 3700 1300 50  0000 C CNN
+F 3 "" H 3700 1300 50  0000 C CNN
+	1    3700 1300
+	1    0    0    -1
+$EndComp
+Wire Wire Line
+	3700 1300 3700 1500
+Wire Wire Line
+	3700 1400 2250 1400
+$Comp
+L CP1 C?
+U 1 1 5B19AB41
+P 3300 1650
+F 0 "C?" H 3325 1750 50  0000 L CNN
+F 1 "CP1" H 3325 1550 50  0000 L CNN
+F 2 "" H 3300 1650 50  0000 C CNN
+F 3 "" H 3300 1650 50  0000 C CNN
+	1    3300 1650
+	1    0    0    -1
+$EndComp
+$Comp
+L C C?
+U 1 1 5B19AB84
+P 3700 1650
+F 0 "C?" H 3725 1750 50  0000 L CNN
+F 1 "C" H 3725 1550 50  0000 L CNN
+F 2 "" H 3738 1500 50  0000 C CNN
+F 3 "" H 3700 1650 50  0000 C CNN
+	1    3700 1650
+	1    0    0    -1
+$EndComp
+$Comp
+L GND #PWR?
+U 1 1 5B19AB9F
+P 3700 2000
+F 0 "#PWR?" H 3700 1750 50  0001 C CNN
+F 1 "GND" H 3700 1850 50  0000 C CNN
+F 2 "" H 3700 2000 50  0000 C CNN
+F 3 "" H 3700 2000 50  0000 C CNN
+	1    3700 2000
+	1    0    0    -1
+$EndComp
+Wire Wire Line
+	3700 2000 3700 1800
+Wire Wire Line
+	3300 1800 3300 1950
+Wire Wire Line
+	3300 1950 3700 1950
+Connection ~ 3700 1950
+Wire Wire Line
+	3300 1500 3300 1400
+Connection ~ 3300 1400
+Connection ~ 3700 1400
 $EndSCHEMATC

Commit message: Removed Supply Sensing from vi_filter.sch
Parts:
- gave numbers to parts that had none: 3
Changed lines of the file:
@@
 v_supply
 $Comp
-L Ferrite_Bead L?
+L Ferrite_Bead L401
 U 1 1 5B19AAF9
 P 2100 1400
-F 0 "L?" V 1950 1425 50  0000 C CNN
+F 0 "L401" V 1950 1425 50  0000 C CNN
 F 1 "Ferrite_Bead" V 2250 1400 50  0000 C CNN
 F 2 "" V 2030 1400 50  0000 C CNN
@@
 	1950 1400 1650 1400
 $Comp
-L +12V #PWR?
+L +12V #PWR045
 U 1 1 5B19AB24
 P 3700 1300
-F 0 "#PWR?" H 3700 1150 50  0001 C CNN
+F 0 "#PWR045" H 3700 1150 50  0001 C CNN
 F 1 "+12V" H 3700 1440 50  0000 C CNN
 F 2 "" H 3700 1300 50  0000 C CNN
@@
 	3700 1400 2250 1400
 $Comp
-L CP1 C?
+L CP1 C401
 U 1 1 5B19AB41
 P 3300 1650
-F 0 "C?" H 3325 1750 50  0000 L CNN
+F 0 "C401" H 3325 1750 50  0000 L CNN
 F 1 "CP1" H 3325 1550 50  0000 L CNN
 F 2 "" H 3300 1650 50  0000 C CNN
@@
 $EndComp
 $Comp
-L C C?
+L C C402
 U 1 1 5B19AB84
 P 3700 1650
-F 0 "C?" H 3725 1750 50  0000 L CNN
+F 0 "C402" H 3725 1750 50  0000 L CNN
 F 1 "C" H 3725 1550 50  0000 L CNN
 F 2 "" H 3738 1500 50  0000 C CNN
@@
 $EndComp
 $Comp
-L GND #PWR?
+L GND #PWR046
 U 1 1 5B19AB9F
 P 3700 2000
-F 0 "#PWR?" H 3700 1750 50  0001 C CNN
+F 0 "#PWR046" H 3700 1750 50  0001 C CNN
 F 1 "GND" H 3700 1850 50  0000 C CNN
 F 2 "" H 3700 2000 50  0000 C CNN

Commit message: Added Supply Schematic
Parts:
- removed C401: CP1, symbol CP1
- removed C402: C, symbol C
- added C? (x17): C_Small, symbol C_Small
- added C? (x9): CP1_Small, symbol CP1_Small
- added D? (x3): D, symbol D
- added D? (x4): LED, symbol LED
- added L? (x2): L, symbol L
- added L? (x2): L_Small, symbol L_Small
- added P? (x4): CONN_01X02, symbol CONN_01X02
- added R? (x14): R_Small, symbol R_Small
- added U? (x2): AOZ1284, symbol AOZ1284
- added U?: MIC39100, symbol MIC39100
- added U?: LT1617, symbol LT1617
- added U?: MC79M05, symbol MC79M05
Connections:
- net +12V: now also C?.1, C?.1, C?.1, C?.1, C?.1, C?.1, D?.2 (A), L?.1, P?.1 (P1), U?.5 (In), U?.9 (VIN), U?.9 (VIN); no longer L401.1
- net GND: now also C?.2, C?.2, C?.2, C?.2, C?.2, C?.2, C?.2, C?.2, C?.2, C?.2, C?.2, C?.2, C?.2, C?.2, C?.2, C?.2, C?.2, C?.2, C?.2, C?.2, C?.2, C?.2, D?.1 (K), D?.2 (A), D?.2 (A), R?.2, R?.2, R?.2, R?.2, R?.2, R?.2, R?.2, R?.2, R?.2, U?.1 (GND), U?.2 (GND), U?.2 (GND), U?.3 (GND), U?.3 (GND), U?.4 (GND)
- new net: C?.1, C?.1, L401.1, P?.2 (P2)
- new net: C?.1, D?.1 (K), L?.1, U?.1 (LX) (x2)
- new net: C?.2, U?.2 (BST) (x2)
- new net: R?.1, U?.4 (FSW) (x2)
- new net: R?.1, U?.5 (COMP) (x2)
- new net: R?.1, R?.2, U?.6 (FB) (x2)
- new net: C?.1, U?.7 (SS) (x2)
- new net: C?.1, C?.1, L?.2, P?.1 (P1), R?.1
- new net: C?.1, R?.2 (x2)
- new net: C?.1, C?.1, L?.2, R?.1, U?.1 (In)
- new net: C?.1, C?.1, P?.1 (P1), U?.3 (Out) (x2)
- new net: D?.1 (K), R?.1 (x3)
- new net: D?.2 (A), R?.1
- new net: C?.2, L?.2, U?.1 (SW)
- new net: C?.2, R?.1, R?.2, U?.3 (NFB)
- new net: C?.1, D?.2 (A), L?.1
- new net: C?.1, C?.1, C?.1, L?.2, R?.1, U?.4 (In)
- new net +3V3: D?.2 (A), P?.2 (P2)
- new net +5V: D?.2 (A), P?.2 (P2)
- new net -5V: D?.1 (K), P?.2 (P2)
Other:
- moved on the sheet: L401

Commit message: Added test points
Parts:
- added D?: D_Zener, symbol D_Zener
- added R?: R_Small, symbol R_Small
- added W? (x4): TEST_1P, symbol TEST_1P
Connections:
- net +12V: now also R?.1, W?.1
- net +3V3: now also W?.1
- net +5V: now also W?.1
- net -5V: now also W?.1
- net GND: now also D?.2 (A)
- net rails_en: now reaches U?.8 (EN)
- net rails_en: now also U?.4 (SHDN), U?.8 (EN), D?.1 (K), R?.2
Changed lines of the file:
@@
 +12V
 Wire Wire Line
-	3550 800  3250 800
+	2900 800  3550 800
 Connection ~ 3250 800
+Text GLabel 2250 3050 0    60   Input ~ 0
+rails_en
+Wire Wire Line
+	2250 3050 2550 3050
+Text GLabel 2400 5050 0    60   Input ~ 0
+rails_en
+Wire Wire Line
+	2400 5050 2600 5050
+Text GLabel 5550 1250 0    60   Input ~ 0
+rails_en
+Wire Wire Line
+	5550 1250 5850 1250
+Text GLabel 4450 6650 2    60   Output ~ 0
+rails_en
+$Comp
+L R_Small R?
+U 1 1 5B3A6C85
+P 4200 6400
+F 0 "R?" H 4230 6420 50  0000 L CNN
+F 1 "R_Small" H 4230 6360 50  0000 L CNN
+F 2 "" H 4200 6400 50  0000 C CNN
+F 3 "" H 4200 6400 50  0000 C CNN
+	1    4200 6400
+	1    0    0    -1
+$EndComp
+$Comp
+L +12V #PWR?
+U 1 1 5B3A6D7E
+P 4200 6150
+F 0 "#PWR?" H 4200 6000 50  0001 C CNN
+F 1 "+12V" H 4200 6290 50  0000 C CNN
+F 2 "" H 4200 6150 50  0000 C CNN
+F 3 "" H 4200 6150 50  0000 C CNN
+	1    4200 6150
+	1    0    0    -1
+$EndComp
+Wire Wire Line
+	4200 6150 4200 6300
+Wire Wire Line
+	4200 6500 4200 6750
+Wire Wire Line
+	4200 6650 4450 6650
+$Comp
+L D_Zener D?
+U 1 1 5B3A7024
+P 4200 6900
+F 0 "D?" H 4200 7000 50  0000 C CNN
+F 1 "D_Zener" H 4200 6800 50  0000 C CNN
+F 2 "" H 4200 6900 50  0000 C CNN
+F 3 "" H 4200 6900 50  0000 C CNN
+	1    4200 6900
+	0    1    1    0
+$EndComp
+$Comp
+L GND #PWR?
+U 1 1 5B3A7112
+P 4200 7250
+F 0 "#PWR?" H 4200 7000 50  0001 C CNN
+F 1 "GND" H 4200 7100 50  0000 C CNN
+F 2 "" H 4200 7250 50  0000 C CNN
+F 3 "" H 4200 7250 50  0000 C CNN
+	1    4200 7250
+	1    0    0    -1
+$EndComp
+Wire Wire Line
+	4200 7250 4200 7050
+Connection ~ 4200 6650
+$Comp
+L TEST_1P W?
+U 1 1 5B3A9159
+P 2900 800
+F 0 "W?" H 2900 1070 50  0000 C CNN
+F 1 "TEST_1P" H 2900 1000 50  0000 C CNN
+F 2 "" H 3100 800 50  0000 C CNN
+F 3 "" H 3100 800 50  0000 C CNN
+	1    2900 800
+	1    0    0    -1
+$EndComp
+$Comp
+L TEST_1P W?
+U 1 1 5B3A96F7
+P 10150 1250
+F 0 "W?" H 10150 1520 50  0000 C CNN
+F 1 "TEST_1P" H 10400 1400 50  0000 C CNN
+F 2 "" H 10350 1250 50  0000 C CNN
+F 3 "" H 10350 1250 50  0000 C CNN
+	1    10150 1250
+	1    0    0    -1
+$EndComp
+$Comp
+L TEST_1P W?
+U 1 1 5B3A98FE
+P 10150 3050
+F 0 "W?" H 10150 3320 50  0000 C CNN
+F 1 "TEST_1P" H 10400 3200 50  0000 C CNN
+F 2 "" H 10350 3050 50  0000 C CNN
+F 3 "" H 10350 3050 50  0000 C CNN
+	1    10150 3050
+	1    0    0    -1
+$EndComp
+$Comp
+L TEST_1P W?
+U 1 1 5B3A9B2A
+P 10150 4450
+F 0 "W?" H 10150 4720 50  0000 C CNN
+F 1 "TEST_1P" H 10400 4600 50  0000 C CNN
+F 2 "" H 10350 4450 50  0000 C CNN
+F 3 "" H 10350 4450 50  0000 C CNN
+	1    10150 4450
+	1    0    0    -1
+$EndComp
+Wire Wire Line
+	10150 4450 10150 4500
+Connection ~ 10150 4500
+Wire Wire Line
+	10150 3050 10150 3100
+Connection ~ 10150 3100
+Wire Wire Line
+	10150 1250 10150 1300
+Connection ~ 10150 1300
 $EndSCHEMATC
