File: components_predev/frontend/hardware/ADC.sch (KiCad schematic (older format))
At the start: 49 parts, among them Q701 Q_NMOS_DGS, U701 MIC7211, U702 ADR4533, U703 LMT88, U704 NCP508, U705 NCP508, U706 MAX11960, U707 LTC2055, U708 NCP508

Commit message: Begun Range Switching Circuitry
Parts:
- removed U708: NCP508, symbol NCP508
- added C?: C_Small, symbol C_Small
- added R? (x2): R_Small, symbol R_Small
- added U?: TSP73001, symbol TSP73001
- U704, U705: Part Number (none) -> NCP508MT33TBG
Connections:
- wire segments 169 -> 177
Other:
- note added: "1.8V"
- note added: "3.6V"
- note added: "V_ref = 3.3V\nV_ref_2 = 1.65V"
Changed lines of the file:
@@
 F 2 "" H 2850 2350 60  0001 C CNN
 F 3 "" H 2850 2350 60  0001 C CNN
+F 4 "NCP508MT33TBG" H 2850 2350 60  0001 C CNN "Part Number"
 	1    2850 2350
 	1    0    0    -1
@@
 F 2 "" H 2850 1300 60  0001 C CNN
 F 3 "" H 2850 1300 60  0001 C CNN
+F 4 "NCP508MT33TBG" H 2850 1300 60  0001 C CNN "Part Number"
 	1    2850 1300
 	1    0    0    -1
@@
 $EndComp
 $Comp
-L NCP508 U708
-U 1 1 5B221D33
-P 6200 1300
-F 0 "U708" H 6300 1450 60  0000 C CNN
-F 1 "NCP508" H 6450 900 60  0000 C CNN
-F 2 "" H 6200 1300 60  0001 C CNN
-F 3 "" H 6200 1300 60  0001 C CNN
-	1    6200 1300
-	-1   0    0    -1
-$EndComp
-$Comp
-L GND #PWR070
-U 1 1 5B221D39
-P 6200 1900
-F 0 "#PWR070" H 6200 1650 50  0001 C CNN
-F 1 "GND" H 6200 1750 50  0000 C CNN
-F 2 "" H 6200 1900 50  0000 C CNN
-F 3 "" H 6200 1900 50  0000 C CNN
-	1    6200 1900
-	-1   0    0    -1
-$EndComp
-$Comp
 L C_Small C717
 U 1 1 5B221D3F
-P 5500 1550
-F 0 "C717" H 5510 1620 50  0000 L CNN
-F 1 "C_Small" H 5510 1470 50  0000 L CNN
-F 2 "" H 5500 1550 50  0000 C CNN
-F 3 "" H 5500 1550 50  0000 C CNN
-	1    5500 1550
+P 5350 1550
+F 0 "C717" H 5360 1620 50  0000 L CNN
+F 1 "C_Small" H 5360 1470 50  0000 L CNN
+F 2 "" H 5350 1550 50  0000 C CNN
+F 3 "" H 5350 1550 50  0000 C CNN
+	1    5350 1550
 	-1   0    0    -1
 $EndComp
@@
 L C_Small C716
 U 1 1 5B221D45
-P 5300 1550
-F 0 "C716" H 5310 1620 50  0000 L CNN
-F 1 "C_Small" H 5310 1470 50  0000 L CNN
-F 2 "" H 5300 1550 50  0000 C CNN
-F 3 "" H 5300 1550 50  0000 C CNN
-	1    5300 1550
+P 5150 1550
+F 0 "C716" H 5160 1620 50  0000 L CNN
+F 1 "C_Small" H 5160 1470 50  0000 L CNN
+F 2 "" H 5150 1550 50  0000 C CNN
+F 3 "" H 5150 1550 50  0000 C CNN
+	1    5150 1550
 	-1   0    0    -1
 $EndComp
@@
 L GND #PWR071
 U 1 1 5B221D4B
-P 5400 1900
-F 0 "#PWR071" H 5400 1650 50  0001 C CNN
-F 1 "GND" H 5400 1750 50  0000 C CNN
-F 2 "" H 5400 1900 50  0000 C CNN
-F 3 "" H 5400 1900 50  0000 C CNN
-	1    5400 1900
+P 5250 1900
+F 0 "#PWR071" H 5250 1650 50  0001 C CNN
+F 1 "GND" H 5250 1750 50  0000 C CNN
+F 2 "" H 5250 1900 50  0000 C CNN
+F 3 "" H 5250 1900 50  0000 C CNN
+	1    5250 1900
 	-1   0    0    -1
 $EndComp
@@
 L C_Small C722
 U 1 1 5B2221D7
-P 7000 1550
-F 0 "C722" H 7010 1620 50  0000 L CNN
-F 1 "C_Small" H 7010 1470 50  0000 L CNN
-F 2 "" H 7000 1550 50  0000 C CNN
-F 3 "" H 7000 1550 50  0000 C CNN
-	1    7000 1550
-	-1   0    0    -1
-$EndComp
-$Comp
-L CP1_Small C723
-U 1 1 5B2221DD
 P 7250 1550
-F 0 "C723" H 7260 1620 50  0000 L CNN
-F 1 "CP1_Small" H 7260 1470 50  0000 L CNN
+F 0 "C722" H 7260 1620 50  0000 L CNN
+F 1 "C_Small" H 7260 1470 50  0000 L CNN
 F 2 "" H 7250 1550 50  0000 C CNN
 F 3 "" H 7250 1550 50  0000 C CNN
@@
 $EndComp
 $Comp
+L CP1_Small C723
+U 1 1 5B2221DD
+P 7500 1550
+F 0 "C723" H 7510 1620 50  0000 L CNN
+F 1 "CP1_Small" H 7510 1470 50  0000 L CNN
+F 2 "" H 7500 1550 50  0000 C CNN
+F 3 "" H 7500 1550 50  0000 C CNN
+	1    7500 1550
+	-1   0    0    -1
+$EndComp
+$Comp
 L GND #PWR072
 U 1 1 5B2221EE
-P 7250 1850
-F 0 "#PWR072" H 7250 1600 50  0001 C CNN
-F 1 "GND" H 7250 1700 50  0000 C CNN
-F 2 "" H 7250 1850 50  0000 C CNN
-F 3 "" H 7250 1850 50  0000 C CNN
-	1    7250 1850
+P 7500 1850
+F 0 "#PWR072" H 7500 1600 50  0001 C CNN
+F 1 "GND" H 7500 1700 50  0000 C CNN
+F 2 "" H 7500 1850 50  0000 C CNN
+F 3 "" H 7500 1850 50  0000 C CNN
+	1    7500 1850
 	-1   0    0    -1
 $EndComp
@@
 L +5V #PWR073
 U 1 1 5B22240B
-P 7250 1200
-F 0 "#PWR073" H 7250 1050 50  0001 C CNN
-F 1 "+5V" H 7250 1340 50  0000 C CNN
-F 2 "" H 7250 1200 50  0000 C CNN
-F 3 "" H 7250 1200 50  0000 C CNN
-	1    7250 1200
+P 7500 1200
+F 0 "#PWR073" H 7500 1050 50  0001 C CNN
+F 1 "+5V" H 7500 1340 50  0000 C CNN
+F 2 "" H 7500 1200 50  0000 C CNN
+F 3 "" H 7500 1200 50  0000 C CNN
+	1    7500 1200
 	1    0    0    -1
 $EndComp
@@
 Connection ~ 1250 1750
 Wire Wire Line
-	6200 1900 6200 1800
-Wire Wire Line
-	5300 1450 5300 1300
-Connection ~ 5300 1300
-Wire Wire Line
-	5500 1300 5500 1450
-Connection ~ 5500 1300
-Wire Wire Line
-	5400 1900 5400 1850
-Wire Wire Line
-	5300 1850 5500 1850
-Wire Wire Line
-	5500 1850 5500 1650
-Wire Wire Line
-	5300 1850 5300 1650
-Connection ~ 5400 1850
-Wire Wire Line
-	6650 1300 7250 1300
-Wire Wire Line
-	6650 1450 6750 1450
-Wire Wire Line
-	6750 1450 6750 1300
-Connection ~ 6750 1300
+	5150 1450 5150 1300
+Connection ~ 5150 1300
+Wire Wire Line
+	5350 1300 5350 1450
+Connection ~ 5350 1300
+Wire Wire Line
+	5250 1900 5250 1850
+Wire Wire Line
+	5150 1850 5350 1850
+Wire Wire Line
+	5350 1850 5350 1650
+Wire Wire Line
+	5150 1850 5150 1650
+Connection ~ 5250 1850
+Wire Wire Line
+	6800 1300 7500 1300
 Wire Wire Line
 	4950 1150 4950 4050
 Wire Wire Line
-	4950 1300 5750 1300
+	4950 1300 5900 1300
 Wire Wire Line
 	4850 4050 4850 3550
@@
 Connection ~ 4950 3550
 Wire Wire Line
-	7000 1300 7000 1450
-Wire Wire Line
-	7250 1200 7250 1450
-Connection ~ 7000 1300
+	7250 1300 7250 1450
+Wire Wire Line
+	7500 1200 7500 1450
 Connection ~ 7250 1300
-Wire Wire Line
-	7250 1650 7250 1850
-Wire Wire Line
-	7250 1750 7000 1750
-Wire Wire Line
-	7000 1750 7000 1650
-Connection ~ 7250 1750
+Connection ~ 7500 1300
+Wire Wire Line
+	7500 1650 7500 1850
+Wire Wire Line
+	7500 1750 7250 1750
+Wire Wire Line
+	7250 1750 7250 1650
+Connection ~ 7500 1750
 Wire Wire Line
 	1300 7800 1300 8050
@@
 	1    0    0    -1
 $EndComp
+Text Notes 6800 8000 0    47   ~ 0
+V_ref = 3.3V\nV_ref_2 = 1.65V
+Text Notes 4100 2250 0    47   ~ 0
+1.8V
+Text Notes 4450 1200 0    47   ~ 0
+1.8V
+Text Notes 5050 1200 0    47   ~ 0
+3.6V
+$Comp
+L TSP73001 U?
+U 1 1 5B4FD42C
+P 6350 1300
+F 0 "U?" H 6500 800 47  0000 C CNN
+F 1 "TSP73001" H 6350 1450 47  0000 C CNN
+F 2 "" H 6350 1300 47  0001 C CNN
+F 3 "" H 6350 1300 47  0001 C CNN
+	1    6350 1300
+	-1   0    0    -1
+$EndComp
+$Comp
+L GND #PWR?
+U 1 1 5B4FD945
+P 6350 2050
+F 0 "#PWR?" H 6350 1800 50  0001 C CNN
+F 1 "GND" H 6350 1900 50  0000 C CNN
+F 2 "" H 6350 2050 50  0000 C CNN
+F 3 "" H 6350 2050 50  0000 C CNN
+	1    6350 2050
+	1    0    0    -1
+$EndComp
+Wire Wire Line
+	6350 2050 6350 1900
+$Comp
+L C_Small C?
+U 1 1 5B4FDACD
+P 5900 1800
+F 0 "C?" H 5910 1870 50  0000 L CNN
+F 1 "C_Small" H 5910 1720 50  0000 L CNN
+F 2 "" H 5900 1800 50  0000 C CNN
+F 3 "" H 5900 1800 50  0000 C CNN
+	1    5900 1800
+	1    0    0    -1
+$EndComp
+Wire Wire Line
+	5900 1700 5900 1600
+Wire Wire Line
+	5900 1900 5900 1950
+Wire Wire Line
+	5650 1950 6350 1950
+Connection ~ 6350 1950
+$Comp
+L R_Small R?
+U 1 1 5B4FDD7B
+P 5650 1450
+F 0 "R?" V 5750 1300 50  0000 L CNN
+F 1 "R_Small" V 5550 1350 50  0000 L CNN
+F 2 "" H 5650 1450 50  0000 C CNN
+F 3 "" H 5650 1450 50  0000 C CNN
+	1    5650 1450
+	0    1    1    0
+$EndComp
+$Comp
+L R_Small R?
+U 1 1 5B4FDE22
+P 5650 1750
+F 0 "R?" H 5680 1770 50  0000 L CNN
+F 1 "R_Small" V 5550 1600 50  0000 L CNN
+F 2 "" H 5650 1750 50  0000 C CNN
+F 3 "" H 5650 1750 50  0000 C CNN
+	1    5650 1750
+	1    0    0    -1
+$EndComp
+Wire Wire Line
+	5650 1850 5650 1950
+Connection ~ 5900 1950
+Wire Wire Line
+	5650 1650 5650 1550
+Wire Wire Line
+	5650 1550 5800 1550
+Wire Wire Line
+	5800 1550 5800 1450
+Wire Wire Line
+	5750 1450 5900 1450
+Connection ~ 5800 1450
+Wire Wire Line
+	5550 1450 5500 1450
+Wire Wire Line
+	5500 1450 5500 1300
+Connection ~ 5500 1300
 $EndSCHEMATC

Commit message: Finished Range Switching/Filters
Parts:
- gave numbers to parts that had none: 11
Connections:
- wire segments 177 -> 179

Commit message: Changed to KiCAD 5
Parts:
- C701, C713, C714, C723: symbol CP1_Small -> Device:CP1_Small
- C702, C703, C704, C705, C706, C707, C708, C709, C710, C711, C712, C715, C716, C717, C718, C719, C720, C721, C722, C724: symbol C_Small -> Device:C_Small
- L701, L702: symbol L_Small -> Device:L_Small
- Q701: symbol Q_NMOS_DGS -> Device:Q_NMOS_DGS
- R701, R702, R704, R705, R706, R707: footprint (none) -> Resistors_SMD:R_0603; symbol R_Small -> Device:R_Small
- R703: footprint (none) -> Resistors_SMD:R_0603; symbol R -> Device:R
- RN701: symbol R_Pack08 -> Device:R_Pack08; Field4 (none) -> test
- RN702: symbol Voltage_Divider -> Device:Voltage_Divider
- RV701: symbol POT_TRIM -> Device:R_POT_TRIM
- U701: symbol MIC7211 -> frontend_additional_components:MIC7211
- U702: symbol AD54xx -> frontend_additional_components:AD54xx
- U703: symbol LMT88 -> frontend_additional_components:LMT88
- U704, U705: symbol NCP508 -> frontend_additional_components:NCP508
- U706: symbol MAX11960 -> frontend_additional_components:MAX11960
- U707: symbol LTC2055 -> frontend_additional_components:LTC2055
- U708: symbol TSP73001 -> frontend_additional_components:TSP73001
- W701, W702, W703, W704, W705, W706, W707: symbol TEST_1P -> Connector:Test_Point
Connections:
- wire segments 179 -> 242

Commit message: Footrpints and Parts Specification
Parts:
- removed RN701: 33, symbol Device:R_Pack08
- added RN701, RN703: 22, Resistor_SMD:R_Array_Convex_4x0402, symbol Device:R_Pack04
- C701, C723: footprint (none) -> Capacitor_SMD:CP_Elec_4x3; Digikey (none) -> 732-8430-1-ND; Manufacturer (none) -> Würth; Mouser (none) -> 710-865080440002; Part Number (none) -> 865080440002
- C702, C703, C704, C705, C706, C707, C708, C709, C710, C711, C712, C715, C716, C717, C722, C724: footprint (none) -> Capacitor_SMD:C_0603_1608Metric
- C713, C714: footprint (none) -> Capacitor_SMD:C_1206_3216Metric
- C718, C719, C720, C721: footprint (none) -> Capacitor_SMD:C_0805_2012Metric
- L701, L702: footprint (none) -> Inductor_SMD:L_0805_2012Metric
- Q701: value Q_NMOS_DGS -> SSM3K329R,LF; footprint (none) -> Package_TO_SOT_SMD:SOT-23; Digikey (none) -> SSM3K329RLFCT-ND; Manufacturer (none) -> Toshiba; Mouser (none) -> 757-SSM3K329RLF; Part Number (none) -> SSM3K329R,LF
- R701, R702, R703, R704, R705, R706, R707: footprint Resistors_SMD:R_0603 -> Resistor_SMD:R_0603_1608Metric
- RV701: footprint (none) -> Potentiometer_SMD:Potentiometer_Bourns_3214X_Vertical; Digikey (none) -> 3214X-1-103ECT-ND; Manufacturer (none) -> Bourns; Mouser (none) -> 652-3214X-1-103E; Part Number (none) -> 3214X-1-103E
- U701: footprint (none) -> Package_TO_SOT_SMD:SOT-23-6
- U702: footprint (none) -> Package_SO:SOIC-8_3.9x4.9mm_P1.27mm
- U703: footprint (none) -> Package_TO_SOT_SMD:SOT-353_SC-70-5; Digikey (none) -> 296-38167-1-ND; Manufacturer (none) -> TI; Mouser (none) -> 595-LMT88DCKR; Part Number (none) -> LMT88DCKR
- U704, U705: footprint (none) -> Package_TO_SOT_SMD:SOT-353_SC-70-5; Digikey (none) -> NCP508SQ18T1GOSCT-ND; Manufacturer (none) -> OnSemi; Mouser (none) -> 863-NCP508SQ18T1G; Part Number NCP508MT33TBG -> NCP508SQ18T1G
- U706: footprint (none) -> Package_DFN_QFN:QFN-32-1EP_5x5mm_P0.5mm_EP3.45x3.45mm; Digikey (none) -> MAX11960ETJ+-ND; Manufacturer (none) -> Maxim; Mouser (none) -> 700-MAX11960ETJ+; Part Number (none) -> MAX11960ETJ+
- U707: footprint (none) -> Package_SO:TSSOP-8_3x3mm_P0.65mm; Digikey (none) -> LTC2055CMS8#PBF-ND; Manufacturer (none) -> Linear Technology; Mouser (none) -> 584-LTC2055CMS8#PBF; Part Number (none) -> LTC2055CMS8#PBF
- U708: footprint (none) -> Package_TO_SOT_SMD:SOT-23-6; symbol frontend_additional_components:TSP73001 -> frontend_additional_components:TPS73001
- W701, W702, W703, W704, W705, W706, W707: footprint (none) -> TestPoint:TestPoint_Pad_D1.0mm
Connections:
- wire segments 242 -> 250

Commit message: Finished Footprints, ERC
Parts:
- removed RN702: Voltage_Divider, symbol Device:Voltage_Divider
- added R708, R709: R_Small, Resistor_SMD:R_0603_1608Metric, symbol Device:R_Small
Connections:
- net labels removed: V_ref
- wire segments 250 -> 257
- no-connect marks 4 -> 2
Changed lines of the file:
@@
 $Descr A4 8268 11693 portrait
 encoding utf-8
-Sheet 7 7
+Sheet 6 7
 Title "Analog-Digital Converter, Reference Voltage"
 Date ""
@@
 L power:GNDPWR #PWR0105
 U 1 1 5B1A5AC8
-P 3950 6600
-F 0 "#PWR0105" H 3950 6400 50  0001 C CNN
-F 1 "GNDPWR" H 3950 6470 50  0000 C CNN
-F 2 "" H 3950 6550 50  0000 C CNN
-F 3 "" H 3950 6550 50  0000 C CNN
-	1    3950 6600
+P 3950 6700
+F 0 "#PWR0105" H 3950 6500 50  0001 C CNN
+F 1 "GNDPWR" H 3950 6570 50  0000 C CNN
+F 2 "" H 3950 6650 50  0000 C CNN
+F 3 "" H 3950 6650 50  0000 C CNN
+	1    3950 6700
 	1    0    0    -1
 $EndComp
@@
 $EndComp
 Text GLabel 6800 8550 2    60   Output ~ 0
-V_ref
+v_ref
 Text GLabel 6700 9150 2    60   Output ~ 0
 v_ref_2
-NoConn ~ 6200 8850
-NoConn ~ 6200 9450
-$Comp
-L Device:Voltage_Divider RN702
-U 1 1 5B21A366
-P 5500 9250
-F 0 "RN702" V 5325 9250 50  0000 C CNN
-F 1 "Voltage_Divider" V 5400 9250 50  0000 C CNN
-F 2 "" V 5975 9250 50  0001 C CNN
-F 3 "" H 5700 9250 50  0000 C CNN
-	1    5500 9250
-	1    0    0    -1
-$EndComp
 $Comp
 L power:GND #PWR0115
@@
 $EndComp
 Text GLabel 6400 5250 2    60   Input ~ 0
-V_ref
+v_ref
 $Comp
 L Device:C_Small C709
@@
 Wire Wire Line
 	4250 6550 4250 6450
-Connection ~ 3950 6550
 Wire Wire Line
 	4150 6450 4150 6550
@@
 Wire Wire Line
 	5500 9500 5500 9550
-Wire Wire Line
-	5950 9250 5650 9250
 Wire Wire Line
 	4850 8050 4850 8150
@@
 	5150 1850 5150 1650
 Connection ~ 5250 1850
-Wire Wire Line
-	6800 1300 6950 1300
 Wire Wire Line
 	4950 1150 4950 1300
@@
 Connection ~ 5500 1300
 Wire Wire Line
-	6800 1450 6950 1450
-Wire Wire Line
-	6950 1450 6950 1300
-Connection ~ 6950 1300
-Wire Wire Line
-	3950 6550 3950 6600
-Wire Wire Line
 	4150 6550 4250 6550
 Wire Wire Line
@@
 Wire Wire Line
 	5500 1300 5900 1300
-Wire Wire Line
-	6950 1300 7250 1300
 $Comp
 L Device:R_Pack04 RN701
@@
 Wire Wire Line
 	3500 4950 3550 4950
+$Comp
+L Device:R_Small R708
+U 1 1 5B57E285
+P 5500 9100
+F 0 "R708" H 5559 9146 50  0000 L CNN
+F 1 "R_Small" H 5559 9055 50  0000 L CNN
+F 2 "Resistor_SMD:R_0603_1608Metric" H 5500 9100 50  0001 C CNN
+F 3 "~" H 5500 9100 50  0001 C CNN
+	1    5500 9100
+	1    0    0    -1
+$EndComp
+$Comp
+L Device:R_Small R709
+U 1 1 5B57E353
+P 5500 9400
+F 0 "R709" H 5559 9446 50  0000 L CNN
+F 1 "R_Small" H 5559 9355 50  0000 L CNN
+F 2 "Resistor_SMD:R_0603_1608Metric" H 5500 9400 50  0001 C CNN
+F 3 "~" H 5500 9400 50  0001 C CNN
+	1    5500 9400
+	1    0    0    -1
+$EndComp
+Wire Wire Line
+	5500 9200 5500 9250
+Wire Wire Line
+	5500 9250 5950 9250
+Connection ~ 5500 9250
+Wire Wire Line
+	5500 9250 5500 9300
+Wire Wire Line
+	6800 1300 7000 1300
+Wire Wire Line
+	6800 1450 7000 1450
+Wire Wire Line
+	7000 1450 7000 1300
+Connection ~ 7000 1300
+Wire Wire Line
+	7000 1300 7250 1300
+Wire Wire Line
+	3950 6700 3950 6550
+Connection ~ 3950 6550
+$Comp
+L power:PWR_FLAG #FLG0103
+U 1 1 5B7AAEF0
+P 1850 8500
+F 0 "#FLG0103" H 1850 8575 50  0001 C CNN
+F 1 "PWR_FLAG" H 1850 8674 50  0000 C CNN
+F 2 "" H 1850 8500 50  0001 C CNN
+F 3 "~" H 1850 8500 50  0001 C CNN
+	1    1850 8500
+	1    0    0    -1
+$EndComp
+Wire Wire Line
+	1850 8500 1850 8650
+$Comp
+L power:+5V #PWR0146
+U 1 1 5B70BEE8
+P 6100 8800
+F 0 "#PWR0146" H 6100 8650 50  0001 C CNN
+F 1 "+5V" H 6100 8940 50  0000 C CNN
+F 2 "" H 6100 8800 50  0000 C CNN
+F 3 "" H 6100 8800 50  0000 C CNN
+	1    6100 8800
+	0    -1   -1   0
+$EndComp
+$Comp
+L power:GND #PWR0147
+U 1 1 5B70BF61
+P 6200 9600
+F 0 "#PWR0147" H 6200 9350 50  0001 C CNN
+F 1 "GND" H 6200 9450 50  0000 C CNN
+F 2 "" H 6200 9600 50  0000 C CNN
+F 3 "" H 6200 9600 50  0000 C CNN
+	1    6200 9600
+	1    0    0    -1
+$EndComp
+Wire Wire Line
+	6100 8800 6200 8800
+Wire Wire Line
+	6200 8800 6200 8850
+Wire Wire Line
+	6200 9600 6200 9450
+$Comp
+L power:PWR_FLAG #FLG0601
+U 1 1 5B72FF50
+P 3750 3400
+F 0 "#FLG0601" H 3750 3475 50  0001 C CNN
+F 1 "PWR_FLAG" H 3750 3574 50  0000 C CNN
+F 2 "" H 3750 3400 50  0001 C CNN
+F 3 "~" H 3750 3400 50  0001 C CNN
+	1    3750 3400
+	1    0    0    -1
+$EndComp
+Wire Wire Line
+	3750 3400 3750 3550
 $EndSCHEMATC

Commit message: Fixed minor net issues, begun routing
Parts:
- R703: footprint Resistor_SMD:R_0603_1608Metric -> Resistor_SMD:R_1206_3216Metric
Changed lines of the file:
@@
 F 0 "R703" V 2730 7900 50  0000 C CNN
 F 1 "R" V 2650 7900 50  0000 C CNN
-F 2 "Resistor_SMD:R_0603_1608Metric" V 2580 7900 50  0001 C CNN
+F 2 "Resistor_SMD:R_1206_3216Metric" V 2580 7900 50  0001 C CNN
 F 3 "" H 2650 7900 50  0000 C CNN
 	1    2650 7900

Commit message: Begun routing
Parts:
- removed C712: C_Small, Capacitor_SMD:C_0603_1608Metric, symbol Device:C_Small
- removed RN701, RN703: 22, Resistor_SMD:R_Array_Convex_4x0402, symbol Device:R_Pack04
- added R603, R604, R605, R606, R607, R608, R609: R_Small, Resistor_SMD:R_0603_1608Metric, symbol Device:R_Small
Connections:
- net labels removed: GNDPWR
- wire segments 257 -> 254
- no-connect marks 2 -> 0
Changed lines of the file:
@@
-$EndComp
-$Comp
-L power:GNDPWR #PWR0105
-U 1 1 5B1A5AC8
-P 3950 6700
-F 0 "#PWR0105" H 3950 6500 50  0001 C CNN
-F 1 "GNDPWR" H 3950 6570 50  0000 C CNN
-F 2 "" H 3950 6650 50  0000 C CNN
-F 3 "" H 3950 6650 50  0000 C CNN
-	1    3950 6700
-	1    0    0    -1
 $EndComp
 $Comp
@@
 $EndComp
 $Comp
-L Device:C_Small C712
-U 1 1 5B21D34E
-P 3750 3800
-F 0 "C712" H 3760 3870 50  0000 L CNN
-F 1 "C_Small" H 3760 3720 50  0000 L CNN
-F 2 "Capacitor_SMD:C_0603_1608Metric" H 3750 3800 50  0001 C CNN
-F 3 "" H 3750 3800 50  0000 C CNN
-	1    3750 3800
-	-1   0    0    1
-$EndComp
-$Comp
 L frontend_additional_components:NCP508 U705
 U 1 1 5B21E4D7
@@
 	3050 5550 3550 5550
 Wire Wire Line
-	1650 4850 2650 4850
-Wire Wire Line
-	2650 4950 1650 4950
-Wire Wire Line
-	1650 5050 2650 5050
-Wire Wire Line
-	2650 5150 1650 5150
-Wire Wire Line
-	1650 5350 2650 5350
-Wire Wire Line
-	2650 5450 1650 5450
-Wire Wire Line
-	1650 5550 2650 5550
-Wire Wire Line
 	6400 5600 5600 5600
 Wire Wire Line
@@
 	4050 3400 4050 3550
 Connection ~ 3950 3550
-Wire Wire Line
-	3750 3700 3750 3550
 Connection ~ 3750 3550
-Wire Wire Line
-	3750 4000 3750 3900
-Connection ~ 3550 4000
 Wire Wire Line
 	2850 2950 2850 2850
@@
 Wire Wire Line
 	2450 6500 3350 6500
-NoConn ~ 3050 5650
-NoConn ~ 2650 5650
 Text HLabel 6800 8300 2    60   Output ~ 0
 v_ref
@@
 	3750 3550 3950 3550
 Wire Wire Line
-	3550 4000 3750 4000
-Wire Wire Line
 	3750 2350 4350 2350
 Wire Wire Line
@@
 Wire Wire Line
 	5500 1300 5900 1300
-$Comp
-L Device:R_Pack04 RN701
-U 1 1 5B67A8F4
-P 2850 5050
-F 0 "RN701" V 2433 5050 50  0000 C CNN
-F 1 "22" V 2524 5050 50  0000 C CNN
-F 2 "Resistor_SMD:R_Array_Convex_4x0402" V 3125 5050 50  0001 C CNN
-F 3 "~" H 2850 5050 50  0001 C CNN
-F 4 "Y10220CT-ND " H 0   0   50  0001 C CNN "Digikey"
-F 5 "Panasonic" H 0   0   50  0001 C CNN "Manufacturer"
-F 6 "667-EXB-N8V220JX " H 0   0   50  0001 C CNN "Mouser"
-F 7 "EXB-N8V220JX " H 0   0   50  0001 C CNN "Part Number"
-	1    2850 5050
-	0    1    1    0
-$EndComp
-$Comp
-L Device:R_Pack04 RN703
-U 1 1 5B67AB13
-P 2850 5550
-F 0 "RN703" V 2433 5550 50  0000 C CNN
-F 1 "22" V 2524 5550 50  0000 C CNN
-F 2 "Resistor_SMD:R_Array_Convex_4x0402" V 3125 5550 50  0001 C CNN
-F 3 "~" H 2850 5550 50  0001 C CNN
-F 4 "Y10220CT-ND " H 0   0   50  0001 C CNN "Digikey"
-F 5 "Panasonic" H 0   0   50  0001 C CNN "Manufacturer"
-F 6 "667-EXB-N8V220JX " H 0   0   50  0001 C CNN "Mouser"
-F 7 "EXB-N8V220JX " H 0   0   50  0001 C CNN "Part Number"
-	1    2850 5550
-	0    1    1    0
-$EndComp
 Wire Wire Line
 	3550 5250 3200 5250
@@
 Wire Wire Line
 	3750 3400 3750 3550
+$Comp
+L Device:R_Small R603
+U 1 1 5B5B145D
+P 2950 4850
+F 0 "R603" V 2754 4850 50  0000 C CNN
+F 1 "R_Small" V 2845 4850 50  0000 C CNN
+F 2 "Resistor_SMD:R_0603_1608Metric" H 2950 4850 50  0001 C CNN
+F 3 "~" H 2950 4850 50  0001 C CNN
+	1    2950 4850
+	0    1    1    0
+$EndComp
+$Comp
+L Device:R_Small R604
+U 1 1 5B5B166A
+P 2950 4950
+F 0 "R604" V 2754 4950 50  0000 C CNN
+F 1 "R_Small" V 2845 4950 50  0000 C CNN
+F 2 "Resistor_SMD:R_0603_1608Metric" H 2950 4950 50  0001 C CNN
+F 3 "~" H 2950 4950 50  0001 C CNN
+	1    2950 4950
+	0    1    1    0
+$EndComp
+$Comp
+L Device:R_Small R605
+U 1 1 5B5B17B2
+P 2950 5050
+F 0 "R605" V 2754 5050 50  0000 C CNN
+F 1 "R_Small" V 2845 5050 50  0000 C CNN
+F 2 "Resistor_SMD:R_0603_1608Metric" H 2950 5050 50  0001 C CNN
+F 3 "~" H 2950 5050 50  0001 C CNN
+	1    2950 5050
+	0    1    1    0
+$EndComp
+$Comp
+L Device:R_Small R606
+U 1 1 5B5B18BF
+P 2950 5150
+F 0 "R606" V 2754 5150 50  0000 C CNN
+F 1 "R_Small" V 2845 5150 50  0000 C CNN
+F 2 "Resistor_SMD:R_0603_1608Metric" H 2950 5150 50  0001 C CNN
+F 3 "~" H 2950 5150 50  0001 C CNN
+	1    2950 5150
+	0    1    1    0
+$EndComp
+$Comp
+L Device:R_Small R607
+U 1 1 5B5B19D0
+P 2950 5350
+F 0 "R607" V 2754 5350 50  0000 C CNN
+F 1 "R_Small" V 2845 5350 50  0000 C CNN
+F 2 "Resistor_SMD:R_0603_1608Metric" H 2950 5350 50  0001 C CNN
+F 3 "~" H 2950 5350 50  0001 C CNN
+	1    2950 5350
+	0    1    1    0
+$EndComp
+$Comp
+L Device:R_Small R608
+U 1 1 5B5B1AE5
+P 2950 5450
+F 0 "R608" V 2754 5450 50  0000 C CNN
+F 1 "R_Small" V 2845 5450 50  0000 C CNN
+F 2 "Resistor_SMD:R_0603_1608Metric" H 2950 5450 50  0001 C CNN
+F 3 "~" H 2950 5450 50  0001 C CNN
+	1    2950 5450
+	0    1    1    0
+$EndComp
+$Comp
+L Device:R_Small R609
+U 1 1 5B5B1BFE
+P 2950 5550
+F 0 "R609" V 2754 5550 50  0000 C CNN
+F 1 "R_Small" V 2845 5550 50  0000 C CNN
+F 2 "Resistor_SMD:R_0603_1608Metric" H 2950 5550 50  0001 C CNN
+F 3 "~" H 2950 5550 50  0001 C CNN
+	1    2950 5550
+	0    1    1    0
+$EndComp
+Wire Wire Line
+	1650 5550 2850 5550
+Wire Wire Line
+	1650 5450 2850 5450
+Wire Wire Line
+	1650 5350 2850 5350
+Wire Wire Line
+	1650 5150 2850 5150
+Wire Wire Line
+	1650 5050 2850 5050
+Wire Wire Line
+	1650 4950 2850 4950
+Wire Wire Line
+	1650 4850 2850 4850
+$Comp
+L power:GND #PWR0105
+U 1 1 5B65641E
+P 3950 6700
+F 0 "#PWR0105" H 3950 6450 50  0001 C CNN
+F 1 "GND" H 3950 6550 50  0000 C CNN
+F 2 "" H 3950 6700 50  0000 C CNN
+F 3 "" H 3950 6700 50  0000 C CNN
+	1    3950 6700
+	1    0    0    -1
+$EndComp
 $EndSCHEMATC
