File: components_predev/frontend/hardware/ADC.sch (KiCad schematic (older format))
At the start: 58 parts, among them Q701 SSM3K329R,LF, U701 MIC7211, U702 ADR4533, U703 LMT88, U704 NCP508, U705 NCP508, U706 MAX11960, U707 LTC2055, U708 TSP73001

Commit message: Finished routing, begun component specification
Parts:
- C701, C723: value CP1_Small -> 22u; Digikey 732-8430-1-ND -> 732-8413-1-ND; Mouser 710-865080440002 -> 710-865080340003; Part Number 865080440002 -> 865080340003; Voltage (none) -> 16 V
- C702, C704, C706, C709, C710, C711, C715, C716, C722: value C_Small -> 100n
- C703, C705, C707, C708, C717: value C_Small -> 10u
- C713, C714: value CP1_Small -> 220u; Dielectric (none) -> X5R; Digikey (none) -> 490-13970-1-ND; Manufacturer (none) -> MuRata; Part Number (none) -> GRM31CR60J227ME11L; Voltage (none) -> 6.3 V
- R603, R604, R605, R606, R607, R608, R609: value R_Small -> 22
- R701: value R_Small -> 10k
Other:
- note added: "Heater"
Changed lines of the file:
@@
 P 1850 9100
 F 0 "C703" H 1860 9170 50  0000 L CNN
-F 1 "C_Small" H 1860 9020 50  0000 L CNN
+F 1 "10u" H 1860 9020 50  0000 L CNN
 F 2 "Capacitor_SMD:C_0603_1608Metric" H 1850 9100 50  0001 C CNN
 F 3 "" H 1850 9100 50  0000 C CNN
@@
 P 3350 3800
 F 0 "C705" H 3360 3870 50  0000 L CNN
-F 1 "C_Small" H 3360 3720 50  0000 L CNN
+F 1 "10u" H 3360 3720 50  0000 L CNN
 F 2 "Capacitor_SMD:C_0603_1608Metric" H 3350 3800 50  0001 C CNN
 F 3 "" H 3350 3800 50  0000 C CNN
@@
 P 3750 8850
 F 0 "C713" H 3760 8920 50  0000 L CNN
-F 1 "CP1_Small" H 3760 8770 50  0000 L CNN
+F 1 "220u" H 3760 8770 50  0000 L CNN
 F 2 "Capacitor_SMD:C_1206_3216Metric" H 3750 8850 50  0001 C CNN
 F 3 "" H 3750 8850 50  0000 C CNN
+F 4 "X5R" H 0   0   50  0001 C CNN "Dielectric"
+F 5 "490-13970-1-ND " H 0   0   50  0001 C CNN "Digikey"
+F 6 "MuRata" H 0   0   50  0001 C CNN "Manufacturer"
+F 7 " 	GRM31CR60J227ME11L " H 0   0   50  0001 C CNN "Part Number"
+F 8 "6.3 V" H 0   0   50  0001 C CNN "Voltage"
 	1    3750 8850
 	1    0    0    -1
@@
 P 3750 9250
 F 0 "C714" H 3760 9320 50  0000 L CNN
-F 1 "CP1_Small" H 3760 9170 50  0000 L CNN
+F 1 "220u" H 3760 9170 50  0000 L CNN
 F 2 "Capacitor_SMD:C_1206_3216Metric" H 3750 9250 50  0001 C CNN
 F 3 "" H 3750 9250 50  0000 C CNN
+F 4 "X5R" H 0   0   50  0001 C CNN "Dielectric"
+F 5 "490-13970-1-ND " H 0   0   50  0001 C CNN "Digikey"
+F 6 "MuRata" H 0   0   50  0001 C CNN "Manufacturer"
+F 7 " 	GRM31CR60J227ME11L " H 0   0   50  0001 C CNN "Part Number"
+F 8 "6.3 V" H 0   0   50  0001 C CNN "Voltage"
 	1    3750 9250
 	1    0    0    -1
@@
 P 5050 8150
 F 0 "C715" H 5060 8220 50  0000 L CNN
-F 1 "C_Small" H 5060 8070 50  0000 L CNN
+F 1 "100n" H 5060 8070 50  0000 L CNN
 F 2 "Capacitor_SMD:C_0603_1608Metric" H 5050 8150 50  0001 C CNN
 F 3 "" H 5050 8150 50  0000 C CNN
@@
 P 3550 3800
 F 0 "C709" H 3560 3870 50  0000 L CNN
-F 1 "C_Small" H 3560 3720 50  0000 L CNN
+F 1 "100n" H 3560 3720 50  0000 L CNN
 F 2 "Capacitor_SMD:C_0603_1608Metric" H 3550 3800 50  0001 C CNN
 F 3 "" H 3550 3800 50  0000 C CNN
@@
 P 3550 2600
 F 0 "C708" H 3560 2670 50  0000 L CNN
-F 1 "C_Small" H 3560 2520 50  0000 L CNN
+F 1 "10u" H 3560 2520 50  0000 L CNN
 F 2 "Capacitor_SMD:C_0603_1608Metric" H 3550 2600 50  0001 C CNN
 F 3 "" H 3550 2600 50  0000 C CNN
@@
 P 3750 2600
 F 0 "C711" H 3760 2670 50  0000 L CNN
-F 1 "C_Small" H 3760 2520 50  0000 L CNN
+F 1 "100n" H 3760 2520 50  0000 L CNN
 F 2 "Capacitor_SMD:C_0603_1608Metric" H 3750 2600 50  0001 C CNN
 F 3 "" H 3750 2600 50  0000 C CNN
@@
 P 3550 1550
 F 0 "C707" H 3560 1620 50  0000 L CNN
-F 1 "C_Small" H 3560 1470 50  0000 L CNN
+F 1 "10u" H 3560 1470 50  0000 L CNN
 F 2 "Capacitor_SMD:C_0603_1608Metric" H 3550 1550 50  0001 C CNN
 F 3 "" H 3550 1550 50  0000 C CNN
@@
 P 3750 1550
 F 0 "C710" H 3760 1620 50  0000 L CNN
-F 1 "C_Small" H 3760 1470 50  0000 L CNN
+F 1 "100n" H 3760 1470 50  0000 L CNN
 F 2 "Capacitor_SMD:C_0603_1608Metric" H 3750 1550 50  0001 C CNN
 F 3 "" H 3750 1550 50  0000 C CNN
@@
 P 1500 1550
 F 0 "C702" H 1510 1620 50  0000 L CNN
-F 1 "C_Small" H 1510 1470 50  0000 L CNN
+F 1 "100n" H 1510 1470 50  0000 L CNN
 F 2 "Capacitor_SMD:C_0603_1608Metric" H 1500 1550 50  0001 C CNN
 F 3 "" H 1500 1550 50  0000 C CNN
@@
 P 1250 1550
 F 0 "C701" H 1260 1620 50  0000 L CNN
-F 1 "CP1_Small" H 1260 1470 50  0000 L CNN
+F 1 "22u" H 1260 1470 50  0000 L CNN
 F 2 "Capacitor_SMD:CP_Elec_4x3" H 1250 1550 50  0001 C CNN
 F 3 "" H 1250 1550 50  0000 C CNN
-F 4 "732-8430-1-ND" H 0   0   50  0001 C CNN "Digikey"
+F 4 "732-8413-1-ND " H 0   0   50  0001 C CNN "Digikey"
 F 5 "Würth" H 0   0   50  0001 C CNN "Manufacturer"
-F 6 "710-865080440002" H 0   0   50  0001 C CNN "Mouser"
-F 7 "865080440002" H 0   0   50  0001 C CNN "Part Number"
+F 6 "710-865080340003 " H 0   0   50  0001 C CNN "Mouser"
+F 7 "865080340003 " H 0   0   50  0001 C CNN "Part Number"
+F 8 "16 V" H 0   0   50  0001 C CNN "Voltage"
 	1    1250 1550
 	1    0    0    -1
@@
 P 5350 1550
 F 0 "C717" H 5360 1620 50  0000 L CNN
-F 1 "C_Small" H 5360 1470 50  0000 L CNN
+F 1 "10u" H 5360 1470 50  0000 L CNN
 F 2 "Capacitor_SMD:C_0603_1608Metric" H 5350 1550 50  0001 C CNN
 F 3 "" H 5350 1550 50  0000 C CNN
@@
 P 5150 1550
 F 0 "C716" H 5160 1620 50  0000 L CNN
-F 1 "C_Small" H 5160 1470 50  0000 L CNN
+F 1 "100n" H 5160 1470 50  0000 L CNN
 F 2 "Capacitor_SMD:C_0603_1608Metric" H 5150 1550 50  0001 C CNN
 F 3 "" H 5150 1550 50  0000 C CNN
@@
 P 7250 1550
 F 0 "C722" H 7260 1620 50  0000 L CNN
-F 1 "C_Small" H 7260 1470 50  0000 L CNN
+F 1 "100n" H 7260 1470 50  0000 L CNN
 F 2 "Capacitor_SMD:C_0603_1608Metric" H 7250 1550 50  0001 C CNN
 F 3 "" H 7250 1550 50  0000 C CNN
@@
 P 7500 1550
 F 0 "C723" H 7510 1620 50  0000 L CNN
-F 1 "CP1_Small" H 7510 1470 50  0000 L CNN
+F 1 "22u" H 7510 1470 50  0000 L CNN
 F 2 "Capacitor_SMD:CP_Elec_4x3" H 7500 1550 50  0001 C CNN
 F 3 "" H 7500 1550 50  0000 C CNN
-F 4 "732-8430-1-ND" H 0   0   50  0001 C CNN "Digikey"
+F 4 "732-8413-1-ND " H 0   0   50  0001 C CNN "Digikey"
 F 5 "Würth" H 0   0   50  0001 C CNN "Manufacturer"
-F 6 "710-865080440002" H 0   0   50  0001 C CNN "Mouser"
-F 7 "865080440002" H 0   0   50  0001 C CNN "Part Number"
+F 6 "710-865080340003 " H 0   0   50  0001 C CNN "Mouser"
+F 7 "865080340003 " H 0   0   50  0001 C CNN "Part Number"
+F 8 "16 V" H 0   0   50  0001 C CNN "Voltage"
 	1    7500 1550
 	-1   0    0    -1
@@
 U 1 1 5B225530
 P 1650 7800
-F 0 "Q701" H 1850 7850 50  0000 L CNN
-F 1 "SSM3K329R,LF" H 1850 7750 50  0000 L CNN
+F 0 "Q701" V 1550 8000 50  0000 L CNN
+F 1 "SSM3K329R,LF" V 1650 8000 50  0000 L CNN
 F 2 "Package_TO_SOT_SMD:SOT-23" H 1850 7900 50  0001 C CNN
 F 3 "" H 1650 7800 50  0000 C CNN
@@
 P 3350 6950
 F 0 "C706" H 3360 7020 50  0000 L CNN
-F 1 "C_Small" H 3360 6870 50  0000 L CNN
+F 1 "100n" H 3360 6870 50  0000 L CNN
 F 2 "Capacitor_SMD:C_0603_1608Metric" H 3350 6950 50  0001 C CNN
 F 3 "" H 3350 6950 50  0000 C CNN
@@
 P 1300 7700
 F 0 "R701" H 1330 7720 50  0000 L CNN
-F 1 "R_Small" H 1330 7660 50  0000 L CNN
+F 1 "10k" H 1330 7660 50  0000 L CNN
 F 2 "Resistor_SMD:R_0603_1608Metric" H 1300 7700 50  0001 C CNN
 F 3 "" H 1300 7700 50  0000 C CNN
@@
 P 2150 7050
 F 0 "C704" H 2160 7120 50  0000 L CNN
-F 1 "C_Small" H 2160 6970 50  0000 L CNN
+F 1 "100n" H 2160 6970 50  0000 L CNN
 F 2 "Capacitor_SMD:C_0603_1608Metric" H 2150 7050 50  0001 C CNN
 F 3 "" H 2150 7050 50  0000 C CNN
@@
 U 1 1 5B5B145D
 P 2950 4850
-F 0 "R603" V 2754 4850 50  0000 C CNN
-F 1 "R_Small" V 2845 4850 50  0000 C CNN
+F 0 "R603" V 2900 4600 50  0000 C CNN
+F 1 "22" V 2950 4850 50  0000 C CNN
 F 2 "Resistor_SMD:R_0603_1608Metric" H 2950 4850 50  0001 C CNN
 F 3 "~" H 2950 4850 50  0001 C CNN
@@
 U 1 1 5B5B166A
 P 2950 4950
-F 0 "R604" V 2754 4950 50  0000 C CNN
-F 1 "R_Small" V 2845 4950 50  0000 C CNN
+F 0 "R604" V 2900 4700 50  0000 C CNN
+F 1 "22" V 2950 4950 50  0000 C CNN
 F 2 "Resistor_SMD:R_0603_1608Metric" H 2950 4950 50  0001 C CNN
 F 3 "~" H 2950 4950 50  0001 C CNN
@@
 U 1 1 5B5B17B2
 P 2950 5050
-F 0 "R605" V 2754 5050 50  0000 C CNN
-F 1 "R_Small" V 2845 5050 50  0000 C CNN
+F 0 "R605" V 2900 4800 50  0000 C CNN
+F 1 "22" V 2950 5050 50  0000 C CNN
 F 2 "Resistor_SMD:R_0603_1608Metric" H 2950 5050 50  0001 C CNN
 F 3 "~" H 2950 5050 50  0001 C CNN
@@
 U 1 1 5B5B18BF
 P 2950 5150
-F 0 "R606" V 2754 5150 50  0000 C CNN
-F 1 "R_Small" V 2845 5150 50  0000 C CNN
+F 0 "R606" V 2900 4900 50  0000 C CNN
+F 1 "22" V 2950 5150 50  0000 C CNN
 F 2 "Resistor_SMD:R_0603_1608Metric" H 2950 5150 50  0001 C CNN
 F 3 "~" H 2950 5150 50  0001 C CNN
@@
 U 1 1 5B5B19D0
 P 2950 5350
-F 0 "R607" V 2754 5350 50  0000 C CNN
-F 1 "R_Small" V 2845 5350 50  0000 C CNN
+F 0 "R607" V 3000 5550 50  0000 C CNN
+F 1 "22" V 2950 5350 50  0000 C CNN
 F 2 "Resistor_SMD:R_0603_1608Metric" H 2950 5350 50  0001 C CNN
 F 3 "~" H 2950 5350 50  0001 C CNN
@@
 U 1 1 5B5B1AE5
 P 2950 5450
-F 0 "R608" V 2754 5450 50  0000 C CNN
-F 1 "R_Small" V 2845 5450 50  0000 C CNN
+F 0 "R608" V 3000 5650 50  0000 C CNN
+F 1 "22" V 2950 5450 50  0000 C CNN
 F 2 "Resistor_SMD:R_0603_1608Metric" H 2950 5450 50  0001 C CNN
 F 3 "~" H 2950 5450 50  0001 C CNN
@@
 U 1 1 5B5B1BFE
 P 2950 5550
-F 0 "R609" V 2754 5550 50  0000 C CNN
-F 1 "R_Small" V 2845 5550 50  0000 C CNN
+F 0 "R609" V 3000 5750 50  0000 C CNN
+F 1 "22" V 2950 5550 50  0000 C CNN
 F 2 "Resistor_SMD:R_0603_1608Metric" H 2950 5550 50  0001 C CNN
 F 3 "~" H 2950 5550 50  0001 C CNN
@@
 	1    0    0    -1
 $EndComp
+Wire Notes Line
+	2650 8100 2650 8400
+Text Notes 2350 8300 0    50   ~ 0
+Heater
 $EndSCHEMATC

Commit message: Some Updates from Testing
Parts:
- C702, C704, C706, C709, C710, C711, C715, C716, C722: Digikey (none) -> 1276-1005-1-ND; Manufacturer (none) -> Samsung; Note (none) -> VH; Part Number (none) -> CL10B104K08NNNC; Voltage (none) -> 16V
- C703, C705, C707, C708, C717: Digikey (none) -> 490-7202-1-ND; Manufacturer (none) -> MuRata; Part Number (none) -> GRM188R61E106MA73D; Voltage (none) -> 25 V
- C713, C714: Part Number GRM31CR60J227ME11L -> GRM31CR60J227ME11L
- C718, C719, C720, C721: Digikey (none) -> 1276-6456-1-ND; Manufacturer (none) -> Samsung; Part Number (none) -> CL21A106KPFNNNG; Voltage (none) -> 10 V
- L701, L702: value L_Small -> 10u; Digikey (none) -> 587-2045-1-ND; Manufacturer (none) -> Taiyo Yuden; Part Number (none) -> LBR2012T100K
- R603, R604, R605, R606, R607, R608, R609: Digikey (none) -> 311-22.0HRCT-ND; Manufacturer (none) -> Yageo; Note (none) -> VH; Part Number (none) -> RC0603FR-0722RL
- R701: Digikey (none) -> 311-10.KHRCT-ND; Manufacturer (none) -> Yageo; Note (none) -> VH; Part Number (none) -> RC0603FR-0710KL
- R703: value R -> 143; Digikey (none) -> 541-143FCT-ND; Manufacturer (none) -> Vishay; Part Number (none) -> CRCW1206143RFKEA
- R704, R705: value R_Small -> 1k
- R708, R709: value R_Small -> 10k; Digikey (none) -> P10KDBCT-ND; Manufacturer (none) -> Panasonic; Part Number (none) -> P10KDBCT-ND
- RV701: value POT_TRIM -> 10k
- U701: Digikey (none) -> 576-1318-1-ND; Manufacturer (none) -> Microchip; Part Number (none) -> MIC7211YM5-TR
- U702: Digikey (none) -> ADR4533ARZ-ND; Manufacturer (none) -> Analog Devices; Part Number (none) -> ADR4533ARZ
- U708: value TSP73001 -> TPS73001; Digikey (none) -> 296-27055-1-ND; Manufacturer (none) -> Texas Instruments; Part Number (none) -> TPS73001DBVR
- W701, W702, W703, W704, W705, W706, W707: Note (none) -> NB
