File: components_predev/frontend/hardware/vi_filter.sch (KiCad schematic (older format))
At the start: 0 parts

Commit message: Begun Filters
Parts:
- added C? (x10): C_Small, symbol C_Small
- added L? (x20): L_Small, symbol L_Small
- added R? (x2): R_Small, symbol R_Small
- added U? (x2): ISL2863x, symbol ISL2863x
Connections:
- net labels added: v_meas+, v_meas-
- wire segments 0 -> 50

Commit message: Begun Range Switching Circuitry
Parts:
- added C? (x12): C_Small, symbol C_Small
- added D?: D, symbol D
- added K?: EE2-12NU-L, symbol EE2-12NU-L
- added K? (x3): HE3600, symbol HE3600
- added Q? (x4): Q_NMOS_DGS, symbol Q_NMOS_DGS
- added R? (x10): R_Small, symbol R_Small
- added R?: 1776-C6217, symbol 1776-C6217
- added U?: 74HC595, symbol 74HC595
- added U?: ISL2863x, symbol ISL2863x
- added U?: TSP73001, symbol TSP73001
- added U?: NCP508, symbol NCP508
Connections:
- net labels added: +12V, +3.3V, +3.3V_lin, +4.2V, +5V, -1.5V, -1V, B0, B1, B2, B3, B4, B5, B6, GND, L1, L2, L3, VCC, i_meas+, i_meas-, v_ref_2, v_sense+, v_sense-, v_sense_ext+, v_sense_ext-
- wire segments 50 -> 202
- no-connect marks 0 -> 10

Commit message: Finished Range Switching/Filters
Parts:
- removed C? (x2): C_Small, symbol C_Small
- removed U?: NCP508, symbol NCP508
- added C512, C521, C? (x2): C_Small, symbol C_Small
- added D?: D, symbol D
- added K?: EE2-12NU-L, symbol EE2-12NU-L
- added Q?: Q_NMOS_DGS, symbol Q_NMOS_DGS
- added R505, R506, R?: R_Small, symbol R_Small
- added U505: MIC5270BM5, symbol MIC5270BM5
- added U?: ISL2863x, symbol ISL2863x
- gave numbers to parts that had none: 67
Connections:
- net labels added: -5V, RCLK, SER, SRCLK, ih_sense+, ih_sense-, il_sense+, il_sense-
- net labels removed: +3.3V_lin, -1V
- wire segments 202 -> 257
- no-connect marks 10 -> 12

Commit message: Changed to KiCAD 5
Parts:
- C501, C502, C503, C504, C505, C506, C507, C508, C509, C510, C511, C512, C513, C514, C515, C516, C517, C519, C520, C521, C522, C523: symbol C_Small -> Device:C_Small
- C518, C524: renamed from C?; symbol C_Small -> Device:C_Small
- D501: symbol D -> Device:D
- D502: renamed from D?; symbol D -> Device:D
- K501, K502, K503: symbol HE3600 -> frontend_additional_components:HE3600
- K504: symbol EE2-12NU-L -> frontend_additional_components:EE2-12NU-L
- K505: renamed from K?; symbol EE2-12NU-L -> frontend_additional_components:EE2-12NU-L
- L501, L502, L503, L504, L505, L506, L507, L508, L509, L510, L511, L512, L513, L514, L515, L516, L517, L518, L519, L520: footprint (none) -> Resistors_SMD:R_0603; symbol L_Small -> Device:L_Small
- Q501, Q502, Q503, Q504: symbol Q_NMOS_DGS -> Device:Q_NMOS_DGS
- Q505: renamed from Q?; symbol Q_NMOS_DGS -> Device:Q_NMOS_DGS
- R501, R502, R503, R504, R505, R506, R507, R508, R509, R510, R511, R512, R514, R515: footprint (none) -> Resistors_SMD:R_0603; symbol R_Small -> Device:R_Small
- R513: footprint (none) -> Air_Coils_SML_NEOSID:Neosid_Air-Coil_SML_2turn_HDM0231A; symbol 1776-C6217 -> frontend_additional_components:1776-C6217
- R516: renamed from R?; footprint (none) -> Resistors_SMD:R_0603; symbol R_Small -> Device:R_Small
- U501, U503: symbol ISL2863x -> frontend_additional_components:ISL2863x
- U502: symbol 74HC595 -> 74xx:74HC595
- U504: symbol TSP73001 -> frontend_additional_components:TSP73001
- U505: symbol MIC5270BM5 -> frontend_additional_components:MIC5270BM5
- U506: renamed from U?; symbol ISL2863x -> frontend_additional_components:ISL2863x
- U507: symbol ISL2863x -> frontend_additional_components:ISL2863x; Field4 (none) -> lug
Connections:
- wire segments 257 -> 323

Commit message: Footrpints and Parts Specification
Parts:
- C501, C502, C503, C504, C505, C506, C507, C508, C509, C510, C511, C512, C513, C514, C515, C516, C517, C518, C519, C520, C521, C522, C523, C524: footprint (none) -> Capacitor_SMD:C_0603_1608Metric
- D501, D502: value D -> FDLL4148; footprint (none) -> Diode_SMD:D_MiniMELF; Digikey (none) -> FDLL4148CT-ND; Manufacturer (none) -> OnSemi; Mouser (none) -> 512-FDLL4148; Part Number (none) -> FDLL4148
- K504, K505: value EE2-12NU-L -> EC2-12NU-L
- L501, L502, L503, L504, L505, L506, L507, L508, L509, L510, L511, L512, L513, L514, L515, L516, L517, L518, L519, L520: footprint Resistors_SMD:R_0603 -> Inductor_SMD:L_0603_1608Metric
- Q501, Q502, Q503, Q504, Q505: value Q_NMOS_DGS -> SSM3K329R,LF; footprint (none) -> Package_TO_SOT_SMD:SOT-23; Digikey (none) -> SSM3K329RLFCT-ND; Manufacturer (none) -> Toshiba; Mouser (none) -> 757-SSM3K329RLF; Part Number (none) -> SSM3K329R,LF
- R501, R502, R503, R504, R505, R506, R507, R508, R509, R510, R511, R512, R514, R515, R516: footprint Resistors_SMD:R_0603 -> Resistor_SMD:R_0603_1608Metric
- R513: footprint Air_Coils_SML_NEOSID:Neosid_Air-Coil_SML_2turn_HDM0231A -> (none)
- U501, U503, U506: footprint (none) -> Package_SO:TSSOP-14_4.4x5mm_P0.65mm
- U502: footprint (none) -> Package_SO:TSSOP-16_4.4x5mm_P0.65mm
- U504: footprint (none) -> Package_TO_SOT_SMD:SOT-23-6; symbol frontend_additional_components:TSP73001 -> frontend_additional_components:TPS73001
- U505: footprint (none) -> Package_TO_SOT_SMD:SOT-23-5
- U507: footprint (none) -> Package_SO:TSSOP-14_4.4x5mm_P0.65mm; Field4 lug -> (none)

Commit message: Finished Footprints, ERC
Parts:
- K501, K502, K503: footprint (none) -> frontend_additional-footprints:HE3600
- K504, K505: footprint (none) -> frontend_additional-footprints:Kemet_EC2-12NU-L
- R513: footprint (none) -> frontend_additional-footprints:1776-C62
Connections:
- net labels added: i_range, v_ext
- net labels removed: VCC
- wire segments 323 -> 329
Changed lines of the file:
@@
 $Descr A4 11693 8268
 encoding utf-8
-Sheet 5 7
+Sheet 4 7
 Title "Voltage/Current Measurement Switching/Filtering"
 Date ""
@@
 F 2 "Package_SO:TSSOP-14_4.4x5mm_P0.65mm" H 6400 2000 60  0001 C CNN
 F 3 "" H 6400 2000 60  0001 C CNN
-F 4 "" H 6400 2000 50  0001 C CNN "Field4"
 	1    6400 2000
 	-1   0    0    -1
@@
 -1.5V
 $Comp
-L power:VCC #PWR079
-U 1 1 5B4BEB8D
-P 1000 6750
-F 0 "#PWR079" H 1000 6600 50  0001 C CNN
-F 1 "VCC" H 1000 6900 50  0000 C CNN
-F 2 "" H 1000 6750 50  0000 C CNN
-F 3 "" H 1000 6750 50  0000 C CNN
-	1    1000 6750
-	1    0    0    -1
-$EndComp
-$Comp
 L power:GND #PWR080
 U 1 1 5B4BEBFD
-P 1000 7350
-F 0 "#PWR080" H 1000 7100 50  0001 C CNN
-F 1 "GND" H 1000 7200 50  0000 C CNN
-F 2 "" H 1000 7350 50  0000 C CNN
-F 3 "" H 1000 7350 50  0000 C CNN
-	1    1000 7350
-	1    0    0    -1
+P 5300 3850
+F 0 "#PWR080" H 5300 3600 50  0001 C CNN
+F 1 "GND" H 5300 3700 50  0000 C CNN
+F 2 "" H 5300 3850 50  0000 C CNN
+F 3 "" H 5300 3850 50  0000 C CNN
+	1    5300 3850
+	-1   0    0    -1
 $EndComp
 $Comp
 L Device:C_Small C501
 U 1 1 5B4BEC6D
-P 1000 7000
-F 0 "C501" H 1010 7070 50  0000 L CNN
-F 1 "C_Small" H 1010 6920 50  0000 L CNN
-F 2 "Capacitor_SMD:C_0603_1608Metric" H 1000 7000 50  0001 C CNN
-F 3 "" H 1000 7000 50  0000 C CNN
-	1    1000 7000
-	-1   0    0    1
+P 5300 3500
+F 0 "C501" H 5310 3570 50  0000 L CNN
+F 1 "C_Small" H 5310 3420 50  0000 L CNN
+F 2 "Capacitor_SMD:C_0603_1608Metric" H 5300 3500 50  0001 C CNN
+F 3 "" H 5300 3500 50  0000 C CNN
+	1    5300 3500
+	1    0    0    1
 $EndComp
 $Comp
 L +3.3V #PWR081
 U 1 1 5B4BF1FE
-P 750 6750
+P 5550 3250
 AR Path="/5B4BF1FE" Ref="#PWR081"  Part="1"
 AR Path="/5B156993/5B4BF1FE" Ref="#PWR081"  Part="1"
-F 0 "#PWR081" H 750 6600 50  0001 C CNN
-F 1 "+3.3V" H 750 6890 50  0000 C CNN
-F 2 "" H 750 6750 50  0000 C CNN
-F 3 "" H 750 6750 50  0000 C CNN
-	1    750  6750
-	1    0    0    -1
+F 0 "#PWR081" H 5550 3100 50  0001 C CNN
+F 1 "+3.3V" H 5550 3390 50  0000 C CNN
+F 2 "" H 5550 3250 50  0000 C CNN
+F 3 "" H 5550 3250 50  0000 C CNN
+	1    5550 3250
+	-1   0    0    -1
 $EndComp
 $Comp
@@
 F 0 "R513" H 9150 1400 47  0000 C CNN
 F 1 "1776-C6217" V 9150 2000 47  0000 C CNN
-F 2 "" H 9050 2000 47  0001 C CNN
+F 2 "frontend_additional-footprints:1776-C62" H 9050 2000 47  0001 C CNN
 F 3 "" H 9050 2000 47  0001 C CNN
 	1    9050 2000
@@
 F 0 "K504" H 10000 1600 47  0000 C CNN
 F 1 "EC2-12NU-L" H 9800 1700 47  0000 C CNN
-F 2 "" H 10000 2000 47  0001 C CNN
+F 2 "frontend_additional-footprints:Kemet_EC2-12NU-L" H 10000 2000 47  0001 C CNN
 F 3 "" H 10000 2000 47  0001 C CNN
 	1    10000 2000
@@
 F 0 "K501" H 7900 1200 47  0000 C CNN
 F 1 "HE3600" H 7950 1100 47  0000 C CNN
-F 2 "" H 7950 1050 47  0001 C CNN
+F 2 "frontend_additional-footprints:HE3600" H 7950 1050 47  0001 C CNN
 F 3 "" H 7950 1050 47  0001 C CNN
 	1    7950 1050
@@
 F 0 "K502" H 7900 1650 47  0000 C CNN
 F 1 "HE3600" H 7950 1550 47  0000 C CNN
-F 2 "" H 7950 1500 47  0001 C CNN
+F 2 "frontend_additional-footprints:HE3600" H 7950 1500 47  0001 C CNN
 F 3 "" H 7950 1500 47  0001 C CNN
 	1    7950 1500
@@
 F 0 "K503" H 7900 2100 47  0000 C CNN
 F 1 "HE3600" H 7950 2000 47  0000 C CNN
-F 2 "" H 7950 1950 47  0001 C CNN
+F 2 "frontend_additional-footprints:HE3600" H 7950 1950 47  0001 C CNN
 F 3 "" H 7950 1950 47  0001 C CNN
 	1    7950 1950
@@
 L3
 $Comp
-L frontend_additional_components:TPS73001 U504
-U 1 1 5B501BC3
-P 2650 6750
-F 0 "U504" H 2800 6250 47  0000 C CNN
-F 1 "TSP73001" H 2650 6900 47  0000 C CNN
-F 2 "Package_TO_SOT_SMD:SOT-23-6" H 2650 6750 47  0001 C CNN
-F 3 "" H 2650 6750 47  0001 C CNN
-	1    2650 6750
-	1    0    0    -1
-$EndComp
-$Comp
 L Device:C_Small C506
 U 1 1 5B505719
@@
 Connection ~ 6250 1000
 Wire Wire Line
-	1000 7100 1000 7350
-Wire Wire Line
-	1000 6750 1000 6850
-Wire Wire Line
-	750  6750 750  6850
-Wire Wire Line
-	750  6850 1000 6850
-Connection ~ 1000 6850
+	5300 3600 5300 3850
+Wire Wire Line
+	5550 3250 5550 3350
+Wire Wire Line
+	5550 3350 5300 3350
+Connection ~ 5300 3350
 Wire Wire Line
 	9550 1450 9550 1600
@@
 	3650 6900 3850 6900
 Connection ~ 3850 6900
-Wire Wire Line
-	2650 7350 2650 7450
 Wire Wire Line
 	3250 7450 3250 7300
@@
 F 0 "K505" H 8650 5050 47  0000 C CNN
 F 1 "EC2-12NU-L" H 8450 5150 47  0000 C CNN
-F 2 "" H 8650 5450 47  0001 C CNN
+F 2 "frontend_additional-footprints:Kemet_EC2-12NU-L" H 8650 5450 47  0001 C CNN
 F 3 "" H 8650 5450 47  0001 C CNN
 	1    8650 5450
@@
 	6250 1000 6250 1300
 Wire Wire Line
-	1000 6850 1000 6900
+	5300 3350 5300 3400
 Wire Wire Line
 	10750 2350 10750 2550
@@
 Wire Wire Line
 	10450 4650 10450 4750
+Text HLabel 10200 2600 0    50   Input ~ 0
+v_ext
+Wire Wire Line
+	10350 2750 10350 2600
+Wire Wire Line
+	10350 2600 10200 2600
+Connection ~ 10350 2750
+Text HLabel 9950 5500 0    50   Input ~ 0
+i_range
+Wire Wire Line
+	9950 5500 10050 5500
+Connection ~ 10050 5500
+$Comp
+L frontend_additional_components:TPS73001 U504
+U 1 1 5B501BC3
+P 2650 6750
+F 0 "U504" H 2800 6250 47  0000 C CNN
+F 1 "TSP73001" H 2650 6900 47  0000 C CNN
+F 2 "Package_TO_SOT_SMD:SOT-23-6" H 2650 6750 47  0001 C CNN
+F 3 "" H 2650 6750 47  0001 C CNN
+	1    2650 6750
+	1    0    0    -1
+$EndComp
+Wire Wire Line
+	2650 7350 2650 7450
+Wire Wire Line
+	4100 2900 4100 3050
+Wire Wire Line
+	5300 2900 4100 2900
+Wire Wire Line
+	5300 2900 5300 3350
+$Comp
+L power:GND #PWR0143
+U 1 1 5B6D5860
+P 4100 4500
+F 0 "#PWR0143" H 4100 4250 50  0001 C CNN
+F 1 "GND" H 4105 4327 50  0000 C CNN
+F 2 "" H 4100 4500 50  0001 C CNN
+F 3 "" H 4100 4500 50  0001 C CNN
+	1    4100 4500
+	1    0    0    -1
+$EndComp
+Wire Wire Line
+	4100 4500 4100 4350
 $EndSCHEMATC

Commit message: Added switchable Gain for ADC Input Drivers
Parts:
- added U406, U407, U408, U409: SN74LVC1G373, Package_TO_SOT_SMD:SOT-363_SC-70-6, symbol frontend_additional_components:SN74LVC1G373
- added U410: 74HC595, Package_SO:TSSOP-16_4.4x5mm_P0.65mm, symbol 74xx:74HC595
Connections:
- net labels added: B10, B11, B12, B13, B14, B15, B7, B8, B9
- wire segments 329 -> 410
- no-connect marks 12 -> 11
