File: components_predev/frontend/hardware/vi_filter.sch (KiCad schematic (older format))
At the start: 84 parts, among them K501 HE3600, K502 HE3600, K503 HE3600, K504 EC2-12NU-L, K505 EC2-12NU-L, Q501 SSM3K329R,LF, Q502 SSM3K329R,LF, Q503 SSM3K329R,LF, Q504 SSM3K329R,LF, Q505 SSM3K329R,LF, U406 SN74LVC1G373, U407 SN74LVC1G373, U408 SN74LVC1G373, U409 SN74LVC1G373, U410 74HC595, U501 ISL2863x, U502 74HC595, U503 ISL2863x, U504 TSP73001, U505 MIC5270BM5, U506 ISL2863x, U507 ISL2863x

Commit message: Finished routing, begun component specification
Parts:
- C501, C502, C503, C504, C505, C506, C512, C513, C518, C521, C522, C523, C524: value C_Small -> 100n
Changed lines of the file:
@@
 P 5850 1150
 F 0 "C523" H 5860 1220 50  0000 L CNN
-F 1 "C_Small" H 5860 1070 50  0000 L CNN
+F 1 "100n" H 5860 1070 50  0000 L CNN
 F 2 "Capacitor_SMD:C_0603_1608Metric" H 5850 1150 50  0001 C CNN
 F 3 "" H 5850 1150 50  0000 C CNN
@@
 P 5600 1000
 F 0 "C522" H 5610 1070 50  0000 L CNN
-F 1 "C_Small" H 5610 920 50  0000 L CNN
+F 1 "100n" H 5610 920 50  0000 L CNN
 F 2 "Capacitor_SMD:C_0603_1608Metric" H 5600 1000 50  0001 C CNN
 F 3 "" H 5600 1000 50  0000 C CNN
@@
 P 6500 3350
 F 0 "C501" H 6510 3420 50  0000 L CNN
-F 1 "C_Small" H 6510 3270 50  0000 L CNN
+F 1 "100n" H 6510 3270 50  0000 L CNN
 F 2 "Capacitor_SMD:C_0603_1608Metric" H 6500 3350 50  0001 C CNN
 F 3 "" H 6500 3350 50  0000 C CNN
@@
 P 1700 1150
 F 0 "C504" H 1710 1220 50  0000 L CNN
-F 1 "C_Small" H 1710 1070 50  0000 L CNN
+F 1 "100n" H 1710 1070 50  0000 L CNN
 F 2 "Capacitor_SMD:C_0603_1608Metric" H 1700 1150 50  0001 C CNN
 F 3 "" H 1700 1150 50  0000 C CNN
@@
 P 1450 1000
 F 0 "C502" H 1460 1070 50  0000 L CNN
-F 1 "C_Small" H 1460 920 50  0000 L CNN
+F 1 "100n" H 1460 920 50  0000 L CNN
 F 2 "Capacitor_SMD:C_0603_1608Metric" H 1450 1000 50  0001 C CNN
 F 3 "" H 1450 1000 50  0000 C CNN
@@
 P 1700 4600
 F 0 "C505" H 1710 4670 50  0000 L CNN
-F 1 "C_Small" H 1710 4520 50  0000 L CNN
+F 1 "100n" H 1710 4520 50  0000 L CNN
 F 2 "Capacitor_SMD:C_0603_1608Metric" H 1700 4600 50  0001 C CNN
 F 3 "" H 1700 4600 50  0000 C CNN
@@
 P 1450 4450
 F 0 "C503" H 1460 4520 50  0000 L CNN
-F 1 "C_Small" H 1460 4370 50  0000 L CNN
+F 1 "100n" H 1460 4370 50  0000 L CNN
 F 2 "Capacitor_SMD:C_0603_1608Metric" H 1450 4450 50  0001 C CNN
 F 3 "" H 1450 4450 50  0000 C CNN
@@
 P 1800 6950
 F 0 "C506" H 1810 7020 50  0000 L CNN
-F 1 "C_Small" H 1810 6870 50  0000 L CNN
+F 1 "100n" H 1810 6870 50  0000 L CNN
 F 2 "Capacitor_SMD:C_0603_1608Metric" H 1800 6950 50  0001 C CNN
 F 3 "" H 1800 6950 50  0000 C CNN
@@
 P 3850 7200
 F 0 "C513" H 3860 7270 50  0000 L CNN
-F 1 "C_Small" H 3860 7120 50  0000 L CNN
+F 1 "100n" H 3860 7120 50  0000 L CNN
 F 2 "Capacitor_SMD:C_0603_1608Metric" H 3850 7200 50  0001 C CNN
 F 3 "" H 3850 7200 50  0000 C CNN
@@
 P 4350 6850
 F 0 "C512" V 4100 6850 50  0000 L CNN
-F 1 "C_Small" V 4200 6700 50  0000 L CNN
+F 1 "100n" V 4200 6700 50  0000 L CNN
 F 2 "Capacitor_SMD:C_0603_1608Metric" H 4350 6850 50  0001 C CNN
 F 3 "" H 4350 6850 50  0000 C CNN
@@
 P 5950 6950
 F 0 "C521" H 5960 7020 50  0000 L CNN
-F 1 "C_Small" H 5960 6870 50  0000 L CNN
+F 1 "100n" H 5960 6870 50  0000 L CNN
 F 2 "Capacitor_SMD:C_0603_1608Metric" H 5950 6950 50  0001 C CNN
 F 3 "" H 5950 6950 50  0000 C CNN
@@
 P 5850 4600
 F 0 "C524" H 5860 4670 50  0000 L CNN
-F 1 "C_Small" H 5860 4520 50  0000 L CNN
+F 1 "100n" H 5860 4520 50  0000 L CNN
 F 2 "Capacitor_SMD:C_0603_1608Metric" H 5850 4600 50  0001 C CNN
 F 3 "" H 5850 4600 50  0000 C CNN
@@
 P 5600 4450
 F 0 "C518" H 5610 4520 50  0000 L CNN
-F 1 "C_Small" H 5610 4370 50  0000 L CNN
+F 1 "100n" H 5610 4370 50  0000 L CNN
 F 2 "Capacitor_SMD:C_0603_1608Metric" H 5600 4450 50  0001 C CNN
 F 3 "" H 5600 4450 50  0000 C CNN

Commit message: More Part Specifications added
Parts:
- R511, R512, R514, R515, R516: value R_Small -> 68k
Changed lines of the file:
@@
 P 10350 3100
 F 0 "R515" H 10380 3120 50  0000 L CNN
-F 1 "R_Small" H 10380 3060 50  0000 L CNN
+F 1 "68k" H 10380 3060 50  0000 L CNN
 F 2 "Resistor_SMD:R_0603_1608Metric" H 10350 3100 50  0001 C CNN
 F 3 "" H 10350 3100 50  0000 C CNN
@@
 P 7350 3800
 F 0 "R511" H 7380 3820 50  0000 L CNN
-F 1 "R_Small" H 7380 3760 50  0000 L CNN
+F 1 "68k" H 7380 3760 50  0000 L CNN
 F 2 "Resistor_SMD:R_0603_1608Metric" H 7350 3800 50  0001 C CNN
 F 3 "" H 7350 3800 50  0000 C CNN
@@
 P 8200 3800
 F 0 "R512" H 8230 3820 50  0000 L CNN
-F 1 "R_Small" H 8230 3760 50  0000 L CNN
+F 1 "68k" H 8230 3760 50  0000 L CNN
 F 2 "Resistor_SMD:R_0603_1608Metric" H 8200 3800 50  0001 C CNN
 F 3 "" H 8200 3800 50  0000 C CNN
@@
 P 9050 3800
 F 0 "R514" H 9080 3820 50  0000 L CNN
-F 1 "R_Small" H 9080 3760 50  0000 L CNN
+F 1 "68k" H 9080 3760 50  0000 L CNN
 F 2 "Resistor_SMD:R_0603_1608Metric" H 9050 3800 50  0001 C CNN
 F 3 "" H 9050 3800 50  0000 C CNN
@@
 P 10050 5850
 F 0 "R516" H 10080 5870 50  0000 L CNN
-F 1 "R_Small" H 10080 5810 50  0000 L CNN
+F 1 "68k" H 10080 5810 50  0000 L CNN
 F 2 "Resistor_SMD:R_0603_1608Metric" H 10050 5850 50  0001 C CNN
 F 3 "" H 10050 5850 50  0000 C CNN

Commit message: Some Updates from Testing
Parts:
- C501, C502, C503, C504, C505, C506, C512, C513, C518, C521, C522, C523, C524: Digikey (none) -> 1276-1005-1-ND; Manufacturer (none) -> Samsung; Note (none) -> VH; Part Number (none) -> CL10B104K08NNNC; Voltage (none) -> 16V
- K501, K502, K503: value HE3600 -> HE3621A1200; Digikey (none) -> HE208-ND; Manufacturer (none) -> Littefluse; Part Number (none) -> HE3621A1200
- K504, K505: value EC2-12NU-L -> EC2-12NU; Digikey (none) -> 399-11029-5-ND; Manufacturer (none) -> Kemet; Part Number (none) -> EC2-12NU
- R511, R512, R514, R515, R516: Digikey (none) -> 311-68.0KHRCT-ND; Manufacturer (none) -> Yageo; Note (none) -> VH; Part Number (none) -> RC0603FR-0768KL
- R513: Digikey (none) -> 1776-C681-ND; Manufacturer (none) -> Caddock; Part Number (none) -> 1776-C681
- U406, U407, U408, U409: Digikey (none) -> 296-18775-1-ND; Manufacturer (none) -> Texas Instruments; Part Number (none) -> SN74LVC1G373DCKR
- U410, U502: Digikey (none) -> 1727-6439-ND; Manufacturer (none) -> NXP; Part Number (none) -> 74HC595PW,112
- U501, U503, U506, U507: Digikey (none) -> ISL28633FVZ-T7ACT-ND; Manufacturer (none) -> Intersil; Part Number (none) -> ISL28633FVZ-T7A
- U504: value TSP73001 -> TPS73001; Digikey (none) -> 296-27055-1-ND; Manufacturer (none) -> Texas Instruments; Part Number (none) -> TPS73001DBVR
- U505: value MIC5270BM5 -> MIC5270YM5; Digikey (none) -> 576-1295-2-ND; Manufacturer (none) -> Microchip; Part Number (none) -> MIC5270YM5-TR
