File: components_predev/frontend/hardware/frontend.sch (KiCad schematic (older format))
At the start: 10 parts, among them K101 PE014005, P101 CONN_01X32, P102 CONN_01X04, P103 CONN_01X02, P104 CONN_01X04, Q101 Q_NMOS_DGS

Commit message: Begun Range Switching Circuitry
Changed lines of the file:
@@
 F16 "ocp" O L 7000 5600 60
 F17 "i_range" I L 7000 5300 60
+F18 "v_ref_2" I L 7000 4850 61
 $EndSheet
 $Sheet
@@
 	1500 3750 1100 3750
 Wire Wire Line
-	4650 4850 5200 4850
+	4650 4850 7000 4850
 Wire Wire Line
 	5200 4850 5200 1950
@@
 Wire Wire Line
 	1100 4050 1700 4050
+Connection ~ 5200 4850
 $EndSCHEMATC

Commit message: Finished Range Switching/Filters
Parts:
- removed P101: CONN_01X32, symbol CONN_01X32
- added P?: CONN_01X40, symbol CONN_01X40
Connections:
- net labels added: RCLK, SER, SRCLK
- net labels removed: v_range
- wire segments 131 -> 136
Changed lines of the file:
@@
 F13 "i_meas-" O L 7000 3950 60
 F14 "v_ext" I L 7000 5200 60
-F15 "v_range" I L 7000 5100 60
-F16 "ocp" O L 7000 5600 60
-F17 "i_range" I L 7000 5300 60
-F18 "v_ref_2" I L 7000 4850 61
+F15 "i_range" I L 7000 5300 60
+F16 "v_ref_2" I L 7000 4850 61
+F17 "SER" I L 7000 4200 60
+F18 "SRCLK" I L 7000 4300 60
+F19 "RCLK" I L 7000 4400 60
 $EndSheet
 $Sheet
@@
 vn
 $Comp
-L PWR_FLAG #FLG012
+L PWR_FLAG #FLG010
 U 1 1 5B162008
 P 1550 5950
-F 0 "#FLG012" H 1550 6045 50  0001 C CNN
+F 0 "#FLG010" H 1550 6045 50  0001 C CNN
 F 1 "PWR_FLAG" H 1550 6130 50  0000 C CNN
 F 2 "" H 1550 5950 50  0000 C CNN
@@
 $EndComp
 $Comp
-L PWR_FLAG #FLG013
+L PWR_FLAG #FLG011
 U 1 1 5B162102
 P 1950 5950
-F 0 "#FLG013" H 1950 6045 50  0001 C CNN
+F 0 "#FLG011" H 1950 6045 50  0001 C CNN
 F 1 "PWR_FLAG" H 1950 6130 50  0000 C CNN
 F 2 "" H 1950 5950 50  0000 C CNN
@@
 $EndComp
 $Comp
-L PWR_FLAG #FLG014
+L PWR_FLAG #FLG012
 U 1 1 5B1621FC
 P 1550 6650
-F 0 "#FLG014" H 1550 6745 50  0001 C CNN
+F 0 "#FLG012" H 1550 6745 50  0001 C CNN
 F 1 "PWR_FLAG" H 1550 6830 50  0000 C CNN
 F 2 "" H 1550 6650 50  0000 C CNN
@@
 $EndComp
 $Comp
-L GND #PWR015
+L GND #PWR013
 U 1 1 5B166631
 P 10600 4450
-F 0 "#PWR015" H 10600 4200 50  0001 C CNN
+F 0 "#PWR013" H 10600 4200 50  0001 C CNN
 F 1 "GND" H 10600 4300 50  0000 C CNN
 F 2 "" H 10600 4450 50  0000 C CNN
@@
 i_range
 $Comp
-L +12V #PWR016
+L +12V #PWR014
 U 1 1 5B16BDB0
 P 3250 6750
-F 0 "#PWR016" H 3250 6600 50  0001 C CNN
+F 0 "#PWR014" H 3250 6600 50  0001 C CNN
 F 1 "+12V" H 3250 6890 50  0000 C CNN
 F 2 "" H 3250 6750 50  0000 C CNN
@@
 $EndComp
 $Comp
-L +5V #PWR017
+L +5V #PWR015
 U 1 1 5B16C00A
 P 3450 6750
-F 0 "#PWR017" H 3450 6600 50  0001 C CNN
+F 0 "#PWR015" H 3450 6600 50  0001 C CNN
 F 1 "+5V" H 3450 6890 50  0000 C CNN
 F 2 "" H 3450 6750 50  0000 C CNN
@@
 $EndComp
 $Comp
-L +3.3V #PWR018
+L +3.3V #PWR016
 U 1 1 5B16C16A
 P 3850 6750
-F 0 "#PWR018" H 3850 6600 50  0001 C CNN
+F 0 "#PWR016" H 3850 6600 50  0001 C CNN
 F 1 "+3.3V" H 3850 6890 50  0000 C CNN
 F 2 "" H 3850 6750 50  0000 C CNN
@@
 $EndComp
 $Comp
-L -5V #PWR107
+L -5V #PWR108
 U 1 1 5B16C931
 P 3650 6750
-F 0 "#PWR107" H 3650 6600 50  0001 C CNN
+F 0 "#PWR108" H 3650 6600 50  0001 C CNN
 F 1 "-5V" H 3650 6890 50  0000 C CNN
 F 2 "" H 3650 6750 50  0000 C CNN
@@
 $EndComp
 $Comp
-L +12V #PWR019
+L +12V #PWR017
 U 1 1 5B16F227
 P 9150 3300
-F 0 "#PWR019" H 9150 3150 50  0001 C CNN
+F 0 "#PWR017" H 9150 3150 50  0001 C CNN
 F 1 "+12V" H 9150 3440 50  0000 C CNN
 F 2 "" H 9150 3300 50  0000 C CNN
@@
 $EndComp
 $Comp
-L GND #PWR020
+L GND #PWR018
 U 1 1 5B170899
 P 1350 3650
-F 0 "#PWR020" H 1350 3400 50  0001 C CNN
+F 0 "#PWR018" H 1350 3400 50  0001 C CNN
 F 1 "GND" H 1350 3500 50  0000 C CNN
 F 2 "" H 1350 3650 50  0000 C CNN
@@
 	0    -1   -1   0
 $EndComp
-Text GLabel 1500 3250 2    47   Input ~ 0
-v_range
 Text GLabel 1500 3350 2    47   Input ~ 0
 i_range
 Text GLabel 1500 3450 2    47   Input ~ 0
 v_extern
-Text GLabel 6600 5100 0    47   Input ~ 0
-v_range
 Text GLabel 6600 5300 0    47   Input ~ 0
 i_range
@@
 v_extern
 $Comp
-L CONN_01X32 P101
-U 1 1 5B242762
-P 900 2700
-F 0 "P101" H 900 4350 50  0000 C CNN
-F 1 "CONN_01X32" V 1000 2700 50  0000 C CNN
-F 2 "" H 900 2700 50  0000 C CNN
-F 3 "" H 900 2700 50  0000 C CNN
-	1    900  2700
-	-1   0    0    -1
-$EndComp
-$Comp
-L GND #PWR021
+L GND #PWR019
 U 1 1 5B2A0FA9
 P 1350 2850
-F 0 "#PWR021" H 1350 2600 50  0001 C CNN
+F 0 "#PWR019" H 1350 2600 50  0001 C CNN
 F 1 "GND" H 1350 2700 50  0000 C CNN
 F 2 "" H 1350 2850 50  0000 C CNN
@@
 	1100 3550 2300 3550
 Wire Wire Line
-	1500 3250 1100 3250
-Wire Wire Line
 	1500 3350 1100 3350
 Wire Wire Line
 	1500 3450 1100 3450
-Wire Wire Line
-	6600 5100 7000 5100
 Wire Wire Line
 	6600 5200 7000 5200
@@
 	1500 4250 1100 4250
 $Comp
-L GND #PWR?
+L GND #PWR020
 U 1 1 5B39AD94
 P 1700 4050
-F 0 "#PWR?" H 1700 3800 50  0001 C CNN
+F 0 "#PWR020" H 1700 3800 50  0001 C CNN
 F 1 "GND" H 1700 3900 50  0000 C CNN
 F 2 "" H 1700 4050 50  0000 C CNN
@@
 	1100 4050 1700 4050
 Connection ~ 5200 4850
+Text GLabel 6700 4200 0    47   Input ~ 0
+SER
+Text GLabel 6700 4300 0    47   Input ~ 0
+SRCLK
+Text GLabel 6700 4400 0    47   Input ~ 0
+RCLK
+Wire Wire Line
+	6700 4200 7000 4200
+Wire Wire Line
+	6700 4300 7000 4300
+Wire Wire Line
+	6700 4400 7000 4400
+$Comp
+L CONN_01X40 P?
+U 1 1 5B4F53AA
+P 900 3100
+F 0 "P?" H 900 5150 50  0000 C CNN
+F 1 "CONN_01X40" V 1000 3100 50  0000 C CNN
+F 2 "" H 900 3100 50  0000 C CNN
+F 3 "" H 900 3100 50  0000 C CNN
+	1    900  3100
+	-1   0    0    -1
+$EndComp
+Text GLabel 1400 4750 2    47   Output ~ 0
+SER
+Text GLabel 1400 4850 2    47   Output ~ 0
+SRCLK
+Text GLabel 1400 4950 2    47   Output ~ 0
+RCLK
+Wire Wire Line
+	1400 4750 1100 4750
+Wire Wire Line
+	1400 4850 1100 4850
+Wire Wire Line
+	1400 4950 1100 4950
+$Comp
+L GND #PWR?
+U 1 1 5B4FD249
+P 1750 5050
+F 0 "#PWR?" H 1750 4800 50  0001 C CNN
+F 1 "GND" H 1750 4900 50  0000 C CNN
+F 2 "" H 1750 5050 50  0000 C CNN
+F 3 "" H 1750 5050 50  0000 C CNN
+	1    1750 5050
+	0    -1   -1   0
+$EndComp
+Wire Wire Line
+	1750 5050 1100 5050
 $EndSCHEMATC

Commit message: Changed to KiCAD 5
Parts:
- D101: symbol D -> Device:D
- K101: symbol PE014005 -> frontend_additional_components:PE014005
- P101: renamed from P?; symbol CONN_01X40 -> Connector_Generic:Conn_01x40
- P102, P104: symbol CONN_01X04 -> Connector_Generic:Conn_01x04
- P103: symbol CONN_01X02 -> Connector_Generic:Conn_01x02
- Q101: symbol Q_NMOS_DGS -> Device:Q_NMOS_DGS
- R101, R102, R103: footprint (none) -> Resistors_SMD:R_0603; symbol R -> Device:R
Connections:
- wire segments 136 -> 150

Commit message: Footrpints and Parts Specification
Parts:
- D101: value D -> FDLL4148; footprint (none) -> Diode_SMD:D_MiniMELF; Digikey (none) -> FDLL4148CT-ND; Manufacturer (none) -> OnSemi; Mouser (none) -> 512-FDLL4148; Part Number (none) -> FDLL4148
- P101: footprint (none) -> Connector_JST:JST_PUD_S40B-PUDSS-1_2x20_P2.00mm_Horizontal; Digikey (none) -> 455-2498-ND; Manufacturer (none) -> JST; Part Number (none) -> S40B-PUDSS-1(LF)(SN)
- P102, P104: footprint (none) -> Connector_Phoenix_MSTB:PhoenixContact_MSTBA_2,5_4-G-5,08_1x04_P5.08mm_Horizontal
- P103: footprint (none) -> Connector_Phoenix_MSTB:PhoenixContact_MSTBA_2,5_2-G-5,08_1x02_P5.08mm_Horizontal
- Q101: value Q_NMOS_DGS -> SSM3K329R,LF; footprint (none) -> Package_TO_SOT_SMD:SOT-23; Digikey (none) -> SSM3K329RLFCT-ND; Manufacturer (none) -> Toshiba; Mouser (none) -> 757-SSM3K329RLF; Part Number (none) -> SSM3K329R,LF
- R101, R102, R103: footprint Resistors_SMD:R_0603 -> Resistor_SMD:R_0603_1608Metric
Changed lines of the file:
@@
 F 0 "P104" H 10350 2050 50  0000 C CNN
 F 1 "CONN_01X04" V 10450 1800 50  0000 C CNN
-F 2 "" H 10350 1800 50  0001 C CNN
+F 2 "Connector_Phoenix_MSTB:PhoenixContact_MSTBA_2,5_4-G-5,08_1x04_P5.08mm_Horizontal" H 10350 1800 50  0001 C CNN
 F 3 "" H 10350 1800 50  0000 C CNN
 	1    10350 1800
@@
 F 0 "R101" V 9480 5300 50  0000 C CNN
 F 1 "R" V 9400 5300 50  0000 C CNN
-F 2 "Resistors_SMD:R_0603" V 9330 5300 50  0001 C CNN
+F 2 "Resistor_SMD:R_0603_1608Metric" V 9330 5300 50  0001 C CNN
 F 3 "" H 9400 5300 50  0000 C CNN
 	1    9400 5300
@@
 F 0 "P102" H 900 6450 50  0000 C CNN
 F 1 "CONN_01X04" V 1000 6200 50  0000 C CNN
-F 2 "" H 900 6200 50  0001 C CNN
+F 2 "Connector_Phoenix_MSTB:PhoenixContact_MSTBA_2,5_4-G-5,08_1x04_P5.08mm_Horizontal" H 900 6200 50  0001 C CNN
 F 3 "" H 900 6200 50  0000 C CNN
 	1    900  6200
@@
 F 0 "R102" V 10580 5300 50  0000 C CNN
 F 1 "R" V 10500 5300 50  0000 C CNN
-F 2 "Resistors_SMD:R_0603" V 10430 5300 50  0001 C CNN
+F 2 "Resistor_SMD:R_0603_1608Metric" V 10430 5300 50  0001 C CNN
 F 3 "" H 10500 5300 50  0000 C CNN
 	1    10500 5300
@@
 F 0 "P103" H 900 6950 50  0000 C CNN
 F 1 "CONN_01X02" V 1000 6800 50  0000 C CNN
-F 2 "" H 900 6800 50  0001 C CNN
+F 2 "Connector_Phoenix_MSTB:PhoenixContact_MSTBA_2,5_2-G-5,08_1x02_P5.08mm_Horizontal" H 900 6800 50  0001 C CNN
 F 3 "" H 900 6800 50  0000 C CNN
 	1    900  6800
@@
 P 10300 4050
 F 0 "Q101" H 10500 4100 50  0000 L CNN
-F 1 "Q_NMOS_DGS" H 9750 4250 50  0000 L CNN
-F 2 "" H 10500 4150 50  0001 C CNN
+F 1 "SSM3K329R,LF" H 9750 4250 50  0000 L CNN
+F 2 "Package_TO_SOT_SMD:SOT-23" H 10500 4150 50  0001 C CNN
 F 3 "" H 10300 4050 50  0000 C CNN
+F 4 "SSM3K329R,LF" H 0   0   50  0001 C CNN "Part Number"
+F 5 "SSM3K329RLFCT-ND" H 0   0   50  0001 C CNN "Digikey"
+F 6 "Toshiba" H 0   0   50  0001 C CNN "Manufacturer"
+F 7 "757-SSM3K329RLF" H 0   0   50  0001 C CNN "Mouser"
 	1    10300 4050
 	-1   0    0    -1
@@
 F 0 "R103" V 10680 4250 50  0000 C CNN
 F 1 "R" V 10600 4250 50  0000 C CNN
-F 2 "Resistors_SMD:R_0603" V 10530 4250 50  0001 C CNN
+F 2 "Resistor_SMD:R_0603_1608Metric" V 10530 4250 50  0001 C CNN
 F 3 "" H 10600 4250 50  0000 C CNN
 	1    10600 4250
@@
 P 9550 3350
 F 0 "D101" H 9550 3450 50  0000 C CNN
-F 1 "D" H 9550 3250 50  0000 C CNN
-F 2 "" H 9550 3350 50  0001 C CNN
+F 1 "FDLL4148" H 9550 3250 50  0000 C CNN
+F 2 "Diode_SMD:D_MiniMELF" H 9550 3350 50  0001 C CNN
 F 3 "" H 9550 3350 50  0000 C CNN
+F 4 "FDLL4148" H 0   0   50  0001 C CNN "Part Number"
+F 5 "FDLL4148CT-ND" H 0   0   50  0001 C CNN "Digikey"
+F 6 "512-FDLL4148" H 0   0   50  0001 C CNN "Mouser"
+F 7 "OnSemi" H 0   0   50  0001 C CNN "Manufacturer"
 	1    9550 3350
 	1    0    0    -1
@@
 F 0 "P101" H 900 5100 50  0000 C CNN
 F 1 "CONN_01X40" V 1000 3050 50  0000 C CNN
-F 2 "" H 900 3050 50  0001 C CNN
+F 2 "Connector_JST:JST_PUD_S40B-PUDSS-1_2x20_P2.00mm_Horizontal" H 900 3050 50  0001 C CNN
 F 3 "" H 900 3050 50  0000 C CNN
+F 4 "455-2498-ND" H 0   0   50  0001 C CNN "Digikey"
+F 5 "JST" H 0   0   50  0001 C CNN "Manufacturer"
+F 6 "S40B-PUDSS-1(LF)(SN)" H 0   0   50  0001 C CNN "Part Number"
 	1    900  3050
 	-1   0    0    -1
@@
 	5200 4850 7000 4850
 $Comp
-L Graphic:Logo_Open_Hardware_Small #LOGO?
+L Graphic:Logo_Open_Hardware_Small #LOGO1
 U 1 1 5B56EA44
 P 7300 6850
-F 0 "#LOGO?" H 7300 7125 50  0001 C CNN
+F 0 "#LOGO1" H 7300 7125 50  0001 C CNN
 F 1 "Logo_Open_Hardware_Small" H 7300 6625 50  0001 C CNN
 F 2 "" H 7300 6850 50  0001 C CNN

Commit message: Finished Footprints, ERC
Parts:
- K101: footprint (none) -> frontend_additional-footprints:PE014005
Connections:
- net labels removed: in, ip
- wire segments 150 -> 147
- no-connect marks 0 -> 10
Changed lines of the file:
@@
 F 0 "K101" H 9300 4375 60  0000 C CNN
 F 1 "PE014005" H 9475 3825 60  0000 C CNN
-F 2 "" H 13350 5700 60  0001 C CNN
+F 2 "frontend_additional-footprints:PE014005" H 13350 5700 60  0001 C CNN
 F 3 "" H 13350 5700 60  0001 C CNN
 	1    9550 4100
@@
 	1    0    0    -1
 $EndComp
-$Sheet
-S 5200 5900 1100 1600
-U 5B0C28A9
-F0 "Inrush Current Limiter" 60
-F1 "inrush_limiter.sch" 60
-F2 "VIn+" I L 5200 6100 60
-F3 "VIn-" I L 5200 6200 60
-F4 "VDD" O R 6300 6100 60
-F5 "VSS" O R 6300 6450 60
-F6 "pwr_enable" I L 5200 7250 60
-F7 "ip" O R 6300 6850 60
-F8 "in" O R 6300 6950 60
-F9 "vp" O R 6300 7150 60
-F10 "vn" O R 6300 7250 60
-$EndSheet
 $Sheet
 S 7000 1000 1100 1650
@@
 Text GLabel 8300 4600 2    47   Input ~ 0
 v_sense+
-Text GLabel 6450 6850 2    47   Output ~ 0
-ip
-Text GLabel 6450 6950 2    47   Output ~ 0
-in
-Text GLabel 6450 7150 2    47   Output ~ 0
-vp
-Text GLabel 6450 7250 2    47   Output ~ 0
-vn
 $Comp
 L power:PWR_FLAG #FLG010
@@
 Wire Wire Line
 	10500 5450 10500 5600
-Connection ~ 10500 5600
 Connection ~ 10500 5000
 Wire Wire Line
 	6300 6450 6450 6450
 Wire Wire Line
-	6300 6100 6450 6100
-Wire Wire Line
 	8100 1800 9700 1800
 Wire Wire Line
@@
 Wire Wire Line
 	8300 4950 8100 4950
-Wire Wire Line
-	6450 6850 6300 6850
-Wire Wire Line
-	6450 7250 6300 7250
-Wire Wire Line
-	6450 7150 6300 7150
-Wire Wire Line
-	6300 6950 6450 6950
 Wire Wire Line
 	4650 3600 7000 3600
@@
 Connection ~ 1550 6100
 Wire Wire Line
-	3250 6750 3250 6800
-Wire Wire Line
-	3250 6800 2900 6800
-Wire Wire Line
 	3850 6750 3850 7250
 Wire Wire Line
@@
 Wire Wire Line
 	3450 6950 3450 6750
-Wire Wire Line
-	3650 6750 3650 7100
 Wire Wire Line
 	3650 7100 2900 7100
@@
 	1500 3450 1100 3450
 Wire Wire Line
-	6600 5200 7000 5200
-Wire Wire Line
-	7000 5300 6600 5300
-Wire Wire Line
 	3550 4300 2100 4300
 Wire Wire Line
@@
 Wire Wire Line
 	2900 2150 1100 2150
-Text GLabel 1500 3850 2    47   Input ~ 0
-ip
-Text GLabel 1500 3950 2    47   Input ~ 0
-in
 Text GLabel 1500 4150 2    47   Input ~ 0
 vp
 Text GLabel 1500 4250 2    47   Input ~ 0
 vn
-Wire Wire Line
-	1500 3850 1100 3850
-Wire Wire Line
-	1500 3950 1100 3950
-Wire Wire Line
-	1500 4150 1100 4150
-Wire Wire Line
-	1500 4250 1100 4250
 $Comp
 L power:GND #PWR020
@@
 	9400 5600 9400 5750
 Wire Wire Line
-	10500 5600 10500 5750
-Wire Wire Line
 	10500 5000 10500 5150
 Wire Wire Line
@@
 	1    0    0    -1
 $EndComp
+Wire Wire Line
+	6600 5200 7000 5200
+Wire Wire Line
+	7000 5300 6600 5300
+NoConn ~ 1100 4650
+NoConn ~ 1100 4550
+NoConn ~ 1100 4450
+NoConn ~ 1100 4350
+NoConn ~ 1100 3250
+NoConn ~ 1100 3150
+NoConn ~ 1100 2250
+NoConn ~ 1100 2050
+Wire Wire Line
+	1100 4150 1500 4150
+Wire Wire Line
+	1500 4250 1100 4250
+Wire Wire Line
+	6450 7150 6300 7150
+Wire Wire Line
+	6450 7250 6300 7250
+Text GLabel 6450 7250 2    47   Output ~ 0
+vn
+Text GLabel 6450 7150 2    47   Output ~ 0
+vp
+Wire Wire Line
+	6450 6100 6300 6100
+Wire Wire Line
+	10500 5600 10500 5750
+Connection ~ 10500 5600
+Wire Wire Line
+	3650 7100 3650 6750
+Wire Wire Line
+	2900 6800 3250 6800
+Wire Wire Line
+	3250 6750 3250 6800
+$Sheet
+S 5200 5900 1100 1600
+U 5B0C28A9
+F0 "Inrush Current Limiter" 60
+F1 "inrush_limiter.sch" 60
+F2 "VIn+" I L 5200 6100 60
+F3 "VIn-" I L 5200 6200 60
+F4 "VDD" O R 6300 6100 60
+F5 "VSS" O R 6300 6450 60
+F6 "pwr_enable" I L 5200 7250 60
+F7 "vp" O R 6300 7150 60
+F8 "vn" O R 6300 7250 60
+$EndSheet
+NoConn ~ 1100 3850
+NoConn ~ 1100 3950
+$Comp
+L power:PWR_FLAG #FLG0104
+U 1 1 5B7CB3A8
+P 9150 3600
+F 0 "#FLG0104" H 9150 3675 50  0001 C CNN
+F 1 "PWR_FLAG" H 9150 3773 50  0000 C CNN
+F 2 "" H 9150 3600 50  0001 C CNN
+F 3 "~" H 9150 3600 50  0001 C CNN
+	1    9150 3600
+	-1   0    0    1
+$EndComp
+Wire Wire Line
+	9150 3600 9150 3450
+Connection ~ 9150 3450
 $EndSCHEMATC

Commit message: Fixed minor net issues, begun routing
Changed lines of the file:
@@
 L Connector_Generic:Conn_01x04 P104
 U 1 1 5B065E90
-P 10350 1800
-F 0 "P104" H 10350 2050 50  0000 C CNN
-F 1 "CONN_01X04" V 10450 1800 50  0000 C CNN
-F 2 "Connector_Phoenix_MSTB:PhoenixContact_MSTBA_2,5_4-G-5,08_1x04_P5.08mm_Horizontal" H 10350 1800 50  0001 C CNN
-F 3 "" H 10350 1800 50  0000 C CNN
-	1    10350 1800
-	1    0    0    -1
+P 10350 1900
+F 0 "P104" H 10350 2150 50  0000 C CNN
+F 1 "CONN_01X04" V 10450 1900 50  0000 C CNN
+F 2 "Connector_Phoenix_MSTB:PhoenixContact_MSTBA_2,5_4-G-5,08_1x04_P5.08mm_Horizontal" H 10350 1900 50  0001 C CNN
+F 3 "" H 10350 1900 50  0000 C CNN
+	1    10350 1900
+	1    0    0    1
 $EndComp
 $Comp
@@
 F 3 "" H 6450 6100 50  0000 C CNN
 	1    6450 6100
-	0    1    1    0
-$EndComp
-$Comp
-L power:VSS #PWR03
-U 1 1 5B084BEC
-P 6450 6450
-F 0 "#PWR03" H 6450 6300 50  0001 C CNN
-F 1 "VSS" H 6450 6600 50  0000 C CNN
-F 2 "" H 6450 6450 50  0000 C CNN
-F 3 "" H 6450 6450 50  0000 C CNN
-	1    6450 6450
 	0    1    1    0
 $EndComp
@@
 Connection ~ 10500 5000
 Wire Wire Line
-	6300 6450 6450 6450
-Wire Wire Line
 	8100 1800 9700 1800
-Wire Wire Line
-	6650 1300 7000 1300
 Wire Wire Line
 	7000 1150 6650 1150
@@
 	9150 3600 9150 3450
 Connection ~ 9150 3450
+Wire Wire Line
+	7000 1300 6650 1300
+$Comp
+L power:VSS #PWR0148
+U 1 1 5B5FAF7F
+P 6450 6450
+F 0 "#PWR0148" H 6450 6300 50  0001 C CNN
+F 1 "VSS" H 6450 6600 50  0000 C CNN
+F 2 "" H 6450 6450 50  0000 C CNN
+F 3 "" H 6450 6450 50  0000 C CNN
+	1    6450 6450
+	0    1    1    0
+$EndComp
+Wire Wire Line
+	6450 6450 6300 6450
 $EndSCHEMATC

Commit message: More routing
Parts:
- R101, R102: footprint Resistor_SMD:R_0603_1608Metric -> Resistor_SMD:R_1206_3216Metric
Connections:
- wire segments 147 -> 148
Changed lines of the file:
@@
 F 0 "R101" V 9480 5300 50  0000 C CNN
 F 1 "R" V 9400 5300 50  0000 C CNN
-F 2 "Resistor_SMD:R_0603_1608Metric" V 9330 5300 50  0001 C CNN
+F 2 "Resistor_SMD:R_1206_3216Metric" V 9330 5300 50  0001 C CNN
 F 3 "" H 9400 5300 50  0000 C CNN
 	1    9400 5300
@@
 F 0 "R102" V 10580 5300 50  0000 C CNN
 F 1 "R" V 10500 5300 50  0000 C CNN
-F 2 "Resistor_SMD:R_0603_1608Metric" V 10430 5300 50  0001 C CNN
+F 2 "Resistor_SMD:R_1206_3216Metric" V 10430 5300 50  0001 C CNN
 F 3 "" H 10500 5300 50  0000 C CNN
 	1    10500 5300
@@
 	9400 5450 9400 5600
 Wire Wire Line
-	1250 6300 1250 6400
-Wire Wire Line
-	1250 6400 1100 6400
-Wire Wire Line
 	1100 6300 1250 6300
-Connection ~ 1250 6400
 Wire Wire Line
 	9700 1550 9700 1800
@@
 Wire Wire Line
 	1950 5950 1950 6200
-Connection ~ 1950 6200
 Wire Wire Line
 	1550 6650 1550 6800
@@
 Wire Wire Line
 	1750 5050 1100 5050
-Wire Wire Line
-	1100 6200 1950 6200
-Wire Wire Line
-	1250 6400 1250 6600
 Wire Wire Line
 	9700 1800 10150 1800
@@
 Wire Wire Line
 	6450 6450 6300 6450
+Wire Wire Line
+	1250 6300 1250 6600
+Wire Wire Line
+	1100 6400 1950 6400
+Wire Wire Line
+	1950 6400 1950 6200
+Connection ~ 1950 6200
+Wire Wire Line
+	1250 6300 1250 6200
+Wire Wire Line
+	1250 6200 1100 6200
+Connection ~ 1250 6300
 $EndSCHEMATC
