File: components_predev/frontend/hardware/frontend.sch (KiCad schematic (older format))
At the start: 10 parts, among them K101 PE014005, P101 CONN_01X40, P102 CONN_01X04, P103 CONN_01X02, P104 CONN_01X04, Q101 SSM3K329R,LF

Commit message: More routing, fixed error in lockstep operation of current range switching relais
Connections:
- net labels added: il_sense+, il_sense-
- net labels removed: ih_sense+, ih_sense-
- wire segments 148 -> 150
Changed lines of the file:
@@
 $EndComp
 Text GLabel 10350 5000 0    47   Output ~ 0
-ih_sense+
+il_sense+
 Text GLabel 10350 5600 0    47   Output ~ 0
-ih_sense-
+il_sense-
 $Comp
 L power:GNDPWR #PWR05
@@
 F14 "v_ref_2" O R 4650 4850 60
 $EndSheet
-Text GLabel 8300 5350 2    47   Input ~ 0
-ih_sense-
-Text GLabel 8300 5250 2    47   Input ~ 0
-ih_sense+
+Text GLabel 8300 5600 2    47   Input ~ 0
+il_sense-
+Text GLabel 8300 5500 2    47   Input ~ 0
+il_sense+
 Text GLabel 8300 4950 2    47   Input ~ 0
 v_sense_ext-
@@
 $EndComp
 Wire Wire Line
-	9400 5450 9400 5600
-Wire Wire Line
 	1100 6300 1250 6300
 Wire Wire Line
@@
 Connection ~ 9700 1900
 Connection ~ 9400 5000
-Connection ~ 9400 5600
 Wire Wire Line
 	9150 5000 9400 5000
-Wire Wire Line
-	8100 5600 9400 5600
 Wire Wire Line
 	10500 5600 10350 5600
@@
 Wire Wire Line
 	1250 6900 1250 7200
-Wire Wire Line
-	9150 5000 9150 5500
-Wire Wire Line
-	9150 5500 8100 5500
-Wire Wire Line
-	8300 5350 8100 5350
-Wire Wire Line
-	8300 5250 8100 5250
 Wire Wire Line
 	8300 4600 8100 4600
@@
 Wire Wire Line
 	9400 5000 9400 5150
-Wire Wire Line
-	9400 5600 9400 5750
 Wire Wire Line
 	10500 5000 10500 5150
@@
 	1250 6200 1100 6200
 Connection ~ 1250 6300
+Wire Wire Line
+	9400 5450 9400 5650
+Wire Wire Line
+	8100 5500 8300 5500
+Wire Wire Line
+	8300 5600 8100 5600
+Wire Wire Line
+	8100 5250 9150 5250
+Wire Wire Line
+	9150 5250 9150 5000
+Wire Wire Line
+	8100 5350 9150 5350
+Wire Wire Line
+	9150 5350 9150 5650
+Wire Wire Line
+	9150 5650 9400 5650
+Connection ~ 9400 5650
+Wire Wire Line
+	9400 5650 9400 5750
 $EndSCHEMATC

Commit message: More Part Specifications added
Parts:
- R103: value R -> 68k
Changed lines of the file:
@@
 P 10600 4250
 F 0 "R103" V 10680 4250 50  0000 C CNN
-F 1 "R" V 10600 4250 50  0000 C CNN
+F 1 "68k" V 10600 4250 50  0000 C CNN
 F 2 "Resistor_SMD:R_0603_1608Metric" V 10530 4250 50  0001 C CNN
 F 3 "" H 10600 4250 50  0000 C CNN

Commit message: Some Updates from Testing
Parts:
- K101: Digikey (none) -> PB353-ND; Manufacturer (none) -> TE Connectivity; Part Number (none) -> PE014005
- P102, P104: value CONN_01X04 -> 1757268; Digikey (none) -> 277-1108-ND; Manufacturer (none) -> Phoenix; Part Number (none) -> 1757268
- P103: value CONN_01X02 -> 1757242; Digikey (none) -> 277-1106-ND; Manufacturer (none) -> Phoenix; Note (none) -> ?; Part Number (none) -> 1757242
- R101: value R -> 200m; Digikey (none) -> WSLC-.20CT-ND; Manufacturer (none) -> Vishay; Part Number (none) -> WSL1206R2000FEA
- R102: value R -> ~
- R103: Digikey (none) -> 311-68.0KHRCT-ND; Manufacturer (none) -> Yageo; Note (none) -> VH; Part Number (none) -> RC0603FR-0768KL
Changed lines of the file:
@@
 P 10350 1900
 F 0 "P104" H 10350 2150 50  0000 C CNN
-F 1 "CONN_01X04" V 10450 1900 50  0000 C CNN
+F 1 "1757268" V 10450 1900 50  0000 C CNN
 F 2 "Connector_Phoenix_MSTB:PhoenixContact_MSTBA_2,5_4-G-5,08_1x04_P5.08mm_Horizontal" H 10350 1900 50  0001 C CNN
 F 3 "" H 10350 1900 50  0000 C CNN
+F 4 "277-1108-ND" H 0   0   50  0001 C CNN "Digikey"
+F 5 "Phoenix" H 0   0   50  0001 C CNN "Manufacturer"
+F 6 "1757268" H 0   0   50  0001 C CNN "Part Number"
 	1    10350 1900
 	1    0    0    1
@@
 P 9400 5300
 F 0 "R101" V 9480 5300 50  0000 C CNN
-F 1 "R" V 9400 5300 50  0000 C CNN
+F 1 "200m" V 9400 5300 50  0000 C CNN
 F 2 "Resistor_SMD:R_1206_3216Metric" V 9330 5300 50  0001 C CNN
 F 3 "" H 9400 5300 50  0000 C CNN
+F 4 "WSLC-.20CT-ND" H 0   0   50  0001 C CNN "Digikey"
+F 5 "Vishay" H 0   0   50  0001 C CNN "Manufacturer"
+F 6 "WSL1206R2000FEA" H 0   0   50  0001 C CNN "Part Number"
 	1    9400 5300
 	-1   0    0    -1
@@
 P 900 6200
 F 0 "P102" H 900 6450 50  0000 C CNN
-F 1 "CONN_01X04" V 1000 6200 50  0000 C CNN
+F 1 "1757268" V 1000 6200 50  0000 C CNN
 F 2 "Connector_Phoenix_MSTB:PhoenixContact_MSTBA_2,5_4-G-5,08_1x04_P5.08mm_Horizontal" H 900 6200 50  0001 C CNN
 F 3 "" H 900 6200 50  0000 C CNN
+F 4 "277-1108-ND" H 0   0   50  0001 C CNN "Digikey"
+F 5 "Phoenix" H 0   0   50  0001 C CNN "Manufacturer"
+F 6 "1757268" H 0   0   50  0001 C CNN "Part Number"
 	1    900  6200
 	-1   0    0    -1
@@
 P 10500 5300
 F 0 "R102" V 10580 5300 50  0000 C CNN
-F 1 "R" V 10500 5300 50  0000 C CNN
+F 1 "~" V 10500 5300 50  0000 C CNN
 F 2 "Resistor_SMD:R_1206_3216Metric" V 10430 5300 50  0001 C CNN
 F 3 "" H 10500 5300 50  0000 C CNN
+F 4 "" H 0   0   50  0001 C CNN "Digikey"
+F 5 "" H 0   0   50  0001 C CNN "Manufacturer"
+F 6 "" H 0   0   50  0001 C CNN "Part Number"
 	1    10500 5300
 	-1   0    0    -1
@@
 F 2 "frontend_additional-footprints:PE014005" H 13350 5700 60  0001 C CNN
 F 3 "" H 13350 5700 60  0001 C CNN
+F 4 "PB353-ND" H 0   0   50  0001 C CNN "Digikey"
+F 5 "TE Connectivity" H 0   0   50  0001 C CNN "Manufacturer"
+F 6 "PE014005" H 0   0   50  0001 C CNN "Part Number"
 	1    9550 4100
 	0    -1   1    0
@@
 P 900 6800
 F 0 "P103" H 900 6950 50  0000 C CNN
-F 1 "CONN_01X02" V 1000 6800 50  0000 C CNN
+F 1 "1757242" V 1000 6800 50  0000 C CNN
 F 2 "Connector_Phoenix_MSTB:PhoenixContact_MSTBA_2,5_2-G-5,08_1x02_P5.08mm_Horizontal" H 900 6800 50  0001 C CNN
 F 3 "" H 900 6800 50  0000 C CNN
+F 4 "?" H 900 6800 50  0001 C CNN "Note"
+F 5 "277-1106-ND" H 0   0   50  0001 C CNN "Digikey"
+F 6 "Phoenix" H 0   0   50  0001 C CNN "Manufacturer"
+F 7 "1757242" H 0   0   50  0001 C CNN "Part Number"
 	1    900  6800
 	-1   0    0    -1
@@
 F 2 "Resistor_SMD:R_0603_1608Metric" V 10530 4250 50  0001 C CNN
 F 3 "" H 10600 4250 50  0000 C CNN
+F 4 "311-68.0KHRCT-ND" H 0   0   50  0001 C CNN "Digikey"
+F 5 "Yageo" H 0   0   50  0001 C CNN "Manufacturer"
+F 6 "VH" H 0   0   50  0001 C CNN "Note"
+F 7 "RC0603FR-0768KL" H 0   0   50  0001 C CNN "Part Number"
 	1    10600 4250
 	1    0    0    -1
