File: components_predev/frontend/hardware/inrush_limiter.sch (KiCad schematic (older format))
At the start: 25 parts, among them Q201 FDMS86263P, Q202 FDMS86252, Q203 MMBT5550L, Q204 MMBT5550L

Commit message: More routing
Parts:
- removed Q201: FDMS86263P, Package_TO_SOT_SMD:TO-252-2, symbol Device:Q_PMOS_DGS
- removed Q202: FDMS86252, Package_TO_SOT_SMD:TO-252-2, symbol Device:Q_NMOS_DGS
- removed R209, R210: 10m, Resistor_SMD:R_0603_1608Metric, symbol Device:R
- added Q702: FDMS86255, Package_TO_SOT_SMD:TDSON-8-1, symbol Transistor_FET:FDMS86255
- added Q703: FQB12P20, Package_TO_SOT_SMD:TO-252-2, symbol Device:Q_PMOS_GDS
- C201, C202: footprint Capacitor_THT:CP_Radial_D8.0mm_P5.00mm -> Capacitor_THT:CP_Radial_D10.0mm_P5.00mm
Connections:
- wire segments 78 -> 76
Changed lines of the file:
@@
 F 0 "C201" H 5475 2450 50  0000 L CNN
 F 1 "100u" H 5475 2250 50  0000 L CNN
-F 2 "Capacitor_THT:CP_Radial_D8.0mm_P5.00mm" H 5450 2350 50  0001 C CNN
+F 2 "Capacitor_THT:CP_Radial_D10.0mm_P5.00mm" H 5450 2350 50  0001 C CNN
 F 3 "" H 5450 2350 50  0000 C CNN
 F 4 "Nichicon" H 5450 2350 60  0001 C CNN "Manufacturer"
@@
 F 0 "C202" H 5475 4500 50  0000 L CNN
 F 1 "100u" H 5475 4300 50  0000 L CNN
-F 2 "Capacitor_THT:CP_Radial_D8.0mm_P5.00mm" H 5450 4400 50  0001 C CNN
+F 2 "Capacitor_THT:CP_Radial_D10.0mm_P5.00mm" H 5450 4400 50  0001 C CNN
 F 3 "" H 5450 4400 50  0000 C CNN
 F 4 "Nichicon" H 5450 4400 60  0001 C CNN "Manufacturer"
@@
 	1    5450 4400
 	-1   0    0    1
-$EndComp
-$Comp
-L Device:Q_PMOS_DGS Q201
-U 1 1 5B0C3B78
-P 4100 2200
-F 0 "Q201" V 4100 2400 50  0000 L CNN
-F 1 "FDMS86263P" V 4000 2400 50  0000 L CNN
-F 2 "Package_TO_SOT_SMD:TO-252-2" H 4300 2300 50  0001 C CNN
-F 3 "" H 4100 2200 50  0000 C CNN
-F 4 "Fairchild" H 4100 2200 60  0001 C CNN "Manufacturer"
-F 5 "FDMS86263PCT-ND" H 4100 2200 60  0001 C CNN "Digikey"
-F 6 "FDMS86263P" H 4100 2200 60  0001 C CNN "Part Number"
-F 7 "512-FDMS86263P" H 4100 2200 60  0001 C CNN "Mouser"
-	1    4100 2200
-	0    1    -1   0
 $EndComp
 $Comp
@@
 	1    5450 2850
 	1    0    0    -1
-$EndComp
-$Comp
-L Device:Q_NMOS_DGS Q202
-U 1 1 5B0C3BC2
-P 4100 4250
-F 0 "Q202" H 4300 4300 50  0000 L CNN
-F 1 "FDMS86252" V 4050 4400 50  0000 L CNN
-F 2 "Package_TO_SOT_SMD:TO-252-2" H 4300 4350 50  0001 C CNN
-F 3 "" H 4100 4250 50  0000 C CNN
-F 4 "Fairchild" H 4100 4250 60  0001 C CNN "Manufacturer"
-F 5 "FDMS86252CT-ND" H 4100 4250 60  0001 C CNN "Digikey"
-F 6 "FDMS86252" H 4100 4250 60  0001 C CNN "Part Number"
-	1    4100 4250
-	0    1    -1   0
 $EndComp
 $Comp
@@
 	5450 4250 5450 4150
 Connection ~ 5450 4150
-$Comp
-L Device:R R209
-U 1 1 5B0C3C5E
-P 6800 2100
-F 0 "R209" V 6880 2100 50  0000 C CNN
-F 1 "10m" V 6800 2100 50  0000 C CNN
-F 2 "Resistor_SMD:R_0603_1608Metric" V 6730 2100 50  0001 C CNN
-F 3 "" H 6800 2100 50  0000 C CNN
-F 4 "Susumu" H 6800 2100 60  0001 C CNN "Manufacturer"
-F 5 "408-1404-1-ND" H 6800 2100 60  0001 C CNN "Digikey"
-F 6 "RL0816T-R010-F" H 6800 2100 60  0001 C CNN "Part Number"
-	1    6800 2100
-	0    1    1    0
-$EndComp
-$Comp
-L Device:R R210
-U 1 1 5B0C3C65
-P 6800 4150
-F 0 "R210" V 6880 4150 50  0000 C CNN
-F 1 "10m" V 6800 4150 50  0000 C CNN
-F 2 "Resistor_SMD:R_0603_1608Metric" V 6730 4150 50  0001 C CNN
-F 3 "" H 6800 4150 50  0000 C CNN
-F 4 "Susumu" H 6800 4150 60  0001 C CNN "Manufacturer"
-F 5 "408-1404-1-ND" H 6800 4150 60  0001 C CNN "Digikey"
-F 6 "RL0816T-R010-F" H 6800 4150 60  0001 C CNN "Part Number"
-	1    6800 4150
-	0    1    1    0
-$EndComp
-Wire Wire Line
-	6950 2100 7050 2100
 Connection ~ 7050 2100
 Text HLabel 3000 2100 0    60   Input ~ 0
@@
 Wire Wire Line
 	7050 3300 7050 3450
-Wire Wire Line
-	6950 4150 7050 4150
 $Comp
 L Device:R_Small R213
@@
 	5450 2500 5450 2850
 Wire Wire Line
-	5450 2100 6650 2100
-Wire Wire Line
 	5450 4550 5450 4900
 Wire Wire Line
-	5450 4150 6650 4150
+	5450 2100 7050 2100
+Wire Wire Line
+	5450 4150 7050 4150
+$Comp
+L Transistor_FET:FDMS86255 Q702
+U 1 1 5B975EBF
+P 4100 4250
+F 0 "Q702" V 4350 4250 50  0000 C CNN
+F 1 "FDMS86255" V 4050 4600 50  0000 C CNN
+F 2 "Package_TO_SOT_SMD:TDSON-8-1" H 4300 4175 50  0001 L CIN
+F 3 "https://www.fairchildsemi.com/datasheets/FD/FDMS86255.pdf" V 4100 4250 50  0001 L CNN
+	1    4100 4250
+	0    1    -1   0
+$EndComp
+$Comp
+L Device:Q_PMOS_GDS Q703
+U 1 1 5B9774E4
+P 4100 2200
+F 0 "Q703" V 4350 2200 50  0000 C CNN
+F 1 "FQB12P20" V 4050 2500 50  0000 C CNN
+F 2 "Package_TO_SOT_SMD:TO-252-2" H 4300 2300 50  0001 C CNN
+F 3 "~" H 4100 2200 50  0001 C CNN
+	1    4100 2200
+	0    1    -1   0
+$EndComp
 $EndSCHEMATC
