File: components_predev/frontend/hardware/inrush_limiter.sch (KiCad schematic (older format))
At the start: 23 parts, among them Q203 MMBT5550L, Q204 MMBT5550L, Q702 FDMS86255, Q703 FQB12P20

Commit message: More routing
Parts:
- added C712, C725: C_Small, Capacitor_SMD:C_0603_1608Metric, symbol Device:C_Small
Connections:
- wire segments 76 -> 86
Changed lines of the file:
@@
 $EndComp
 Wire Wire Line
-	7050 3300 7050 3450
+	7050 3300 7050 3400
 $Comp
 L Device:R_Small R213
@@
 $EndComp
 Wire Wire Line
-	7050 5350 7050 5500
+	7050 5350 7050 5450
 Wire Wire Line
 	7050 4850 7050 4150
@@
 	0    1    -1   0
 $EndComp
+$Comp
+L Device:C_Small C725
+U 1 1 5BA0DAD8
+P 6850 5250
+F 0 "C725" H 6758 5204 50  0000 R CNN
+F 1 "C_Small" H 6758 5295 50  0000 R CNN
+F 2 "Capacitor_SMD:C_0603_1608Metric" H 6850 5250 50  0001 C CNN
+F 3 "~" H 6850 5250 50  0001 C CNN
+	1    6850 5250
+	1    0    0    1
+$EndComp
+$Comp
+L Device:C_Small C712
+U 1 1 5BA0DBFF
+P 6850 3200
+F 0 "C712" H 6942 3246 50  0000 L CNN
+F 1 "C_Small" H 6942 3155 50  0000 L CNN
+F 2 "Capacitor_SMD:C_0603_1608Metric" H 6850 3200 50  0001 C CNN
+F 3 "~" H 6850 3200 50  0001 C CNN
+	1    6850 3200
+	1    0    0    -1
+$EndComp
+Wire Wire Line
+	7050 3050 6850 3050
+Wire Wire Line
+	6850 3050 6850 3100
+Wire Wire Line
+	6850 3300 6850 3400
+Wire Wire Line
+	6850 3400 7050 3400
+Connection ~ 7050 3400
+Wire Wire Line
+	7050 3400 7050 3450
+Wire Wire Line
+	7050 5100 6850 5100
+Wire Wire Line
+	6850 5100 6850 5150
+Wire Wire Line
+	6850 5350 6850 5450
+Wire Wire Line
+	6850 5450 7050 5450
+Connection ~ 7050 5450
+Wire Wire Line
+	7050 5450 7050 5500
 $EndSCHEMATC

Commit message: Some Updates from Testing
Parts:
- Q702: Digikey (none) -> FDMS86255CT-ND; Manufacturer (none) -> Fairchild; Part Number (none) -> FDMS86255
- Q703: Digikey (none) -> FQB12P20TMCT-ND; Manufacturer (none) -> OnSemi; Part Number (none) -> FQB12P20TM
- R203, R204: Digikey (none) -> 311-220HRCT-ND; Manufacturer (none) -> Yageo; Note (none) -> VH; Part Number (none) -> RC0603FR-07220RL
- R205, R206, R207, R208: Digikey (none) -> 311-68.0KHRCT-ND; Manufacturer (none) -> Yageo; Note (none) -> VH; Part Number (none) -> RC0603FR-0768KL
- W201, W202: Note (none) -> NB
Changed lines of the file:
@@
 F 2 "Resistor_SMD:R_0603_1608Metric" V 4330 2750 50  0001 C CNN
 F 3 "" H 4400 2750 50  0000 C CNN
+F 4 "311-68.0KHRCT-ND" H 0   0   50  0001 C CNN "Digikey"
+F 5 "Yageo" H 0   0   50  0001 C CNN "Manufacturer"
+F 6 "VH" H 0   0   50  0001 C CNN "Note"
+F 7 "RC0603FR-0768KL" H 0   0   50  0001 C CNN "Part Number"
 	1    4400 2750
 	0    1    1    0
@@
 F 2 "Resistor_SMD:R_0603_1608Metric" V 4330 4850 50  0001 C CNN
 F 3 "" H 4400 4850 50  0000 C CNN
+F 4 "311-68.0KHRCT-ND" H 0   0   50  0001 C CNN "Digikey"
+F 5 "Yageo" H 0   0   50  0001 C CNN "Manufacturer"
+F 6 "VH" H 0   0   50  0001 C CNN "Note"
+F 7 "RC0603FR-0768KL" H 0   0   50  0001 C CNN "Part Number"
 	1    4400 4850
 	0    1    1    0
@@
 F 2 "Resistor_SMD:R_1206_3216Metric" V 4030 1750 50  0001 C CNN
 F 3 "" H 4100 1750 50  0000 C CNN
+F 4 "311-220HRCT-ND" H 0   0   50  0001 C CNN "Digikey"
+F 5 "Yageo" H 0   0   50  0001 C CNN "Manufacturer"
+F 6 "VH" H 0   0   50  0001 C CNN "Note"
+F 7 "RC0603FR-07220RL" H 0   0   50  0001 C CNN "Part Number"
 	1    4100 1750
 	0    1    1    0
@@
 F 2 "Resistor_SMD:R_1206_3216Metric" V 4030 3800 50  0001 C CNN
 F 3 "" H 4100 3800 50  0000 C CNN
+F 4 "311-220HRCT-ND" H 0   0   50  0001 C CNN "Digikey"
+F 5 "Yageo" H 0   0   50  0001 C CNN "Manufacturer"
+F 6 "VH" H 0   0   50  0001 C CNN "Note"
+F 7 "RC0603FR-07220RL" H 0   0   50  0001 C CNN "Part Number"
 	1    4100 3800
 	0    1    1    0
@@
 F 2 "Resistor_SMD:R_0603_1608Metric" V 4230 3150 50  0001 C CNN
 F 3 "" H 4300 3150 50  0000 C CNN
+F 4 "311-68.0KHRCT-ND" H 0   0   50  0001 C CNN "Digikey"
+F 5 "Yageo" H 0   0   50  0001 C CNN "Manufacturer"
+F 6 "VH" H 0   0   50  0001 C CNN "Note"
+F 7 "RC0603FR-0768KL" H 0   0   50  0001 C CNN "Part Number"
 	1    4300 3150
 	0    1    1    0
@@
 F 2 "Resistor_SMD:R_0603_1608Metric" V 4230 5250 50  0001 C CNN
 F 3 "" H 4300 5250 50  0000 C CNN
+F 4 "311-68.0KHRCT-ND" H 0   0   50  0001 C CNN "Digikey"
+F 5 "Yageo" H 0   0   50  0001 C CNN "Manufacturer"
+F 6 "VH" H 0   0   50  0001 C CNN "Note"
+F 7 "RC0603FR-0768KL" H 0   0   50  0001 C CNN "Part Number"
 	1    4300 5250
 	0    1    1    0
@@
 F 2 "TestPoint:TestPoint_Pad_D1.0mm" H 7700 2000 50  0001 C CNN
 F 3 "" H 7700 2000 50  0000 C CNN
+F 4 "NB" H 0   0   50  0001 C CNN "Note"
 	1    7500 2000
 	1    0    0    -1
@@
 F 2 "TestPoint:TestPoint_Pad_D1.0mm" H 7700 4050 50  0001 C CNN
 F 3 "" H 7700 4050 50  0000 C CNN
+F 4 "NB" H 0   0   50  0001 C CNN "Note"
 	1    7500 4050
 	1    0    0    -1
@@
 F 2 "Package_TO_SOT_SMD:TDSON-8-1" H 4300 4175 50  0001 L CIN
 F 3 "https://www.fairchildsemi.com/datasheets/FD/FDMS86255.pdf" V 4100 4250 50  0001 L CNN
+F 4 "FDMS86255CT-ND" H 0   0   50  0001 C CNN "Digikey"
+F 5 "Fairchild" H 0   0   50  0001 C CNN "Manufacturer"
+F 6 "FDMS86255" H 0   0   50  0001 C CNN "Part Number"
 	1    4100 4250
 	0    1    -1   0
@@
 F 2 "Package_TO_SOT_SMD:TO-252-2" H 4300 2300 50  0001 C CNN
 F 3 "~" H 4100 2200 50  0001 C CNN
+F 4 "FQB12P20TMCT-ND" H 0   0   50  0001 C CNN "Digikey"
+F 5 "OnSemi" H 0   0   50  0001 C CNN "Manufacturer"
+F 6 "FQB12P20TM" H 0   0   50  0001 C CNN "Part Number"
 	1    4100 2200
 	0    1    -1   0
