File: components_predev/frontend/hardware/frontend.kicad_pcb (KiCad board)
At the start: 2 copper layers, 300 parts, among them J601 Conn_01x03, K101 PE014005, K301 PE014005, K501 HE3600, K502 HE3600, K503 HE3600, K504 EC2-12NU-L, K505 EC2-12NU-L, P101 CONN_01X40, P102 CONN_01X04, P103 CONN_01X02, P104 CONN_01X04, P401 CONN_01X02, P402 CONN_01X02, P403 CONN_01X02, P404 CONN_01X02, Q101 SSM3K329R,LF, Q201 FDMS86263P, Q202 FDMS86252, Q203 MMBT5550L, Q204 MMBT5550L, Q301 MMBT5550L, Q302 MMBT5550L, Q303 MMBT5401-7-F, Q304 MMBT5550L, Q305 MMBT5401-7-F, Q306 2SA1962OTU, Q307 2SC5242OTU, Q308 SSM3K329R,LF, Q501 SSM3K329R,LF, Q502 SSM3K329R,LF, Q503 SSM3K329R,LF, Q504 SSM3K329R,LF, Q505 SSM3K329R,LF, Q701 SSM3K329R,LF, U301 LTC6090-5, U302 LTC6090-5, U303 LTC6090-5, U401 AOZ1284, U402 LT1617, U403 AOZ1284, U404 MIC39100, U405 MC79M05, U501 ISL2863x, U502 74HC595, U503 ISL2863x, U504 TSP73001, U505 MIC5270BM5, U506 ISL2863x, U507 ISL2863x, U601 MAX5318, U701 MIC7211, U702 ADR4533, U703 LMT88, U704 NCP508, U705 NCP508, U706 MAX11960, U707 LTC2055, U708 TSP73001

Commit message: Fixed minor net issues, begun routing
Parts:
- removed C205, C206: 100u, frontend_additional-footprints:UVR2C101MHD
- removed C302: 100n, Capacitor_SMD:C_1206_3216Metric
- added C300: C_Small, Capacitor_SMD:C_1206_3216Metric, F.Cu at (495.0, 95.0)
- added REF**: MountingHole_3.2mm_M3_Pad_Via, MountingHole:MountingHole_3.2mm_M3_Pad_Via, F.Cu at (234.0, 144.0)
- added REF**: MountingHole_3.2mm_M3_Pad_Via, MountingHole:MountingHole_3.2mm_M3_Pad_Via, F.Cu at (106.0, 144.0)
- added REF**: MountingHole_3.2mm_M3_Pad_Via, MountingHole:MountingHole_3.2mm_M3_Pad_Via, F.Cu at (234.0, 56.0)
- added REF**: MountingHole_3.2mm_M3_Pad_Via, MountingHole:MountingHole_3.2mm_M3_Pad_Via, F.Cu at (106.0, 56.0)
- D101, D302, Q101, Q306, Q307, Q308, R103, R318: moved to B.Cu
- R316, R317: footprint Resistor_SMD:R_0603_1608Metric -> Resistor_SMD:R_2512_6332Metric
- R703: footprint Resistor_SMD:R_0603_1608Metric -> Resistor_SMD:R_1206_3216Metric; moved to B.Cu
- U301, U302, U303: value LTC6090-5 -> LTC6090
- moved RN701 362.0 mm to (132.5, 123.0)
- moved RN703 349.9 mm to (132.5, 126.0)
- moved R703 349.7 mm to (141.0, 110.0), turned to 90 degrees
- moved U706 349.6 mm to (143.0, 131.0), turned to 225 degrees
- moved W701 346.6 mm to (150.5, 105.5)
- moved R704 345.5 mm to (151.0, 108.0)
- moved R705 344.6 mm to (151.0, 111.0)
- moved W702 342.5 mm to (152.5, 105.5)
- moved W707 341.3 mm to (158.5, 107.0)
- moved U702 336.2 mm to (141.0, 110.0)
- moved R708 335.3 mm to (159.0, 113.0)
- moved R709 332.4 mm to (159.0, 114.5), turned to 180 degrees
- moved C714 330.5 mm to (152.0, 113.5)
- moved C713 329.2 mm to (154.0, 109.5), turned to 270 degrees
- moved U707 325.4 mm to (159.0, 110.5)
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Connections:
- P104 pad 1: v_sense_ext+ -> v_sense_ext-
- P104 pad 2: output -> v_sense-
- P104 pad 3: v_sense- -> output
- P104 pad 4: v_sense_ext- -> v_sense_ext+
- Q307 pad 3: GND -> VSS
- R210 pad 1: GND -> VSS
- R213 pad 1: GND -> VSS
- R307 pad 1: GND -> VSS
- R311 pad 2: GND -> VSS
- R315 pad 2: GND -> VSS
- U301 pad 9: GND -> Net-(U301-Pad4)
- U302 pad 4: GND -> VSS
- U302 pad 9: GND -> VSS
- W202 pad 1: GND -> VSS
Other:
- board outline added: 140 x 100 mm
- copper layers 2 -> 4

Commit message: Begun routing
Parts:
- removed C203, C204: 100u, frontend_additional-footprints:UVR2C101MHD
- removed C401, C411: CP1_Small, Capacitor_SMD:CP_Elec_4x3
- removed C712: C_Small, Capacitor_SMD:C_0603_1608Metric
- removed RN601, RN602, RN603, RN701, RN703: 22, Resistor_SMD:R_Array_Convex_4x0402
- added R517: R_Small, Resistor_SMD:R_0603_1608Metric, F.Cu at (132.0, 85.5)
- added R518: R_Small, Resistor_SMD:R_0603_1608Metric, F.Cu at (132.0, 91.5)
- added R519: R_Small, Resistor_SMD:R_0603_1608Metric, F.Cu at (132.0, 87.0)
- added R520: R_Small, Resistor_SMD:R_0603_1608Metric, F.Cu at (132.0, 90.0)
- added R521: R_Small, Resistor_SMD:R_0603_1608Metric, F.Cu at (132.0, 88.5)
- added R522: R_Small, Resistor_SMD:R_0603_1608Metric, F.Cu at (132.0, 99.0)
- added R523: R_Small, Resistor_SMD:R_0603_1608Metric, F.Cu at (132.0, 100.5)
- added R524: R_Small, Resistor_SMD:R_0603_1608Metric, F.Cu at (132.0, 97.5)
- added R525: R_Small, Resistor_SMD:R_0603_1608Metric, F.Cu at (132.0, 96.0)
- added R526: R_Small, Resistor_SMD:R_0603_1608Metric, F.Cu at (132.0, 94.5)
- added R527: R_Small, Resistor_SMD:R_0603_1608Metric, F.Cu at (132.0, 93.0)
- added R603: R_Small, Resistor_SMD:R_0603_1608Metric, F.Cu at (132.0, 120.0)
- added R604: R_Small, Resistor_SMD:R_0603_1608Metric, F.Cu at (132.0, 127.5)
- added R605: R_Small, Resistor_SMD:R_0603_1608Metric, F.Cu at (132.0, 124.5)
- added R606: R_Small, Resistor_SMD:R_0603_1608Metric, F.Cu at (132.0, 121.5)
- added R607: R_Small, Resistor_SMD:R_0603_1608Metric, F.Cu at (132.0, 118.5)
- added R608: R_Small, Resistor_SMD:R_0603_1608Metric, F.Cu at (132.0, 126.0)
- added R609: R_Small, Resistor_SMD:R_0603_1608Metric, F.Cu at (132.0, 123.0)
- added REF**: KiCAD Logo, Symbol:Symbol_KiCAD-Logo_CopperAndSilkScreenTop, F.Cu at (222.0, 143.8)
- C201, C202: footprint frontend_additional-footprints:UVR2C101MHD -> Capacitor_THT:CP_Radial_D8.0mm_P5.00mm
- C403, C409, C412, C420, C704, C706, D406, Q701, R403, R407, R412, R701, R702, U701: moved to B.Cu
- R301, R302, R304, R305, R306, R307, R308, R309, R310, R311, R312, R313, R314, R315: footprint Resistor_SMD:R_0603_1608Metric -> Resistor_SMD:R_1206_3216Metric
- moved C708 386.4 mm to (122.5, 138.5), turned to 180 degrees
- moved W704 384.1 mm to (123.5, 136.5)
- moved U705 383.6 mm to (122.5, 141.0)
- moved C702 378.1 mm to (119.0, 143.0), turned to 270 degrees
- moved R702 377.8 mm to (124.5, 104.5)
- moved R701 376.6 mm to (120.5, 114.0), turned to 180 degrees
- moved W703 373.3 mm to (132.5, 136.5)
- moved C701 373.2 mm to (115.0, 143.0), turned to 270 degrees
- moved W705 373.2 mm to (128.0, 136.5)
- moved C722 372.7 mm to (135.0, 140.0), turned to 270 degrees
- moved C704 370.8 mm to (125.0, 114.0)
- moved U701 369.4 mm to (125.0, 111.0)
- moved L702 367.1 mm to (131.5, 141.0)
- moved Q701 366.7 mm to (120.5, 111.0), turned to 180 degrees
- moved C705 366.3 mm to (131.4, 138.5)
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Connections:
- U706 pad 16: ih_sense- -> GND
- U706 pad 19: ih_sense- -> GND
- U706 pad 20: ih_sense- -> GND
- U706 pad 33: ih_sense- -> GND
Routing:
- net Net-(C708-Pad1): track 0.00 -> 40.9 mm, vias 0 -> 3
- net /ADC/DINA: track 0.00 -> 35.8 mm, vias 0 -> 1
- net GND: track 0.00 -> 33.8 mm, vias 0 -> 38
- net /DAC/~LDAC: track 0.00 -> 28.0 mm, vias 0 -> 2
- net /ADC/i_meas+: track 0.00 -> 27.9 mm
- net /ADC/DINB: track 0.00 -> 27.8 mm, vias 0 -> 1
- net /DAC/~READY: track 0.00 -> 27.6 mm
- net /ADC/i_meas-: track 0.00 -> 26.9 mm
- net /DAC/~RST: track 0.00 -> 26.7 mm
- net /DAC/PD: track 0.00 -> 25.6 mm, vias 0 -> 1
- net /ADC/CNVSTB: track 0.00 -> 23.4 mm
- net /ADC/DOUTB: track 0.00 -> 23.1 mm
- net /DAC/DIN: track 0.00 -> 22.7 mm
- net +3V3: track 0.00 -> 22.3 mm, vias 0 -> 2
- net /DAC/~CS: track 0.00 -> 21.3 mm, vias 0 -> 1
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- added copper zone on F.Cu, net GND
- added copper zone on In1.Cu, net GND
- added copper zone on F.Cu, net Net-(C708-Pad1)
- added copper zone on F.Cu, net Net-(C716-Pad1)
Other:
- outline, holes or cut-outs redrawn
- net class HV added: clearance 0.2, trace_width 0.25, via_dia 0.8, via_drill 0.4

Commit message: Added switchable Gain for ADC Input Drivers
Parts:
- removed the REF** at (222.0, 143.8)
- added U406: SN74LVC1G373, Package_TO_SOT_SMD:SOT-363_SC-70-6, F.Cu at (259.4, 129.7)
- added U407: SN74LVC1G373, Package_TO_SOT_SMD:SOT-363_SC-70-6, F.Cu at (262.7, 129.7)
- added U408: SN74LVC1G373, Package_TO_SOT_SMD:SOT-363_SC-70-6, F.Cu at (259.4, 132.5)
- added U409: SN74LVC1G373, Package_TO_SOT_SMD:SOT-363_SC-70-6, F.Cu at (262.7, 132.5)
- added U410: 74HC595, Package_SO:TSSOP-16_4.4x5mm_P0.65mm, F.Cu at (180.3, 40.6)
- moved Q203 112.3 mm to (265.5, 87.8)
- moved Q204 112.3 mm to (262.0, 87.8)
- moved W201 112.3 mm to (272.5, 73.0)
- moved W202 112.3 mm to (272.5, 75.0)
- moved D201 68.3 mm to (273.2, 101.2)
- moved D202 68.3 mm to (276.4, 101.2)
- moved NT701 68.3 mm to (263.3, 103.1)
- moved R201 68.3 mm to (288.1, 101.0)
- moved R202 68.3 mm to (285.1, 101.0)
- moved R203 68.3 mm to (269.2, 101.4)
- moved R204 68.3 mm to (264.6, 101.4)
- moved R205 68.3 mm to (276.1, 102.9)
- moved R206 68.3 mm to (279.5, 101.0)
- moved R207 68.3 mm to (291.1, 102.5)
- moved R208 68.3 mm to (288.1, 102.5)
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Connections:
- Q501 pad 2: B4 -> B0
- Q502 pad 2: B5 -> B1
- Q503 pad 2: B6 -> B2
- R511 pad 1: B4 -> B0
- R512 pad 1: B5 -> B1
- R514 pad 1: B6 -> B2
- U501 pad 1: B0 -> Net-(U408-Pad4)
- U501 pad 2: B1 -> Net-(U409-Pad4)
- U502 pad 7: Net-(U502-Pad7) -> B7
- U503 pad 1: B2 -> Net-(U406-Pad4)
- U503 pad 2: B3 -> Net-(U407-Pad4)

Commit message: A little more routing
Parts:
- added REF**: MountingHole_6.5mm, MountingHole:MountingHole_6.5mm, F.Cu at (183.9, 81.0)
- added REF**: MountingHole_6.5mm, MountingHole:MountingHole_6.5mm, F.Cu at (183.9, 62.0)
- C501, D201, D202, Q203, Q204, R201, R202, R203, R204, R207, R208, U406, U407, U408, U409: moved to B.Cu
- moved R303 122.8 mm to (167.1, 80.3), turned to 90 degrees
- moved R207 120.3 mm to (180.1, 56.1)
- moved R201 118.6 mm to (180.1, 52.1), turned to 180 degrees
- moved W301 110.8 mm to (169.9, 91.2)
- moved U407 109.2 mm to (154.2, 142.2), turned to 90 degrees
- moved U409 109.0 mm to (154.2, 122.1), turned to 90 degrees
- moved R208 106.4 mm to (191.8, 57.4)
- moved R203 106.2 mm to (174.2, 53.8), turned to 270 degrees
- moved W302 105.5 mm to (167.6, 91.2)
- moved R202 104.8 mm to (191.8, 53.3), turned to 180 degrees
- moved D201 104.4 mm to (180.1, 53.8)
- moved U406 103.0 mm to (157.2, 142.2), turned to 90 degrees
- moved U408 102.7 mm to (157.2, 122.2), turned to 90 degrees
- moved NT701 100.8 mm to (162.6, 100.8), turned to 180 degrees
- moved D301 99.9 mm to (167.1, 77.0), turned to 90 degrees
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Routing:
- net +4.2V: track 6.54 -> 51.2 mm, vias 0 -> 9
- net -1.5V: track 6.99 -> 45.8 mm, vias 0 -> 6
- net B10: track 0.00 -> 30.5 mm, vias 0 -> 1
- net B9: track 0.00 -> 29.7 mm, vias 0 -> 3
- net B5: track 0.00 -> 22.9 mm, vias 0 -> 1
- net SRCLK: track 0.00 -> 22.8 mm, vias 0 -> 4
- net B6: track 0.00 -> 18.8 mm, vias 0 -> 1
- net B7: track 0.00 -> 18.0 mm, vias 0 -> 1
- net B4: track 0.00 -> 17.5 mm, vias 0 -> 1
- net B8: track 0.00 -> 17.3 mm, vias 0 -> 1
- net B3: track 0.00 -> 17.1 mm, vias 0 -> 1
- net Net-(U410-Pad14): track 0.00 -> 15.5 mm
- net B0: track 0.00 -> 9.85 mm, vias 0 -> 1
- net +5V: track 0.00 -> 5.73 mm
- net GND: track 33.8 -> 29.2 mm, vias 38 -> 51
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
Commit message: More routing
Parts:
- removed Q201: FDMS86263P, Package_TO_SOT_SMD:TO-252-2
- removed Q202: FDMS86252, Package_TO_SOT_SMD:TO-252-2
- removed R209, R210: 10m, Resistor_SMD:R_0603_1608Metric
- added G***: repo_url, frontend_additional-footprints:repo_url, F.Cu at (122.5, 124.3)
- added Q702: FDMS86255, Package_TO_SOT_SMD:TDSON-8-1, B.Cu at (202.7, 69.3)
- added Q703: FQB12P20, Package_TO_SOT_SMD:TO-252-2, B.Cu at (231.9, 70.4)
- C201, C202: footprint Capacitor_THT:CP_Radial_D8.0mm_P5.00mm -> Capacitor_THT:CP_Radial_D10.0mm_P5.00mm
- D501, D502, Q501, Q502, Q503, Q504, Q505, R211, R212, R213, R214, R511, R512, R514, R515, R516, R602: moved to B.Cu
- Q203, Q204, R207, R208: moved to F.Cu
- R101, R102: footprint Resistor_SMD:R_0603_1608Metric -> Resistor_SMD:R_1206_3216Metric
- moved R601 152.7 mm to (132.0, 83.7)
- moved R211 142.8 mm to (159.3, 54.0), turned to 180 degrees
- moved R602 138.2 mm to (147.4, 93.4), turned to 180 degrees
- moved R212 137.7 mm to (156.2, 54.0), turned to 180 degrees
- moved C608 136.0 mm to (148.1, 90.0), turned to 180 degrees
- moved C607 136.0 mm to (148.1, 88.6), turned to 180 degrees
- moved C602 134.1 mm to (152.2, 90.8), turned to 270 degrees
- moved R214 132.8 mm to (156.2, 52.4), turned to 180 degrees
- moved C601 132.7 mm to (153.7, 90.8), turned to 270 degrees
- moved R213 132.6 mm to (159.3, 52.4), turned to 180 degrees
- moved C605 131.1 mm to (153.7, 93.8), turned to 90 degrees
- moved Q505 128.8 mm to (193.6, 143.5), turned to 90 degrees
- moved C604 127.4 mm to (149.5, 99.9), turned to 180 degrees
- moved C603 124.1 mm to (149.5, 101.4), turned to 180 degrees
- moved C606 121.4 mm to (152.2, 93.8), turned to 90 degrees
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Connections:
- C201 pad 1: Net-(C201-Pad1) -> VDD
- C202 pad 2: Net-(C202-Pad2) -> VSS
- P102 pad 2: /Inrush Current Limiter/VIn- -> ih_sense-
- P102 pad 4: ih_sense- -> /Inrush Current Limiter/VIn-
- R203 pad 1: Net-(C201-Pad1) -> VDD
- R204 pad 1: Net-(C202-Pad2) -> VSS
Routing:
- net i_range: track 0.00 -> 97.2 mm
- net B0: track 9.85 -> 87.9 mm, vias 1 -> 3
- net B1: track 1.84 -> 74.6 mm
- net ih_sense-: track 0.00 -> 71.8 mm, vias 0 -> 2
- net Net-(K501-Pad4): track 0.00 -> 57.1 mm
- net B2: track 2.47 -> 52.5 mm
- net /vi_filter/il_sense+: track 0.00 -> 49.3 mm, vias 0 -> 1
- net v_sense-: track 0.00 -> 49.1 mm
- net ih_sense+: track 0.00 -> 45.8 mm, vias 0 -> 1
- net Net-(K504-Pad4): track 0.00 -> 37.6 mm
- net Net-(K501-Pad1): track 0.00 -> 28.4 mm
- net v_sense_ext+: track 0.00 -> 25.0 mm
- net output: track 0.00 -> 18.1 mm
- net +5V: track 5.73 -> 21.4 mm
- net Net-(C708-Pad1): track 40.9 -> 25.9 mm
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- added copper zone on F.Cu, net ih_sense-
- added copper zone on In1.Cu, net ih_sense-
Other:
- board text added: "±125 V"

Commit message: More routing (power supplies)
Parts:
- C408: moved to B.Cu
- moved G*** 86.9 mm to (181.3, 60.4)
- moved C423 50.5 mm to (154.1, 73.8), turned to 0 degrees
- moved C421 48.4 mm to (152.8, 70.3), turned to 0 degrees
- moved U404 47.6 mm to (155.2, 65.8), turned to 0 degrees
- moved P402 45.6 mm to (148.4, 73.8)
- moved C426 28.3 mm to (128.9, 54.6), turned to 90 degrees
- moved C414 26.3 mm to (150.7, 57.7)
- moved R415 25.8 mm to (146.5, 57.7)
- moved C415 25.7 mm to (150.7, 53.6)
- moved R413 25.7 mm to (150.7, 56.1)
- moved C420 25.7 mm to (139.3, 53.2)
- moved D408 25.7 mm to (139.3, 53.2)
- moved L405 25.7 mm to (134.8, 54.7)
- moved P404 25.7 mm to (140.8, 60.7)
- moved R412 25.7 mm to (138.3, 55.7)
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Routing:
- net +12V: track 4.80 -> 87.3 mm, vias 0 -> 11
- net rails_en: track 0.00 -> 69.6 mm, vias 0 -> 2
- net SRCLK: track 22.8 -> 85.0 mm, vias 4 -> 6
- net RCLK: track 0.00 -> 47.9 mm, vias 0 -> 2
- net SER: track 0.00 -> 46.0 mm, vias 0 -> 1
- net +5V: track 21.4 -> 55.4 mm, vias 0 -> 1
- net Net-(C705-Pad2): track 2.56 -> 29.7 mm, vias 0 -> 2
- net GND: track 35.8 -> 58.5 mm, vias 52 -> 65
- net +3V3: track 22.3 -> 43.4 mm, vias 2 -> 3
- net Net-(C716-Pad1): track 0.00 -> 20.4 mm, vias 1 -> 2
- net Net-(C707-Pad1): track 1.92 -> 18.9 mm
- net i_range: track 97.2 -> 112.6 mm
- net Net-(C407-Pad1): track 0.00 -> 14.1 mm
- net Net-(C708-Pad1): track 25.9 -> 38.2 mm
- net Net-(R414-Pad2): track 0.00 -> 11.7 mm, vias 0 -> 2
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- added copper zone on B.Cu, net +12V
- added copper zone on F.Cu, net +12V
- added copper zone on In2.Cu, net +12V
- added copper zone on B.Cu, net Net-(C409-Pad1)
- added copper zone on F.Cu, net Net-(C409-Pad1)
- added copper zone on F.Cu, net Net-(C417-Pad1)
- added copper zone on B.Cu, net Net-(C420-Pad1)
- added copper zone on F.Cu, net Net-(C420-Pad1)
- added copper zone on F.Cu, net Net-(C425-Pad1)

Commit message: More routing
Parts:
- added C712: C_Small, Capacitor_SMD:C_0603_1608Metric, B.Cu at (166.1, 71.0)
- added C725: C_Small, Capacitor_SMD:C_0603_1608Metric, B.Cu at (166.1, 66.2)
- added G***: temp_symbol, frontend_additional-footprints:temp_symbol, F.Cu at (170.8, 113.2)
- moved W302 9.48 mm to (184.8, 105.6)
- moved W202 6.72 mm to (194.2, 78.4)
- moved J601 2.49 mm to (158.4, 96.5)
- moved R302 1.70 mm to (166.3, 90.9)
- moved R516 0.59 mm to (190.7, 142.6)
- moved R602 0.30 mm to (147.7, 93.4)
- moved R212 0.07 mm to (166.1, 69.4)
- moved R211 0.05 mm to (169.2, 69.4)
Routing:
- net +3V3: track 43.4 -> 295.4 mm, vias 3 -> 10
- net vn: track 0.00 -> 125.4 mm, vias 0 -> 1
- net +5V: track 55.4 -> 180.5 mm, vias 1 -> 8
- net vp: track 0.00 -> 115.4 mm, vias 0 -> 1
- net GND: track 58.5 -> 132.0 mm, vias 65 -> 92
- net Net-(K301-Pad11): track 0.00 -> 57.8 mm
- net Net-(C303-Pad1): track 0.00 -> 56.9 mm
- net output: track 18.1 -> 70.4 mm, vias 0 -> 1
- net VSS: track 0.00 -> 43.8 mm, vias 0 -> 5
- net Net-(U301-Pad7): track 0.00 -> 38.3 mm, vias 0 -> 4
- net temp: track 0.00 -> 34.3 mm, vias 0 -> 4
- net Net-(R305-Pad2): track 0.00 -> 30.6 mm, vias 0 -> 2
- net VDD: track 0.00 -> 29.3 mm, vias 0 -> 1
- net Net-(R304-Pad1): track 0.00 -> 27.3 mm
- net RCLK: track 47.9 -> 72.8 mm
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- added copper zone on B.Cu, net GND
- added copper zone on F.Cu, net Net-(C410-Pad1)
- added copper zone on F.Cu, net Net-(C410-Pad2)
- added copper zone on F.Cu, net Net-(C413-Pad1)
- added copper zone on F.Cu, net Net-(K301-Pad11)
- added copper zone on B.Cu, net Net-(U301-Pad4)
- added copper zone on F.Cu, net Net-(U301-Pad4)
- added copper zone on B.Cu, net VSS
- added copper zone on F.Cu, net VSS

Commit message: More routing, fixed error in lockstep operation of current range switching relais
Parts:
- removed the G*** at (170.8, 113.2)
- moved NT701 2.50 mm to (195.3, 135.1)
- moved C524 1.75 mm to (186.2, 137.4), turned to 180 degrees
- moved C421 0.45 mm to (153.2, 70.3)
- moved C415 0.11 mm to (150.8, 53.6)
Connections:
- net ih_sense- renamed il_sense-
- K101 pad 12: /vi_filter/il_sense+ -> /vi_filter/ih_sense+
- K101 pad 14: ih_sense+ -> il_sense+
- K505 pad 10: ih_sense+ -> /vi_filter/ih_sense+
- K505 pad 8: /vi_filter/il_sense+ -> il_sense+
- R101 pad 1: /vi_filter/il_sense+ -> /vi_filter/ih_sense+
- R102 pad 1: ih_sense+ -> il_sense+
Routing:
- net +12V: track 97.5 -> 295.9 mm, vias 11 -> 14
- net pwr_enable: track 0.00 -> 162.7 mm, vias 0 -> 2
- net +5V: track 180.5 -> 319.9 mm, vias 8 -> 12
- net /output_stage/disengage: track 2.14 -> 140.0 mm, vias 0 -> 2
- net v_extern: track 1.69 -> 134.0 mm
- net v_ref_2: track 4.25 -> 89.1 mm, vias 0 -> 4
- net VSS: track 43.8 -> 107.6 mm, vias 5 -> 9
- net Net-(C417-Pad1): track 0.00 -> 62.2 mm, vias 0 -> 7
- net -1.5V: track 45.8 -> 106.7 mm, vias 6 -> 9
- net /vi_filter/ih_sense+: track 0.00 -> 58.7 mm, vias 0 -> 1
- net temp: track 34.3 -> 91.9 mm, vias 4 -> 5
- net /vi_filter/il_sense+: track 49.1 -> 0.00 mm, vias 1 -> 0
- net ih_sense+: track 45.8 -> 0.00 mm, vias 1 -> 0
- net il_sense+: track 0.00 -> 40.6 mm, vias 0 -> 1
- net i_range: track 117.5 -> 146.3 mm
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- added copper zone on B.Cu, net /Inrush Current Limiter/VIn-
- added copper zone on F.Cu, net Net-(C422-Pad1)
