File: components_predev/frontend/hardware/frontend.kicad_pcb (KiCad board)
At the start: 4 copper layers, 140 x 100 mm, 318 parts, among them J601 Conn_01x03, K101 PE014005, K301 PE014005, K501 HE3600, K502 HE3600, K503 HE3600, K504 EC2-12NU-L, K505 EC2-12NU-L, P101 CONN_01X40, P102 CONN_01X04, P103 CONN_01X02, P104 CONN_01X04, P401 CONN_01X02, P402 CONN_01X02, P403 CONN_01X02, P404 CONN_01X02, Q101 SSM3K329R,LF, Q203 MMBT5550L, Q204 MMBT5550L, Q301 MMBT5550L, Q302 MMBT5550L, Q303 MMBT5401-7-F, Q304 MMBT5550L, Q305 MMBT5401-7-F, Q306 2SA1962OTU, Q307 2SC5242OTU, Q308 SSM3K329R,LF, Q501 SSM3K329R,LF, Q502 SSM3K329R,LF, Q503 SSM3K329R,LF, Q504 SSM3K329R,LF, Q505 SSM3K329R,LF, Q701 SSM3K329R,LF, Q702 FDMS86255, Q703 FQB12P20, U301 LTC6090, U302 LTC6090, U303 LTC6090, U401 AOZ1284, U402 LT1617, U403 AOZ1284, U404 MIC39100, U405 MC79M05, U406 SN74LVC1G373, U407 SN74LVC1G373, U408 SN74LVC1G373, U409 SN74LVC1G373, U410 74HC595, U501 ISL2863x, U502 74HC595, U503 ISL2863x, U504 TSP73001, U505 MIC5270BM5, U506 ISL2863x, U507 ISL2863x, U601 MAX5318, U701 MIC7211, U702 ADR4533, U703 LMT88, U704 NCP508, U705 NCP508, U706 MAX11960, U707 LTC2055, U708 TSP73001

Commit message: Routing done
Parts:
- added G***: temp_symbol, frontend_additional-footprints:temp_symbol, F.Cu at (170.6, 112.8)
- added REF**: Symbol_HighVoltage_Type2_CopperTop_VerySmall, frontend_additional-footprints:Symbol_HighVoltage_Type2_CopperTop_VerySmall, F.Cu at (181.2, 61.9)
- moved G*** 43.1 mm to (144.4, 82.6)
Routing:
- net GND: track 155.7 -> 301.0 mm, vias 104 -> 122
- net -5V: track 12.0 -> 153.8 mm, vias 1 -> 6
- net +5V: track 319.9 -> 406.9 mm, vias 12 -> 13
- net VDD: track 29.3 -> 112.3 mm, vias 1 -> 5
- net +4.2V: track 81.8 -> 163.6 mm, vias 9 -> 11
- net v_ref_2: track 89.1 -> 165.7 mm, vias 4 -> 6
- net i_range: track 146.3 -> 198.2 mm
- net +12V: track 295.9 -> 342.8 mm
- net pwr_enable: track 162.7 -> 201.9 mm
- net il_sense-: track 79.9 -> 110.7 mm
- net -1.5V: track 106.7 -> 136.7 mm
- net v_ref: track 25.6 -> 53.4 mm
- net Net-(C305-Pad2): track 4.95 -> 24.0 mm, vias 0 -> 2
- net temp: track 91.9 -> 107.8 mm, vias 5 -> 8
- net Net-(D201-Pad2): track 0.00 -> 7.19 mm, vias 0 -> 1
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- added copper zone on B.Cu, net /Inrush Current Limiter/VIn+
- added copper zone on B.Cu, net VDD
Other:
- board text added: "+12V"
- board text added: "+3.3V"
- board text added: "+5V"
- board text added: "-5V"
- board text added: "DANGER! HIGH VOLTAGE!"
- board text added: "openSMU Frontend 09/2018"

Commit message: Finished routing, begun component specification
Parts:
- moved C504 0.50 mm to (153.0, 116.9)
- moved C523 0.40 mm to (186.0, 117.0)
- moved C503 0.32 mm to (159.0, 147.1)
- moved C522 0.30 mm to (193.2, 125.2)
- moved C505 0.27 mm to (155.0, 137.3)
Routing:
- net v_ref_2: track 165.7 -> 162.5 mm
- net -1.5V: track 136.7 -> 139.6 mm
- net Net-(U301-Pad4): track 17.9 -> 19.4 mm
- net GND: track 301.0 -> 299.8 mm, vias 122 -> 120
- net v_extern: track 134.0 -> 132.9 mm
- net VSS: track 106.7 -> 105.7 mm
- net +12V: track 342.8 -> 342.0 mm
- net Net-(C708-Pad1): track 39.1 -> 38.4 mm
- net il_sense-: vias 5 -> 11
- added copper zone on In2.Cu, net GND

Commit message: Some Updates from Testing
Parts:
- removed the G*** at (170.6, 112.8)
- removed the REF** at (181.2, 61.9)
- C300, C403, C404, C408, C412, C416, C417, C421, C422, C425, C501, C502, C503, C504, C505, C506, C512, C513, C518, C521, C522, C523, C524, C602, C604, C606, C608, C702, C704, C706, C709, C710, C711, C715, C716, C722: value C_Small -> 100n
- C402, C407, C418, C419, C423, C424, C426, C701, C723: value CP1_Small -> 22u
- C601, C603, C605, C703, C705, C707, C708, C717: value C_Small -> 10u
- C607: value C_Small -> 22u
- C713, C714: value CP1_Small -> 220u
- R103: value R -> 68k
- R302: value 132k -> 130k
- R318, R511, R512, R514, R515, R516: value R_Small -> 68k
- R517, R518, R519, R520, R521, R522, R523, R524, R525, R526, R527, R603, R604, R605, R606, R607, R608, R609: value R_Small -> 22
- R601: value R_Small -> 2k
- R701: value R_Small -> 10k
- U301: value LTC6090 -> LTC6090-5
- U504, U708: value TSP73001 -> TPS73001
- U505: value MIC5270BM5 -> MIC5270YM5
