File: components_predev/frontend/hardware/output_stage.sch (KiCad schematic (older format))
At the start: 43 parts, among them K301 PE014005, Q301 MMBT5550L, Q302 MMBT5550L, Q303 MMBT5401-7-F, Q304 MMBT5550L, Q305 MMBT5401-7-F, Q306 2SA1962OTU, Q307 2SC5242OTU, Q308 Q_NMOS_DGS, U301 LTC6090-5, U302 LTC6091

Commit message: Finished Range Switching/Filters
Parts:
- gave numbers to parts that had none: 5
Changed lines of the file:
@@
 $EndComp
 $Comp
-L VDD #PWR026
+L VDD #PWR025
 U 1 1 5B0EA219
 P 8300 800
-F 0 "#PWR026" H 8300 650 50  0001 C CNN
+F 0 "#PWR025" H 8300 650 50  0001 C CNN
 F 1 "VDD" H 8300 950 50  0000 C CNN
 F 2 "" H 8300 800 50  0000 C CNN
@@
 $EndComp
 $Comp
-L VSS #PWR027
+L VSS #PWR026
 U 1 1 5B0EA25A
 P 6000 6250
-F 0 "#PWR027" H 6000 6100 50  0001 C CNN
+F 0 "#PWR026" H 6000 6100 50  0001 C CNN
 F 1 "VSS" H 6000 6400 50  0000 C CNN
 F 2 "" H 6000 6250 50  0000 C CNN
@@
 VSS
 $Comp
-L VDD #PWR028
+L VDD #PWR027
 U 1 1 5B0ED212
 P 1300 1050
-F 0 "#PWR028" H 1300 900 50  0001 C CNN
+F 0 "#PWR027" H 1300 900 50  0001 C CNN
 F 1 "VDD" H 1300 1200 50  0000 C CNN
 F 2 "" H 1300 1050 50  0000 C CNN
@@
 $EndComp
 $Comp
-L VSS #PWR029
+L VSS #PWR028
 U 1 1 5B0ED37D
 P 1300 1250
-F 0 "#PWR029" H 1300 1100 50  0001 C CNN
+F 0 "#PWR028" H 1300 1100 50  0001 C CNN
 F 1 "VSS" H 1300 1400 50  0000 C CNN
 F 2 "" H 1300 1250 50  0000 C CNN
@@
 Connection ~ 7700 5550
 $Comp
-L GNDPWR #PWR030
+L GNDPWR #PWR029
 U 1 1 5B118A91
 P 7600 3750
-F 0 "#PWR030" H 7600 3550 50  0001 C CNN
+F 0 "#PWR029" H 7600 3550 50  0001 C CNN
 F 1 "GNDPWR" H 7600 3620 50  0000 C CNN
 F 2 "" H 7600 3700 50  0000 C CNN
@@
 	10000 4450 9650 4450
 $Comp
-L GND #PWR031
+L GND #PWR030
 U 1 1 5B29F8CE
 P 10000 5350
-F 0 "#PWR031" H 10000 5100 50  0001 C CNN
+F 0 "#PWR030" H 10000 5100 50  0001 C CNN
 F 1 "GND" H 10000 5200 50  0000 C CNN
 F 2 "" H 10000 5350 50  0000 C CNN
@@
 Connection ~ 10000 5300
 $Comp
-L +12V #PWR032
+L +12V #PWR031
 U 1 1 5B29FBBB
 P 9100 4450
-F 0 "#PWR032" H 9100 4300 50  0001 C CNN
+F 0 "#PWR031" H 9100 4300 50  0001 C CNN
 F 1 "+12V" H 9100 4590 50  0000 C CNN
 F 2 "" H 9100 4450 50  0000 C CNN
@@
 Connection ~ 4400 5900
 $Comp
-L VDD #PWR033
+L VDD #PWR032
 U 1 1 5B33DC6E
 P 4400 6600
-F 0 "#PWR033" H 4400 6450 50  0001 C CNN
+F 0 "#PWR032" H 4400 6450 50  0001 C CNN
 F 1 "VDD" H 4400 6750 50  0000 C CNN
 F 2 "" H 4400 6600 50  0000 C CNN
@@
 	4400 6600 4400 6350
 $Comp
-L VDD #PWR034
+L VDD #PWR033
 U 1 1 5B33E01C
 P 3500 5050
-F 0 "#PWR034" H 3500 4900 50  0001 C CNN
+F 0 "#PWR033" H 3500 4900 50  0001 C CNN
 F 1 "VDD" H 3500 5200 50  0000 C CNN
 F 2 "" H 3500 5050 50  0000 C CNN
@@
 $EndComp
 $Comp
-L GND #PWR035
+L GND #PWR034
 U 1 1 5B33E1D8
 P 3950 5250
-F 0 "#PWR035" H 3950 5000 50  0001 C CNN
+F 0 "#PWR034" H 3950 5000 50  0001 C CNN
 F 1 "GND" H 3950 5100 50  0000 C CNN
 F 2 "" H 3950 5250 50  0000 C CNN
@@
 	2150 5750 2700 5750
 $Comp
-L GND #PWR036
+L GND #PWR035
 U 1 1 5B33E42B
 P 3500 6350
-F 0 "#PWR036" H 3500 6100 50  0001 C CNN
+F 0 "#PWR035" H 3500 6100 50  0001 C CNN
 F 1 "GND" H 3500 6200 50  0000 C CNN
 F 2 "" H 3500 6350 50  0000 C CNN
@@
 	1350 3650 1450 3650
 $Comp
-L GND #PWR037
+L GND #PWR036
 U 1 1 5B33ECC1
 P 4000 1300
-F 0 "#PWR037" H 4000 1050 50  0001 C CNN
+F 0 "#PWR036" H 4000 1050 50  0001 C CNN
 F 1 "GND" H 4000 1150 50  0000 C CNN
 F 2 "" H 4000 1300 50  0000 C CNN
@@
 	3500 1200 3500 1400
 $Comp
-L VSS #PWR038
+L VSS #PWR037
 U 1 1 5B33EF8A
 P 3500 2550
-F 0 "#PWR038" H 3500 2400 50  0001 C CNN
+F 0 "#PWR037" H 3500 2400 50  0001 C CNN
 F 1 "VSS" H 3500 2700 50  0000 C CNN
 F 2 "" H 3500 2550 50  0000 C CNN
@@
 $EndComp
 $Comp
-L GND #PWR039
+L GND #PWR038
 U 1 1 5B33F1B7
 P 4000 2550
-F 0 "#PWR039" H 4000 2300 50  0001 C CNN
+F 0 "#PWR038" H 4000 2300 50  0001 C CNN
 F 1 "GND" H 4000 2400 50  0000 C CNN
 F 2 "" H 4000 2550 50  0000 C CNN
@@
 	4850 1100 4850 1350
 $Comp
-L VSS #PWR040
+L VSS #PWR039
 U 1 1 5B340542
 P 4850 1100
-F 0 "#PWR040" H 4850 950 50  0001 C CNN
+F 0 "#PWR039" H 4850 950 50  0001 C CNN
 F 1 "VSS" H 4850 1250 50  0000 C CNN
 F 2 "" H 4850 1100 50  0000 C CNN
@@
 	2750 7300 2600 7300
 $Comp
-L +5V #PWR041
+L +5V #PWR040
 U 1 1 5B343BDA
 P 2100 7300
-F 0 "#PWR041" H 2100 7150 50  0001 C CNN
+F 0 "#PWR040" H 2100 7150 50  0001 C CNN
 F 1 "+5V" H 2100 7440 50  0000 C CNN
 F 2 "" H 2100 7300 50  0000 C CNN
@@
 	2100 7300 2300 7300
 $Comp
-L GND #PWR042
+L GND #PWR041
 U 1 1 5B3448FD
 P 3250 6500
-F 0 "#PWR042" H 3250 6250 50  0001 C CNN
+F 0 "#PWR041" H 3250 6250 50  0001 C CNN
 F 1 "GND" H 3250 6350 50  0000 C CNN
 F 2 "" H 3250 6500 50  0000 C CNN
@@
 $EndComp
 $Comp
-L GND #PWR043
+L GND #PWR042
 U 1 1 5B344A22
 P 3050 4500
-F 0 "#PWR043" H 3050 4250 50  0001 C CNN
+F 0 "#PWR042" H 3050 4250 50  0001 C CNN
 F 1 "GND" H 3050 4350 50  0000 C CNN
 F 2 "" H 3050 4500 50  0000 C CNN
@@
 	3250 6500 3250 6100
 $Comp
-L GND #PWR044
+L GND #PWR043
 U 1 1 5B344F7A
 P 3250 2600
-F 0 "#PWR044" H 3250 2350 50  0001 C CNN
+F 0 "#PWR043" H 3250 2350 50  0001 C CNN
 F 1 "GND" H 3250 2450 50  0000 C CNN
 F 2 "" H 3250 2600 50  0000 C CNN
@@
 	1350 4600 1750 4600
 $Comp
-L TEST_1P W?
+L TEST_1P W303
 U 1 1 5B3ABE63
 P 4800 3650
-F 0 "W?" H 4800 3920 50  0000 C CNN
+F 0 "W303" H 4800 3920 50  0000 C CNN
 F 1 "TEST_1P" H 4800 3850 50  0000 C CNN
 F 2 "" H 5000 3650 50  0000 C CNN
@@
 Connection ~ 4800 3800
 $Comp
-L TEST_1P W?
+L TEST_1P W302
 U 1 1 5B3ABFD1
 P 2800 2900
-F 0 "W?" H 2800 3170 50  0000 C CNN
+F 0 "W302" H 2800 3170 50  0000 C CNN
 F 1 "TEST_1P" H 2800 3100 50  0000 C CNN
 F 2 "" H 3000 2900 50  0000 C CNN
@@
 $EndComp
 $Comp
-L TEST_1P W?
+L TEST_1P W301
 U 1 1 5B3AC0BA
 P 1700 2900
-F 0 "W?" H 1700 3170 50  0000 C CNN
+F 0 "W301" H 1700 3170 50  0000 C CNN
 F 1 "TEST_1P" H 1700 3100 50  0000 C CNN
 F 2 "" H 1900 2900 50  0000 C CNN
@@
 Connection ~ 2800 3000
 $Comp
-L TEST_1P W?
+L TEST_1P W305
 U 1 1 5B3AC35A
 P 8850 3500
-F 0 "W?" H 8850 3770 50  0000 C CNN
+F 0 "W305" H 8850 3770 50  0000 C CNN
 F 1 "TEST_1P" H 8850 3700 50  0000 C CNN
 F 2 "" H 9050 3500 50  0000 C CNN
@@
 Connection ~ 8850 3600
 $Comp
-L TEST_1P W?
+L TEST_1P W304
 U 1 1 5B3AC54F
 P 6650 1950
-F 0 "W?" H 6650 2220 50  0000 C CNN
+F 0 "W304" H 6650 2220 50  0000 C CNN
 F 1 "TEST_1P" H 6650 2150 50  0000 C CNN
 F 2 "" H 6850 1950 50  0000 C CNN

Commit message: Changed to KiCAD 5
Parts:
- C301, C302: footprint (none) -> Capacitors_SMD:C_1206; symbol C_Small -> Device:C_Small; Dielectric (none) -> X7R; Digikey (none) -> 1276-3084-1-ND; Manufacturer (none) -> Samsung; Part Number (none) -> CL31B104KEHSNNE; Voltage (none) -> 250 V
- C303: footprint (none) -> Capacitors_SMD:C_0603; symbol C -> Device:C; Dielectric (none) -> X7R; Digikey (none) -> 1276-1000-1-ND; Manufacturer (none) -> Samsung; Part Number (none) -> CL10B104KB8NNNC; Voltage (none) -> 50 V
- C304, C305: value C -> 33p; symbol C -> Device:C
- D301: symbol LED -> Device:LED
- D302: symbol D -> Device:D
- K301: symbol PE014005 -> frontend_additional_components:PE014005
- L301: symbol Ferrite_Bead -> Device:Ferrite_Bead
- Q301, Q302, Q304: footprint (none) -> TO_SOT_Packages_SMD:SOT-23; symbol Q_NPN_BCE -> Device:Q_NPN_BCE
- Q303, Q305, Q306: symbol Q_PNP_BCE -> Device:Q_PNP_BCE
- Q307: symbol Q_NPN_BCE -> Device:Q_NPN_BCE
- Q308: symbol Q_NMOS_DGS -> Device:Q_NMOS_DGS
- R301, R302, R303, R304, R305, R306, R307, R308, R309, R310, R311, R312, R313, R314, R315, R316, R317: footprint (none) -> Resistors_SMD:R_0603; symbol R -> Device:R
- R318: footprint (none) -> Resistors_SMD:R_0603; symbol R_Small -> Device:R_Small
- RV301: symbol POT_TRIM -> Device:R_POT_TRIM
- U301: symbol LTC6090 -> frontend_additional_components:LTC6090
- U302: symbol LTC6091 -> frontend_additional_components:LTC6091
- W301, W302, W303, W304, W305: symbol TEST_1P -> Connector:Test_Point
Connections:
- wire segments 124 -> 164

Commit message: Footrpints and Parts Specification
Parts:
- C304, C305: footprint (none) -> Capacitor_SMD:C_0805_2012Metric; Digikey (none) -> 311-4249-1-ND; Manufacturer (none) -> Yageo; Mouser (none) -> 603-CC805JRNPOABN330; Part Number (none) -> CC0805JRNPOABN330
- D301: footprint (none) -> LED_SMD:LED_0603_1608Metric
- D302: value D -> FDLL4148; footprint (none) -> Diode_SMD:D_MiniMELF; Digikey (none) -> FDLL4148CT-ND; Manufacturer (none) -> OnSemi; Mouser (none) -> 512-FDLL4148; Part Number (none) -> FDLL4148
- L301: value Ferrite_Bead -> HI1206T500R-10; footprint (none) -> Inductor_SMD:L_1206_3216Metric; Digikey (none) -> 240-2412-1-ND; Manufacturer (none) -> Laird; Mouser (none) -> 875-HI1206T500R-10; Part Number (none) -> HI1206T500R-10
- Q303, Q305: footprint (none) -> Package_TO_SOT_SMD:SOT-23
- Q304: Digikey (none) -> MMBT5550LT1GOSCT-ND; Manufacturer (none) -> OnSemi
- Q306, Q307: footprint (none) -> Package_TO_SOT_THT:TO-3P-3_Vertical
- Q308: value Q_NMOS_DGS -> SSM3K329R,LF; footprint (none) -> Package_TO_SOT_SMD:SOT-23; Digikey (none) -> SSM3K329RLFCT-ND; Manufacturer (none) -> Toshiba; Mouser (none) -> 757-SSM3K329RLF; Part Number (none) -> SSM3K329R,LF
- R301, R302, R303, R304, R305, R306, R307, R308, R309, R310, R311, R312, R313, R314, R315, R316, R317, R318: footprint Resistors_SMD:R_0603 -> Resistor_SMD:R_0603_1608Metric
- RV301: footprint (none) -> Potentiometer_SMD:Potentiometer_Bourns_3214X_Vertical; Digikey (none) -> 3214X-1-501ECT-ND; Manufacturer (none) -> Bourns; Mouser (none) -> 652-3214X-1-501E; Part Number (none) -> 3214X-1-501E
- U301: footprint (none) -> Package_SO:TI_SO-PowerPAD-8; Digikey (none) -> LTC6090IS8E-5#PBF-ND; Manufacturer (none) -> Linear Technology; Part Number (none) -> LTC6090IS8E-5#PBF
- W301, W302, W303, W304, W305: footprint (none) -> TestPoint:TestPoint_Pad_D1.0mm

Commit message: Finished Footprints, ERC
Parts:
- removed U302: LTC6091, symbol frontend_additional_components:LTC6091
- added U302, U303: LTC6090-5, Package_SO:TI_SO-PowerPAD-8, symbol frontend_additional_components:LTC6090
- C301, C302: footprint Capacitors_SMD:C_1206 -> Capacitor_SMD:C_1206_3216Metric
- C303: footprint Capacitors_SMD:C_0603 -> Capacitor_SMD:C_0603_1608Metric
- K301: footprint (none) -> frontend_additional-footprints:PE014005
- Q301, Q302, Q304: footprint TO_SOT_Packages_SMD:SOT-23 -> Package_TO_SOT_SMD:SOT-23
Connections:
- wire segments 164 -> 168
Changed lines of the file:
@@
 $Descr A4 11693 8268
 encoding utf-8
-Sheet 3 7
+Sheet 2 7
 Title "Output Amplifier"
 Date ""
@@
 F 0 "Q302" H 7800 2100 50  0000 L CNN
 F 1 "MMBT5550L" H 7800 2000 50  0000 L CNN
-F 2 "TO_SOT_Packages_SMD:SOT-23" H 7800 2150 50  0001 C CNN
+F 2 "Package_TO_SOT_SMD:SOT-23" H 7800 2150 50  0001 C CNN
 F 3 "" H 7600 2050 50  0000 C CNN
 F 4 "OnSemi" H 7600 2050 60  0001 C CNN "Manufacturer"
@@
 F 0 "Q304" H 8200 3100 50  0000 L CNN
 F 1 "MMBT5550L" H 7150 3050 50  0000 L CNN
-F 2 "TO_SOT_Packages_SMD:SOT-23" H 8200 3150 50  0001 C CNN
+F 2 "Package_TO_SOT_SMD:SOT-23" H 8200 3150 50  0001 C CNN
 F 3 "" H 8000 3050 50  0000 C CNN
 F 4 "MMBT5550L" H 8000 3050 60  0001 C CNN "Part Number"
@@
 F 0 "Q301" H 6750 3650 50  0000 L CNN
 F 1 "MMBT5550L" H 6750 3550 50  0000 L CNN
-F 2 "TO_SOT_Packages_SMD:SOT-23" H 6750 3700 50  0001 C CNN
+F 2 "Package_TO_SOT_SMD:SOT-23" H 6750 3700 50  0001 C CNN
 F 3 "" H 6550 3600 50  0000 C CNN
 F 4 "OnSemi" H 6550 3600 60  0001 C CNN "Manufacturer"
@@
 F 0 "C303" H 5575 3700 50  0000 L CNN
 F 1 "100n" H 5575 3500 50  0000 L CNN
-F 2 "Capacitors_SMD:C_0603" H 5588 3450 50  0001 C CNN
+F 2 "Capacitor_SMD:C_0603_1608Metric" H 5588 3450 50  0001 C CNN
 F 3 "" H 5550 3600 50  0000 C CNN
 F 4 "Samsung" H 5550 3600 60  0001 C CNN "Manufacturer"
@@
 	1    0    0    -1
 $EndComp
-Wire Wire Line
-	7600 3750 7600 3600
 Wire Wire Line
 	7600 3600 7350 3600
@@
 F 0 "K301" H 9250 3975 60  0000 C CNN
 F 1 "PE014005" H 9425 3425 60  0000 C CNN
-F 2 "" H 13300 5300 60  0001 C CNN
+F 2 "frontend_additional-footprints:PE014005" H 13300 5300 60  0001 C CNN
 F 3 "" H 13300 5300 60  0001 C CNN
 	1    9500 3700
@@
 $EndComp
 $Comp
-L frontend_additional_components:LTC6091 U302
-U 2 1 5B33CC17
-P 3750 1850
-F 0 "U302" H 4400 2150 60  0000 C CNN
-F 1 "LTC6091" H 4550 2050 60  0000 C CNN
-F 2 "" H 3750 1850 60  0001 C CNN
-F 3 "" H 3750 1850 60  0001 C CNN
-	2    3750 1850
-	-1   0    0    -1
-$EndComp
-$Comp
-L frontend_additional_components:LTC6091 U302
-U 1 1 5B33CCAA
-P 3750 5750
-F 0 "U302" H 4400 6050 60  0000 C CNN
-F 1 "LTC6091" H 4550 5950 60  0000 C CNN
-F 2 "" H 3750 5750 60  0001 C CNN
-F 3 "" H 3750 5750 60  0001 C CNN
-	1    3750 5750
-	-1   0    0    -1
-$EndComp
-$Comp
 L Device:R R304
 U 1 1 5B33D296
@@
 F 0 "C301" H 3710 5220 50  0000 L CNN
 F 1 "100n" H 3710 5070 50  0000 L CNN
-F 2 "Capacitors_SMD:C_1206" H 3700 5150 50  0001 C CNN
+F 2 "Capacitor_SMD:C_1206_3216Metric" H 3700 5150 50  0001 C CNN
 F 3 "" H 3700 5150 50  0000 C CNN
 F 4 "Samsung" H 3700 5150 60  0001 C CNN "Manufacturer"
@@
 $EndComp
 Wire Wire Line
-	3500 6350 3500 6200
+	3500 6350 3500 6300
 Wire Wire Line
 	3950 2000 4400 2000
@@
 F 0 "C302" H 3760 2520 50  0000 L CNN
 F 1 "100n" H 3760 2370 50  0000 L CNN
-F 2 "Capacitors_SMD:C_1206" H 3750 2450 50  0001 C CNN
+F 2 "Capacitor_SMD:C_1206_3216Metric" H 3750 2450 50  0001 C CNN
 F 3 "" H 3750 2450 50  0000 C CNN
 F 4 "Samsung" H 3750 2450 60  0001 C CNN "Manufacturer"
@@
 	4000 2450 3850 2450
 Wire Wire Line
-	3650 2450 3500 2450
+	3650 2450 3600 2450
 Connection ~ 3500 2450
 Wire Wire Line
 	4000 1200 4000 1300
-Wire Wire Line
-	2800 4250 2800 4450
-Wire Wire Line
-	2800 4450 2050 4450
-Wire Wire Line
-	2050 4450 2050 3000
-Wire Wire Line
-	2050 1850 2700 1850
-Wire Wire Line
-	3950 1700 4400 1700
-Wire Wire Line
-	4400 1700 4400 950
-Wire Wire Line
-	4400 950  2050 950
-Connection ~ 2050 1850
 $Comp
 L Device:R R307
@@
 	0    -1   -1   0
 $EndComp
-Wire Wire Line
-	2100 7300 2300 7300
 $Comp
 L power:GND #PWR042
@@
 	1    0    0    -1
 $EndComp
-Wire Wire Line
-	1700 2900 1700 3000
-Wire Wire Line
-	1700 3000 2050 3000
-Connection ~ 2050 3000
 Connection ~ 2800 3000
 $Comp
@@
 	3500 2450 3500 2550
 Wire Wire Line
-	2050 1850 2050 950
-Wire Wire Line
 	4400 2000 4850 2000
 Wire Wire Line
@@
 	4800 3800 5150 3800
 Wire Wire Line
-	2050 3000 2050 1850
-Wire Wire Line
 	2800 3000 2800 3350
 Wire Wire Line
@@
 Wire Wire Line
 	6650 2050 6650 2850
+Wire Wire Line
+	7600 3750 7600 3600
+$Comp
+L frontend_additional_components:LTC6090 U302
+U 1 1 5B798560
+P 3750 1850
+F 0 "U302" H 4400 2150 60  0000 C CNN
+F 1 "LTC6090-5" H 4550 2050 60  0000 C CNN
+F 2 "Package_SO:TI_SO-PowerPAD-8" H 3750 1850 60  0001 C CNN
+F 3 "" H 3750 1850 60  0001 C CNN
+F 4 "LTC6090IS8E-5#PBF-ND" H 1200 -1950 50  0001 C CNN "Digikey"
+F 5 "Linear Technology" H 1200 -1950 50  0001 C CNN "Manufacturer"
+F 6 "LTC6090IS8E-5#PBF" H 1200 -1950 50  0001 C CNN "Part Number"
+	1    3750 1850
+	-1   0    0    -1
+$EndComp
+Wire Wire Line
+	3600 2350 3600 2450
+Connection ~ 3600 2450
+Wire Wire Line
+	3600 2450 3500 2450
+$Comp
+L frontend_additional_components:LTC6090 U303
+U 1 1 5B7A1262
+P 3750 5750
+F 0 "U303" H 4400 6050 60  0000 C CNN
+F 1 "LTC6090-5" H 4550 5950 60  0000 C CNN
+F 2 "Package_SO:TI_SO-PowerPAD-8" H 3750 5750 60  0001 C CNN
+F 3 "" H 3750 5750 60  0001 C CNN
+F 4 "LTC6090IS8E-5#PBF-ND" H 1200 1950 50  0001 C CNN "Digikey"
+F 5 "Linear Technology" H 1200 1950 50  0001 C CNN "Manufacturer"
+F 6 "LTC6090IS8E-5#PBF" H 1200 1950 50  0001 C CNN "Part Number"
+	1    3750 5750
+	-1   0    0    -1
+$EndComp
+Wire Wire Line
+	3600 6250 3600 6300
+Wire Wire Line
+	3600 6300 3500 6300
+Connection ~ 3500 6300
+Wire Wire Line
+	3500 6300 3500 6200
+Wire Wire Line
+	2300 7300 2100 7300
+Wire Wire Line
+	3950 1700 4400 1700
+Wire Wire Line
+	4400 1700 4400 950
+Wire Wire Line
+	4400 950  2050 950
+Wire Wire Line
+	2050 950  2050 1850
+Wire Wire Line
+	2050 1850 2700 1850
+Wire Wire Line
+	2050 1850 2050 2900
+Wire Wire Line
+	2050 4500 2800 4500
+Wire Wire Line
+	2800 4500 2800 4250
+Connection ~ 2050 1850
+Wire Wire Line
+	1700 2900 2050 2900
+Connection ~ 2050 2900
+Wire Wire Line
+	2050 2900 2050 4500
 $EndSCHEMATC
