File: components_predev/frontend/hardware/output_stage.sch (KiCad schematic (older format))
At the start: 44 parts, among them K301 PE014005, Q301 MMBT5550L, Q302 MMBT5550L, Q303 MMBT5401-7-F, Q304 MMBT5550L, Q305 MMBT5401-7-F, Q306 2SA1962OTU, Q307 2SC5242OTU, Q308 SSM3K329R,LF, U301 LTC6090, U302 LTC6090, U303 LTC6090

Commit message: More Part Specifications added
Parts:
- R301: Digikey (none) -> P2.00KFCT-ND; Manufacturer (none) -> Panasonic; Part Number (none) -> ERJ-8ENF2001V
- R302: value 132k -> 130k; Digikey (none) -> P130KFCT-ND; Manufacturer (none) -> Panasonic; Part Number (none) -> ERJ-8ENF1303V
- R304, R305: Digikey (none) -> P120KFCT-ND; Manufacturer (none) -> Panasonic; Part Number (none) -> ERJ-8ENF1203V
- R306, R307: Digikey (none) -> P100KFCT-ND; Manufacturer (none) -> Panasonic; Part Number (none) -> ERJ-8ENF1003V
- R308: Digikey (none) -> P68.0FCT-ND; Manufacturer (none) -> Panasonic; Part Number (none) -> ERJ-8ENF68R0V
- R309, R310: Digikey (none) -> P523FCT-ND; Manufacturer (none) -> Panasonic; Part Number (none) -> ERJ-8ENF5230V
- R311: Digikey (none) -> P68.0KFCT-ND; Manufacturer (none) -> Panasonic; Part Number (none) -> ERJ-8ENF6802V
- R312, R313: Digikey (none) -> P3.32KFCT-ND; Manufacturer (none) -> Panasonic; Part Number (none) -> ERJ-8ENF3321V
- R314, R315: Digikey (none) -> P1.02KFCT-ND; Manufacturer (none) -> Panasonic; Part Number (none) -> ERJ-8ENF1021V
- R316, R317: Digikey (none) -> P17684CT-ND; Manufacturer (none) -> Panasonic; Part Number (none) -> ERJ-8BSFR20V
- R318: value R_Small -> 68k
- U301: value LTC6090 -> LTC6090-5; Digikey (none) -> LTC6090CS8E-5#PBF-ND; Manufacturer (none) -> Linear Technology; Part Number (none) -> LTC6090CS8E-5#PBF
- U302, U303: Digikey (none) -> LTC6090CS8E#PBF-ND; Manufacturer (none) -> Linear Technology; Part Number (none) -> LTC6090CS8E#PBF
Changed lines of the file:
@@
 F 2 "Resistor_SMD:R_1206_3216Metric" V 7630 1300 50  0001 C CNN
 F 3 "" H 7700 1300 50  0000 C CNN
+F 4 "P1.02KFCT-ND" H 0   0   50  0001 C CNN "Digikey"
+F 5 "Panasonic" H 0   0   50  0001 C CNN "Manufacturer"
+F 6 "ERJ-8ENF1021V" H 0   0   50  0001 C CNN "Part Number"
 	1    7700 1300
 	1    0    0    -1
@@
 F 2 "Resistor_SMD:R_2512_6332Metric" V 8230 3300 50  0001 C CNN
 F 3 "" H 8300 3300 50  0000 C CNN
+F 4 "P17684CT-ND" H 0   0   50  0001 C CNN "Digikey"
+F 5 "Panasonic" H 0   0   50  0001 C CNN "Manufacturer"
+F 6 "ERJ-8BSFR20V" H 0   0   50  0001 C CNN "Part Number"
 	1    8300 3300
 	1    0    0    -1
@@
 F 2 "Resistor_SMD:R_2512_6332Metric" V 8230 3900 50  0001 C CNN
 F 3 "" H 8300 3900 50  0000 C CNN
+F 4 "P17684CT-ND" H 0   0   50  0001 C CNN "Digikey"
+F 5 "Panasonic" H 0   0   50  0001 C CNN "Manufacturer"
+F 6 "ERJ-8BSFR20V" H 0   0   50  0001 C CNN "Part Number"
 	1    8300 3900
 	1    0    0    -1
@@
 F 2 "Resistor_SMD:R_1206_3216Metric" V 7630 5900 50  0001 C CNN
 F 3 "" H 7700 5900 50  0000 C CNN
+F 4 "P1.02KFCT-ND" H 0   0   50  0001 C CNN "Digikey"
+F 5 "Panasonic" H 0   0   50  0001 C CNN "Manufacturer"
+F 6 "ERJ-8ENF1021V" H 0   0   50  0001 C CNN "Part Number"
 	1    7700 5900
 	1    0    0    -1
@@
 F 2 "Resistor_SMD:R_1206_3216Metric" V 6980 2050 50  0001 C CNN
 F 3 "" H 7050 2050 50  0000 C CNN
+F 4 "P3.32KFCT-ND " H 0   0   50  0001 C CNN "Digikey"
+F 5 "Panasonic" H 0   0   50  0001 C CNN "Manufacturer"
+F 6 "ERJ-8ENF3321V " H 0   0   50  0001 C CNN "Part Number"
 	1    7050 2050
 	0    1    1    0
@@
 F 2 "Resistor_SMD:R_1206_3216Metric" V 7030 5150 50  0001 C CNN
 F 3 "" H 7100 5150 50  0000 C CNN
+F 4 "P3.32KFCT-ND " H 0   0   50  0001 C CNN "Digikey"
+F 5 "Panasonic" H 0   0   50  0001 C CNN "Manufacturer"
+F 6 "ERJ-8ENF3321V " H 0   0   50  0001 C CNN "Part Number"
 	1    7100 5150
 	0    1    1    0
@@
 F 2 "Resistor_SMD:R_1206_3216Metric" V 5930 3150 50  0001 C CNN
 F 3 "" H 6000 3150 50  0000 C CNN
+F 4 "P523FCT-ND" H 0   0   50  0001 C CNN "Digikey"
+F 5 "Panasonic" H 0   0   50  0001 C CNN "Manufacturer"
+F 6 "ERJ-8ENF5230V" H 0   0   50  0001 C CNN "Part Number"
 	1    6000 3150
 	1    0    0    -1
@@
 F 2 "Resistor_SMD:R_1206_3216Metric" V 5930 4050 50  0001 C CNN
 F 3 "" H 6000 4050 50  0000 C CNN
+F 4 "P523FCT-ND" H 0   0   50  0001 C CNN "Digikey"
+F 5 "Panasonic" H 0   0   50  0001 C CNN "Manufacturer"
+F 6 "ERJ-8ENF5230V" H 0   0   50  0001 C CNN "Part Number"
 	1    6000 4050
 	1    0    0    -1
@@
 F 2 "Resistor_SMD:R_1206_3216Metric" V 6580 5900 50  0001 C CNN
 F 3 "" H 6650 5900 50  0000 C CNN
+F 4 "P68.0KFCT-ND" H 0   0   50  0001 C CNN "Digikey"
+F 5 "Panasonic" H 0   0   50  0001 C CNN "Manufacturer"
+F 6 "ERJ-8ENF6802V" H 0   0   50  0001 C CNN "Part Number"
 	1    6650 5900
 	1    0    0    -1
@@
 F 2 "Resistor_SMD:R_1206_3216Metric" V 5380 2350 50  0001 C CNN
 F 3 "" H 5450 2350 50  0000 C CNN
+F 4 "P68.0FCT-ND " H 0   0   50  0001 C CNN "Digikey"
+F 5 "Panasonic" H 0   0   50  0001 C CNN "Manufacturer"
+F 6 "ERJ-8ENF68R0V " H 0   0   50  0001 C CNN "Part Number"
 	1    5450 2350
 	0    1    1    0
@@
 P 9550 5150
 F 0 "R318" H 9580 5170 50  0000 L CNN
-F 1 "R_Small" H 9580 5110 50  0000 L CNN
+F 1 "68k" H 9580 5110 50  0000 L CNN
 F 2 "Resistor_SMD:R_0603_1608Metric" H 9550 5150 50  0001 C CNN
 F 3 "" H 9550 5150 50  0000 C CNN
@@
 F 2 "Resistor_SMD:R_1206_3216Metric" V 4330 3550 50  0001 C CNN
 F 3 "" H 4400 3550 50  0000 C CNN
+F 4 "Panasonic" H 0   0   50  0001 C CNN "Manufacturer"
+F 5 "ERJ-8ENF1203V " H 0   0   50  0001 C CNN "Part Number"
+F 6 "P120KFCT-ND " H 0   0   50  0001 C CNN "Digikey"
 	1    4400 3550
 	1    0    0    -1
@@
 F 2 "Resistor_SMD:R_1206_3216Metric" V 4330 4050 50  0001 C CNN
 F 3 "" H 4400 4050 50  0000 C CNN
+F 4 "Panasonic" H 0   0   50  0001 C CNN "Manufacturer"
+F 5 "ERJ-8ENF1203V " H 0   0   50  0001 C CNN "Part Number"
+F 6 "P120KFCT-ND " H 0   0   50  0001 C CNN "Digikey"
 	1    4400 4050
 	1    0    0    -1
@@
 F 2 "Resistor_SMD:R_1206_3216Metric" V 4330 6200 50  0001 C CNN
 F 3 "" H 4400 6200 50  0000 C CNN
+F 4 "Panasonic" H 0   0   50  0001 C CNN "Manufacturer"
+F 5 "ERJ-8ENF1003V" H 0   0   50  0001 C CNN "Part Number"
+F 6 "P100KFCT-ND " H 0   0   50  0001 C CNN "Digikey"
 	1    4400 6200
 	1    0    0    -1
@@
 F 2 "Resistor_SMD:R_1206_3216Metric" V 1530 3650 50  0001 C CNN
 F 3 "" H 1600 3650 50  0000 C CNN
+F 4 "P2.00KFCT-ND " H 0   0   50  0001 C CNN "Digikey"
+F 5 "Panasonic" H 0   0   50  0001 C CNN "Manufacturer"
+F 6 "ERJ-8ENF2001V " H 0   0   50  0001 C CNN "Part Number"
 	1    1600 3650
 	0    1    1    0
@@
 F 2 "Resistor_SMD:R_1206_3216Metric" V 4780 1500 50  0001 C CNN
 F 3 "" H 4850 1500 50  0000 C CNN
+F 4 "Panasonic" H 0   0   50  0001 C CNN "Manufacturer"
+F 5 "ERJ-8ENF1003V" H 0   0   50  0001 C CNN "Part Number"
+F 6 "P100KFCT-ND " H 0   0   50  0001 C CNN "Digikey"
 	1    4850 1500
 	1    0    0    -1
@@
 P 2300 3100
 F 0 "R302" V 2380 3100 50  0000 C CNN
-F 1 "132k" V 2300 3100 50  0000 C CNN
+F 1 "130k" V 2300 3100 50  0000 C CNN
 F 2 "Resistor_SMD:R_1206_3216Metric" V 2230 3100 50  0001 C CNN
 F 3 "" H 2300 3100 50  0000 C CNN
+F 4 "P130KFCT-ND" H 0   0   50  0001 C CNN "Digikey"
+F 5 "Panasonic" H 0   0   50  0001 C CNN "Manufacturer"
+F 6 "ERJ-8ENF1303V " H 0   0   50  0001 C CNN "Part Number"
 	1    2300 3100
 	1    0    0    -1
@@
 P 2550 3800
 F 0 "U301" H 3641 3828 60  0000 L CNN
-F 1 "LTC6090" H 3641 3722 60  0000 L CNN
+F 1 "LTC6090-5" H 3641 3722 60  0000 L CNN
 F 2 "Package_SO:TI_SO-PowerPAD-8" H 2550 3800 60  0001 C CNN
 F 3 "" H 2550 3800 60  0001 C CNN
+F 4 "LTC6090CS8E-5#PBF-ND " H 0   0   50  0001 C CNN "Digikey"
+F 5 "Linear Technology" H 0   0   50  0001 C CNN "Manufacturer"
+F 6 "LTC6090CS8E-5#PBF" H 0   0   50  0001 C CNN "Part Number"
 	1    2550 3800
 	1    0    0    -1
@@
 F 2 "Package_SO:TI_SO-PowerPAD-8" H 3750 5750 60  0001 C CNN
 F 3 "" H 3750 5750 60  0001 C CNN
+F 4 "LTC6090CS8E#PBF-ND " H 0   0   50  0001 C CNN "Digikey"
+F 5 "Linear Technology" H 0   0   50  0001 C CNN "Manufacturer"
+F 6 "LTC6090CS8E#PBF" H 0   0   50  0001 C CNN "Part Number"
 	1    3750 5750
 	-1   0    0    -1
@@
 F 2 "Package_SO:TI_SO-PowerPAD-8" H 3750 1850 60  0001 C CNN
 F 3 "" H 3750 1850 60  0001 C CNN
+F 4 "LTC6090CS8E#PBF-ND " H 0   0   50  0001 C CNN "Digikey"
+F 5 "Linear Technology" H 0   0   50  0001 C CNN "Manufacturer"
+F 6 "LTC6090CS8E#PBF" H 0   0   50  0001 C CNN "Part Number"
 	1    3750 1850
 	-1   0    0    -1

Commit message: Some Updates from Testing
Parts:
- D301: value LED -> RED; Digikey (none) -> SML-D12V1WT86CT-ND; Manufacturer (none) -> Rohm; Part Number (none) -> SML-D12V1WT86
- K301: Digikey (none) -> PB353-ND; Manufacturer (none) -> TE Connectivity; Part Number (none) -> PE014005
- Q303, Q305: Digikey (none) -> MMBT5401-FDICT-ND
- R303: value R -> 2; Digikey (none) -> RL16R2.0FCT-ND; Manufacturer (none) -> Susumu; Part Number (none) -> RL1632R-2R00-F
- R318: Digikey (none) -> 311-68.0KHRCT-ND; Manufacturer (none) -> Yageo; Note (none) -> VH; Part Number (none) -> RC0603FR-0768KL
- W301, W302, W303, W304, W305: Note (none) -> NB
Changed lines of the file:
@@
 F 4 "Diodes" H 8000 4200 60  0001 C CNN "Manufacturer"
 F 5 "MMBT5401-7-F" H 8000 4200 60  0001 C CNN "Part Number"
+F 6 "MMBT5401-FDICT-ND" H 0   0   50  0001 C CNN "Digikey"
 	1    8000 4200
 	-1   0    0    1
@@
 F 4 "Diodes" H 7600 5150 60  0001 C CNN "Manufacturer"
 F 5 "MMBT5401-7-F" H 7600 5150 60  0001 C CNN "Part Number"
+F 6 "MMBT5401-FDICT-ND" H 0   0   50  0001 C CNN "Digikey"
 	1    7600 5150
 	1    0    0    1
@@
 F 2 "frontend_additional-footprints:PE014005" H 13300 5300 60  0001 C CNN
 F 3 "" H 13300 5300 60  0001 C CNN
+F 4 "PB353-ND" H 0   0   50  0001 C CNN "Digikey"
+F 5 "TE Connectivity" H 0   0   50  0001 C CNN "Manufacturer"
+F 6 "PE014005" H 0   0   50  0001 C CNN "Part Number"
 	1    9500 3700
 	0    -1   -1   0
@@
 F 2 "Resistor_SMD:R_0603_1608Metric" H 9550 5150 50  0001 C CNN
 F 3 "" H 9550 5150 50  0000 C CNN
+F 4 "311-68.0KHRCT-ND" H 0   0   50  0001 C CNN "Digikey"
+F 5 "Yageo" H 0   0   50  0001 C CNN "Manufacturer"
+F 6 "VH" H 0   0   50  0001 C CNN "Note"
+F 7 "RC0603FR-0768KL" H 0   0   50  0001 C CNN "Part Number"
 	1    9550 5150
 	1    0    0    -1
@@
 P 2450 7300
 F 0 "D301" H 2450 7400 50  0000 C CNN
-F 1 "LED" H 2450 7200 50  0000 C CNN
+F 1 "RED" H 2450 7200 50  0000 C CNN
 F 2 "LED_SMD:LED_0603_1608Metric" H 2450 7300 50  0001 C CNN
 F 3 "" H 2450 7300 50  0000 C CNN
+F 4 "SML-D12V1WT86CT-ND" H 0   0   50  0001 C CNN "Digikey"
+F 5 "Rohm" H 0   0   50  0001 C CNN "Manufacturer"
+F 6 "SML-D12V1WT86" H 0   0   50  0001 C CNN "Part Number"
 	1    2450 7300
 	-1   0    0    1
@@
 P 2900 7300
 F 0 "R303" V 2980 7300 50  0000 C CNN
-F 1 "R" V 2900 7300 50  0000 C CNN
+F 1 "2" V 2900 7300 50  0000 C CNN
 F 2 "Resistor_SMD:R_0603_1608Metric" V 2830 7300 50  0001 C CNN
 F 3 "" H 2900 7300 50  0000 C CNN
+F 4 "RL16R2.0FCT-ND" H 0   0   50  0001 C CNN "Digikey"
+F 5 "Susumu" H 0   0   50  0001 C CNN "Manufacturer"
+F 6 "RL1632R-2R00-F" H 0   0   50  0001 C CNN "Part Number"
 	1    2900 7300
 	0    1    1    0
@@
 F 2 "TestPoint:TestPoint_Pad_D1.0mm" H 5000 3650 50  0001 C CNN
 F 3 "" H 5000 3650 50  0000 C CNN
+F 4 "NB" H 0   0   50  0001 C CNN "Note"
 	1    4800 3650
 	1    0    0    -1
@@
 F 2 "TestPoint:TestPoint_Pad_D1.0mm" H 3000 2900 50  0001 C CNN
 F 3 "" H 3000 2900 50  0000 C CNN
+F 4 "NB" H 0   0   50  0001 C CNN "Note"
 	1    2800 2900
 	1    0    0    -1
@@
 F 2 "TestPoint:TestPoint_Pad_D1.0mm" H 1900 2900 50  0001 C CNN
 F 3 "" H 1900 2900 50  0000 C CNN
+F 4 "NB" H 0   0   50  0001 C CNN "Note"
 	1    1700 2900
 	1    0    0    -1
@@
 F 2 "TestPoint:TestPoint_Pad_D1.0mm" H 9050 3500 50  0001 C CNN
 F 3 "" H 9050 3500 50  0000 C CNN
+F 4 "NB" H 0   0   50  0001 C CNN "Note"
 	1    8850 3500
 	1    0    0    -1
@@
 F 2 "TestPoint:TestPoint_Pad_D1.0mm" H 6850 1950 50  0001 C CNN
 F 3 "" H 6850 1950 50  0000 C CNN
+F 4 "NB" H 0   0   50  0001 C CNN "Note"
 	1    6650 1950
 	1    0    0    -1
