File: components_predev/frontend/hardware/supplies.sch (KiCad schematic (older format))
At the start: 67 parts

Commit message: Finished Range Switching/Filters
Parts:
- gave numbers to parts that had none: 66

Commit message: Changed to KiCAD 5
Parts:
- C401, C402, C411, C418, C419, C423, C424, C426: symbol CP1_Small -> Device:CP1_Small
- C403, C404, C405, C406: footprint (none) -> Capacitors_SMD:C_0603; symbol C_Small -> Device:C_Small
- C407: footprint (none) -> Capacitors_SMD:C_0603; symbol CP1_Small -> Device:CP1_Small
- C408, C409, C410, C412, C413, C414, C415, C416, C417, C420, C421, C422, C425: symbol C_Small -> Device:C_Small
- D401, D402, D403, D404: symbol LED -> Device:LED
- D405, D407, D408: symbol D -> Device:D
- D406: symbol D_Zener -> Device:D_Zener
- L401: symbol Ferrite_Bead -> Device:Ferrite_Bead
- L402, L404: symbol L_Small -> Device:L_Small
- L403, L405: symbol L -> Device:L
- P401, P402, P403, P404: symbol CONN_01X02 -> Connector_Generic:Conn_01x02
- R401, R402, R403, R404, R405, R406, R407, R408, R409, R410, R411, R412, R413, R414, R415: footprint (none) -> Resistors_SMD:R_0603; symbol R_Small -> Device:R_Small
- U401, U403: symbol AOZ1284 -> frontend_additional_components:AOZ1284
- U402: symbol LT1617 -> frontend_additional_components:LT1617
- U404: symbol MIC39100 -> frontend_additional_components:MIC39100
- U405: symbol MC79M05 -> frontend_additional_components:MC79M05
- W401, W402, W403, W404: symbol TEST_1P -> Connector:Test_Point
Connections:
- wire segments 162 -> 221

Commit message: Footrpints and Parts Specification
Parts:
- C401, C402, C411, C418, C419, C423, C424, C426: footprint (none) -> Capacitor_SMD:CP_Elec_4x3; Digikey (none) -> 732-8430-1-ND; Manufacturer (none) -> Würth; Mouser (none) -> 710-865080440002; Part Number (none) -> 865080440002
- C403, C404, C405, C406: footprint Capacitors_SMD:C_0603 -> Capacitor_SMD:C_0603_1608Metric
- C408, C409, C410, C412, C413, C414, C415, C416, C417, C420, C421, C422, C425: footprint (none) -> Capacitor_SMD:C_0603_1608Metric
- D401, D402, D403, D404: footprint (none) -> LED_SMD:LED_0603_1608Metric
- D405, D407, D408: value D -> NSR0530HT1G; footprint (none) -> Diode_SMD:D_SOD-323; Digikey (none) -> NSR0530HT1GOSCT-ND; Manufacturer (none) -> OnSemi; Mouser (none) -> 863-NSR0530HT1G; Part Number (none) -> NSR0530HT1G
- D406: footprint (none) -> Diode_SMD:D_SOD-323; Digikey (none) -> 863-MM3Z4V7ST1G; Manufacturer (none) -> OnSemi; Mouser (none) -> MM3Z4V7ST1GOSCT-ND; Part Number (none) -> MM3Z4V7ST1G
- L401: footprint (none) -> Inductor_SMD:L_0603_1608Metric
- L402, L403, L404, L405: footprint (none) -> Inductor_SMD:L_Bourns-SRN6028
- P401, P402, P403, P404: footprint (none) -> Connector_PinHeader_2.54mm:PinHeader_1x02_P2.54mm_Vertical
- R401, R402, R403, R404, R405, R406, R407, R408, R409, R410, R411, R412, R413, R414, R415: footprint Resistors_SMD:R_0603 -> Resistor_SMD:R_0603_1608Metric
- U401, U403: footprint (none) -> Package_SO:TI_SO-PowerPAD-8
- U402: footprint (none) -> Package_TO_SOT_SMD:SOT-23-5
- U404: footprint (none) -> Package_TO_SOT_SMD:SOT-223
- U405: footprint (none) -> Package_TO_SOT_SMD:TO-252-2
- W401, W402, W403, W404: footprint (none) -> TestPoint:TestPoint_Pad_D1.0mm

Commit message: Finished Footprints, ERC
Parts:
- C407: footprint Capacitors_SMD:C_0603 -> Capacitor_SMD:CP_Elec_4x3
Connections:
- wire segments 221 -> 231
Changed lines of the file:
@@
 $Descr A4 11693 8268
 encoding utf-8
-Sheet 4 7
+Sheet 3 7
 Title "Power Supplies"
 Date "2018-07-09"
@@
 	4750 1050 4750 1350
 Wire Wire Line
-	4500 900  4500 1050
-Wire Wire Line
 	4750 1550 4750 1950
 Wire Wire Line
@@
 	1    0    0    -1
 $EndComp
-Connection ~ 4500 1050
 $Comp
 L Device:C_Small C408
@@
 F 0 "C407" H 2860 1570 50  0000 L CNN
 F 1 "CP1_Small" H 2860 1420 50  0000 L CNN
-F 2 "Capacitors_SMD:C_0603" H 2850 1500 50  0001 C CNN
+F 2 "Capacitor_SMD:CP_Elec_4x3" H 2850 1500 50  0001 C CNN
 F 3 "" H 2850 1500 50  0000 C CNN
 	1    2850 1500
@@
 Wire Wire Line
 	1200 2850 1450 2850
-Connection ~ 1450 2850
 $Comp
 L power:GND #PWR060
@@
 	6000 3700 6150 3700
 Wire Wire Line
-	6150 3100 6850 3100
+	6150 3100 6650 3100
 Wire Wire Line
 	4900 3500 4900 3550
@@
 	2150 3750 2400 3750
 Wire Wire Line
-	1450 2850 2550 2850
-Wire Wire Line
 	1200 3750 1200 3800
 Wire Wire Line
@@
 	5750 4500 6050 4500
 Wire Wire Line
-	6050 4500 6900 4500
+	6050 4500 6650 4500
 Wire Wire Line
 	8350 5100 8500 5100
@@
 Wire Wire Line
 	10150 1300 10200 1300
+Wire Wire Line
+	4500 1050 4500 900
+Connection ~ 4500 1050
+Wire Wire Line
+	2550 2850 1450 2850
+Connection ~ 1450 2850
+$Comp
+L power:PWR_FLAG #FLG0105
+U 1 1 5B7E0BD1
+P 6650 2950
+F 0 "#FLG0105" H 6650 3025 50  0001 C CNN
+F 1 "PWR_FLAG" H 6650 3124 50  0000 C CNN
+F 2 "" H 6650 2950 50  0001 C CNN
+F 3 "~" H 6650 2950 50  0001 C CNN
+	1    6650 2950
+	1    0    0    -1
+$EndComp
+Wire Wire Line
+	6650 2950 6650 3100
+Connection ~ 6650 3100
+Wire Wire Line
+	6650 3100 6850 3100
+$Comp
+L power:PWR_FLAG #FLG0101
+U 1 1 5B5CECF1
+P 6650 4300
+F 0 "#FLG0101" H 6650 4375 50  0001 C CNN
+F 1 "PWR_FLAG" H 6650 4474 50  0000 C CNN
+F 2 "" H 6650 4300 50  0001 C CNN
+F 3 "~" H 6650 4300 50  0001 C CNN
+	1    6650 4300
+	1    0    0    -1
+$EndComp
+Wire Wire Line
+	6650 4300 6650 4500
+Connection ~ 6650 4500
+Wire Wire Line
+	6650 4500 6900 4500
+$Comp
+L power:PWR_FLAG #FLG0301
+U 1 1 5B5DD5A7
+P 9950 1450
+F 0 "#FLG0301" H 9950 1525 50  0001 C CNN
+F 1 "PWR_FLAG" V 9950 1578 50  0000 L CNN
+F 2 "" H 9950 1450 50  0001 C CNN
+F 3 "~" H 9950 1450 50  0001 C CNN
+	1    9950 1450
+	0    1    1    0
+$EndComp
+$Comp
+L power:PWR_FLAG #FLG0302
+U 1 1 5B5DD824
+P 10000 3250
+F 0 "#FLG0302" H 10000 3325 50  0001 C CNN
+F 1 "PWR_FLAG" V 10000 3378 50  0000 L CNN
+F 2 "" H 10000 3250 50  0001 C CNN
+F 3 "~" H 10000 3250 50  0001 C CNN
+	1    10000 3250
+	0    1    1    0
+$EndComp
+$Comp
+L power:PWR_FLAG #FLG0303
+U 1 1 5B5DDA1B
+P 10000 4700
+F 0 "#FLG0303" H 10000 4775 50  0001 C CNN
+F 1 "PWR_FLAG" V 10000 4828 50  0000 L CNN
+F 2 "" H 10000 4700 50  0001 C CNN
+F 3 "~" H 10000 4700 50  0001 C CNN
+	1    10000 4700
+	0    1    1    0
+$EndComp
+Wire Wire Line
+	10000 4700 9900 4700
+Wire Wire Line
+	9900 4700 9900 4500
+Wire Wire Line
+	10000 3250 9900 3250
+Wire Wire Line
+	9900 3250 9900 3100
+Wire Wire Line
+	9950 1450 9900 1450
+Wire Wire Line
+	9900 1450 9900 1300
 $EndSCHEMATC

Commit message: Fixed minor net issues, begun routing
Changed lines of the file:
@@
 Connection ~ 2000 7150
-Wire Wire Line
-	1800 7150 1800 7250
-Connection ~ 1800 7150
 Wire Wire Line
 	1200 6850 1200 6650
@@
 	1200 2850 1200 3150
 Wire Wire Line
-	1600 7150 1800 7150
-Wire Wire Line
 	2000 7150 2400 7150
-Wire Wire Line
-	1800 7150 2000 7150
 Wire Wire Line
 	8350 3700 8500 3700
@@
 Wire Wire Line
 	9900 1450 9900 1300
+Wire Wire Line
+	1600 7150 1800 7150
+Wire Wire Line
+	1800 7250 1800 7150
+Connection ~ 1800 7150
+Wire Wire Line
+	1800 7150 2000 7150
 $EndSCHEMATC

Commit message: Begun routing
Parts:
- removed C401, C411: CP1_Small, Capacitor_SMD:CP_Elec_4x3, symbol Device:CP1_Small
Connections:
- wire segments 231 -> 227
Changed lines of the file:
@@
 Wire Wire Line
 	4750 1550 4750 1950
-Wire Wire Line
-	4500 1550 4500 1950
 $Comp
 L Device:C_Small C412
@@
 	1    0    0    -1
 $EndComp
-$Comp
-L Device:CP1_Small C411
-U 1 1 5B3A28A1
-P 4500 1450
-F 0 "C411" H 4510 1520 50  0000 L CNN
-F 1 "CP1_Small" H 4510 1370 50  0000 L CNN
-F 2 "Capacitor_SMD:CP_Elec_4x3" H 4500 1450 50  0001 C CNN
-F 3 "" H 4500 1450 50  0000 C CNN
-F 4 "732-8430-1-ND" H 0   0   50  0001 C CNN "Digikey"
-F 5 "Würth" H 0   0   50  0001 C CNN "Manufacturer"
-F 6 "710-865080440002" H 0   0   50  0001 C CNN "Mouser"
-F 7 "865080440002" H 0   0   50  0001 C CNN "Part Number"
-	1    4500 1450
-	1    0    0    -1
-$EndComp
 Wire Wire Line
 	4500 1050 4750 1050
@@
 Wire Wire Line
 	4750 1950 4500 1950
-Connection ~ 4500 1950
 $Comp
 L power:+12V #PWR054
@@
 Wire Wire Line
 	1450 3350 1450 3750
-Wire Wire Line
-	1200 3350 1200 3750
 $Comp
 L Device:C_Small C403
@@
 	1    0    0    -1
 $EndComp
-$Comp
-L Device:CP1_Small C401
-U 1 1 5B3A4EB8
-P 1200 3250
-F 0 "C401" H 1210 3320 50  0000 L CNN
-F 1 "CP1_Small" H 1210 3170 50  0000 L CNN
-F 2 "Capacitor_SMD:CP_Elec_4x3" H 1200 3250 50  0001 C CNN
-F 3 "" H 1200 3250 50  0000 C CNN
-F 4 "732-8430-1-ND" H 0   0   50  0001 C CNN "Digikey"
-F 5 "Würth" H 0   0   50  0001 C CNN "Manufacturer"
-F 6 "710-865080440002" H 0   0   50  0001 C CNN "Mouser"
-F 7 "865080440002" H 0   0   50  0001 C CNN "Part Number"
-	1    1200 3250
-	1    0    0    -1
-$EndComp
 Wire Wire Line
 	1200 2850 1450 2850
@@
 Wire Wire Line
 	1450 3750 1200 3750
-Connection ~ 1200 3750
 $Comp
 L power:+12V #PWR061
@@
 	1    0    0    -1
 $EndComp
-Connection ~ 1200 2850
 $Comp
 L Device:LED D401
@@
 	4500 1950 4500 2000
 Wire Wire Line
-	4500 1050 4500 1350
-Wire Wire Line
 	4250 3100 4500 3100
 Wire Wire Line
@@
 	1200 3750 1200 3800
 Wire Wire Line
-	1200 2850 1200 3150
-Wire Wire Line
 	2000 7150 2400 7150
 Wire Wire Line
@@
 Wire Wire Line
 	4500 1050 4500 900
-Connection ~ 4500 1050
 Wire Wire Line
 	2550 2850 1450 2850

Commit message: Finished routing, begun component specification
Parts:
- C402, C418, C419, C423, C424, C426: value CP1_Small -> 22u; Digikey 732-8430-1-ND -> 732-8413-1-ND; Mouser 710-865080440002 -> 710-865080340003; Part Number 865080440002 -> 865080340003; Voltage (none) -> 16 V
- C403, C404, C408, C412, C416, C417, C421, C422, C425: value C_Small -> 100n
- C407: value CP1_Small -> 22u; Digikey (none) -> 732-8413-1-ND; Manufacturer (none) -> Würth; Mouser (none) -> 710-865080340003; Part Number (none) -> 865080340003; Voltage (none) -> 16 V
Changed lines of the file:
@@
 P 8750 1600
 F 0 "C425" H 8760 1670 50  0000 L CNN
-F 1 "C_Small" H 8760 1520 50  0000 L CNN
+F 1 "100n" H 8760 1520 50  0000 L CNN
 F 2 "Capacitor_SMD:C_0603_1608Metric" H 8750 1600 50  0001 C CNN
 F 3 "" H 8750 1600 50  0000 C CNN
@@
 P 9050 1600
 F 0 "C426" H 9060 1670 50  0000 L CNN
-F 1 "CP1_Small" H 9060 1520 50  0000 L CNN
+F 1 "22u" H 9060 1520 50  0000 L CNN
 F 2 "Capacitor_SMD:CP_Elec_4x3" H 9050 1600 50  0001 C CNN
 F 3 "" H 9050 1600 50  0000 C CNN
-F 4 "732-8430-1-ND" H 0   0   50  0001 C CNN "Digikey"
+F 4 "732-8413-1-ND " H 0   0   50  0001 C CNN "Digikey"
 F 5 "Würth" H 0   0   50  0001 C CNN "Manufacturer"
-F 6 "710-865080440002" H 0   0   50  0001 C CNN "Mouser"
-F 7 "865080440002" H 0   0   50  0001 C CNN "Part Number"
+F 6 "710-865080340003 " H 0   0   50  0001 C CNN "Mouser"
+F 7 "865080340003 " H 0   0   50  0001 C CNN "Part Number"
+F 8 "16 V" H 0   0   50  0001 C CNN "Voltage"
 	1    9050 1600
 	1    0    0    -1
@@
 P 4750 1450
 F 0 "C412" H 4760 1520 50  0000 L CNN
-F 1 "C_Small" H 4760 1370 50  0000 L CNN
+F 1 "100n" H 4760 1370 50  0000 L CNN
 F 2 "Capacitor_SMD:C_0603_1608Metric" H 4750 1450 50  0001 C CNN
 F 3 "" H 4750 1450 50  0000 C CNN
@@
 P 3250 1500
 F 0 "C408" H 3260 1570 50  0000 L CNN
-F 1 "C_Small" H 3260 1420 50  0000 L CNN
+F 1 "100n" H 3260 1420 50  0000 L CNN
 F 2 "Capacitor_SMD:C_0603_1608Metric" H 3250 1500 50  0001 C CNN
 F 3 "" H 3250 1500 50  0000 C CNN
@@
 P 2850 1500
 F 0 "C407" H 2860 1570 50  0000 L CNN
-F 1 "CP1_Small" H 2860 1420 50  0000 L CNN
+F 1 "22u" H 2860 1420 50  0000 L CNN
 F 2 "Capacitor_SMD:CP_Elec_4x3" H 2850 1500 50  0001 C CNN
 F 3 "" H 2850 1500 50  0000 C CNN
+F 4 "732-8413-1-ND " H 0   0   50  0001 C CNN "Digikey"
+F 5 "Würth" H 0   0   50  0001 C CNN "Manufacturer"
+F 6 "710-865080340003 " H 0   0   50  0001 C CNN "Mouser"
+F 7 "865080340003 " H 0   0   50  0001 C CNN "Part Number"
+F 8 "16 V" H 0   0   50  0001 C CNN "Voltage"
 	1    2850 1500
 	1    0    0    -1
@@
 P 5850 3400
 F 0 "C417" H 5860 3470 50  0000 L CNN
-F 1 "C_Small" H 5860 3320 50  0000 L CNN
+F 1 "100n" H 5860 3320 50  0000 L CNN
 F 2 "Capacitor_SMD:C_0603_1608Metric" H 5850 3400 50  0001 C CNN
 F 3 "" H 5850 3400 50  0000 C CNN
@@
 P 6150 3400
 F 0 "C419" H 6160 3470 50  0000 L CNN
-F 1 "CP1_Small" H 6160 3320 50  0000 L CNN
+F 1 "22u" H 6160 3320 50  0000 L CNN
 F 2 "Capacitor_SMD:CP_Elec_4x3" H 6150 3400 50  0001 C CNN
 F 3 "" H 6150 3400 50  0000 C CNN
-F 4 "732-8430-1-ND" H 0   0   50  0001 C CNN "Digikey"
+F 4 "732-8413-1-ND " H 0   0   50  0001 C CNN "Digikey"
 F 5 "Würth" H 0   0   50  0001 C CNN "Manufacturer"
-F 6 "710-865080440002" H 0   0   50  0001 C CNN "Mouser"
-F 7 "865080440002" H 0   0   50  0001 C CNN "Part Number"
+F 6 "710-865080340003 " H 0   0   50  0001 C CNN "Mouser"
+F 7 "865080340003 " H 0   0   50  0001 C CNN "Part Number"
+F 8 "16 V" H 0   0   50  0001 C CNN "Voltage"
 	1    6150 3400
 	1    0    0    -1
@@
 P 1450 3250
 F 0 "C403" H 1460 3320 50  0000 L CNN
-F 1 "C_Small" H 1460 3170 50  0000 L CNN
+F 1 "100n" H 1460 3170 50  0000 L CNN
 F 2 "Capacitor_SMD:C_0603_1608Metric" H 1450 3250 50  0001 C CNN
 F 3 "" H 1450 3250 50  0000 C CNN
@@
 P 8200 3400
 F 0 "C421" H 8210 3470 50  0000 L CNN
-F 1 "C_Small" H 8210 3320 50  0000 L CNN
+F 1 "100n" H 8210 3320 50  0000 L CNN
 F 2 "Capacitor_SMD:C_0603_1608Metric" H 8200 3400 50  0001 C CNN
 F 3 "" H 8200 3400 50  0000 C CNN
@@
 P 8500 3400
 F 0 "C423" H 8510 3470 50  0000 L CNN
-F 1 "CP1_Small" H 8510 3320 50  0000 L CNN
+F 1 "22u" H 8510 3320 50  0000 L CNN
 F 2 "Capacitor_SMD:CP_Elec_4x3" H 8500 3400 50  0001 C CNN
 F 3 "" H 8500 3400 50  0000 C CNN
-F 4 "732-8430-1-ND" H 0   0   50  0001 C CNN "Digikey"
+F 4 "732-8413-1-ND " H 0   0   50  0001 C CNN "Digikey"
 F 5 "Würth" H 0   0   50  0001 C CNN "Manufacturer"
-F 6 "710-865080440002" H 0   0   50  0001 C CNN "Mouser"
-F 7 "865080440002" H 0   0   50  0001 C CNN "Part Number"
+F 6 "710-865080340003 " H 0   0   50  0001 C CNN "Mouser"
+F 7 "865080340003 " H 0   0   50  0001 C CNN "Part Number"
+F 8 "16 V" H 0   0   50  0001 C CNN "Voltage"
 	1    8500 3400
 	1    0    0    -1
@@
 P 1450 4900
 F 0 "C404" H 1460 4970 50  0000 L CNN
-F 1 "C_Small" H 1460 4820 50  0000 L CNN
+F 1 "100n" H 1460 4820 50  0000 L CNN
 F 2 "Capacitor_SMD:C_0603_1608Metric" H 1450 4900 50  0001 C CNN
 F 3 "" H 1450 4900 50  0000 C CNN
@@
 P 1200 4900
 F 0 "C402" H 1210 4970 50  0000 L CNN
-F 1 "CP1_Small" H 1210 4820 50  0000 L CNN
+F 1 "22u" H 1210 4820 50  0000 L CNN
 F 2 "Capacitor_SMD:CP_Elec_4x3" H 1200 4900 50  0001 C CNN
 F 3 "" H 1200 4900 50  0000 C CNN
-F 4 "732-8430-1-ND" H 0   0   50  0001 C CNN "Digikey"
+F 4 "732-8413-1-ND " H 0   0   50  0001 C CNN "Digikey"
 F 5 "Würth" H 0   0   50  0001 C CNN "Manufacturer"
-F 6 "710-865080440002" H 0   0   50  0001 C CNN "Mouser"
-F 7 "865080440002" H 0   0   50  0001 C CNN "Part Number"
+F 6 "710-865080340003 " H 0   0   50  0001 C CNN "Mouser"
+F 7 "865080340003 " H 0   0   50  0001 C CNN "Part Number"
+F 8 "16 V" H 0   0   50  0001 C CNN "Voltage"
 	1    1200 4900
 	1    0    0    -1
@@
 P 5750 4750
 F 0 "C416" H 5760 4820 50  0000 L CNN
-F 1 "C_Small" H 5760 4670 50  0000 L CNN
+F 1 "100n" H 5760 4670 50  0000 L CNN
 F 2 "Capacitor_SMD:C_0603_1608Metric" H 5750 4750 50  0001 C CNN
 F 3 "" H 5750 4750 50  0000 C CNN
@@
 P 6050 4750
 F 0 "C418" H 6060 4820 50  0000 L CNN
-F 1 "CP1_Small" H 6060 4670 50  0000 L CNN
+F 1 "22u" H 6060 4670 50  0000 L CNN
 F 2 "Capacitor_SMD:CP_Elec_4x3" H 6050 4750 50  0001 C CNN
 F 3 "" H 6050 4750 50  0000 C CNN
-F 4 "732-8430-1-ND" H 0   0   50  0001 C CNN "Digikey"
+F 4 "732-8413-1-ND " H 0   0   50  0001 C CNN "Digikey"
 F 5 "Würth" H 0   0   50  0001 C CNN "Manufacturer"
-F 6 "710-865080440002" H 0   0   50  0001 C CNN "Mouser"
-F 7 "865080440002" H 0   0   50  0001 C CNN "Part Number"
+F 6 "710-865080340003 " H 0   0   50  0001 C CNN "Mouser"
+F 7 "865080340003 " H 0   0   50  0001 C CNN "Part Number"
+F 8 "16 V" H 0   0   50  0001 C CNN "Voltage"
 	1    6050 4750
 	1    0    0    -1
@@
 U 1 1 5B3B1731
 P 8200 4800
-F 0 "C422" H 8210 4870 50  0000 L CNN
-F 1 "C_Small" H 8210 4720 50  0000 L CNN
+F 0 "C422" H 7950 4700 50  0000 L CNN
+F 1 "100n" H 7950 4900 50  0000 L CNN
 F 2 "Capacitor_SMD:C_0603_1608Metric" H 8200 4800 50  0001 C CNN
 F 3 "" H 8200 4800 50  0000 C CNN
@@
 U 1 1 5B3B1737
 P 8500 4800
-F 0 "C424" H 8510 4870 50  0000 L CNN
-F 1 "CP1_Small" H 8510 4720 50  0000 L CNN
+F 0 "C424" H 8250 4900 50  0000 L CNN
+F 1 "22u" H 8300 4700 50  0000 L CNN
 F 2 "Capacitor_SMD:CP_Elec_4x3" H 8500 4800 50  0001 C CNN
 F 3 "" H 8500 4800 50  0000 C CNN
-F 4 "732-8430-1-ND" H 0   0   50  0001 C CNN "Digikey"
+F 4 "732-8413-1-ND " H 0   0   50  0001 C CNN "Digikey"
 F 5 "Würth" H 0   0   50  0001 C CNN "Manufacturer"
-F 6 "710-865080440002" H 0   0   50  0001 C CNN "Mouser"
-F 7 "865080440002" H 0   0   50  0001 C CNN "Part Number"
+F 6 "710-865080340003 " H 0   0   50  0001 C CNN "Mouser"
+F 7 "865080340003 " H 0   0   50  0001 C CNN "Part Number"
+F 8 "16 V" H 0   0   50  0001 C CNN "Voltage"
 	1    8500 4800
 	-1   0    0    1
