File: components_predev/frontend/hardware/supplies.sch (KiCad schematic (older format))
At the start: 65 parts, among them P401 CONN_01X02, P402 CONN_01X02, P403 CONN_01X02, P404 CONN_01X02, U401 AOZ1284, U402 LT1617, U403 AOZ1284, U404 MIC39100, U405 MC79M05

Commit message: Some Updates from Testing
Parts:
- C403, C404, C408, C412, C416, C417, C421, C422, C425: Digikey (none) -> 1276-1005-1-ND; Manufacturer (none) -> Samsung; Note (none) -> VH; Part Number (none) -> CL10B104K08NNNC; Voltage (none) -> 16V
- C406, C415: value C_Small -> 4n7
- C410: value C_Small -> 4u7; Digikey (none) -> 1276-1784-1-ND; Manufacturer (none) -> Samsung; Part Number (none) -> CL10A475KO8NNNC; Voltage (none) -> 16 V
- D401, D402, D403, D404: value LED -> GREEN; Digikey (none) -> SML-D12M1WT86CT-ND; Manufacturer (none) -> Rohm; Part Number (none) -> SML-D12M1WT86
- D406: value D_Zener -> UDZ4V7B-7; Digikey 863-MM3Z4V7ST1G -> UDZ4V7B-7DICT-ND; Manufacturer OnSemi -> Diodes; Mouser MM3Z4V7ST1GOSCT-ND -> (none); Part Number MM3Z4V7ST1G -> UDZ4V7B-7
- L401: Digikey (none) -> 732-1591-1-ND; Manufacturer (none) -> Würth; Part Number (none) -> 742792609
- L402, L404: value L_Small -> 22u; Digikey (none) -> 587-2103-1-ND; Manufacturer (none) -> Taiyo Yuden; Part Number (none) -> NR6028T220M
- L403, L405: value L -> 330u; Digikey (none) -> 240-2744-1-ND; Manufacturer (none) -> Laird; Part Number (none) -> TYS6045331M-10
- P401, P402, P403, P404: Digikey (none) -> 952-2262-ND; Manufacturer (none) -> Harwin; Part Number (none) -> M20-9990246
- R401: value R_Small -> 990
- R402: value R_Small -> 120
- R404, R406: value R_Small -> 290
- R407: value R_Small -> 1k5
- R412: value R_Small -> 62k
- U401, U403: Digikey (none) -> 785-1689-1-ND; Manufacturer (none) -> Alpha & Omega; Part Number (none) -> AOZ1284PI
- U402: Digikey (none) -> LT1617ES5#TRMPBFCT-ND; Manufacturer (none) -> Linear Technology; Part Number (none) -> LT1617ES5#TRMPBF
- U404: Digikey (none) -> 576-1173-ND; Manufacturer (none) -> Microchip; Part Number (none) -> MIC39100-5.0WS
- U405: Digikey (none) -> MC79M05CDTRKGOSCT-ND; Manufacturer (none) -> OnSemi; Part Number (none) -> MC79M05CDTRKG
- W401, W402, W403, W404: Note (none) -> NB
Other:
- note added: "-6V"
- note added: "6V"
- note added: "all LEDs 10 mA each"
- note added: "f_sw = 746 kHz"
