File: components_predev/frontend/hardware/DAC.sch (KiCad schematic (older format))
At the start: 8 parts, among them U601 MAX5318

Commit message: Changed to KiCAD 5
Parts:
- JP601, JP602: symbol Jumper_NC_Dual -> Device:Jumper_NC_Dual
- R601, R602: footprint (none) -> Resistors_SMD:R_0603; symbol R_Small -> Device:R_Small
- RN601, RN602, RN603: symbol R_Pack04 -> Device:R_Pack04
- U601: symbol MAX5318 -> frontend_additional_components:MAX5318
Connections:
- wire segments 45 -> 50
Changed lines of the file:
@@
-EESchema Schematic File Version 2
-LIBS:power
-LIBS:device
-LIBS:transistors
-LIBS:conn
-LIBS:linear
-LIBS:regul
-LIBS:74xx
-LIBS:cmos4000
-LIBS:adc-dac
-LIBS:memory
-LIBS:xilinx
-LIBS:microcontrollers
-LIBS:dsp
-LIBS:microchip
-LIBS:analog_switches
-LIBS:motorola
-LIBS:texas
-LIBS:intel
-LIBS:audio
-LIBS:interface
-LIBS:digital-audio
-LIBS:philips
-LIBS:display
-LIBS:cypress
-LIBS:siliconi
-LIBS:opto
-LIBS:atmel
-LIBS:contrib
-LIBS:valves
-LIBS:frontend_additional_components
+EESchema Schematic File Version 4
 LIBS:frontend-cache
-EELAYER 25 0
+EELAYER 26 0
 EELAYER END
 $Descr A4 11693 8268
@@
 $EndDescr
 $Comp
-L MAX5318 U601
+L frontend_additional_components:MAX5318 U601
 U 1 1 5B296E71
 P 5150 3800
@@
 	6350 3400 7300 3400
 $Comp
-L GND #PWR0102
+L power:GND #PWR0103
 U 1 1 5B299996
 P 4900 4950
-F 0 "#PWR0102" H 4900 4700 50  0001 C CNN
+F 0 "#PWR0103" H 4900 4700 50  0001 C CNN
 F 1 "GND" H 4900 4800 50  0000 C CNN
 F 2 "" H 4900 4950 50  0000 C CNN
@@
 	4900 4950 4900 4750
 Wire Wire Line
-	3950 2950 3950 3300
+	3950 2950 3950 3100
 Wire Wire Line
 	3950 3300 4250 3300
@@
 ~BUSY
 $Comp
-L R_Small R602
+L Device:R_Small R602
 U 1 1 5B29C829
 P 3950 2850
 F 0 "R602" H 3980 2870 50  0000 L CNN
 F 1 "2k" H 3980 2810 50  0000 L CNN
-F 2 "" H 3950 2850 50  0000 C CNN
+F 2 "Resistors_SMD:R_0603" H 3950 2850 50  0001 C CNN
 F 3 "" H 3950 2850 50  0000 C CNN
 	1    3950 2850
@@
 	4900 2600 4900 2950
 Wire Wire Line
-	3100 2600 4900 2600
+	3100 2600 3350 2600
 Wire Wire Line
 	3950 2600 3950 2750
 Connection ~ 3950 3100
 $Comp
-L Jumper_NC_Dual JP602
+L Device:Jumper_NC_Dual JP602
 U 1 1 5B29C8D3
 P 2850 2600
 F 0 "JP602" H 2900 2500 50  0000 L CNN
 F 1 "Jumper_NC_Dual" H 2850 2700 50  0000 C BNN
-F 2 "" H 2850 2600 50  0000 C CNN
+F 2 "" H 2850 2600 50  0001 C CNN
 F 3 "" H 2850 2600 50  0000 C CNN
 	1    2850 2600
@@
 	2850 3200 2850 2700
 $Comp
-L GND #PWR0103
+L power:GND #PWR0104
 U 1 1 5B29C959
 P 2500 2800
-F 0 "#PWR0103" H 2500 2550 50  0001 C CNN
+F 0 "#PWR0104" H 2500 2550 50  0001 C CNN
 F 1 "GND" H 2500 2650 50  0000 C CNN
 F 2 "" H 2500 2800 50  0000 C CNN
@@
 $EndComp
 $Comp
-L Jumper_NC_Dual JP601
+L Device:Jumper_NC_Dual JP601
 U 1 1 5B29C9AC
 P 2850 2150
 F 0 "JP601" H 2900 2050 50  0000 L CNN
 F 1 "Jumper_NC_Dual" H 2850 2250 50  0000 C BNN
-F 2 "" H 2850 2150 50  0000 C CNN
+F 2 "" H 2850 2150 50  0001 C CNN
 F 3 "" H 2850 2150 50  0000 C CNN
 	1    2850 2150
@@
 Connection ~ 3350 2600
 Wire Wire Line
-	2500 2150 2500 2800
+	2500 2150 2500 2600
 Wire Wire Line
 	2500 2600 2600 2600
@@
 DOUT
 $Comp
-L R_Small R601
+L Device:R_Small R601
 U 1 1 5B29D046
 P 2100 2700
 F 0 "R601" H 2130 2720 50  0000 L CNN
 F 1 "R_Small" H 2130 2660 50  0000 L CNN
-F 2 "" H 2100 2700 50  0000 C CNN
+F 2 "Resistors_SMD:R_0603" H 2100 2700 50  0001 C CNN
 F 3 "" H 2100 2700 50  0000 C CNN
 	1    2100 2700
@@
 output
 $Comp
-L R_Pack04 RN602
+L Device:R_Pack04 RN602
 U 1 1 5B2A27DD
 P 3350 3300
@@
 $EndComp
 $Comp
-L R_Pack04 RN603
+L Device:R_Pack04 RN603
 U 1 1 5B2A2862
 P 3350 4300
@@
 $EndComp
 $Comp
-L R_Pack04 RN601
+L Device:R_Pack04 RN601
 U 1 1 5B2A28B9
 P 2900 3800
@@
 $EndComp
 Wire Wire Line
-	2000 3700 2700 3700
+	2000 3700 2100 3700
 Wire Wire Line
 	2700 3800 2000 3800
@@
 	2100 2800 2100 3700
 Connection ~ 2100 3700
+Wire Wire Line
+	3950 3100 3950 3300
+Wire Wire Line
+	3950 2600 4900 2600
+Wire Wire Line
+	3350 2600 3950 2600
+Wire Wire Line
+	2500 2600 2500 2800
+Wire Wire Line
+	2100 3700 2700 3700
 $EndSCHEMATC

Commit message: Footrpints and Parts Specification
Parts:
- JP601, JP602: footprint (none) -> Jumper:SolderJumper-3_P1.3mm_Open_RoundedPad1.0x1.5mm
- R601, R602: footprint Resistors_SMD:R_0603 -> Resistor_SMD:R_0603_1608Metric
- RN601, RN602, RN603: value R_Pack04 -> 22; footprint (none) -> Resistor_SMD:R_Array_Convex_4x0402; Digikey (none) -> Y10220CT-ND; Manufacturer (none) -> Panasonic; Mouser (none) -> 667-EXB-N8V220JX; Part Number (none) -> EXB-N8V220JX
- U601: footprint (none) -> Package_SO:TSSOP-24_4.4x7.8mm_P0.65mm
Changed lines of the file:
@@
 F 0 "U601" H 5950 4550 60  0000 C CNN
 F 1 "MAX5318" H 5300 3800 60  0000 C CNN
-F 2 "" H 5150 3800 60  0001 C CNN
+F 2 "Package_SO:TSSOP-24_4.4x7.8mm_P0.65mm" H 5150 3800 60  0001 C CNN
 F 3 "" H 5150 3800 60  0001 C CNN
 	1    5150 3800
@@
 F 0 "R602" H 3980 2870 50  0000 L CNN
 F 1 "2k" H 3980 2810 50  0000 L CNN
-F 2 "Resistors_SMD:R_0603" H 3950 2850 50  0001 C CNN
+F 2 "Resistor_SMD:R_0603_1608Metric" H 3950 2850 50  0001 C CNN
 F 3 "" H 3950 2850 50  0000 C CNN
 	1    3950 2850
@@
 F 0 "JP602" H 2900 2500 50  0000 L CNN
 F 1 "Jumper_NC_Dual" H 2850 2700 50  0000 C BNN
-F 2 "" H 2850 2600 50  0001 C CNN
+F 2 "Jumper:SolderJumper-3_P1.3mm_Open_RoundedPad1.0x1.5mm" H 2850 2600 50  0001 C CNN
 F 3 "" H 2850 2600 50  0000 C CNN
 	1    2850 2600
@@
 F 0 "JP601" H 2900 2050 50  0000 L CNN
 F 1 "Jumper_NC_Dual" H 2850 2250 50  0000 C BNN
-F 2 "" H 2850 2150 50  0001 C CNN
+F 2 "Jumper:SolderJumper-3_P1.3mm_Open_RoundedPad1.0x1.5mm" H 2850 2150 50  0001 C CNN
 F 3 "" H 2850 2150 50  0000 C CNN
 	1    2850 2150
@@
 F 0 "R601" H 2130 2720 50  0000 L CNN
 F 1 "R_Small" H 2130 2660 50  0000 L CNN
-F 2 "Resistors_SMD:R_0603" H 2100 2700 50  0001 C CNN
+F 2 "Resistor_SMD:R_0603_1608Metric" H 2100 2700 50  0001 C CNN
 F 3 "" H 2100 2700 50  0000 C CNN
 	1    2100 2700
@@
 P 3350 3300
 F 0 "RN602" V 3050 3300 50  0000 C CNN
-F 1 "R_Pack04" V 3550 3300 50  0000 C CNN
-F 2 "" V 3625 3300 50  0001 C CNN
+F 1 "22" V 3550 3300 50  0000 C CNN
+F 2 "Resistor_SMD:R_Array_Convex_4x0402" V 3625 3300 50  0001 C CNN
 F 3 "" H 3350 3300 50  0000 C CNN
+F 4 "Y10220CT-ND " H 0   0   50  0001 C CNN "Digikey"
+F 5 "Panasonic" H 0   0   50  0001 C CNN "Manufacturer"
+F 6 "667-EXB-N8V220JX " H 0   0   50  0001 C CNN "Mouser"
+F 7 "EXB-N8V220JX " H 0   0   50  0001 C CNN "Part Number"
 	1    3350 3300
 	0    1    1    0
@@
 P 3350 4300
 F 0 "RN603" V 3050 4300 50  0000 C CNN
-F 1 "R_Pack04" V 3550 4300 50  0000 C CNN
-F 2 "" V 3625 4300 50  0001 C CNN
+F 1 "22" V 3550 4300 50  0000 C CNN
+F 2 "Resistor_SMD:R_Array_Convex_4x0402" V 3625 4300 50  0001 C CNN
 F 3 "" H 3350 4300 50  0000 C CNN
+F 4 "Y10220CT-ND " H 0   0   50  0001 C CNN "Digikey"
+F 5 "Panasonic" H 0   0   50  0001 C CNN "Manufacturer"
+F 6 "667-EXB-N8V220JX " H 0   0   50  0001 C CNN "Mouser"
+F 7 "EXB-N8V220JX " H 0   0   50  0001 C CNN "Part Number"
 	1    3350 4300
 	0    1    1    0
@@
 P 2900 3800
 F 0 "RN601" V 2600 3800 50  0000 C CNN
-F 1 "R_Pack04" V 3100 3800 50  0000 C CNN
-F 2 "" V 3175 3800 50  0001 C CNN
+F 1 "22" V 3100 3800 50  0000 C CNN
+F 2 "Resistor_SMD:R_Array_Convex_4x0402" V 3175 3800 50  0001 C CNN
 F 3 "" H 2900 3800 50  0000 C CNN
+F 4 "Y10220CT-ND " H 0   0   50  0001 C CNN "Digikey"
+F 5 "Panasonic" H 0   0   50  0001 C CNN "Manufacturer"
+F 6 "667-EXB-N8V220JX " H 0   0   50  0001 C CNN "Mouser"
+F 7 "EXB-N8V220JX " H 0   0   50  0001 C CNN "Part Number"
 	1    2900 3800
 	0    1    1    0

Commit message: Finished Footprints, ERC
Parts:
- added C601, C602, C603, C604, C605, C606, C607, C608: C_Small, Capacitor_SMD:C_0603_1608Metric, symbol Device:C_Small
- added J601: Conn_01x03, Connector_PinHeader_2.54mm:PinHeader_1x03_P2.54mm_Vertical, symbol Connector_Generic:Conn_01x03
Connections:
- net labels added: +3.3V, +5V
- wire segments 50 -> 102
- no-connect marks 2 -> 3

Commit message: Begun routing
Parts:
- removed RN601, RN602, RN603: 22, Resistor_SMD:R_Array_Convex_4x0402, symbol Device:R_Pack04
- added R517, R518, R519, R520, R521, R522, R523, R524, R525, R526, R527: R_Small, Resistor_SMD:R_0603_1608Metric, symbol Device:R_Small
Connections:
- no-connect marks 3 -> 1
Changed lines of the file:
@@
 $Descr A4 11693 8268
 encoding utf-8
-Sheet 6 7
+Sheet 5 7
 Title "Digital-Analog Converter"
 Date ""
@@
 Wire Wire Line
 	3750 3800 4150 3800
-NoConn ~ 3300 4300
-NoConn ~ 2900 4300
 Text HLabel 2200 3800 0    60   BiDi ~ 0
 ~BUSY
@@
 Text HLabel 8700 4850 2    60   Output ~ 0
 output
-$Comp
-L Device:R_Pack04 RN602
-U 1 1 5B2A27DD
-P 3550 4000
-F 0 "RN602" V 3250 4000 50  0000 C CNN
-F 1 "22" V 3750 4000 50  0000 C CNN
-F 2 "Resistor_SMD:R_Array_Convex_4x0402" V 3825 4000 50  0001 C CNN
-F 3 "" H 3550 4000 50  0000 C CNN
-F 4 "Y10220CT-ND " H 200 700 50  0001 C CNN "Digikey"
-F 5 "Panasonic" H 200 700 50  0001 C CNN "Manufacturer"
-F 6 "667-EXB-N8V220JX " H 200 700 50  0001 C CNN "Mouser"
-F 7 "EXB-N8V220JX " H 200 700 50  0001 C CNN "Part Number"
-	1    3550 4000
-	0    1    1    0
-$EndComp
-$Comp
-L Device:R_Pack04 RN603
-U 1 1 5B2A2862
-P 3550 5000
-F 0 "RN603" V 3250 5000 50  0000 C CNN
-F 1 "22" V 3750 5000 50  0000 C CNN
-F 2 "Resistor_SMD:R_Array_Convex_4x0402" V 3825 5000 50  0001 C CNN
-F 3 "" H 3550 5000 50  0000 C CNN
-F 4 "Y10220CT-ND " H 200 700 50  0001 C CNN "Digikey"
-F 5 "Panasonic" H 200 700 50  0001 C CNN "Manufacturer"
-F 6 "667-EXB-N8V220JX " H 200 700 50  0001 C CNN "Mouser"
-F 7 "EXB-N8V220JX " H 200 700 50  0001 C CNN "Part Number"
-	1    3550 5000
-	0    1    1    0
-$EndComp
-$Comp
-L Device:R_Pack04 RN601
-U 1 1 5B2A28B9
-P 3100 4500
-F 0 "RN601" V 2800 4500 50  0000 C CNN
-F 1 "22" V 3300 4500 50  0000 C CNN
-F 2 "Resistor_SMD:R_Array_Convex_4x0402" V 3375 4500 50  0001 C CNN
-F 3 "" H 3100 4500 50  0000 C CNN
-F 4 "Y10220CT-ND " H 200 700 50  0001 C CNN "Digikey"
-F 5 "Panasonic" H 200 700 50  0001 C CNN "Manufacturer"
-F 6 "667-EXB-N8V220JX " H 200 700 50  0001 C CNN "Mouser"
-F 7 "EXB-N8V220JX " H 200 700 50  0001 C CNN "Part Number"
-	1    3100 4500
-	0    1    1    0
-$EndComp
 Wire Wire Line
 	2200 4400 2300 4400
-Wire Wire Line
-	2900 4500 2200 4500
-Wire Wire Line
-	2200 4600 2900 4600
-Wire Wire Line
-	2200 3800 3350 3800
-Wire Wire Line
-	3350 3900 3050 3900
-Wire Wire Line
-	3350 4000 2500 4000
-Wire Wire Line
-	3350 4100 2200 4100
-Wire Wire Line
-	3350 5100 2200 5100
-Wire Wire Line
-	2200 5000 3350 5000
-Wire Wire Line
-	3350 4900 2200 4900
-Wire Wire Line
-	2200 4800 3350 4800
 Wire Wire Line
 	2300 3500 2300 4400
@@
 Wire Wire Line
 	2700 3300 2700 3500
-Wire Wire Line
-	2300 4400 2900 4400
 $Comp
 L power:GND #PWR0138
@@
 	6800 4500 8300 4500
 NoConn ~ 6550 4900
+$Comp
+L Device:R_Small R520
+U 1 1 5B632256
+P 3650 3800
+F 0 "R520" V 3454 3800 50  0000 C CNN
+F 1 "R_Small" V 3545 3800 50  0000 C CNN
+F 2 "Resistor_SMD:R_0603_1608Metric" H 3650 3800 50  0001 C CNN
+F 3 "~" H 3650 3800 50  0001 C CNN
+	1    3650 3800
+	0    1    1    0
+$EndComp
+$Comp
+L Device:R_Small R521
+U 1 1 5B6322DF
+P 3650 3900
+F 0 "R521" V 3454 3900 50  0000 C CNN
+F 1 "R_Small" V 3545 3900 50  0000 C CNN
+F 2 "Resistor_SMD:R_0603_1608Metric" H 3650 3900 50  0001 C CNN
+F 3 "~" H 3650 3900 50  0001 C CNN
+	1    3650 3900
+	0    1    1    0
+$EndComp
+$Comp
+L Device:R_Small R522
+U 1 1 5B63234C
+P 3650 4000
+F 0 "R522" V 3454 4000 50  0000 C CNN
+F 1 "R_Small" V 3545 4000 50  0000 C CNN
+F 2 "Resistor_SMD:R_0603_1608Metric" H 3650 4000 50  0001 C CNN
+F 3 "~" H 3650 4000 50  0001 C CNN
+	1    3650 4000
+	0    1    1    0
+$EndComp
+$Comp
+L Device:R_Small R523
+U 1 1 5B6323BD
+P 3650 4100
+F 0 "R523" V 3454 4100 50  0000 C CNN
+F 1 "R_Small" V 3545 4100 50  0000 C CNN
+F 2 "Resistor_SMD:R_0603_1608Metric" H 3650 4100 50  0001 C CNN
+F 3 "~" H 3650 4100 50  0001 C CNN
+	1    3650 4100
+	0    1    1    0
+$EndComp
+$Comp
+L Device:R_Small R517
+U 1 1 5B632432
+P 3200 4400
+F 0 "R517" V 3004 4400 50  0000 C CNN
+F 1 "R_Small" V 3095 4400 50  0000 C CNN
+F 2 "Resistor_SMD:R_0603_1608Metric" H 3200 4400 50  0001 C CNN
+F 3 "~" H 3200 4400 50  0001 C CNN
+	1    3200 4400
+	0    1    1    0
+$EndComp
+$Comp
+L Device:R_Small R518
+U 1 1 5B6324AD
+P 3200 4500
+F 0 "R518" V 3004 4500 50  0000 C CNN
+F 1 "R_Small" V 3095 4500 50  0000 C CNN
+F 2 "Resistor_SMD:R_0603_1608Metric" H 3200 4500 50  0001 C CNN
+F 3 "~" H 3200 4500 50  0001 C CNN
+	1    3200 4500
+	0    1    1    0
+$EndComp
+$Comp
+L Device:R_Small R519
+U 1 1 5B63252A
+P 3200 4600
+F 0 "R519" V 3004 4600 50  0000 C CNN
+F 1 "R_Small" V 3095 4600 50  0000 C CNN
+F 2 "Resistor_SMD:R_0603_1608Metric" H 3200 4600 50  0001 C CNN
+F 3 "~" H 3200 4600 50  0001 C CNN
+	1    3200 4600
+	0    1    1    0
+$EndComp
+$Comp
+L Device:R_Small R524
+U 1 1 5B6325AB
+P 3650 4800
+F 0 "R524" V 3454 4800 50  0000 C CNN
+F 1 "R_Small" V 3545 4800 50  0000 C CNN
+F 2 "Resistor_SMD:R_0603_1608Metric" H 3650 4800 50  0001 C CNN
+F 3 "~" H 3650 4800 50  0001 C CNN
+	1    3650 4800
+	0    1    1    0
+$EndComp
+$Comp
+L Device:R_Small R525
+U 1 1 5B632630
+P 3650 4900
+F 0 "R525" V 3454 4900 50  0000 C CNN
+F 1 "R_Small" V 3545 4900 50  0000 C CNN
+F 2 "Resistor_SMD:R_0603_1608Metric" H 3650 4900 50  0001 C CNN
+F 3 "~" H 3650 4900 50  0001 C CNN
+	1    3650 4900
+	0    1    1    0
+$EndComp
+$Comp
+L Device:R_Small R526
+U 1 1 5B6326B9
+P 3650 5000
+F 0 "R526" V 3454 5000 50  0000 C CNN
+F 1 "R_Small" V 3545 5000 50  0000 C CNN
+F 2 "Resistor_SMD:R_0603_1608Metric" H 3650 5000 50  0001 C CNN
+F 3 "~" H 3650 5000 50  0001 C CNN
+	1    3650 5000
+	0    1    1    0
+$EndComp
+$Comp
+L Device:R_Small R527
+U 1 1 5B632746
+P 3650 5100
+F 0 "R527" V 3454 5100 50  0000 C CNN
+F 1 "R_Small" V 3545 5100 50  0000 C CNN
+F 2 "Resistor_SMD:R_0603_1608Metric" H 3650 5100 50  0001 C CNN
+F 3 "~" H 3650 5100 50  0001 C CNN
+	1    3650 5100
+	0    1    1    0
+$EndComp
+Wire Wire Line
+	2200 5100 3550 5100
+Wire Wire Line
+	2200 5000 3550 5000
+Wire Wire Line
+	2200 4800 3550 4800
+Wire Wire Line
+	2200 4600 3100 4600
+Wire Wire Line
+	2200 4500 3100 4500
+Wire Wire Line
+	2300 4400 3100 4400
+Wire Wire Line
+	2200 4100 3550 4100
+Wire Wire Line
+	2500 4000 3550 4000
+Wire Wire Line
+	3050 3900 3550 3900
+Wire Wire Line
+	2200 3800 3550 3800
+Wire Wire Line
+	2200 4900 3550 4900
 $EndSCHEMATC

Commit message: Finished routing, begun component specification
Parts:
- C601, C603, C605: value C_Small -> 10u
- C602, C604, C606, C608: value C_Small -> 100n
- C607: value C_Small -> 22u
- R517, R518, R519, R520, R521, R522, R523, R524, R525, R526, R527: value R_Small -> 22
- R601: value R_Small -> 2k
Changed lines of the file:
@@
 P 2300 3400
 F 0 "R601" H 2330 3420 50  0000 L CNN
-F 1 "R_Small" H 2330 3360 50  0000 L CNN
+F 1 "2k" H 2330 3360 50  0000 L CNN
 F 2 "Resistor_SMD:R_0603_1608Metric" H 2300 3400 50  0001 C CNN
 F 3 "" H 2300 3400 50  0000 C CNN
@@
 P 4800 2950
 F 0 "C602" V 4571 2950 50  0000 C CNN
-F 1 "C_Small" V 4662 2950 50  0000 C CNN
+F 1 "100n" V 4662 2950 50  0000 C CNN
 F 2 "Capacitor_SMD:C_0603_1608Metric" H 4800 2950 50  0001 C CNN
 F 3 "~" H 4800 2950 50  0001 C CNN
@@
 P 4800 2600
 F 0 "C601" V 4571 2600 50  0000 C CNN
-F 1 "C_Small" V 4662 2600 50  0000 C CNN
+F 1 "10u" V 4662 2600 50  0000 C CNN
 F 2 "Capacitor_SMD:C_0603_1608Metric" H 4800 2600 50  0001 C CNN
 F 3 "~" H 4800 2600 50  0001 C CNN
@@
 P 6350 3550
 F 0 "C608" V 6121 3550 50  0000 C CNN
-F 1 "C_Small" V 6212 3550 50  0000 C CNN
+F 1 "100n" V 6212 3550 50  0000 C CNN
 F 2 "Capacitor_SMD:C_0603_1608Metric" H 6350 3550 50  0001 C CNN
 F 3 "~" H 6350 3550 50  0001 C CNN
@@
 P 6350 3200
 F 0 "C607" V 6121 3200 50  0000 C CNN
-F 1 "C_Small" V 6212 3200 50  0000 C CNN
+F 1 "22u" V 6212 3200 50  0000 C CNN
 F 2 "Capacitor_SMD:C_0603_1608Metric" H 6350 3200 50  0001 C CNN
 F 3 "~" H 6350 3200 50  0001 C CNN
@@
 P 6350 2800
 F 0 "C606" V 6121 2800 50  0000 C CNN
-F 1 "C_Small" V 6212 2800 50  0000 C CNN
+F 1 "100n" V 6212 2800 50  0000 C CNN
 F 2 "Capacitor_SMD:C_0603_1608Metric" H 6350 2800 50  0001 C CNN
 F 3 "~" H 6350 2800 50  0001 C CNN
@@
 P 6350 2450
 F 0 "C605" V 6121 2450 50  0000 C CNN
-F 1 "C_Small" V 6212 2450 50  0000 C CNN
+F 1 "10u" V 6212 2450 50  0000 C CNN
 F 2 "Capacitor_SMD:C_0603_1608Metric" H 6350 2450 50  0001 C CNN
 F 3 "~" H 6350 2450 50  0001 C CNN
@@
 P 6350 2150
 F 0 "C604" V 6121 2150 50  0000 C CNN
-F 1 "C_Small" V 6212 2150 50  0000 C CNN
+F 1 "100n" V 6212 2150 50  0000 C CNN
 F 2 "Capacitor_SMD:C_0603_1608Metric" H 6350 2150 50  0001 C CNN
 F 3 "~" H 6350 2150 50  0001 C CNN
@@
 P 6350 1800
 F 0 "C603" V 6121 1800 50  0000 C CNN
-F 1 "C_Small" V 6212 1800 50  0000 C CNN
+F 1 "10u" V 6212 1800 50  0000 C CNN
 F 2 "Capacitor_SMD:C_0603_1608Metric" H 6350 1800 50  0001 C CNN
 F 3 "~" H 6350 1800 50  0001 C CNN
@@
 U 1 1 5B632256
 P 3650 3800
-F 0 "R520" V 3454 3800 50  0000 C CNN
-F 1 "R_Small" V 3545 3800 50  0000 C CNN
+F 0 "R520" V 3700 4000 50  0000 C CNN
+F 1 "22" V 3650 3800 50  0000 C CNN
 F 2 "Resistor_SMD:R_0603_1608Metric" H 3650 3800 50  0001 C CNN
 F 3 "~" H 3650 3800 50  0001 C CNN
@@
 U 1 1 5B6322DF
 P 3650 3900
-F 0 "R521" V 3454 3900 50  0000 C CNN
-F 1 "R_Small" V 3545 3900 50  0000 C CNN
+F 0 "R521" V 3700 4100 50  0000 C CNN
+F 1 "22" V 3650 3900 50  0000 C CNN
 F 2 "Resistor_SMD:R_0603_1608Metric" H 3650 3900 50  0001 C CNN
 F 3 "~" H 3650 3900 50  0001 C CNN
@@
 U 1 1 5B63234C
 P 3650 4000
-F 0 "R522" V 3454 4000 50  0000 C CNN
-F 1 "R_Small" V 3545 4000 50  0000 C CNN
+F 0 "R522" V 3700 4200 50  0000 C CNN
+F 1 "22" V 3650 4000 50  0000 C CNN
 F 2 "Resistor_SMD:R_0603_1608Metric" H 3650 4000 50  0001 C CNN
 F 3 "~" H 3650 4000 50  0001 C CNN
@@
 U 1 1 5B6323BD
 P 3650 4100
-F 0 "R523" V 3454 4100 50  0000 C CNN
-F 1 "R_Small" V 3545 4100 50  0000 C CNN
+F 0 "R523" V 3700 4300 50  0000 C CNN
+F 1 "22" V 3650 4100 50  0000 C CNN
 F 2 "Resistor_SMD:R_0603_1608Metric" H 3650 4100 50  0001 C CNN
 F 3 "~" H 3650 4100 50  0001 C CNN
@@
 U 1 1 5B632432
 P 3200 4400
-F 0 "R517" V 3004 4400 50  0000 C CNN
-F 1 "R_Small" V 3095 4400 50  0000 C CNN
+F 0 "R517" V 3250 4600 50  0000 C CNN
+F 1 "22" V 3200 4400 50  0000 C CNN
 F 2 "Resistor_SMD:R_0603_1608Metric" H 3200 4400 50  0001 C CNN
 F 3 "~" H 3200 4400 50  0001 C CNN
@@
 U 1 1 5B6324AD
 P 3200 4500
-F 0 "R518" V 3004 4500 50  0000 C CNN
-F 1 "R_Small" V 3095 4500 50  0000 C CNN
+F 0 "R518" V 3250 4700 50  0000 C CNN
+F 1 "22" V 3200 4500 50  0000 C CNN
 F 2 "Resistor_SMD:R_0603_1608Metric" H 3200 4500 50  0001 C CNN
 F 3 "~" H 3200 4500 50  0001 C CNN
@@
 U 1 1 5B63252A
 P 3200 4600
-F 0 "R519" V 3004 4600 50  0000 C CNN
-F 1 "R_Small" V 3095 4600 50  0000 C CNN
+F 0 "R519" V 3250 4800 50  0000 C CNN
+F 1 "22" V 3200 4600 50  0000 C CNN
 F 2 "Resistor_SMD:R_0603_1608Metric" H 3200 4600 50  0001 C CNN
 F 3 "~" H 3200 4600 50  0001 C CNN
@@
 U 1 1 5B6325AB
 P 3650 4800
-F 0 "R524" V 3454 4800 50  0000 C CNN
-F 1 "R_Small" V 3545 4800 50  0000 C CNN
+F 0 "R524" V 3700 5000 50  0000 C CNN
+F 1 "22" V 3650 4800 50  0000 C CNN
 F 2 "Resistor_SMD:R_0603_1608Metric" H 3650 4800 50  0001 C CNN
 F 3 "~" H 3650 4800 50  0001 C CNN
@@
 U 1 1 5B632630
 P 3650 4900
-F 0 "R525" V 3454 4900 50  0000 C CNN
-F 1 "R_Small" V 3545 4900 50  0000 C CNN
+F 0 "R525" V 3700 5100 50  0000 C CNN
+F 1 "22" V 3650 4900 50  0000 C CNN
 F 2 "Resistor_SMD:R_0603_1608Metric" H 3650 4900 50  0001 C CNN
 F 3 "~" H 3650 4900 50  0001 C CNN
@@
 U 1 1 5B6326B9
 P 3650 5000
-F 0 "R526" V 3454 5000 50  0000 C CNN
-F 1 "R_Small" V 3545 5000 50  0000 C CNN
+F 0 "R526" V 3700 5200 50  0000 C CNN
+F 1 "22" V 3650 5000 50  0000 C CNN
 F 2 "Resistor_SMD:R_0603_1608Metric" H 3650 5000 50  0001 C CNN
 F 3 "~" H 3650 5000 50  0001 C CNN
@@
 U 1 1 5B632746
 P 3650 5100
-F 0 "R527" V 3454 5100 50  0000 C CNN
-F 1 "R_Small" V 3545 5100 50  0000 C CNN
+F 0 "R527" V 3700 5300 50  0000 C CNN
+F 1 "22" V 3650 5100 50  0000 C CNN
 F 2 "Resistor_SMD:R_0603_1608Metric" H 3650 5100 50  0001 C CNN
 F 3 "~" H 3650 5100 50  0001 C CNN
