File: components_predev/frontend/hardware/DAC.sch (KiCad schematic (older format))
At the start: 25 parts, among them J601 Conn_01x03, U601 MAX5318

Commit message: Some Updates from Testing
Parts:
- C601, C603, C605: Digikey (none) -> 490-7202-1-ND; Manufacturer (none) -> MuRata; Part Number (none) -> GRM188R61E106MA73D; Voltage (none) -> 25 V
- C602, C604, C606, C608: Digikey (none) -> 1276-1005-1-ND; Manufacturer (none) -> Samsung; Note (none) -> VH; Part Number (none) -> CL10B104K08NNNC; Voltage (none) -> 16V
- C607: Digikey (none) -> 490-10476-1-ND; Manufacturer (none) -> MuRata; Part Number (none) -> GRM188R61A226ME15D
- J601: Note (none) -> VH
- JP601, JP602: Note (none) -> NB
- R517, R518, R519, R520, R521, R522, R523, R524, R525, R526, R527: Digikey (none) -> 311-22.0HRCT-ND; Manufacturer (none) -> Yageo; Note (none) -> VH; Part Number (none) -> RC0603FR-0722RL
- R601, R602: Digikey (none) -> P2.00KHCT-ND; Manufacturer (none) -> Panasonic; Note (none) -> VH; Part Number (none) -> ERJ-3EKF2001V
- U601: Digikey (none) -> MAX5318GUG+-ND; Manufacturer (none) -> Maxim; Part Number (none) -> MAX5318GUG+
Changed lines of the file:
@@
 F 2 "Package_SO:TSSOP-24_4.4x7.8mm_P0.65mm" H 5350 4500 60  0001 C CNN
 F 3 "" H 5350 4500 60  0001 C CNN
+F 4 "MAX5318GUG+-ND" H 0   0   50  0001 C CNN "Digikey"
+F 5 "Maxim" H 0   0   50  0001 C CNN "Manufacturer"
+F 6 "MAX5318GUG+" H 0   0   50  0001 C CNN "Part Number"
 	1    5350 4500
 	1    0    0    -1
@@
 F 2 "Resistor_SMD:R_0603_1608Metric" H 4150 3550 50  0001 C CNN
 F 3 "" H 4150 3550 50  0000 C CNN
+F 4 "P2.00KHCT-ND" H 0   0   50  0001 C CNN "Digikey"
+F 5 "Panasonic" H 0   0   50  0001 C CNN "Manufacturer"
+F 6 "VH" H 0   0   50  0001 C CNN "Note"
+F 7 "ERJ-3EKF2001V" H 0   0   50  0001 C CNN "Part Number"
 	1    4150 3550
 	1    0    0    -1
@@
 F 2 "Jumper:SolderJumper-3_P1.3mm_Open_RoundedPad1.0x1.5mm" H 3050 3300 50  0001 C CNN
 F 3 "" H 3050 3300 50  0000 C CNN
+F 4 "NB" H 0   0   50  0001 C CNN "Note"
 	1    3050 3300
 	1    0    0    -1
@@
 F 2 "Jumper:SolderJumper-3_P1.3mm_Open_RoundedPad1.0x1.5mm" H 3050 2850 50  0001 C CNN
 F 3 "" H 3050 2850 50  0000 C CNN
+F 4 "NB" H 0   0   50  0001 C CNN "Note"
 	1    3050 2850
 	1    0    0    -1
@@
 F 2 "Resistor_SMD:R_0603_1608Metric" H 2300 3400 50  0001 C CNN
 F 3 "" H 2300 3400 50  0000 C CNN
+F 4 "P2.00KHCT-ND" H 0   0   50  0001 C CNN "Digikey"
+F 5 "Panasonic" H 0   0   50  0001 C CNN "Manufacturer"
+F 6 "VH" H 0   0   50  0001 C CNN "Note"
+F 7 "ERJ-3EKF2001V" H 0   0   50  0001 C CNN "Part Number"
 	1    2300 3400
 	-1   0    0    1
@@
 F 2 "Capacitor_SMD:C_0603_1608Metric" H 4800 2950 50  0001 C CNN
 F 3 "~" H 4800 2950 50  0001 C CNN
+F 4 "1276-1005-1-ND" H 0   0   50  0001 C CNN "Digikey"
+F 5 "Samsung" H 0   0   50  0001 C CNN "Manufacturer"
+F 6 "VH" H 0   0   50  0001 C CNN "Note"
+F 7 "CL10B104K08NNNC" H 0   0   50  0001 C CNN "Part Number"
+F 8 "16V" H 0   0   50  0001 C CNN "Voltage"
 	1    4800 2950
 	0    1    1    0
@@
 F 2 "Capacitor_SMD:C_0603_1608Metric" H 4800 2600 50  0001 C CNN
 F 3 "~" H 4800 2600 50  0001 C CNN
+F 4 "490-7202-1-ND" H 0   0   50  0001 C CNN "Digikey"
+F 5 "MuRata" H 0   0   50  0001 C CNN "Manufacturer"
+F 6 "GRM188R61E106MA73D" H 0   0   50  0001 C CNN "Part Number"
+F 7 "25 V" H 0   0   50  0001 C CNN "Voltage"
 	1    4800 2600
 	0    1    1    0
@@
 F 2 "Connector_PinHeader_2.54mm:PinHeader_1x03_P2.54mm_Vertical" H 8400 4150 50  0001 C CNN
 F 3 "~" H 8400 4150 50  0001 C CNN
+F 4 "VH" H 0   0   50  0001 C CNN "Note"
 	1    8400 4150
 	0    -1   -1   0
@@
 F 2 "Capacitor_SMD:C_0603_1608Metric" H 6350 3550 50  0001 C CNN
 F 3 "~" H 6350 3550 50  0001 C CNN
+F 4 "1276-1005-1-ND" H 0   0   50  0001 C CNN "Digikey"
+F 5 "Samsung" H 0   0   50  0001 C CNN "Manufacturer"
+F 6 "VH" H 0   0   50  0001 C CNN "Note"
+F 7 "CL10B104K08NNNC" H 0   0   50  0001 C CNN "Part Number"
+F 8 "16V" H 0   0   50  0001 C CNN "Voltage"
 	1    6350 3550
 	0    1    1    0
@@
 F 2 "Capacitor_SMD:C_0603_1608Metric" H 6350 3200 50  0001 C CNN
 F 3 "~" H 6350 3200 50  0001 C CNN
+F 4 "490-10476-1-ND" H 0   0   50  0001 C CNN "Digikey"
+F 5 "MuRata" H 0   0   50  0001 C CNN "Manufacturer"
+F 6 "GRM188R61A226ME15D" H 0   0   50  0001 C CNN "Part Number"
 	1    6350 3200
 	0    1    1    0
@@
 F 2 "Capacitor_SMD:C_0603_1608Metric" H 6350 2800 50  0001 C CNN
 F 3 "~" H 6350 2800 50  0001 C CNN
+F 4 "1276-1005-1-ND" H 0   0   50  0001 C CNN "Digikey"
+F 5 "Samsung" H 0   0   50  0001 C CNN "Manufacturer"
+F 6 "VH" H 0   0   50  0001 C CNN "Note"
+F 7 "CL10B104K08NNNC" H 0   0   50  0001 C CNN "Part Number"
+F 8 "16V" H 0   0   50  0001 C CNN "Voltage"
 	1    6350 2800
 	0    1    1    0
@@
 F 2 "Capacitor_SMD:C_0603_1608Metric" H 6350 2450 50  0001 C CNN
 F 3 "~" H 6350 2450 50  0001 C CNN
+F 4 "490-7202-1-ND" H 0   0   50  0001 C CNN "Digikey"
+F 5 "MuRata" H 0   0   50  0001 C CNN "Manufacturer"
+F 6 "GRM188R61E106MA73D" H 0   0   50  0001 C CNN "Part Number"
+F 7 "25 V" H 0   0   50  0001 C CNN "Voltage"
 	1    6350 2450
 	0    1    1    0
@@
 F 2 "Capacitor_SMD:C_0603_1608Metric" H 6350 2150 50  0001 C CNN
 F 3 "~" H 6350 2150 50  0001 C CNN
+F 4 "1276-1005-1-ND" H 0   0   50  0001 C CNN "Digikey"
+F 5 "Samsung" H 0   0   50  0001 C CNN "Manufacturer"
+F 6 "VH" H 0   0   50  0001 C CNN "Note"
+F 7 "CL10B104K08NNNC" H 0   0   50  0001 C CNN "Part Number"
+F 8 "16V" H 0   0   50  0001 C CNN "Voltage"
 	1    6350 2150
 	0    1    1    0
@@
 F 2 "Capacitor_SMD:C_0603_1608Metric" H 6350 1800 50  0001 C CNN
 F 3 "~" H 6350 1800 50  0001 C CNN
+F 4 "490-7202-1-ND" H 0   0   50  0001 C CNN "Digikey"
+F 5 "MuRata" H 0   0   50  0001 C CNN "Manufacturer"
+F 6 "GRM188R61E106MA73D" H 0   0   50  0001 C CNN "Part Number"
+F 7 "25 V" H 0   0   50  0001 C CNN "Voltage"
 	1    6350 1800
 	0    1    1    0
@@
 F 2 "Resistor_SMD:R_0603_1608Metric" H 3650 3800 50  0001 C CNN
 F 3 "~" H 3650 3800 50  0001 C CNN
+F 4 "311-22.0HRCT-ND" H 0   0   50  0001 C CNN "Digikey"
+F 5 "Yageo" H 0   0   50  0001 C CNN "Manufacturer"
+F 6 "RC0603FR-0722RL" H 0   0   50  0001 C CNN "Part Number"
+F 7 "VH" H 0   0   50  0001 C CNN "Note"
 	1    3650 3800
 	0    1    1    0
@@
 F 2 "Resistor_SMD:R_0603_1608Metric" H 3650 3900 50  0001 C CNN
 F 3 "~" H 3650 3900 50  0001 C CNN
+F 4 "311-22.0HRCT-ND" H 0   0   50  0001 C CNN "Digikey"
+F 5 "Yageo" H 0   0   50  0001 C CNN "Manufacturer"
+F 6 "RC0603FR-0722RL" H 0   0   50  0001 C CNN "Part Number"
+F 7 "VH" H 0   0   50  0001 C CNN "Note"
 	1    3650 3900
 	0    1    1    0
@@
 F 2 "Resistor_SMD:R_0603_1608Metric" H 3650 4000 50  0001 C CNN
 F 3 "~" H 3650 4000 50  0001 C CNN
+F 4 "311-22.0HRCT-ND" H 0   0   50  0001 C CNN "Digikey"
+F 5 "Yageo" H 0   0   50  0001 C CNN "Manufacturer"
+F 6 "RC0603FR-0722RL" H 0   0   50  0001 C CNN "Part Number"
+F 7 "VH" H 0   0   50  0001 C CNN "Note"
 	1    3650 4000
 	0    1    1    0
@@
 F 2 "Resistor_SMD:R_0603_1608Metric" H 3650 4100 50  0001 C CNN
 F 3 "~" H 3650 4100 50  0001 C CNN
+F 4 "311-22.0HRCT-ND" H 0   0   50  0001 C CNN "Digikey"
+F 5 "Yageo" H 0   0   50  0001 C CNN "Manufacturer"
+F 6 "RC0603FR-0722RL" H 0   0   50  0001 C CNN "Part Number"
+F 7 "VH" H 0   0   50  0001 C CNN "Note"
 	1    3650 4100
 	0    1    1    0
@@
 F 2 "Resistor_SMD:R_0603_1608Metric" H 3200 4400 50  0001 C CNN
 F 3 "~" H 3200 4400 50  0001 C CNN
+F 4 "311-22.0HRCT-ND" H 0   0   50  0001 C CNN "Digikey"
+F 5 "Yageo" H 0   0   50  0001 C CNN "Manufacturer"
+F 6 "RC0603FR-0722RL" H 0   0   50  0001 C CNN "Part Number"
+F 7 "VH" H 0   0   50  0001 C CNN "Note"
 	1    3200 4400
 	0    1    1    0
@@
 F 2 "Resistor_SMD:R_0603_1608Metric" H 3200 4500 50  0001 C CNN
 F 3 "~" H 3200 4500 50  0001 C CNN
+F 4 "311-22.0HRCT-ND" H 0   0   50  0001 C CNN "Digikey"
+F 5 "Yageo" H 0   0   50  0001 C CNN "Manufacturer"
+F 6 "RC0603FR-0722RL" H 0   0   50  0001 C CNN "Part Number"
+F 7 "VH" H 0   0   50  0001 C CNN "Note"
 	1    3200 4500
 	0    1    1    0
@@
 F 2 "Resistor_SMD:R_0603_1608Metric" H 3200 4600 50  0001 C CNN
 F 3 "~" H 3200 4600 50  0001 C CNN
+F 4 "311-22.0HRCT-ND" H 0   0   50  0001 C CNN "Digikey"
+F 5 "Yageo" H 0   0   50  0001 C CNN "Manufacturer"
+F 6 "RC0603FR-0722RL" H 0   0   50  0001 C CNN "Part Number"
+F 7 "VH" H 0   0   50  0001 C CNN "Note"
 	1    3200 4600
 	0    1    1    0
@@
 F 2 "Resistor_SMD:R_0603_1608Metric" H 3650 4800 50  0001 C CNN
 F 3 "~" H 3650 4800 50  0001 C CNN
+F 4 "311-22.0HRCT-ND" H 0   0   50  0001 C CNN "Digikey"
+F 5 "Yageo" H 0   0   50  0001 C CNN "Manufacturer"
+F 6 "RC0603FR-0722RL" H 0   0   50  0001 C CNN "Part Number"
+F 7 "VH" H 0   0   50  0001 C CNN "Note"
 	1    3650 4800
 	0    1    1    0
@@
 F 2 "Resistor_SMD:R_0603_1608Metric" H 3650 4900 50  0001 C CNN
 F 3 "~" H 3650 4900 50  0001 C CNN
+F 4 "311-22.0HRCT-ND" H 0   0   50  0001 C CNN "Digikey"
+F 5 "Yageo" H 0   0   50  0001 C CNN "Manufacturer"
+F 6 "RC0603FR-0722RL" H 0   0   50  0001 C CNN "Part Number"
+F 7 "VH" H 0   0   50  0001 C CNN "Note"
 	1    3650 4900
 	0    1    1    0
@@
 F 2 "Resistor_SMD:R_0603_1608Metric" H 3650 5000 50  0001 C CNN
 F 3 "~" H 3650 5000 50  0001 C CNN
+F 4 "311-22.0HRCT-ND" H 0   0   50  0001 C CNN "Digikey"
+F 5 "Yageo" H 0   0   50  0001 C CNN "Manufacturer"
+F 6 "RC0603FR-0722RL" H 0   0   50  0001 C CNN "Part Number"
+F 7 "VH" H 0   0   50  0001 C CNN "Note"
 	1    3650 5000
 	0    1    1    0
@@
 F 2 "Resistor_SMD:R_0603_1608Metric" H 3650 5100 50  0001 C CNN
 F 3 "~" H 3650 5100 50  0001 C CNN
+F 4 "311-22.0HRCT-ND" H 0   0   50  0001 C CNN "Digikey"
+F 5 "Yageo" H 0   0   50  0001 C CNN "Manufacturer"
+F 6 "RC0603FR-0722RL" H 0   0   50  0001 C CNN "Part Number"
+F 7 "VH" H 0   0   50  0001 C CNN "Note"
 	1    3650 5100
 	0    1    1    0
